Commit message: Controller and OPC UA Server added

File: pm_robot_description/urdf/ros2_control.xacro (robot description, xacro)
@@ -6,14 +6,21 @@
         </hardware>
         <joint name="X_Axis_Joint">
-            <command_interface name="velocity">
+            <command_interface name="position">
                 <param name="min">-10000</param>
                 <param name="max">10000</param>
             </command_interface>
-            <state_interface name="velocity"/>
+            <state_interface name="position"/>
+        </joint>
+        <joint name="Y_Axis_Joint">
+            <command_interface name="position">
+                <param name="min">-10000</param>
+                <param name="max">10000</param>
+            </command_interface>
+            <state_interface name="position"/>
         </joint>
     </ros2_control>
     <gazebo>
         <plugin name="gazebo_ros2_control" filename="libgazebo_ros2_control.so">
-            <parameters>$(find pm_robot_description)/config/controller.yaml</parameters>
+            <parameters>$(find pm_robot_description)/config/control.yaml</parameters>
         </plugin>
     </gazebo>

Commit message: Joint Trajectory controller is working

File: pm_robot_description/urdf/ros2_control.xacro (robot description, xacro)
@@ -19,4 +19,11 @@
             <state_interface name="position"/>
         </joint>
+        <joint name="Z_Axis_Joint">
+            <command_interface name="position">
+                <param name="min">-10000</param>
+                <param name="max">10000</param>
+            </command_interface>
+            <state_interface name="position"/>
+        </joint>
     </ros2_control>
     <gazebo>
