Commit message: Gazebo launch file added

File: pm_robot_description/urdf/pm_robot.urdf (robot description, URDF)
Before this commit: robot pm_robot, 29 links, 28 joints
Links:
- removed link Component
- link Camera_Calibration: geometry collision mesh filename=file://$(find pm_robot_description)/meshes/Camera_Calibrati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; visual mesh filename=file://$(find pm_robot_description)/meshes/Camera_Calibrati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
- link Camera_Module_Z_Axis: geometry collision mesh filename=file://$(find pm_robot_description)/meshes/Camera_Module_Z_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; visual mesh filename=file://$(find pm_robot_description)/meshes/Camera_Module_Z_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
- link Camera_System: geometry collision mesh filename=file://$(find pm_robot_description)/meshes/Camera_System.STL; visual mesh filename=file://$(find pm_robot_description)/meshes/Camera_System.STL
- link EQ: geometry collision mesh filename=file://$(find pm_robot_description)/meshes/EQ.STL; visual mesh filename=file://$(find pm_robot_description)/meshes/EQ.STL
- link Glue_Cartridge: geometry collision mesh filename=file://$(find pm_robot_description)/meshes/Glue_Cartridge.S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; visual mesh filename=file://$(find pm_robot_description)/meshes/Glue_Cartridge.S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
- link Glue_Cartridge_Flap: geometry collision mesh filename=file://$(find pm_robot_description)/meshes/Glue_Cartridge_F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; visual mesh filename=file://$(find pm_robot_description)/meshes/Glue_Cartridge_F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
- link Gonio_Base_Left: geometry collision mesh filename=file://$(find pm_robot_description)/meshes/Gonio_Base_Left.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; visual mesh filename=file://$(find pm_robot_description)/meshes/Gonio_Base_Left.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
- link Gonio_Base_Rigth: geometry collision mesh filename=file://$(find pm_robot_description)/meshes/Gonio_Base_Rigth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; visual mesh filename=file://$(find pm_robot_description)/meshes/Gonio_Base_Rigth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
- link Gonio_Left_Stage_1_Upper: geometry collision mesh filename=file://$(find pm_robot_description)/meshes/Gonio_Left_Stage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; visual mesh filename=file://$(find pm_robot_description)/meshes/Gonio_Left_Stage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
- link Gonio_Left_Stage_2_Upper: geometry collision mesh filename=file://$(find pm_robot_description)/meshes/Gonio_Left_Stage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; visual mesh filename=file://$(find pm_robot_description)/meshes/Gonio_Left_Stage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
- link Gonio_Right_Mount_Lower: geometry collision mesh filename=file://$(find pm_robot_description)/meshes/Gonio_Right_Moun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; visual mesh filename=file://$(find pm_robot_description)/meshes/Gonio_Right_Moun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
- link Gonio_Right_Mount_Upper: geometry collision mesh filename=file://$(find pm_robot_description)/meshes/Gonio_Right_Moun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; visual mesh filename=file://$(find pm_robot_description)/meshes/Gonio_Right_Moun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
- link Gonio_Right_Stage_1_Upper: geometry collision mesh filename=file://$(find pm_robot_description)/meshes/Gonio_Right_Stag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; visual mesh filename=file://$(find pm_robot_description)/meshes/Gonio_Right_Stag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
- link Gonio_Right_Stage_2_Upper: geometry collision mesh filename=file://$(find pm_robot_description)/meshes/Gonio_Right_Stag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; visual mesh filename=file://$(find pm_robot_description)/meshes/Gonio_Right_Stag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
- link Gripper: geometry collision mesh filename=file://$(find pm_robot_description)/meshes/Gripper.STL; visual mesh filename=file://$(find pm_robot_description)/meshes/Gripper.STL
- link Gripper_Rot_Plate: geometry collision mesh filename=file://$(find pm_robot_description)/meshes/Gripper_Rot_Plat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; visual mesh filename=file://$(find pm_robot_description)/meshes/Gripper_Rot_Plat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
- link Nest: geometry collision mesh filename=file://$(find pm_robot_description)/meshes/Nest.STL; visual mesh filename=file://$(find pm_robot_description)/meshes/Nest.STL
- link Stage_1_Gonio_Right: geometry collision mesh filename=file://$(find pm_robot_description)/meshes/Stage_1_Gonio_Ri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; visual mesh filename=file://$(find pm_robot_description)/meshes/Stage_1_Gonio_Ri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
- link Test_Station: geometry collision mesh filename=file://$(find pm_robot_description)/meshes/Test_Station.STL; visual mesh filename=file://$(find pm_robot_description)/meshes/Test_Station.STL
- link UV_Cart_Left: geometry collision mesh filename=file://$(find pm_robot_description)/meshes/UV_Cart_Left.STL; visual mesh filename=file://$(find pm_robot_description)/meshes/UV_Cart_Left.STL
- link UV_Cart_Right: geometry collision mesh filename=file://$(find pm_robot_description)/meshes/UV_Cart_Right.STL; visual mesh filename=file://$(find pm_robot_description)/meshes/UV_Cart_Right.STL
- link UV_Module_Left: geometry collision mesh filename=file://$(find pm_robot_description)/meshes/UV_Module_Left.S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; visual mesh filename=file://$(find pm_robot_description)/meshes/UV_Module_Left.S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
- link UV_Module_Right: geometry collision mesh filename=file://$(find pm_robot_description)/meshes/UV_Module_Right.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; visual mesh filename=file://$(find pm_robot_description)/meshes/UV_Module_Right.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
- link X_Axis: geometry collision mesh filename=file://$(find pm_robot_description)/meshes/X_Axis.STL; visual mesh filename=file://$(find pm_robot_description)/meshes/X_Axis.STL
- link Y_Axis: geometry collision mesh filename=file://$(find pm_robot_description)/meshes/Y_Axis.STL; visual mesh filename=file://$(find pm_robot_description)/meshes/Y_Axis.STL
- link Z_Axis: geometry collision mesh filename=file://$(find pm_robot_description)/meshes/Z_Axis.STL; visual mesh filename=file://$(find pm_robot_description)/meshes/Z_Axis.STL
- link base_link: geometry collision mesh filename=file://$(find pm_robot_description)/meshes/base_link.STL; visual mesh filename=file://$(find pm_robot_description)/meshes/base_link.STL
Joints:
- removed joint Component_Joint

Commit message: controller publisher added

File: pm_robot_description/urdf/pm_robot.urdf (robot description, URDF)
Before this commit: robot pm_robot, 28 links, 27 joints
Joints:
- removed joint Gonio_Right_Stage_1_Upper_joint
- added joint Gonio_Right_Stage_1_Upper_Joint: type revolute, parent Stage_1_Gonio_Right, child Gonio_Right_Stage_1_Upper, origin xyz=0.0125000000000001 0.0325000000000001 0.281999999999999 rpy=0 0 0, axis 1 0 0, limit lower=-0.087266 upper=0.087266 effort=100 velocity=0.1
- joint X_Axis_Joint: limit lower=-0.745 upper=0.055 effort=100 velocity=0.05 -> lower=-0.745 upper=0.055 effort=1 velocity=100
- joint Y_Axis_Joint: limit lower=-0.425 upper=0.2505 effort=100 velocity=0.05 -> lower=-0.425 upper=0.2505 effort=100 velocity=100

File: pm_robot_description/urdf/ros2_control.xacro (robot description, xacro)
@@ -7,6 +7,4 @@
         <joint name="X_Axis_Joint">
             <command_interface name="position">
-                <param name="min">-10000</param>
-                <param name="max">10000</param>
             </command_interface>
             <state_interface name="position"/>
@@ -14,6 +12,4 @@
         <joint name="Y_Axis_Joint">
             <command_interface name="position">
-                <param name="min">-10000</param>
-                <param name="max">10000</param>
             </command_interface>
             <state_interface name="position"/>
@@ -21,6 +17,69 @@
         <joint name="Z_Axis_Joint">
             <command_interface name="position">
-                <param name="min">-10000</param>
-                <param name="max">10000</param>
+            </command_interface>
+            <state_interface name="position"/>
+        </joint>
+        <joint name="Gripper_Rot_Plate_Joint">
+            <command_interface name="position">
+            </command_interface>
+            <state_interface name="position"/>
+        </joint>
+        <joint name="Glue_Cartridge_Flap_Joint">
+            <command_interface name="position">
+            </command_interface>
+            <state_interface name="position"/>
+        </joint>
+        <joint name="Glue_Cartridge_Joint">
+            <command_interface name="position">
+            </command_interface>
+            <state_interface name="position"/>
+        </joint>
+        <joint name="EQ_Joint">
+            <command_interface name="position">
+            </command_interface>
+            <state_interface name="position"/>
+        </joint>
+        <joint name="Gonio_Right_Stage_1_Upper_Joint">
+            <command_interface name="position">
+            </command_interface>
+            <state_interface name="position"/>
+        </joint>
+        <joint name="Gonio_Right_Stage_2_Upper_Joint">
+            <command_interface name="position">
+            </command_interface>
+            <state_interface name="position"/>
+        </joint>
+        <joint name="Camera_Calibartion_Joint">
+            <command_interface name="position">
+            </command_interface>
+            <state_interface name="position"/>
+        </joint>
+        <joint name="Gonio_Left_Stage_1_Upper_Joint">
+            <command_interface name="position">
+            </command_interface>
+            <state_interface name="position"/>
+        </joint>
+        <joint name="Gonio_Left_Stage_2_Upper_Joint">
+            <command_interface name="position">
+            </command_interface>
+            <state_interface name="position"/>
+        </joint>
+        <joint name="UV_Cart_Left_Joint">
+            <command_interface name="position">
+            </command_interface>
+            <state_interface name="position"/>
+        </joint>
+        <joint name="UV_Module_Left_Joint">
+            <command_interface name="position">
+            </command_interface>
+            <state_interface name="position"/>
+        </joint>
+        <joint name="UV_Cart_Right_Joint">
+            <command_interface name="position">
+            </command_interface>
+            <state_interface name="position"/>
+        </joint>
+        <joint name="UV_Module_Right_Joint">
+            <command_interface name="position">
             </command_interface>
             <state_interface name="position"/>

Commit message: urdf model modified

File: pm_robot_description/urdf/pm_robot.urdf (robot description, URDF)
Before this commit: robot pm_robot, 28 links, 27 joints
Links:
- removed link Camera_Module_Z_Axis
- removed link EQ
- removed link Glue_Cartridge
- removed link Glue_Cartridge_Flap
- removed link Gonio_Base_Left
- removed link Gonio_Base_Rigth
- removed link Gonio_Left_Stage_1_Upper
- removed link Gonio_Left_Stage_2_Upper
- removed link Gonio_Right_Mount_Lower
- removed link Gonio_Right_Mount_Upper
- removed link Gonio_Right_Stage_1_Upper
- removed link Gonio_Right_Stage_2_Upper
- removed link Nest
- removed link Stage_1_Gonio_Right
- removed link UV_Cart_Left
- removed link UV_Cart_Right
- removed link UV_Module_Left
- removed link UV_Module_Right
- added link 1K_Dispenser, mass 0.0725671789847037; collision mesh filename=file://$(find pm_robot_description)/meshes/1K_Dispenser.STL; visual mesh filename=file://$(find pm_robot_description)/meshes/1K_Dispenser.STL
- added link 1K_Dispenser_Flap, mass 0.0179277924431146; collision mesh filename=file://$(find pm_robot_description)/meshes/1K_Dispenser_Fla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; visual mesh filename=file://$(find pm_robot_description)/meshes/1K_Dispenser_Fla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
- added link 2K_Dispenser, mass 0.313852053537918; collision mesh filename=file://$(find pm_robot_description)/meshes/2K_Dispenser.STL; visual mesh filename=file://$(find pm_robot_description)/meshes/2K_Dispenser.STL
- added link Camera_Top_View, mass 0.0744906107551854; collision mesh filename=file://$(find pm_robot_description)/meshes/Camera_Top_View.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; visual mesh filename=file://$(find pm_robot_description)/meshes/Camera_Top_View.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
- added link Gonio_Left_Holder, mass 0.0867575149913971; collision mesh filename=file://$(find pm_robot_description)/meshes/Gonio_Left_Holde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; visual mesh filename=file://$(find pm_robot_description)/meshes/Gonio_Left_Holde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
- added link Gonio_Left_Stage_1_Top, mass 0.578798857286943; collision mesh filename=file://$(find pm_robot_description)/meshes/Gonio_Left_Stage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; visual mesh filename=file://$(find pm_robot_description)/meshes/Gonio_Left_Stage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
- added link Gonio_Left_Stage_2_Bottom, mass 0.0270626702476316; collision mesh filename=file://$(find pm_robot_description)/meshes/Gonio_Left_Stage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; visual mesh filename=file://$(find pm_robot_description)/meshes/Gonio_Left_Stage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
- added link Gonio_Right, mass 0.735149712395274; collision mesh filename=file://$(find pm_robot_description)/meshes/Gonio_Right.STL; visual mesh filename=file://$(find pm_robot_description)/meshes/Gonio_Right.STL
- added link Gonio_Right_Holder, mass 0.133934804202608; collision mesh filename=file://$(find pm_robot_description)/meshes/Gonio_Right_Hold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; visual mesh filename=file://$(find pm_robot_description)/meshes/Gonio_Right_Hold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
- added link Gonio_Right_Stage_1_Bottom, mass 0.0706349432835735; collision mesh filename=file://$(find pm_robot_description)/meshes/Gonio_Right_Stag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; visual mesh filename=file://$(find pm_robot_description)/meshes/Gonio_Right_Stag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
- added link Gonio_Right_Stage_1_Top, mass 0.13548582818363; collision mesh filename=file://$(find pm_robot_description)/meshes/Gonio_Right_Stag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; visual mesh filename=file://$(find pm_robot_description)/meshes/Gonio_Right_Stag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
- added link Gonio_Right_Stage_2_Bottom, mass 0.0546397543064686; collision mesh filename=file://$(find pm_robot_description)/meshes/Gonio_Right_Stag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; visual mesh filename=file://$(find pm_robot_description)/meshes/Gonio_Right_Stag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
- added link Gonio_Station_Left, mass 4.82459847582554; collision mesh filename=file://$(find pm_robot_description)/meshes/Gonio_Station_Le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; visual mesh filename=file://$(find pm_robot_description)/meshes/Gonio_Station_Le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
- added link UV_LED_Back, mass 0.119915229322348; collision mesh filename=file://$(find pm_robot_description)/meshes/UV_LED_Back.STL; visual mesh filename=file://$(find pm_robot_description)/meshes/UV_LED_Back.STL
- added link UV_LED_Front, mass 0.119915229322347; collision mesh filename=file://$(find pm_robot_description)/meshes/UV_LED_Front.STL; visual mesh filename=file://$(find pm_robot_description)/meshes/UV_LED_Front.STL
- added link UV_Slider_X_Back, mass 0.127959263593804; collision mesh filename=file://$(find pm_robot_description)/meshes/UV_Slider_X_Back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; visual mesh filename=file://$(find pm_robot_description)/meshes/UV_Slider_X_Back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
- added link UV_Slider_X_Front, mass 0.127959263611524; collision mesh filename=file://$(find pm_robot_description)/meshes/UV_Slider_X_Fron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; visual mesh filename=file://$(find pm_robot_description)/meshes/UV_Slider_X_Fron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
- link Gripper: mass 0.127647896986229 -> 0.123801210587509
Joints:
- removed joint Camera_Module_Z_Axis_Joint
- removed joint EQ_Joint
- removed joint Glue_Cartridge_Flap_Joint
- removed joint Glue_Cartridge_Joint
- removed joint Gonio_Base_Left_Joint
- removed joint Gonio_Left_Stage_1_Upper_Joint
- removed joint Gonio_Left_Stage_2_Upper_Joint
- removed joint Gonio_Right_Mount_Lower_joint
- removed joint Gonio_Right_Mount_Upper_Joint
- removed joint Gonio_Right_Stage_1_Upper_Joint
- removed joint Gonio_Right_Stage_2_Upper_Joint
- removed joint Gonio_base_Rigth_Joint
- removed joint Nest_Joint
- removed joint Stage_1_Gonio_Right_Joint
- removed joint UV_Cart_Left_Joint
- removed joint UV_Cart_Right_Joint
- removed joint UV_Module_Left_Joint
- removed joint UV_Module_Right_Joint
- added joint 1K_Dispenser_Flap_Joint: type prismatic, parent Z_Axis, child 1K_Dispenser_Flap, origin xyz=0.075 0.0545 -0.4125 rpy=0 0 0, axis -1 0 0, limit lower=0 upper=0.02 effort=100 velocity=0.05
- added joint 1K_Dispenser_Joint: type prismatic, parent Z_Axis, child 1K_Dispenser, origin xyz=0.1725 0.09 -0.4655 rpy=0 0 0, axis 0 0 -1, limit lower=0 upper=0.04 effort=100 velocity=0.05
- added joint 2K_Dispenser_Joint: type prismatic, parent Z_Axis, child 2K_Dispenser, origin xyz=0.2365 0.0618 -0.4695 rpy=0 0 0, axis 0 0 1, limit lower=0 upper=0.02 effort=100 velocity=0.05
- added joint Camera_Top_View_Joint: type fixed, parent Z_Axis, child Camera_Top_View, origin xyz=0.0795000000000243 0.068500020970708 -0.233999999999991 rpy=0 0 0, axis 0 0 0
- added joint Gonio_Left_Holder_Joint: type fixed, parent Gonio_Left_Stage_2_Bottom, child Gonio_Left_Holder, origin xyz=-1.8727E-05 -0.025 -0.015 rpy=0 0.00124847209372143 0, axis 0 0 0
- added joint Gonio_Left_Stage_1_Top_Joint: type revolute, parent Gonio_Station_Left, child Gonio_Left_Stage_1_Top, origin xyz=-0.385 0.0855 0.1847 rpy=0 0 0, axis 1 0 0, limit lower=-0.78539816339745 upper=0.78539816339745 effort=100 velocity=0.1
- added joint Gonio_Left_Stage_2_Bottom_Joint: type revolute, parent Gonio_Left_Stage_1_Top, child Gonio_Left_Stage_2_Bottom, origin xyz=0.5015 0.0495 0.0278 rpy=0 0 0, axis 0 -1 0, limit lower=-0.78539816339745 upper=0.78539816339745 effort=100 velocity=0.1
- added joint Gonio_Right_Holder_Joint: type fixed, parent Gonio_Right_Stage_2_Bottom, child Gonio_Right_Holder, origin xyz=-0.0325 -0.065 -0.05 rpy=0 0 0, axis 0 0 0
- added joint Gonio_Right_Joint: type fixed, parent base_link, child Gonio_Right, origin xyz=0.355 0.77 0.1127 rpy=0 0 0, axis 0 0 0
- added joint Gonio_Right_Stage_1_Bottom_Joint: type fixed, parent Gonio_Right, child Gonio_Right_Stage_1_Bottom, origin xyz=0.0125 0 0.172 rpy=0 0 0, axis 0 0 0
- added joint Gonio_Right_Stage_1_Top_Joint: type revolute, parent Gonio_Right_Stage_1_Bottom, child Gonio_Right_Stage_1_Top, origin xyz=0 0.0325 0.11 rpy=0 0 0, axis 1 0 0, limit lower=-0.087266 upper=0.087266 effort=100 velocity=0.1
- added joint Gonio_Right_Stage_2_Bottom_Joint: type revolute, parent Gonio_Right_Stage_1_Top, child Gonio_Right_Stage_2_Bottom, origin xyz=0.0325 0.0325 0 rpy=0 0 0, axis 0 -1 0, limit lower=-0.17453 upper=0.17453 effort=100 velocity=0.1
- added joint Gonio_Station_Left_Joint: type fixed, parent base_link, child Gonio_Station_Left, origin xyz=0.7525 0.6845 0.1 rpy=0 0 0, axis 0 0 0
- added joint UV_LED_Back_Joint: type prismatic, parent UV_Slider_X_Back, child UV_LED_Back, origin xyz=0.11 -0.08618 0.0276 rpy=0 0 0, axis 0 -1 0, limit lower=0 upper=0.05 effort=100 velocity=0.05
- added joint UV_LED_Front_Joint: type prismatic, parent UV_Slider_X_Front, child UV_LED_Front, origin xyz=0.11 0.02382 0.0276 rpy=0 0 0, axis 0 1 0, limit lower=0.045 upper=0.045 effort=100 velocity=0.05
- added joint UV_Slider_X_Back_Joint: type prismatic, parent Gonio_Station_Left, child UV_Slider_X_Back, origin xyz=0.0065 0.05118 0.2526 rpy=0 0 0, axis 1 0 0, limit lower=-0.045 upper=0.045 effort=0.05 velocity=100
- added joint UV_Slider_X_Front_Joint: type prismatic, parent Gonio_Station_Left, child UV_Slider_X_Front, origin xyz=0.0065 0.23118 0.2526 rpy=0 0 0, axis -1 0 0, limit lower=-0.05 upper=0.095 effort=100 velocity=0.05
- joint Gripper_Joint: origin xyz=0 0 -0.0255000000000101 rpy=0 0 0 -> xyz=0 0 -0.096 rpy=0 0 0

File: pm_robot_description/urdf/ros2_control.xacro (robot description, xacro)
@@ -25,25 +25,25 @@
             <state_interface name="position"/>
         </joint>
-        <joint name="Glue_Cartridge_Flap_Joint">
+        <joint name="1K_Dispenser_Flap_Joint">
             <command_interface name="position">
             </command_interface>
             <state_interface name="position"/>
         </joint>
-        <joint name="Glue_Cartridge_Joint">
+        <joint name="1K_Dispenser_Joint">
             <command_interface name="position">
             </command_interface>
             <state_interface name="position"/>
         </joint>
-        <joint name="EQ_Joint">
+        <joint name="2K_Dispenser_Joint">
             <command_interface name="position">
             </command_interface>
             <state_interface name="position"/>
         </joint>
-        <joint name="Gonio_Right_Stage_1_Upper_Joint">
+        <joint name="Gonio_Right_Stage_1_Top_Joint">
             <command_interface name="position">
             </command_interface>
             <state_interface name="position"/>
         </joint>
-        <joint name="Gonio_Right_Stage_2_Upper_Joint">
+        <joint name="Gonio_Right_Stage_2_Bottom_Joint">
             <command_interface name="position">
             </command_interface>
@@ -55,30 +55,30 @@
             <state_interface name="position"/>
         </joint>
-        <joint name="Gonio_Left_Stage_1_Upper_Joint">
+        <joint name="Gonio_Left_Stage_1_Top_Joint">
             <command_interface name="position">
             </command_interface>
             <state_interface name="position"/>
         </joint>
-        <joint name="Gonio_Left_Stage_2_Upper_Joint">
+        <joint name="Gonio_Left_Stage_2_Bottom_Joint">
             <command_interface name="position">
             </command_interface>
             <state_interface name="position"/>
         </joint>
-        <joint name="UV_Cart_Left_Joint">
+        <joint name="UV_Slider_X_Front_Joint">
             <command_interface name="position">
             </command_interface>
             <state_interface name="position"/>
         </joint>
-        <joint name="UV_Module_Left_Joint">
+        <joint name="UV_LED_Front_Joint">
             <command_interface name="position">
             </command_interface>
             <state_interface name="position"/>
         </joint>
-        <joint name="UV_Cart_Right_Joint">
+        <joint name="UV_Slider_X_Back_Joint">
             <command_interface name="position">
             </command_interface>
             <state_interface name="position"/>
         </joint>
-        <joint name="UV_Module_Right_Joint">
+        <joint name="UV_LED_Back_Joint">
             <command_interface name="position">
             </command_interface>

File: pm_robot_description/urdf/sensors.urdf (robot description, URDF)
Before this commit: robot pm_robot, 3 links, 3 joints
Joints:
- joint camera_joint: parent Camera_Module_Z_Axis -> Camera_Top_View
- joint camera_optical_joint: parent Camera_Module_Z_Axis -> Camera_Top_View
