Commit message: Gripper

File: pm_robot_description/urdf/pm_robot.urdf (robot description, URDF)
Before this commit: robot pm_robot, 27 links, 26 joints
Links:
- removed link Gripper
- added link Tool_Gripper_MPG_10_3mm_Lens_Jaw_1, mass 0.123801210587509; collision mesh filename=file://$(find pm_robot_description)/meshes/Tools/MPG_10_plu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; visual mesh filename=file://$(find pm_robot_description)/meshes/Tools/MPG_10_plu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
- added link Tool_Gripper_MPG_10_Body, mass 0.123801210587509; collision mesh filename=file://$(find pm_robot_description)/meshes/Tools/MPG_10_plu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; visual mesh filename=file://$(find pm_robot_description)/meshes/Tools/MPG_10_plu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
Joints:
- removed joint Gripper_Joint
- added joint Tool_Gripper_MPG_10_3mm_Lens_Jaw_1_Joint: type prismatic, parent Tool_Gripper_MPG_10_Body, child Tool_Gripper_MPG_10_3mm_Lens_Jaw_1, origin xyz=0 -0.04 0 rpy=0 0 3.1416, axis -1 0 0, limit lower=0 upper=0.02 effort=100 velocity=0.05
- added joint Tool_Gripper_MPG_10_Body_Joint: type fixed, parent Gripper_Rot_Plate, child Tool_Gripper_MPG_10_Body, origin xyz=0 0 -0.06 rpy=1.5708 0 0, axis 0 0 0

File: pm_robot_description/urdf/ros2_control.xacro (robot description, xacro)
@@ -21,4 +21,9 @@
         </joint>
         <joint name="Gripper_Rot_Plate_Joint">
+            <command_interface name="position">
+            </command_interface>
+            <state_interface name="position"/>
+        </joint>
+        <joint name="Tool_Gripper_MPG_10_3mm_Lens_Jaw_1_Joint">
             <command_interface name="position">
             </command_interface>
