Commit message: Structure Tests

File: pm_robot_description/urdf/main.xacro (robot description, xacro)
@@ -2,6 +2,8 @@
 <robot name="pm_robot"
   xmlns:xacro="https://ros.org/wiki/xacro">
-  <xacro:include filename="$(find pm_robot_description)/urdf/pm_robot.urdf" />
+  <xacro:include filename="$(find pm_robot_description)/urdf/pm_robot.xacro" />
+  <xacro:include filename="$(find pm_robot_description)/urdf/pm_Schunk_Tools/MPG_10_plus.xacro" />
+  <xacro:include filename="$(find pm_robot_description)/urdf/ros2_control.xacro" />
+  <!--xacro:include filename="$(find pm_robot_description)/urdf/MPG_10_plus_control.xacro" /-->
   <xacro:include filename="$(find pm_robot_description)/urdf/sensors.urdf" />
-  <xacro:include filename="$(find pm_robot_description)/urdf/ros2_control.xacro" />
 </robot>

File: pm_robot_description/urdf/pm_robot.xacro (robot description, xacro)
@@ -4,7 +4,4 @@
      For more information, please see http://wiki.ros.org/sw_urdf_exporter -->
 <robot name="pm_robot">
-  <material name="white">
-    <color rgba="1 1 0.5 1"/>
-  </material>
   <link name="world">
   </link>
@@ -32,13 +29,13 @@
         <mesh filename="file://$(find pm_robot_description)/meshes/base_link.STL" />
       </geometry>
-    </visual>
-    <collision>
-      <origin xyz="0 0 0" rpy="0 0 0" />
-      <geometry>
-        <mesh filename="file://$(find pm_robot_description)/meshes/base_link.STL" />
-      </geometry>
       <material name="">
         <color rgba="0.792156862745098 0.819607843137255 0.933333333333333 1" />
       </material>
+    </visual>
+    <collision>
+      <origin xyz="0 0 0" rpy="0 0 0" />
+      <geometry>
+        <mesh filename="file://$(find pm_robot_description)/meshes/base_link.STL" />
+      </geometry>
     </collision>
   </link>
@@ -157,13 +154,11 @@
     <child link="Gripper_Rot_Plate" />
     <axis xyz="0 0 1" />
-    <limit lower="0" upper="628319" effort="100" velocity="0.05" />
+    <limit lower="0" upper="12" effort="100" velocity="2" />
   </joint>
   <!--
   Gripper Definitions
   <link name="Gripper">
-    <inertial>
-      <origin xyz="-3.43029364781033E-05 -2.0382712019356E-05 0.0426309002703344" rpy="0 0 0" />
-      <mass value="0.123801210587509" />
-      <inertia ixx="2.48847691501343E-05" ixy="-1.96701975168782E-08" ixz="3.35250198834726E-09" iyy="2.52844539238953E-05" iyz="4.55516572819596E-10" izz="4.09732369514151E-05" />
+    <inertial>            </command_interface>
+" ixy="-1.96701975168782E-08" ixz="3.35250198834726E-09" iyy="2.52844539238953E-05" iyz="4.55516572819596E-10" izz="4.09732369514151E-05" />
     </inertial>
     <visual>
@@ -190,68 +185,4 @@
   </joint>
 -->
-  <!--%%%%%%%%%%%%% MPG 10-plus Base Parallel Gripper Definitions %%%%%%%%%%%%%-->
-  <link name="Tool_Gripper_MPG_10_Body">
-    <inertial>
-      <origin xyz="-3.43029364781033E-05 -2.0382712019356E-05 0.0426309002703344" rpy="0 0 0" />
-      <mass value="0.123801210587509" />
-      <inertia ixx="2.48847691501343E-05" ixy="-1.96701975168782E-08" ixz="3.35250198834726E-09" iyy="2.52844539238953E-05" iyz="4.55516572819596E-10" izz="4.09732369514151E-05" />
-    </inertial>
-    <visual>
-      <origin xyz="0 0 0" rpy="0 0 0" />
-      <geometry>
-        <mesh filename="file://$(find pm_robot_description)/meshes/Tools/MPG_10_plus/Tool_MPG_10_Base.STL" />
-      </geometry>
-      <material name="white"/>
-    </visual>
-    <collision>
-      <origin xyz="0 0 0" rpy="0 0 0" />
-      <geometry>
-        <mesh filename="file://$(find pm_robot_description)/meshes/Tools/MPG_10_plus/Tool_MPG_10_Base.STL" />
-      </geometry>
-    </collision>
-  </link>
-  <!---Gravity off-->
-  <gazebo reference="Tool_Gripper_MPG_10_Body">
-    <turnGravityOff>true</turnGravityOff>
-    <color>1.0 0 0.5 1.0</color>
-  </gazebo>
-  <joint name="Tool_Gripper_MPG_10_Body_Joint" type="fixed">
-    <origin xyz="0 0 -0.06" rpy="1.5708 0 0" />
-    <parent link="Gripper_Rot_Plate" />
-    <child link="Tool_Gripper_MPG_10_Body" />
-    <axis xyz="0 0 0" />
-  </joint>
-<!--%%%%%%%%%%%%% MPG 10-plus Jaw 1 Parallel Gripper Definitions %%%%%%%%%%%%%-->
-  <link name="Tool_Gripper_MPG_10_3mm_Lens_Jaw_1">
-    <inertial>
-      <origin xyz="-3.43029364781033E-05 -2.0382712019356E-05 0.0426309002703344" rpy="0 0 0" />
-      <mass value="0.123801210587509" />
-      <inertia ixx="2.48847691501343E-05" ixy="-1.96701975168782E-08" ixz="3.35250198834726E-09" iyy="2.52844539238953E-05" iyz="4.55516572819596E-10" izz="4.09732369514151E-05" />
-    </inertial>
-    <visual>
-      <origin xyz="0 0 0" rpy="0 0 0" />
-      <geometry>
-        <mesh filename="file://$(find pm_robot_description)/meshes/Tools/MPG_10_plus/SCHUNK_MPG-plus_Gripper_Jaw_3MM_Lens_1_Part_scaled.STL" />
-      </geometry>
-      <color rgba="1 1 0.5 1"/>
-    </visual>
-    <collision>
-      <origin xyz="0 0 0" rpy="0 0 0" />
-      <geometry>
-        <mesh filename="file://$(find pm_robot_description)/meshes/Tools/MPG_10_plus/SCHUNK_MPG-plus_Gripper_Jaw_3MM_Lens_1_Part_scaled.STL" />
-      </geometry>
-    </collision>
-  </link>
-  <!---Gravity off-->
-  <gazebo reference="Tool_Gripper_MPG_10_3mm_Lens_Jaw_1">
-    <turnGravityOff>true</turnGravityOff>
-  </gazebo>
-  <joint name="Tool_Gripper_MPG_10_3mm_Lens_Jaw_1_Joint" type="prismatic">
-    <origin xyz="0 -0.04 0" rpy="0 0 3.1416" />
-    <parent link="Tool_Gripper_MPG_10_Body" />
-    <child link="Tool_Gripper_MPG_10_3mm_Lens_Jaw_1" />
-    <axis xyz="-1 0 0" />
-    <limit lower="0" upper="0.02" effort="100" velocity="0.05" />
-  </joint>
    <!--%%%%%%%%%%%%% 1K Dispenser Flap Definitions %%%%%%%%%%%%%-->
   <link name="1K_Dispenser_Flap">

File: pm_robot_description/urdf/ros2_control.xacro (robot description, xacro)
@@ -1,4 +1,4 @@
 <?xml version="1.0"?>
-<robot xmlns:xacro="http://www.ros.org/wiki/xacro">
+<robot name="pm_robot">
     <ros2_control name="GazeboSystem" type="system">
         <hardware>
@@ -21,9 +21,4 @@
         </joint>
         <joint name="Gripper_Rot_Plate_Joint">
-            <command_interface name="position">
-            </command_interface>
-            <state_interface name="position"/>
-        </joint>
-        <joint name="Tool_Gripper_MPG_10_3mm_Lens_Jaw_1_Joint">
             <command_interface name="position">
             </command_interface>
@@ -90,4 +85,15 @@
             <state_interface name="position"/>
         </joint>
+        <!--
+        <joint name="Tool_Gripper_MPG_10_3mm_Lens_Jaw_1_Joint">
+            <command_interface name="position">
+            </command_interface>
+            <state_interface name="position"/>
+        </joint>
+        <joint name="Tool_Gripper_MPG_10_3mm_Lens_Jaw_2_Joint">
+            <command_interface name="position">
+            </command_interface>
+            <state_interface name="position"/>
+        </joint>-->
     </ros2_control>
     <gazebo>

Commit message: test

File: pm_robot_description/urdf/main.xacro (robot description, xacro)
@@ -2,6 +2,11 @@
 <robot name="pm_robot"
   xmlns:xacro="https://ros.org/wiki/xacro">
+  <!-- Configurations -->
+  <xacro:arg name="with_Tool_MPG_10" default="true" />
   <xacro:include filename="$(find pm_robot_description)/urdf/pm_robot.xacro" />
-  <xacro:include filename="$(find pm_robot_description)/urdf/pm_Schunk_Tools/MPG_10_plus.xacro" />
+  <!-- Tool Defines-->
+    <xacro:if value="$(arg with_Tool_MPG_10)">
+      <xacro:include filename="$(find pm_robot_description)/urdf/pm_Schunk_Tools/MPG_10_plus.xacro" />
+    </xacro:if>
   <xacro:include filename="$(find pm_robot_description)/urdf/ros2_control.xacro" />
   <!--xacro:include filename="$(find pm_robot_description)/urdf/MPG_10_plus_control.xacro" /-->

File: pm_robot_description/urdf/pm_Schunk_Tools/MPG_10_plus.xacro (robot description, xacro)
@@ -3,5 +3,5 @@
      Commit Version: 1.6.0-1-g15f4949  Build Version: 1.6.7594.29634
      For more information, please see http://wiki.ros.org/sw_urdf_exporter -->
-<robot name="pm_robot_MPG_10_Lens_Gripper">
+<robot name="pm_robot">
  <!--%%%%%%%%%%%%% MPG 10-plus Base Parallel Gripper Definitions %%%%%%%%%%%%%-->
   <link name="Tool_Gripper_MPG_10_Body">
@@ -119,5 +119,4 @@
     </collision>
   </link>
-  <!---Gravity off-->
   <gazebo reference="Tool_Gripper_MPG_10_3mm_Lens_Jaw_2">
     <turnGravityOff>true</turnGravityOff>

File: pm_robot_description/urdf/ros2_control.xacro (robot description, xacro)
@@ -85,5 +85,4 @@
             <state_interface name="position"/>
         </joint>
-        <!--
         <joint name="Tool_Gripper_MPG_10_3mm_Lens_Jaw_1_Joint">
             <command_interface name="position">
@@ -95,9 +94,13 @@
             </command_interface>
             <state_interface name="position"/>
-        </joint>-->
+        </joint>
     </ros2_control>
     <gazebo>
         <plugin name="gazebo_ros2_control" filename="libgazebo_ros2_control.so">
             <parameters>$(find pm_robot_description)/config/control.yaml</parameters>
+            <parameters>$(find pm_robot_description)/config/control_gripper.yaml</parameters>
+            <!--robot_param>robot_description</robot_param--> <!--The location of the robot_description (URDF) on the parameter server, defaults to robot_description-->
+            <!--robot_param_node>robot_state_publisher</robot_param_node--> <!-- Name of the node where the robot_param is located, defauls to robot_state_publisher-->
+            <!--robotNamespace>${arm_id}</robotNamespace-->
         </plugin>
     </gazebo>
