Commit message: Changes from Niklas applied

File: pm_robot_description/urdf/pm_robot_backup_copy.xacro (robot description, xacro)
@@ -17,4 +17,5 @@
     <material>Gazebo/White</material>
 </gazebo> -->
+ <!--%%%%%%%%%%%%% Base Link Definitions %%%%%%%%%%%%%-->
   <link name="base_link">
     <inertial>
@@ -28,15 +29,16 @@
         <mesh filename="file://$(find pm_robot_description)/meshes/base_link.STL" />
       </geometry>
-    </visual>
-    <collision>
-      <origin xyz="0 0 0" rpy="0 0 0" />
-      <geometry>
-        <mesh filename="file://$(find pm_robot_description)/meshes/base_link.STL" />
-      </geometry>
       <material name="">
         <color rgba="0.792156862745098 0.819607843137255 0.933333333333333 1" />
       </material>
-    </collision>
-  </link>
+    </visual>
+    <collision>
+      <origin xyz="0 0 0" rpy="0 0 0" />
+      <geometry>
+        <mesh filename="file://$(find pm_robot_description)/meshes/base_link.STL" />
+      </geometry>
+    </collision>
+  </link>
+ <!--%%%%%%%%%%%%% X Axis Definitions %%%%%%%%%%%%%-->
   <link name="X_Axis">
     <inertial>
@@ -65,4 +67,5 @@
     <limit lower="-0.745" upper="0.055" effort="1" velocity="100" />
   </joint>
+ <!--%%%%%%%%%%%%% Y Axis Definitions %%%%%%%%%%%%%-->
   <link name="Y_Axis">
     <inertial>
@@ -91,4 +94,5 @@
     <limit lower="-0.425" upper="0.2505" effort="100" velocity="100" />
   </joint>
+ <!--%%%%%%%%%%%%% Z Axis Definitions %%%%%%%%%%%%%-->
   <link name="Z_Axis">
     <inertial>
@@ -121,4 +125,5 @@
     <limit lower="-0.05262" upper="0.055" effort="100" velocity="0.05" />
   </joint>
+   <!--%%%%%%%%%%%%% T Axis Definitions %%%%%%%%%%%%%-->
   <link name="Gripper_Rot_Plate">
     <inertial>
@@ -149,11 +154,11 @@
     <child link="Gripper_Rot_Plate" />
     <axis xyz="0 0 1" />
-    <limit lower="0" upper="628319" effort="100" velocity="0.05" />
-  </joint>
+    <limit lower="0" upper="12" effort="100" velocity="2" />
+  </joint>
+  <!--
+  Gripper Definitions
   <link name="Gripper">
-    <inertial>
-      <origin xyz="-3.43029364781033E-05 -2.0382712019356E-05 0.0426309002703344" rpy="0 0 0" />
-      <mass value="0.123801210587509" />
-      <inertia ixx="2.48847691501343E-05" ixy="-1.96701975168782E-08" ixz="3.35250198834726E-09" iyy="2.52844539238953E-05" iyz="4.55516572819596E-10" izz="4.09732369514151E-05" />
+    <inertial>            </command_interface>
+" ixy="-1.96701975168782E-08" ixz="3.35250198834726E-09" iyy="2.52844539238953E-05" iyz="4.55516572819596E-10" izz="4.09732369514151E-05" />
     </inertial>
     <visual>
@@ -170,5 +175,4 @@
     </collision>
   </link>
-  <!---Gravity off-->
   <gazebo reference="Gripper">
     <turnGravityOff>true</turnGravityOff>
@@ -180,4 +184,6 @@
     <axis xyz="0 0 0" />
   </joint>
+-->
+   <!--%%%%%%%%%%%%% 1K Dispenser Flap Definitions %%%%%%%%%%%%%-->
   <link name="1K_Dispenser_Flap">
     <inertial>
@@ -210,4 +216,5 @@
     <limit lower="0" upper="0.02" effort="100" velocity="0.05" />
   </joint>
+   <!--%%%%%%%%%%%%% 1K Dispenser Definitions %%%%%%%%%%%%%-->
   <link name="1K_Dispenser">
     <inertial>
@@ -240,4 +247,5 @@
     <limit lower="0" upper="0.04" effort="100" velocity="0.05" />
   </joint>
+   <!--%%%%%%%%%%%%% 2K Dispenser Definitions-->
   <link name="2K_Dispenser">
     <inertial>
@@ -270,4 +278,5 @@
     <limit lower="0" upper="0.02" effort="100" velocity="0.05" />
   </joint>
+   <!--%%%%%%%%%%%%% Top Camera Definitions-->
   <link name="Camera_Top_View">
     <inertial>
@@ -299,4 +308,5 @@
     <axis xyz="0 0 0" />
   </joint>
+  <!--%%%%%%%%%%%%% Test Station Definitions-->
   <link name="Test_Station">
     <inertial>
@@ -324,4 +334,5 @@
     <axis xyz="0 0 0" />
   </joint>
+  <!-- %%%%%%%%%%%%% Gonio_Right Definitions-->
   <link name="Gonio_Right">
     <inertial>
@@ -349,4 +360,5 @@
     <axis xyz="0 0 0" />
   </joint>
+  <!--%%%%%%%%%%%%% Gonio_Right Stage Bottom Definitions-->
   <link name="Gonio_Right_Stage_1_Bottom">
     <inertial>
@@ -378,4 +390,5 @@
     <axis xyz="0 0 0" />
   </joint>
+  <!--%%%%%%%%%%%%% Gonio_Right Stage 1 Top Definitions-->
   <link name="Gonio_Right_Stage_1_Top">
     <inertial>
@@ -408,4 +421,5 @@
     <limit lower="-0.087266" upper="0.087266" effort="100" velocity="0.1" />
   </joint>
+   <!--%%%%%%%%%%%%% Gonio_Right Stage 2 Bottom Definitions-->
   <link name="Gonio_Right_Stage_2_Bottom">
     <inertial>
@@ -434,4 +448,5 @@
     <limit lower="-0.17453" upper="0.17453" effort="100" velocity="0.1" />
   </joint>
+  <!--%%%%%%%%%%%%% Gonio Right Holder Definitions-->
   <link name="Gonio_Right_Holder">
     <inertial>
@@ -463,6 +478,5 @@
     <axis xyz="0 0 0" />
   </joint>
-  <!--
-  <link name="Component">
+  <!-- <link name="Component">
     <inertial>
       <origin xyz="0.0347500000000016 0.0327000000000096 0.0533550000000003" rpy="0 0 0" />
@@ -492,4 +506,5 @@
     <axis xyz="0 0 0" />
   </joint> -->
+  <!--%%%%%%%%%%%%% Camera Definitions-->
   <link name="Camera_System">
     <inertial>
@@ -517,4 +532,5 @@
     <axis xyz="0 0 0" />
   </joint>
+  <!--%%%%%%%%%%%%% Camera Calibration Definitions-->
   <link name="Camera_Calibration">
     <inertial>
@@ -543,4 +559,5 @@
     <limit lower="-0.04" upper="0.0" effort="100" velocity="0.05" />
   </joint>
+  <!--%%%%%%%%%%%%% Gonio Station Left Definitions-->
   <link name="Gonio_Station_Left">
     <inertial>
@@ -568,4 +585,5 @@
     <axis xyz="0 0 0" />
   </joint>
+<!--%%%%%%%%%%%%% Gonio Left Stage 1 Top Definitions-->
   <link name="Gonio_Left_Stage_1_Top">
     <inertial>
@@ -598,4 +616,5 @@
     <limit lower="-0.78539816339745" upper="0.78539816339745" effort="100" velocity="0.1" />
   </joint>
+<!--%%%%%%%%%%%%% Gonio Left Stage 2 Bottom Definitions-->
   <link name="Gonio_Left_Stage_2_Bottom">
     <inertial>
@@ -628,4 +647,5 @@
     <limit lower="-0.78539816339745" upper="0.78539816339745" effort="100" velocity="0.1" />
   </joint>
+  <!--%%%%%%%%%%%%% Gonio Left Holder Definitions-->
   <link name="Gonio_Left_Holder">
     <inertial>
@@ -657,4 +677,5 @@
     <axis xyz="0 0 0" />
   </joint>
+  <!--%%%%%%%%%%%%% UV Slider X Front Definitions-->
   <link name="UV_Slider_X_Front">
     <inertial>
@@ -683,4 +704,5 @@
     <limit lower="-0.05" upper="0.095" effort="100" velocity="0.05" />
   </joint>
+  <!--%%%%%%%%%%%%% UV LED Front Definitions-->
   <link name="UV_LED_Front">
     <inertial>
@@ -709,4 +731,5 @@
     <limit lower="0.045" upper="0.045" effort="100" velocity="0.05" />
   </joint>
+  <!--%%%%%%%%%%%%% UV Slider X Back Definitions-->
   <link name="UV_Slider_X_Back">
     <inertial>
@@ -735,4 +758,5 @@
     <limit lower="-0.045" upper="0.045" effort="0.05" velocity="100" />
   </joint>
+   <!--%%%%%%%%%%%%% UV LED Back Definitions-->
   <link name="UV_LED_Back">
     <inertial>

File: pm_robot_description/urdf/ros2_control.xacro (robot description, xacro)
@@ -1,4 +1,4 @@
 <?xml version="1.0"?>
-<robot xmlns:xacro="http://www.ros.org/wiki/xacro">
+<robot name="pm_robot">
     <ros2_control name="GazeboSystem" type="system">
         <hardware>
@@ -6,7 +6,8 @@
         </hardware>
         <joint name="X_Axis_Joint">
-            <command_interface name="position">
-            </command_interface>
+            <command_interface name="position"/>
+            <!-- <command_interface name="velocity"/> -->
             <state_interface name="position"/>
+            <state_interface name="velocity"/>
         </joint>
         <joint name="Y_Axis_Joint">
@@ -14,4 +15,5 @@
             </command_interface>
             <state_interface name="position"/>
+            <state_interface name="velocity"/>
         </joint>
         <joint name="Z_Axis_Joint">
@@ -19,4 +21,5 @@
             </command_interface>
             <state_interface name="position"/>
+            <state_interface name="velocity"/>
         </joint>
         <joint name="Gripper_Rot_Plate_Joint">
@@ -24,4 +27,5 @@
             </command_interface>
             <state_interface name="position"/>
+            <state_interface name="velocity"/>
         </joint>
         <joint name="1K_Dispenser_Flap_Joint">
@@ -85,8 +89,26 @@
             <state_interface name="position"/>
         </joint>
+        <joint name="Tool_Gripper_MPG_10_Jaw_1_Joint">
+            <command_interface name="position">
+            </command_interface>
+            <state_interface name="position"/>
+        </joint>
+        <joint name="Tool_Gripper_MPG_10_Jaw_2_Joint">
+            <param name="mimic">Tool_Gripper_MPG_10_Jaw_1_Joint</param>
+            <param name="mulltiplier">1</param>
+            <command_interface name="position">
+            </command_interface>
+            <state_interface name="position"/>
+        </joint>
     </ros2_control>
     <gazebo>
         <plugin name="gazebo_ros2_control" filename="libgazebo_ros2_control.so">
-            <parameters>$(find pm_robot_description)/config/control.yaml</parameters>
+            <parameters>$(find pm_robot_description)/config/pm_robot_control.yaml</parameters>
+            <parameters>$(find pm_robot_description)/config/pm_robot_control_gonio_right.yaml</parameters>
+            <parameters>$(find pm_robot_description)/config/pm_robot_control_gonio_left.yaml</parameters>
+            <parameters>$(find pm_robot_description)/config/pm_robot_control_gripper.yaml</parameters>
+            <!--robot_param>robot_description</robot_param--> <!--The location of the robot_description (URDF) on the parameter server, defaults to robot_description-->
+            <!--robot_param_node>robot_state_publisher</robot_param_node--> <!-- Name of the node where the robot_param is located, defauls to robot_state_publisher-->
+            <!--robotNamespace>${arm_id}</robotNamespace-->
         </plugin>
     </gazebo>
