Commit message: Bottom View Cam added

File: pm_robot_description/urdf/sensors.urdf (robot description, URDF)
Before this commit: robot pm_robot, 3 links, 3 joints
Links:
- removed link camera_link
- removed link camera_link_optical
- added link Camera_Bottom_View_Link
- added link Camera_Bottom_View_Link_Optical
- added link Camera_Top_View_Link
- added link Camera_Top_View_Link_Optical
Joints:
- removed joint camera_joint
- removed joint camera_optical_joint
- added joint Camera_Bottom_View_Joint: type fixed, parent Camera_System, child Camera_Bottom_View_Link, origin xyz=0.0645 0.287 0.246 rpy=0 -1.570796 0 
- added joint Camera_Bottom_View_Link_Optical_Joint: type fixed, parent Camera_Bottom_View_Link, child Camera_Bottom_View_Link_Optical, origin xyz=0 0 0 rpy=-1.570796 0 -1.570796 
- added joint Camera_Top_View_Link_Joint: type fixed, parent Camera_Top_View, child Camera_Top_View_Link, origin xyz=0.02 0.021 -0.16 rpy=0 1.570796 0 
- added joint Camera_Top_View_Link_Optical_Joint: type fixed, parent Camera_Top_View_Link, child Camera_Top_View_Link_Optical, origin xyz=0 0 0 rpy=-1.570796 0 -1.570796 

Commit message: h_fov bottom cam

File: pm_robot_description/urdf/sensors.urdf (robot description, URDF)
Before this commit: robot pm_robot, 5 links, 5 joints
Joints:
- joint Camera_Bottom_View_Joint: origin xyz=0.0645 0.287 0.246 rpy=0 -1.570796 0  -> xyz=0.0645 0.287 -2.754 rpy=0 -1.570796 0 

Commit message: bottom light

File: pm_robot_description/urdf/sensors.urdf (robot description, URDF)
Before this commit: robot pm_robot, 5 links, 5 joints
Joints:
- joint Camera_Bottom_View_Joint: origin xyz=0.0645 0.287 -2.754 rpy=0 -1.570796 0  -> xyz=0.0645 0.287 -0.754 rpy=0 -1.570796 0 
