Commit message: troubleshoot

File: pm_robot_description/urdf/ros2_control_fake_HW.xacro (robot description, xacro)
@@ -2,5 +2,5 @@
 <robot xmlns:xacro="http://www.ros.org/wiki/xacro">
     <xacro:macro name="pm_robot_ros2_control_hw_fake" params="name initial_positions_file">
-        <xacro:property name="initial_positions" value="${load_yaml(initial_positions_file)['initial_positions']}"/>
+        <xacro:property name="initial_positions" value="${xacro.load_yaml(initial_positions_file)['initial_positions']}"/>
         <ros2_control name="${name}" type="system">
             <hardware>

File: pm_robot_description/urdf/ros2_control_sim_HW.xacro (robot description, xacro)
@@ -2,5 +2,5 @@
 <robot xmlns:xacro="http://www.ros.org/wiki/xacro">
     <xacro:macro name="pm_robot_ros2_control_hw_sim" params="name initial_positions_file">
-        <xacro:property name="initial_positions" value="${load_yaml(initial_positions_file)['initial_positions']}"/>
+        <xacro:property name="initial_positions" value="${xacro.load_yaml(initial_positions_file)['initial_positions']}"/>
         <ros2_control name="GazeboSystem" type="system">
             <hardware>
@@ -10,5 +10,7 @@
                 <command_interface name="position"/>
                 <!-- <command_interface name="velocity"/> -->
-                <state_interface name="position"/>
+                <state_interface name="position">
+                    <param name="initial_value">${initial_positions['X_Axis_Joint']}</param>
+                </state_interface>
                 <state_interface name="velocity"/>
             </joint>
@@ -16,5 +18,7 @@
                 <command_interface name="position">
                 </command_interface>
-                <state_interface name="position"/>
+                <state_interface name="position">
+                    <param name="initial_value">${initial_positions['Y_Axis_Joint']}</param>
+                </state_interface>
                 <state_interface name="velocity"/>
             </joint>
@@ -22,5 +26,7 @@
                 <command_interface name="position">
                 </command_interface>
-                <state_interface name="position"/>
+                <state_interface name="position">
+                    <param name="initial_value">${initial_positions['Z_Axis_Joint']}</param>
+                </state_interface>
                 <state_interface name="velocity"/>
             </joint>
@@ -28,5 +34,7 @@
                 <command_interface name="position">
                 </command_interface>
-                <state_interface name="position"/>
+                <state_interface name="position">
+                    <param name="initial_value">${initial_positions['T_Axis_Joint']}</param>
+                </state_interface>
                 <state_interface name="velocity"/>
             </joint>
