Commit message: moveit.srdf

File: pm_robot_description/urdf/match_logo.urdf.xacro (robot description, xacro)
@@ -10,4 +10,11 @@
                 <material name="match_green"/>
 			</visual>
+			<collision>
+				<origin xyz="0 0 0" rpy="0 0 0" />
+				<geometry>
+					<mesh filename="file://$(find pm_robot_description)/meshes/Housing/match_background.dae" scale="0.001 0.001 0.001" />
+				</geometry>
+                <material name="match_green"/>
+			</collision>
 		</link>
 		<joint name="${locationprefix}_match_logo_joint" type="fixed">
@@ -24,4 +31,11 @@
                 <material name="white"/>
 			</visual>
+			<collision>
+				<origin xyz="0 0 0 " rpy="${pi/2} 0 ${pi}" />
+				<geometry>
+					<mesh filename="file://$(find pm_robot_description)/meshes/Housing/match_font.stl" scale="0.01 0.01 0.01" />
+				</geometry>
+                <material name="white"/>
+			</collision>
 		</link>
 		<joint name="${locationprefix}_match_logo_font_joint" type="fixed">

File: pm_robot_description/urdf/pm_robot.xacro (robot description, xacro)
@@ -196,5 +196,5 @@
         <origin xyz="-1.74281094778017E-07 2.03483659588777E-07 0.00907792340584457" rpy="0 0 0" />
         <mass value="0.110297257842221" />
-        <inertia ixx="8.79759467929701E-05" ixy="1.90651210379881E-10" ixz="1.25536613370482E-10" iyy="8.79764882626525E-05" iyz="-1.50065581017382E-10" izz="0.00016565987032676" />
+        <inertia ixx="8.79759467929701E-05" ixy="1.90651210379881E-6" ixz="1.25536613370482E-6" iyy="8.79764882626525E-05" iyz="-1.50065581017382E-6" izz="0.00016565987032676" />
       </inertial>
       <visual>
@@ -227,5 +227,5 @@
         <origin xyz="2.66657822625138E-05 -6.51697797860451E-05 -0.0173989628147272" rpy="0 0 0" />
         <mass value="0.0741175653990944" />
-        <inertia ixx="1.38724675369177E-05" ixy="-2.81065278601148E-08" ixz="-4.32931581160332E-09" iyy="1.28173377099281E-05" iyz="-3.69738102041932E-10" izz="2.32495071670115E-05" />
+        <inertia ixx="1.38724675369177E-05" ixy="-2.81065278601148E-08" ixz="-4.32931581160332E-09" iyy="1.28173377099281E-05" iyz="-3.69738102041932E-6" izz="2.32495071670115E-05" />
       </inertial>
       <visual>
@@ -560,5 +560,5 @@
         <origin xyz="0.0250000000000002 0.0791274046351475 -0.154851137332961" rpy="0 0 0" />
         <mass value="1.39099524679326" />
-        <inertia ixx="0.00780193904512034" ixy="-2.61717009512019E-14" ixz="-4.79910370720457E-20" iyy="0.00547600691976027" iyz="9.87499782602546E-10" izz="0.00281708795214926" />
+        <inertia ixx="0.00780193904512034" ixy="-2.61717009512019E-6" ixz="-4.79910370720457E-6" iyy="0.00547600691976027" iyz="9.87499782602546E-6" izz="0.00281708795214926" />
       </inertial>
       <visual>
@@ -676,5 +676,5 @@
         <origin xyz="-0.000344499007125409 0.0696122748122424 0.000295151280628292" rpy="0 0 0" />
         <mass value="0.0334016358510876" />
-        <inertia ixx="2.05104945364406E-05" ixy="-1.61006130053269E-08" ixz="-7.42638002033627E-11" iyy="2.64967112268826E-06" iyz="4.64472618194223E-07" izz="2.23824646029018E-05" />
+        <inertia ixx="2.05104945364406E-05" ixy="-1.61006130053269E-08" ixz="-7.42638002033627E-6" iyy="2.64967112268826E-06" iyz="4.64472618194223E-07" izz="2.23824646029018E-05" />
       </inertial>
       <visual>
@@ -702,7 +702,7 @@
     <link name="Calibration_Qube">
       <inertial>
-        <origin xyz="0 -5.55111512312578E-17 -0.007418215969486" rpy="0 0 0" />
+        <origin xyz="0 -5.55111512312578E-6 -0.007418215969486" rpy="0 0 0" />
         <mass value="0.000608132735199849" />
-        <inertia ixx="3.05434929012605E-04" ixy="2.70098962651108E-25" ixz="-1.09265340380468E-24" iyy="3.05434929012605E-04" iyz="6.45610037231024E-25" izz="5.52989859299796E-04" />
+        <inertia ixx="3.05434929012605E-04" ixy="2.70098962651108E-6" ixz="-1.09265340380468E-6" iyy="3.05434929012605E-04" iyz="6.45610037231024E-6" izz="5.52989859299796E-04" />
       </inertial>
       <visual>
