Commit message: Gonio real HW

File: pm_robot_description/urdf/ros2_control_real_HW.xacro (robot description, xacro)
@@ -10,6 +10,6 @@
             </hardware>
             <joint name="X_Axis_Joint">
-                <command_interface name="position"/>
-                <!-- <command_interface name="velocity"/> -->
+                <command_interface name="position">
+                </command_interface>
                 <state_interface name="position"/>
                 <state_interface name="velocity"/>
@@ -47,9 +47,10 @@
                 </command_interface>
                 <state_interface name="position"/>
-            </joint>
-            <joint name="Gonio_Right_Stage_1_Joint">
+            </joint> -->
+            <!-- <joint name="Gonio_Right_Stage_1_Joint">
                 <command_interface name="position">
                 </command_interface>
                 <state_interface name="position"/>
+                <state_interface name="velocity"/>
             </joint>
             <joint name="Gonio_Right_Stage_2_Joint">
@@ -57,11 +58,12 @@
                 </command_interface>
                 <state_interface name="position"/>
-            </joint>
-            <joint name="Camera_Calibration_Platelet_Joint">
+                <state_interface name="velocity"/>
+            </joint> -->
+            <!-- <joint name="Camera_Calibration_Platelet_Joint">
                 <command_interface name="position">
                 </command_interface>
                 <state_interface name="position"/>
-            </joint>
-            <joint name="Gonio_Left_Stage_1_Joint">
+            </joint> -->
+            <!-- <joint name="Gonio_Left_Stage_1_Joint">
                 <command_interface name="position">
                 </command_interface>
@@ -72,6 +74,6 @@
                 </command_interface>
                 <state_interface name="position"/>
-            </joint>
-            <joint name="UV_Slider_X_Front_Joint">
+            </joint> -->
+            <!-- <joint name="UV_Slider_X_Front_Joint">
                 <command_interface name="position">
                 </command_interface>

Commit message: urdf changes hw_interface fix

File: pm_robot_description/urdf/ros2_control_real_HW.xacro (robot description, xacro)
@@ -69,11 +69,11 @@
                 </command_interface>
                 <state_interface name="position"/>
-            </joint> -->
-            <!-- <joint name="Camera_Calibration_Platelet_Joint">
+            </joint>
+            <joint name="Camera_Calibration_Platelet_Joint">
                 <command_interface name="position">
                 </command_interface>
                 <state_interface name="position"/>
-            </joint> -->
-            <!-- <joint name="UV_Slider_X_Front_Joint">
+            </joint>
+            <joint name="UV_Slider_X_Front_Joint">
                 <command_interface name="position">
                 </command_interface>
@@ -99,6 +99,6 @@
                 </command_interface>
                 <state_interface name="position"/>
-            </joint>
-            <xacro:if value="$(arg with_Tool_MPG_10)">
+            </joint> -->
+            <!-- <xacro:if value="$(arg with_Tool_MPG_10)">
                 <joint name="pm_robot_Tool_Parallel_Joint">
                     <command_interface name="position">
@@ -115,5 +115,6 @@
                     <state_interface name="velocity"/>
                 </joint>
-            </xacro:if> -->
+            </xacro:if>  -->
+            <!-- Only if gripper with two jaws is selected -->
             <xacro:if value="${current_pm_robot_bringup_config['pm_robot_tools']['pm_robot_tool_parallel_gripper_2_jaws']['use_paralell_gripper']}">
                 <joint name="Tool_Parallel_Gripper_Jaw_1_Joint">
@@ -123,5 +124,5 @@
                     <state_interface name="velocity"/>
                 </joint>
-               <joint name="Tool_Parallel_Gripper_Jaw_2_Joint">
+                <joint name="Tool_Parallel_Gripper_Jaw_2_Joint">
                     <command_interface name="position">
                     </command_interface>
