Commit message: modular Launch Files, Axis renaming

File: pm_robot_description/urdf/pm_robot_gonio_left.xacro (robot description, xacro)
@@ -56,4 +56,5 @@
     <turnGravityOff>true</turnGravityOff>
   </gazebo>
+<<<<<<< HEAD
   <joint name="Gonio_Left_Stage_1_Top_Joint" type="revolute">
     <origin xyz="-0.385 0.0855 0.1847" rpy="0 0 0" />
@@ -61,4 +62,18 @@
     <child link="Gonio_Left_Stage_1_Top" />
     <axis xyz="1 0 0" />
+=======
+  <joint
+    name="Gonio_Left_Stage_1_Joint"
+    type="revolute">
+    <origin
+      xyz="0.188500000000042 0.110000000000054 0.212499999999997"
+      rpy="0 0 0" />
+    <parent
+      link="Gonio_Left_Base" />
+    <child
+      link="Gonio_Left_Stage_1_Top" />
+    <axis
+      xyz="1 0 0" />
+>>>>>>> f5d9834 (modular Launch Files, Axis renaming)
     <limit lower="-0.17453" upper="0.17453" effort="100" velocity="0.1" />
   </joint>
@@ -85,7 +100,8 @@
   </link>
   <!---Gravity off-->
-  <gazebo reference="Gonio_Left_Stage_2_Bottom">
+  <gazebo reference="Gonio_Left_Stage_2_Joint">
     <turnGravityOff>true</turnGravityOff>
   </gazebo>
+<<<<<<< HEAD
   <joint name="Gonio_Left_Stage_2_Bottom_Joint" type="revolute">
     <origin xyz="0.5015 0.0495 0.0278" rpy="0 0 0" />
@@ -97,4 +113,56 @@
   <!--%%%%%%%%%%%%% Gonio Left Holder Definitions-->
   <link name="Gonio_Left_Holder">
+=======
+  <joint
+    name="Gonio_Left_Stage_2_Joint"
+    type="revolute">
+    <origin
+      xyz="0 0 0"
+      rpy="0 0 0" />
+    <parent
+      link="Gonio_Left_Stage_1_Top" />
+    <child
+      link="Gonio_Left_Stage_2_Bottom" />
+    <axis
+      xyz="0.0334865202089474 -0.999439169216564 0" />
+    <limit lower="-0.17453" upper="0.17453" effort="100" velocity="0.1" />
+  </joint>
+  <!--%%%%%%%%%%%%% Gonio Left Chuck Definitions-->
+  <link
+    name="Gonio_Left_Chuck">
+  </link>
+  <joint
+    name="Gonio_Left_Chuck_Joint"
+    type="fixed">
+    <origin
+      xyz="0 0 -0.015"
+      rpy="0 0 0" />
+    <parent
+      link="Gonio_Left_Stage_2_Bottom" />
+    <child
+      link="Gonio_Left_Chuck" />
+    <axis
+      xyz="0 0 0" />
+  </joint>
+  <link
+    name="Gonio_Left_Part_Origin">
+  </link>
+  <joint
+    name="Gonio_Left_Part_Origin_Joint"
+    type="fixed">
+    <origin
+      xyz="0 0 0"
+      rpy="0 0 0" />
+    <parent
+      link="Gonio_Left_Chuck" />
+    <child
+      link="Gonio_Left_Part_Origin" />
+    <axis
+      xyz="0 0 0" />
+  </joint>
+  <!--%%%%%%%%%%%%% Gonio Left Example Chuck Definitions-->
+  <link
+    name="Gonio_Left_Example_Chuck">
+>>>>>>> f5d9834 (modular Launch Files, Axis renaming)
     <inertial>
       <origin xyz="-8.16234952583095E-06 0.000868103725036456 0.0372986798808728" rpy="0 0 0" />

File: pm_robot_description/urdf/pm_robot_gonio_right.xacro (robot description, xacro)
@@ -87,4 +87,5 @@
     <turnGravityOff>true</turnGravityOff>
   </gazebo>
+<<<<<<< HEAD
   <joint name="Gonio_Right_Stage_1_Top_Joint" type="revolute">
     <origin xyz="0 0.0325 0.11" rpy="0 0 0" />
@@ -92,4 +93,18 @@
     <child link="Gonio_Right_Stage_1_Top" />
     <axis xyz="1 0 0" />
+=======
+  <joint
+    name="Gonio_Right_Stage_1_Joint"
+    type="revolute">
+    <origin
+      xyz="0.0324999999999993 0.0326774999999999 0.11"
+      rpy="0 0 0" />
+    <parent
+      link="Gonio_Right_Stage_1_Bottom" />
+    <child
+      link="Gonio_Right_Stage_1_Top" />
+    <axis
+      xyz="0 -1 0" />
+>>>>>>> f5d9834 (modular Launch Files, Axis renaming)
     <limit lower="-0.087266" upper="0.087266" effort="100" velocity="0.1" />
   </joint>
@@ -119,4 +134,5 @@
     <turnGravityOff>true</turnGravityOff>
   </gazebo>
+<<<<<<< HEAD
   <joint name="Gonio_Right_Stage_2_Bottom_Joint" type="revolute">
     <origin xyz="0.0325 0.0325 0" rpy="0 0 0" />
@@ -124,4 +140,18 @@
     <child link="Gonio_Right_Stage_2_Bottom" />
     <axis xyz="0 -1 0" />
+=======
+  <joint
+    name="Gonio_Right_Stage_2_Joint"
+    type="revolute">
+    <origin
+      xyz="0 0 0"
+      rpy="0 0 0" />
+    <parent
+      link="Gonio_Right_Stage_1_Top" />
+    <child
+      link="Gonio_Right_Stage_2_Bottom" />
+    <axis
+      xyz="-1 0 0" />
+>>>>>>> f5d9834 (modular Launch Files, Axis renaming)
     <limit lower="-0.17453" upper="0.17453" effort="100" velocity="0.1" />
   </joint>

File: pm_robot_description/urdf/ros2_control_gazebo.xacro (robot description, xacro)
@@ -89,4 +89,5 @@
             <state_interface name="position"/>
         </joint>
+<<<<<<< HEAD
         <joint name="Tool_Gripper_MPG_10_Jaw_1_Joint">
             <command_interface name="position">
@@ -94,4 +95,84 @@
             <state_interface name="position"/>
         </joint>
+=======
+            </joint>
+            <joint name="Z_Axis_Joint">
+                <command_interface name="position">
+                </command_interface>
+                <state_interface name="position"/>
+                <state_interface name="velocity"/>
+            </joint>
+            <joint name="T_Axis_Joint">
+                <command_interface name="position">
+                </command_interface>
+                <state_interface name="position"/>
+                <state_interface name="velocity"/>
+            </joint>
+            <joint name="1K_Dispenser_Flap_Joint">
+                <command_interface name="position">
+                </command_interface>
+                <state_interface name="position"/>
+            </joint>
+            <joint name="1K_Dispenser_Joint">
+                <command_interface name="position">
+                </command_interface>
+                <state_interface name="position"/>
+            </joint>
+            <joint name="2K_Dispenser_Joint">
+                <command_interface name="position">
+                </command_interface>
+                <state_interface name="position"/>
+            </joint>
+            <joint name="Gonio_Right_Stage_1_Joint">
+                <command_interface name="position">
+                </command_interface>
+                <state_interface name="position"/>
+            </joint>
+            <joint name="Gonio_Right_Stage_2_Joint">
+                <command_interface name="position">
+                </command_interface>
+                <state_interface name="position"/>
+            </joint>
+            <joint name="Camera_Calibration_Platelet_Joint">
+                <command_interface name="position">
+                </command_interface>
+                <state_interface name="position"/>
+            </joint>
+            <joint name="Gonio_Left_Stage_1_Joint">
+                <command_interface name="position">
+                </command_interface>
+                <state_interface name="position"/>
+            </joint>
+            <joint name="Gonio_Left_Stage_2_Joint">
+                <command_interface name="position">
+                </command_interface>
+                <state_interface name="position"/>
+            </joint>
+            <joint name="UV_Slider_X_Front_Joint">
+                <command_interface name="position">
+                </command_interface>
+                <state_interface name="position"/>
+            </joint>
+            <joint name="UV_LED_Front_Joint">
+                <command_interface name="position">
+                </command_interface>
+                <state_interface name="position"/>
+            </joint>
+            <joint name="UV_Slider_X_Back_Joint">
+                <command_interface name="position">
+                </command_interface>
+                <state_interface name="position"/>
+            </joint>
+            <joint name="UV_LED_Back_Joint">
+                <command_interface name="position">
+                </command_interface>
+                <state_interface name="position"/>
+            </joint>
+            <joint name="Calibration_Qube_Joint">
+                <command_interface name="position">
+                </command_interface>
+                <state_interface name="position"/>
+            </joint>
+>>>>>>> f5d9834 (modular Launch Files, Axis renaming)
         <joint name="Tool_Gripper_MPG_10_Jaw_2_Joint">
             <param name="mimic">Tool_Gripper_MPG_10_Jaw_1_Joint</param>

Commit message: modular Launch Files, Axis renaming

File: pm_robot_description/urdf/pm_robot_gonio_left.xacro (robot description, xacro)
@@ -92,5 +92,5 @@
   </gazebo>
   <joint
-    name="Gonio_Left_Stage_1_Top_Joint"
+    name="Gonio_Left_Stage_1_Joint"
     type="revolute">
     <origin
@@ -141,9 +141,9 @@
   </link>
   <!---Gravity off-->
-  <gazebo reference="Gonio_Left_Stage_2_Bottom">
+  <gazebo reference="Gonio_Left_Stage_2_Joint">
     <turnGravityOff>true</turnGravityOff>
   </gazebo>
   <joint
-    name="Gonio_Left_Stage_2_Bottom_Joint"
+    name="Gonio_Left_Stage_2_Joint"
     type="revolute">
     <origin
@@ -176,8 +176,8 @@
   </joint>
   <link
-    name="Gonio_Left_Part_Base">
-  </link>
-  <joint
-    name="Gonio_Left_Part_Base_Joint"
+    name="Gonio_Left_Part_Origin">
+  </link>
+  <joint
+    name="Gonio_Left_Part_Origin_Joint"
     type="fixed">
     <origin
@@ -187,5 +187,5 @@
       link="Gonio_Left_Chuck" />
     <child
-      link="Gonio_Left_Part_Base" />
+      link="Gonio_Left_Part_Origin" />
     <axis
       xyz="0 0 0" />

File: pm_robot_description/urdf/pm_robot_gonio_right.xacro (robot description, xacro)
@@ -144,5 +144,5 @@
   </gazebo>
   <joint
-    name="Gonio_Right_Stage_1_Top_Joint"
+    name="Gonio_Right_Stage_1_Joint"
     type="revolute">
     <origin
@@ -197,5 +197,5 @@
   </gazebo>
   <joint
-    name="Gonio_Right_Stage_2_Bottom_Joint"
+    name="Gonio_Right_Stage_2_Joint"
     type="revolute">
     <origin

File: pm_robot_description/urdf/pm_robot_housing.xacro (robot description, xacro)
@@ -216,5 +216,5 @@
         <mesh filename="file://$(find pm_robot_description)/meshes/Housing/housing.STL" />
       </geometry>
-      <material name="black"/>
+      <material name="grey"/>
     </visual>
     <collision>

File: pm_robot_description/urdf/ros2_control_fake.xacro (robot description, xacro)
@@ -47,10 +47,10 @@
                 <state_interface name="position"/>
             </joint>
-            <joint name="Gonio_Right_Stage_1_Top_Joint">
+            <joint name="Gonio_Right_Stage_1_Joint">
                 <command_interface name="position">
                 </command_interface>
                 <state_interface name="position"/>
             </joint>
-            <joint name="Gonio_Right_Stage_2_Bottom_Joint">
+            <joint name="Gonio_Right_Stage_2_Joint">
                 <command_interface name="position">
                 </command_interface>
@@ -62,10 +62,10 @@
                 <state_interface name="position"/>
             </joint>
-            <joint name="Gonio_Left_Stage_1_Top_Joint">
+            <joint name="Gonio_Left_Stage_1_Joint">
                 <command_interface name="position">
                 </command_interface>
                 <state_interface name="position"/>
             </joint>
-            <joint name="Gonio_Left_Stage_2_Bottom_Joint">
+            <joint name="Gonio_Left_Stage_2_Joint">
                 <command_interface name="position">
                 </command_interface>

File: pm_robot_description/urdf/ros2_control_gazebo.xacro (robot description, xacro)
@@ -46,10 +46,10 @@
                 <state_interface name="position"/>
             </joint>
-            <joint name="Gonio_Right_Stage_1_Top_Joint">
+            <joint name="Gonio_Right_Stage_1_Joint">
                 <command_interface name="position">
                 </command_interface>
                 <state_interface name="position"/>
             </joint>
-            <joint name="Gonio_Right_Stage_2_Bottom_Joint">
+            <joint name="Gonio_Right_Stage_2_Joint">
                 <command_interface name="position">
                 </command_interface>
@@ -61,10 +61,10 @@
                 <state_interface name="position"/>
             </joint>
-            <joint name="Gonio_Left_Stage_1_Top_Joint">
+            <joint name="Gonio_Left_Stage_1_Joint">
                 <command_interface name="position">
                 </command_interface>
                 <state_interface name="position"/>
             </joint>
-            <joint name="Gonio_Left_Stage_2_Bottom_Joint">
+            <joint name="Gonio_Left_Stage_2_Joint">
                 <command_interface name="position">
                 </command_interface>

File: pm_robot_description/urdf/ros2_control_real.xacro (robot description, xacro)
@@ -46,10 +46,10 @@
                 <state_interface name="position"/>
             </joint>
-            <joint name="Gonio_Right_Stage_1_Top_Joint">
+            <joint name="Gonio_Right_Stage_1_Joint">
                 <command_interface name="position">
                 </command_interface>
                 <state_interface name="position"/>
             </joint>
-            <joint name="Gonio_Right_Stage_2_Bottom_Joint">
+            <joint name="Gonio_Right_Stage_2_Joint">
                 <command_interface name="position">
                 </command_interface>
@@ -61,10 +61,10 @@
                 <state_interface name="position"/>
             </joint>
-            <joint name="Gonio_Left_Stage_1_Top_Joint">
+            <joint name="Gonio_Left_Stage_1_Joint">
                 <command_interface name="position">
                 </command_interface>
                 <state_interface name="position"/>
             </joint>
-            <joint name="Gonio_Left_Stage_2_Bottom_Joint">
+            <joint name="Gonio_Left_Stage_2_Joint">
                 <command_interface name="position">
                 </command_interface>
@@ -87,9 +87,4 @@
             </joint>
             <joint name="UV_LED_Back_Joint">
-                <command_interface name="position">
-                </command_interface>
-                <state_interface name="position"/>
-            </joint>
-            <joint name="Tool_Gripper_MPG_10_Jaw_1_Joint">
                 <command_interface name="position">
                 </command_interface>

Commit message: Revert "modular Launch Files, Axis renaming"
This reverts commit e68d30bb21ecd78b5d3f6222b4a81be18c2a7f21.

File: pm_robot_description/urdf/pm_robot_gonio_left.xacro (robot description, xacro)
@@ -56,5 +56,4 @@
     <turnGravityOff>true</turnGravityOff>
   </gazebo>
-<<<<<<< HEAD
   <joint name="Gonio_Left_Stage_1_Top_Joint" type="revolute">
     <origin xyz="-0.385 0.0855 0.1847" rpy="0 0 0" />
@@ -62,18 +61,4 @@
     <child link="Gonio_Left_Stage_1_Top" />
     <axis xyz="1 0 0" />
-=======
-  <joint
-    name="Gonio_Left_Stage_1_Joint"
-    type="revolute">
-    <origin
-      xyz="0.188500000000042 0.110000000000054 0.212499999999997"
-      rpy="0 0 0" />
-    <parent
-      link="Gonio_Left_Base" />
-    <child
-      link="Gonio_Left_Stage_1_Top" />
-    <axis
-      xyz="1 0 0" />
->>>>>>> f5d9834 (modular Launch Files, Axis renaming)
     <limit lower="-0.17453" upper="0.17453" effort="100" velocity="0.1" />
   </joint>
@@ -100,8 +85,7 @@
   </link>
   <!---Gravity off-->
-  <gazebo reference="Gonio_Left_Stage_2_Joint">
+  <gazebo reference="Gonio_Left_Stage_2_Bottom">
     <turnGravityOff>true</turnGravityOff>
   </gazebo>
-<<<<<<< HEAD
   <joint name="Gonio_Left_Stage_2_Bottom_Joint" type="revolute">
     <origin xyz="0.5015 0.0495 0.0278" rpy="0 0 0" />
@@ -113,56 +97,4 @@
   <!--%%%%%%%%%%%%% Gonio Left Holder Definitions-->
   <link name="Gonio_Left_Holder">
-=======
-  <joint
-    name="Gonio_Left_Stage_2_Joint"
-    type="revolute">
-    <origin
-      xyz="0 0 0"
-      rpy="0 0 0" />
-    <parent
-      link="Gonio_Left_Stage_1_Top" />
-    <child
-      link="Gonio_Left_Stage_2_Bottom" />
-    <axis
-      xyz="0.0334865202089474 -0.999439169216564 0" />
-    <limit lower="-0.17453" upper="0.17453" effort="100" velocity="0.1" />
-  </joint>
-  <!--%%%%%%%%%%%%% Gonio Left Chuck Definitions-->
-  <link
-    name="Gonio_Left_Chuck">
-  </link>
-  <joint
-    name="Gonio_Left_Chuck_Joint"
-    type="fixed">
-    <origin
-      xyz="0 0 -0.015"
-      rpy="0 0 0" />
-    <parent
-      link="Gonio_Left_Stage_2_Bottom" />
-    <child
-      link="Gonio_Left_Chuck" />
-    <axis
-      xyz="0 0 0" />
-  </joint>
-  <link
-    name="Gonio_Left_Part_Origin">
-  </link>
-  <joint
-    name="Gonio_Left_Part_Origin_Joint"
-    type="fixed">
-    <origin
-      xyz="0 0 0"
-      rpy="0 0 0" />
-    <parent
-      link="Gonio_Left_Chuck" />
-    <child
-      link="Gonio_Left_Part_Origin" />
-    <axis
-      xyz="0 0 0" />
-  </joint>
-  <!--%%%%%%%%%%%%% Gonio Left Example Chuck Definitions-->
-  <link
-    name="Gonio_Left_Example_Chuck">
->>>>>>> f5d9834 (modular Launch Files, Axis renaming)
     <inertial>
       <origin xyz="-8.16234952583095E-06 0.000868103725036456 0.0372986798808728" rpy="0 0 0" />

File: pm_robot_description/urdf/pm_robot_gonio_right.xacro (robot description, xacro)
@@ -87,5 +87,4 @@
     <turnGravityOff>true</turnGravityOff>
   </gazebo>
-<<<<<<< HEAD
   <joint name="Gonio_Right_Stage_1_Top_Joint" type="revolute">
     <origin xyz="0 0.0325 0.11" rpy="0 0 0" />
@@ -93,18 +92,4 @@
     <child link="Gonio_Right_Stage_1_Top" />
     <axis xyz="1 0 0" />
-=======
-  <joint
-    name="Gonio_Right_Stage_1_Joint"
-    type="revolute">
-    <origin
-      xyz="0.0324999999999993 0.0326774999999999 0.11"
-      rpy="0 0 0" />
-    <parent
-      link="Gonio_Right_Stage_1_Bottom" />
-    <child
-      link="Gonio_Right_Stage_1_Top" />
-    <axis
-      xyz="0 -1 0" />
->>>>>>> f5d9834 (modular Launch Files, Axis renaming)
     <limit lower="-0.087266" upper="0.087266" effort="100" velocity="0.1" />
   </joint>
@@ -134,5 +119,4 @@
     <turnGravityOff>true</turnGravityOff>
   </gazebo>
-<<<<<<< HEAD
   <joint name="Gonio_Right_Stage_2_Bottom_Joint" type="revolute">
     <origin xyz="0.0325 0.0325 0" rpy="0 0 0" />
@@ -140,18 +124,4 @@
     <child link="Gonio_Right_Stage_2_Bottom" />
     <axis xyz="0 -1 0" />
-=======
-  <joint
-    name="Gonio_Right_Stage_2_Joint"
-    type="revolute">
-    <origin
-      xyz="0 0 0"
-      rpy="0 0 0" />
-    <parent
-      link="Gonio_Right_Stage_1_Top" />
-    <child
-      link="Gonio_Right_Stage_2_Bottom" />
-    <axis
-      xyz="-1 0 0" />
->>>>>>> f5d9834 (modular Launch Files, Axis renaming)
     <limit lower="-0.17453" upper="0.17453" effort="100" velocity="0.1" />
   </joint>

File: pm_robot_description/urdf/ros2_control_gazebo.xacro (robot description, xacro)
@@ -89,5 +89,4 @@
             <state_interface name="position"/>
         </joint>
-<<<<<<< HEAD
         <joint name="Tool_Gripper_MPG_10_Jaw_1_Joint">
             <command_interface name="position">
@@ -95,84 +94,4 @@
             <state_interface name="position"/>
         </joint>
-=======
-            </joint>
-            <joint name="Z_Axis_Joint">
-                <command_interface name="position">
-                </command_interface>
-                <state_interface name="position"/>
-                <state_interface name="velocity"/>
-            </joint>
-            <joint name="T_Axis_Joint">
-                <command_interface name="position">
-                </command_interface>
-                <state_interface name="position"/>
-                <state_interface name="velocity"/>
-            </joint>
-            <joint name="1K_Dispenser_Flap_Joint">
-                <command_interface name="position">
-                </command_interface>
-                <state_interface name="position"/>
-            </joint>
-            <joint name="1K_Dispenser_Joint">
-                <command_interface name="position">
-                </command_interface>
-                <state_interface name="position"/>
-            </joint>
-            <joint name="2K_Dispenser_Joint">
-                <command_interface name="position">
-                </command_interface>
-                <state_interface name="position"/>
-            </joint>
-            <joint name="Gonio_Right_Stage_1_Joint">
-                <command_interface name="position">
-                </command_interface>
-                <state_interface name="position"/>
-            </joint>
-            <joint name="Gonio_Right_Stage_2_Joint">
-                <command_interface name="position">
-                </command_interface>
-                <state_interface name="position"/>
-            </joint>
-            <joint name="Camera_Calibration_Platelet_Joint">
-                <command_interface name="position">
-                </command_interface>
-                <state_interface name="position"/>
-            </joint>
-            <joint name="Gonio_Left_Stage_1_Joint">
-                <command_interface name="position">
-                </command_interface>
-                <state_interface name="position"/>
-            </joint>
-            <joint name="Gonio_Left_Stage_2_Joint">
-                <command_interface name="position">
-                </command_interface>
-                <state_interface name="position"/>
-            </joint>
-            <joint name="UV_Slider_X_Front_Joint">
-                <command_interface name="position">
-                </command_interface>
-                <state_interface name="position"/>
-            </joint>
-            <joint name="UV_LED_Front_Joint">
-                <command_interface name="position">
-                </command_interface>
-                <state_interface name="position"/>
-            </joint>
-            <joint name="UV_Slider_X_Back_Joint">
-                <command_interface name="position">
-                </command_interface>
-                <state_interface name="position"/>
-            </joint>
-            <joint name="UV_LED_Back_Joint">
-                <command_interface name="position">
-                </command_interface>
-                <state_interface name="position"/>
-            </joint>
-            <joint name="Calibration_Qube_Joint">
-                <command_interface name="position">
-                </command_interface>
-                <state_interface name="position"/>
-            </joint>
->>>>>>> f5d9834 (modular Launch Files, Axis renaming)
         <joint name="Tool_Gripper_MPG_10_Jaw_2_Joint">
             <param name="mimic">Tool_Gripper_MPG_10_Jaw_1_Joint</param>
