Commit message: calibration

File: pm_robot_description/urdf/pm_robot_gonio_left.xacro (robot description, xacro)
@@ -51,6 +51,19 @@
       </collision>
     </link>
+    <xacro:property name="gonio_base_Cal_x" value="${calibration_dict['Gonio_Left_Base_Joint']['x_offset']}"/>
+    <xacro:property name="gonio_base_Cal_y" value="${calibration_dict['Gonio_Left_Base_Joint']['y_offset']}"/>
+    <xacro:property name="gonio_base_Cal_z" value="${calibration_dict['Gonio_Left_Base_Joint']['z_offset']}"/>
+    <xacro:property name="gonio_base_Cal_rx" value="${calibration_dict['Gonio_Left_Base_Joint']['rx_offset']}"/>
+    <xacro:property name="gonio_base_Cal_ry" value="${calibration_dict['Gonio_Left_Base_Joint']['ry_offset']}"/>
+    <xacro:property name="gonio_base_Cal_rz" value="${calibration_dict['Gonio_Left_Base_Joint']['rz_offset']}"/>
     <joint name="Gonio_Left_Base_Joint" type="fixed">
-      <origin xyz="0.14249999999998 0.295499999999939 0" rpy="0 0 0" />
+      <origin xyz="
+        ${0.14249999999998 + gonio_base_Cal_x * 0.000001}
+        ${0.295499999999939 + gonio_base_Cal_y * 0.000001}
+        ${0 + gonio_base_Cal_z * 0.000001}"
+        rpy="
+        ${0 + gonio_base_Cal_rx * 3.14159265359/180}
+        ${0 + gonio_base_Cal_ry * 3.14159265359/180}
+        ${0 + gonio_base_Cal_rz * 3.14159265359/180}" />
       <parent link="pm_robot_base_link" />
       <child link="Gonio_Left_Base" />
@@ -161,4 +174,10 @@
     <xacro:property name="gonio_chuck_visual_filename" value="${gonio_left_configs_dict[current_gonio_left_chuck]['visual_filename']}"/>
     <xacro:property name="gonio_chuck_collision_filename" value="${gonio_left_configs_dict[current_gonio_left_chuck]['collision_filename']}"/>
+    <xacro:property name="Gonio_Left_Chuck_Cal_x" value="${calibration_dict['Gonio_Left_Chuck_Joint']['x_offset']}"/>
+    <xacro:property name="Gonio_Left_Chuck_Cal_y" value="${calibration_dict['Gonio_Left_Chuck_Joint']['y_offset']}"/>
+    <xacro:property name="Gonio_Left_Chuck_Cal_z" value="${calibration_dict['Gonio_Left_Chuck_Joint']['z_offset']}"/>
+    <xacro:property name="Gonio_Left_Chuck_Cal_rx" value="${calibration_dict['Gonio_Left_Chuck_Joint']['rx_offset']}"/>
+    <xacro:property name="Gonio_Left_Chuck_Cal_ry" value="${calibration_dict['Gonio_Left_Chuck_Joint']['ry_offset']}"/>
+    <xacro:property name="Gonio_Left_Chuck_Cal_rz" value="${calibration_dict['Gonio_Left_Chuck_Joint']['rz_offset']}"/>
     <link name="Gonio_Left_Chuck">
       <inertial>
@@ -183,5 +202,12 @@
     </link>
     <joint name="Gonio_Left_Chuck_Joint" type="fixed">
-      <origin xyz="0 0 0" rpy="0 0 0" />
+        <origin xyz="
+        ${0.0 + Gonio_Left_Chuck_Cal_x * 0.000001}
+        ${0.0 + Gonio_Left_Chuck_Cal_y * 0.000001}
+        ${0.0 + Gonio_Left_Chuck_Cal_z * 0.000001}"
+        rpy="
+        ${0 + Gonio_Left_Chuck_Cal_rx * 3.14159265359/180}
+        ${0 + Gonio_Left_Chuck_Cal_ry * 3.14159265359/180}
+        ${0 + Gonio_Left_Chuck_Cal_rz * 3.14159265359/180}" />
       <parent link="Gonio_Left_Chuck_Origin" />
       <child link="Gonio_Left_Chuck" />

File: pm_robot_description/urdf/pm_robot_gonio_right.xacro (robot description, xacro)
@@ -70,10 +70,21 @@
     </collision>
   </link>
+  <xacro:property name="gonio_base_Cal_x" value="${calibration_dict['Gonio_Right_Base_Joint']['x_offset']}"/>
+  <xacro:property name="gonio_base_Cal_y" value="${calibration_dict['Gonio_Right_Base_Joint']['y_offset']}"/>
+  <xacro:property name="gonio_base_Cal_z" value="${calibration_dict['Gonio_Right_Base_Joint']['z_offset']}"/>
+  <xacro:property name="gonio_base_Cal_rx" value="${calibration_dict['Gonio_Right_Base_Joint']['rx_offset']}"/>
+  <xacro:property name="gonio_base_Cal_ry" value="${calibration_dict['Gonio_Right_Base_Joint']['ry_offset']}"/>
+  <xacro:property name="gonio_base_Cal_rz" value="${calibration_dict['Gonio_Right_Base_Joint']['rz_offset']}"/>
   <joint
     name="Gonio_Base_Right_Joint"
     type="fixed">
-    <origin
-      xyz="${0.750000000000003+gonio_offset_smarpod_x} ${0.31+gonio_offset_smarpod_y} 0"
-      rpy="0 0 0" />
+    <origin xyz="
+        ${0.750000000000003 + gonio_base_Cal_x * 0.000001 + gonio_offset_smarpod_x}
+        ${0.31 + gonio_base_Cal_y * 0.000001 + gonio_offset_smarpod_y}
+        ${0 + gonio_base_Cal_z * 0.000001}"
+        rpy="
+        ${0 + gonio_base_Cal_rx * 3.14159265359/180}
+        ${0 + gonio_base_Cal_ry * 3.14159265359/180}
+        ${0 + gonio_base_Cal_rz * 3.14159265359/180}" />
     <parent
       link="pm_robot_base_link" />
@@ -279,87 +290,98 @@
   <xacro:property name="gonio_chuck_visual_filename" value="${gonio_right_configs_dict[current_gonio_right_chuck]['visual_filename']}"/>
   <xacro:property name="gonio_chuck_collision_filename" value="${gonio_right_configs_dict[current_gonio_right_chuck]['collision_filename']}"/>
-<link
-  name="Gonio_Right_Chuck">
-  <inertial>
-    <origin
-      xyz="${gonio_chuck_xyz}"
-      rpy="${gonio_chuck_rpy}"/>
-    <mass
-      value="${gonio_chuck_mass}"/>
-    <inertia
-      ixx="${gonio_chuck_inertia_ixx}"
-      ixy="${gonio_chuck_inertia_ixy}"
-      ixz="${gonio_chuck_inertia_ixz}"
-      iyy="${gonio_chuck_inertia_iyy}"
-      iyz="${gonio_chuck_inertia_iyz}"
-      izz="${gonio_chuck_inertia_izz}" />
-  </inertial>
-  <visual>
-    <origin
-      xyz="0 0 0"
-      rpy="0 0 0" />
-    <geometry>
-      <mesh filename="file://$(find pm_robot_description)/meshes/Gonio_Right/Gonio_Right_Chucks/${gonio_chuck_visual_filename}" />
-    </geometry>
-    <material
-      name="${gonio_chuck_color}">
-    </material>
-  </visual>
-  <collision>
-    <origin
-      xyz="0 0 0"
-      rpy="0 0 0" />
-    <geometry>
-      <mesh filename="file://$(find pm_robot_description)/meshes/Gonio_Right/Gonio_Right_Chucks/${gonio_chuck_collision_filename}" />
-    </geometry>
-  </collision>
-</link>
-<joint
-  name="Gonio_Right_Chuck_Joint"
-  type="fixed">
-  <origin
-    xyz="0 0 0"
-    rpy="0 0 0" />
-  <parent
-    link="Gonio_Right_Chuck_Origin" />
-  <child
-    link="Gonio_Right_Chuck" />
-  <axis
-    xyz="0 0 0" />
-</joint>
-  <!--%%%%%%%%%%%%% Gonio Right Part 1 Origin -->
-  <link
-    name="Gonio_Right_Part_1_Origin">
-  </link>
-  <joint
-    name="Gonio_Right_Part_1_Origin_Joint"
+  <xacro:property name="Gonio_Right_Chuck_Cal_x" value="${calibration_dict['Gonio_Right_Chuck_Joint']['x_offset']}"/>
+  <xacro:property name="Gonio_Right_Chuck_Cal_y" value="${calibration_dict['Gonio_Right_Chuck_Joint']['y_offset']}"/>
+  <xacro:property name="Gonio_Right_Chuck_Cal_z" value="${calibration_dict['Gonio_Right_Chuck_Joint']['z_offset']}"/>
+  <xacro:property name="Gonio_Right_Chuck_Cal_rx" value="${calibration_dict['Gonio_Right_Chuck_Joint']['rx_offset']}"/>
+  <xacro:property name="Gonio_Right_Chuck_Cal_ry" value="${calibration_dict['Gonio_Right_Chuck_Joint']['ry_offset']}"/>
+  <xacro:property name="Gonio_Right_Chuck_Cal_rz" value="${calibration_dict['Gonio_Right_Chuck_Joint']['rz_offset']}"/>
+  <link
+    name="Gonio_Right_Chuck">
+    <inertial>
+      <origin
+        xyz="${gonio_chuck_xyz}"
+        rpy="${gonio_chuck_rpy}"/>
+      <mass
+        value="${gonio_chuck_mass}"/>
+      <inertia
+        ixx="${gonio_chuck_inertia_ixx}"
+        ixy="${gonio_chuck_inertia_ixy}"
+        ixz="${gonio_chuck_inertia_ixz}"
+        iyy="${gonio_chuck_inertia_iyy}"
+        iyz="${gonio_chuck_inertia_iyz}"
+        izz="${gonio_chuck_inertia_izz}" />
+    </inertial>
+    <visual>
+      <origin
+        xyz="0 0 0"
+        rpy="0 0 0" />
+      <geometry>
+        <mesh filename="file://$(find pm_robot_description)/meshes/Gonio_Right/Gonio_Right_Chucks/${gonio_chuck_visual_filename}" />
+      </geometry>
+      <material
+        name="${gonio_chuck_color}">
+      </material>
+    </visual>
+    <collision>
+      <origin
+        xyz="0 0 0"
+        rpy="0 0 0" />
+      <geometry>
+        <mesh filename="file://$(find pm_robot_description)/meshes/Gonio_Right/Gonio_Right_Chucks/${gonio_chuck_collision_filename}" />
+      </geometry>
+    </collision>
+  </link>
+  <joint
+    name="Gonio_Right_Chuck_Joint"
     type="fixed">
-    <origin
-      xyz="${gonio_chuck_tcp_offset_x_1} ${gonio_chuck_tcp_offset_y_1} ${gonio_chuck_tcp_offset_z_1}"
-      rpy="0 0 0" />
+    <origin xyz="
+      ${0.0 + Gonio_Right_Chuck_Cal_x * 0.000001}
+      ${0.0 + Gonio_Right_Chuck_Cal_y * 0.000001}
+      ${0.0 + Gonio_Right_Chuck_Cal_z * 0.000001}"
+      rpy="
+      ${0 + Gonio_Right_Chuck_Cal_rx * 3.14159265359/180}
+      ${0 + Gonio_Right_Chuck_Cal_ry * 3.14159265359/180}
+      ${0 + Gonio_Right_Chuck_Cal_rz * 3.14159265359/180}" />
     <parent
       link="Gonio_Right_Chuck_Origin" />
     <child
-      link="Gonio_Right_Part_1_Origin" />
+      link="Gonio_Right_Chuck" />
     <axis
       xyz="0 0 0" />
   </joint>
-  <!--%%%%%%%%%%%%% Gonio Right Part 2 Origin -->
-  <link
-    name="Gonio_Right_Part_2_Origin">
-  </link>
-  <joint
-    name="Gonio_Right_Part_2_Origin_Joint"
-    type="fixed">
-    <origin
-      xyz="${gonio_chuck_tcp_offset_x_2} ${gonio_chuck_tcp_offset_y_2} ${gonio_chuck_tcp_offset_z_2}"
-      rpy="0 0 0" />
-    <parent
-      link="Gonio_Right_Chuck_Origin" />
-    <child
-      link="Gonio_Right_Part_2_Origin" />
-    <axis
-      xyz="0 0 0" />
-  </joint>
-</xacro:macro>
+    <!--%%%%%%%%%%%%% Gonio Right Part 1 Origin -->
+    <link
+      name="Gonio_Right_Part_1_Origin">
+    </link>
+    <joint
+      name="Gonio_Right_Part_1_Origin_Joint"
+      type="fixed">
+      <origin
+        xyz="${gonio_chuck_tcp_offset_x_1} ${gonio_chuck_tcp_offset_y_1} ${gonio_chuck_tcp_offset_z_1}"
+        rpy="0 0 0" />
+      <parent
+        link="Gonio_Right_Chuck_Origin" />
+      <child
+        link="Gonio_Right_Part_1_Origin" />
+      <axis
+        xyz="0 0 0" />
+    </joint>
+    <!--%%%%%%%%%%%%% Gonio Right Part 2 Origin -->
+    <link
+      name="Gonio_Right_Part_2_Origin">
+    </link>
+    <joint
+      name="Gonio_Right_Part_2_Origin_Joint"
+      type="fixed">
+      <origin
+        xyz="${gonio_chuck_tcp_offset_x_2} ${gonio_chuck_tcp_offset_y_2} ${gonio_chuck_tcp_offset_z_2}"
+        rpy="0 0 0" />
+      <parent
+        link="Gonio_Right_Chuck_Origin" />
+      <child
+        link="Gonio_Right_Part_2_Origin" />
+      <axis
+        xyz="0 0 0" />
+    </joint>
+  </xacro:macro>
 </robot>

Commit message: uv cart manaul service

File: pm_robot_description/urdf/pm_robot_gonio_left.xacro (robot description, xacro)
@@ -254,5 +254,5 @@
       <child link="UV_Slider_X_Front" />
       <axis xyz="1 0 0" />
-      <limit lower="0" upper="0.095" effort="100" velocity="0.05" />
+      <limit lower="-0.06" upper="0.06" effort="100" velocity="0.05" />
     </joint>
     <!--%%%%%%%%%%%%% UV LED Front Definitions-->
@@ -311,5 +311,5 @@
       <child link="UV_Slider_X_Back" />
       <axis xyz="1 0 0" />
-      <limit lower="0" upper="0.045" effort="0.05" velocity="100" />
+      <limit lower="-0.06" upper="0.06" effort="100" velocity="0.05" />
     </joint>
     <!--%%%%%%%%%%%%% UV LED Back Definitions-->

File: pm_robot_description/urdf/ros2_control_real_HW.xacro (robot description, xacro)
@@ -72,4 +72,14 @@
                 <state_interface name="velocity"/>
             </joint>
+            <joint name="UV_Slider_X_Front_Joint">
+                <command_interface name="position">
+                </command_interface>
+                <state_interface name="position"/>
+            </joint>
+            <joint name="UV_Slider_X_Back_Joint">
+                <command_interface name="position">
+                </command_interface>
+                <state_interface name="position"/>
+            </joint>
 <!--
             <joint name="1K_Dispenser_Protection_Joint">
