Commit message: Differentiation between simulation and real robot controller

File: pm_robot_description/urdf/pm_robot.xacro (robot description, xacro)
@@ -151,5 +151,5 @@
     <turnGravityOff>true</turnGravityOff>
   </gazebo>
-  <joint name="Gripper_Rot_Plate_Joint" type="revolute">
+  <joint name="T_Axis_Joint" type="revolute">
     <origin xyz="0.00750000000002338 0.0900000062570287 -0.389499999999991" rpy="0 0 0" />
     <parent link="Z_Axis" />

File: pm_robot_description/urdf/pm_robot_main.xacro (robot description, xacro)
@@ -4,4 +4,5 @@
   <!-- Configurations -->
   <xacro:include filename="$(find pm_robot_description)/urdf/materials.xacro" />
+  <xacro:arg name="sim_mode"                 default="false" />
   <xacro:arg name="with_Gonio_Left"                 default="true" />
   <xacro:arg name="with_Gonio_Right"                default="true" />
@@ -29,5 +30,11 @@
       <xacro:include filename="$(find pm_robot_description)/urdf/pm_robot_gonio_left.xacro" />
     </xacro:if>
-  <xacro:include filename="$(find pm_robot_description)/urdf/ros2_control.xacro" />
+  <!-- Switch between Gazebo-Simulation and Real Robot -->
+    <xacro:if value="$(arg sim_mode)">
+      <xacro:include filename="$(find pm_robot_description)/urdf/ros2_control_gazebo.xacro" />
+    </xacro:if>
+    <xacro:unless value="$(arg sim_mode)">
+      <xacro:include filename="$(find pm_robot_description)/urdf/ros2_control.xacro" />
+    </xacro:unless>
   <!--xacro:include filename="$(find pm_robot_description)/urdf/MPG_10_plus_control.xacro" /-->
   <xacro:include filename="$(find pm_robot_description)/urdf/sensors.urdf" />

File: pm_robot_description/urdf/ros2_control_gazebo.xacro (robot description, xacro)
@@ -1,9 +1,7 @@
 <?xml version="1.0"?>
 <robot name="pm_robot">
-    <!-- <ros2_control name="GazeboSystem" type="system"> -->
-    <ros2_control name="PMSystem" type="system">
+    <ros2_control name="GazeboSystem" type="system">
         <hardware>
-            <!-- <plugin>gazebo_ros2_control/GazeboSystem</plugin> -->
-            <plugin>pm_hardware_interface/PMSystem</plugin>
+            <plugin>gazebo_ros2_control/GazeboSystem</plugin>
         </hardware>
         <joint name="X_Axis_Joint">

File: pm_robot_moveit_config/config/pm_robot.ros2_control.xacro (robot description, xacro)
@@ -64,8 +64,8 @@
                 <state_interface name="velocity"/>
             </joint>
-            <joint name="Gripper_Rot_Plate_Joint">
+            <joint name="T_Axis_Joint">
                 <command_interface name="position"/>
                 <state_interface name="position">
-                  <param name="initial_value">${initial_positions['Gripper_Rot_Plate_Joint']}</param>
+                  <param name="initial_value">${initial_positions['T_Axis_Joint']}</param>
                 </state_interface>
                 <state_interface name="velocity"/>

Commit message: moveit edited

File: pm_robot_description/urdf/pm_robot.xacro (robot description, xacro)
@@ -231,5 +231,5 @@
         <mesh filename="file://$(find pm_robot_description)/meshes/1K_Dispenser.STL" />
       </geometry>
-      <material name="red"/>
+      <material name="grey"/>
     </visual>
     <collision>
@@ -263,5 +263,5 @@
         <mesh filename="file://$(find pm_robot_description)/meshes/2K_Dispenser.STL" />
       </geometry>
-      <material name="orange"/>
+      <material name="white"/>
     </visual>
     <collision>

File: pm_robot_description/urdf/pm_robot_gonio_left.xacro (robot description, xacro)
@@ -16,4 +16,5 @@
         <mesh filename="file://$(find pm_robot_description)/meshes/Gonio_Left/Gonio_Station_Left.STL" />
       </geometry>
+      <material name="white"/>
     </visual>
     <collision>
@@ -42,4 +43,5 @@
         <mesh filename="file://$(find pm_robot_description)/meshes/Gonio_Left/Gonio_Left_Stage_1_Top.STL" />
       </geometry>
+      <material name="grey"/>
     </visual>
     <collision>
@@ -73,4 +75,5 @@
         <mesh filename="file://$(find pm_robot_description)/meshes/Gonio_Left/Gonio_Left_Stage_2_Bottom.STL" />
       </geometry>
+      <material name="white"/>
     </visual>
     <collision>
@@ -104,4 +107,5 @@
         <mesh filename="file://$(find pm_robot_description)/meshes/Gonio_Left/Gonio_Left_Chucks/Chuck_Siemens_Carrier_Gonio_Left.STL" />
       </geometry>
+      <material name="grey"/>
     </visual>
     <collision>
@@ -134,4 +138,5 @@
         <mesh filename="file://$(find pm_robot_description)/meshes/UV_Slider_X_Front.STL" />
       </geometry>
+      <material name="white"/>
     </visual>
     <collision>
@@ -161,4 +166,5 @@
         <mesh filename="file://$(find pm_robot_description)/meshes/UV_LED_Front.STL" />
       </geometry>
+      <material name="grey"/>
     </visual>
     <collision>
@@ -188,4 +194,5 @@
         <mesh filename="file://$(find pm_robot_description)/meshes/UV_Slider_X_Back.STL" />
       </geometry>
+      <material name="white"/>
     </visual>
     <collision>
@@ -215,4 +222,5 @@
         <mesh filename="file://$(find pm_robot_description)/meshes/UV_LED_Back.STL" />
       </geometry>
+      <material name="grey"/>
     </visual>
     <collision>

File: pm_robot_description/urdf/pm_robot_gonio_right.xacro (robot description, xacro)
@@ -16,4 +16,5 @@
         <mesh filename="file://$(find pm_robot_description)/meshes/Gonio_Right/Gonio_Right.STL" />
       </geometry>
+      <material name="white"/>
     </visual>
     <collision>
@@ -42,4 +43,5 @@
         <mesh filename="file://$(find pm_robot_description)/meshes/Gonio_Right/Gonio_Right_Stage_1_Bottom.STL" />
       </geometry>
+      <material name="grey"/>
     </visual>
     <collision>
@@ -72,4 +74,5 @@
         <mesh filename="file://$(find pm_robot_description)/meshes/Gonio_Right/Gonio_Right_Stage_1_Top.STL" />
       </geometry>
+      <material name="white"/>
     </visual>
     <collision>
@@ -103,4 +106,5 @@
         <mesh filename="file://$(find pm_robot_description)/meshes/Gonio_Right/Gonio_Right_Stage_2_Bottom.STL" />
       </geometry>
+      <material name="grey"/>
     </visual>
     <collision>
@@ -134,4 +138,5 @@
         <mesh filename="file://$(find pm_robot_description)/meshes/Gonio_Right/Gonio_Right_Chucks/Chuck_Siemens_UFC_Gonio_Right.STL" />
       </geometry>
+      <material name="white"/>
     </visual>
     <collision>

File: pm_robot_description/urdf/pm_robot_main_copy.xacro (robot description, xacro)
@@ -31,10 +31,10 @@
     </xacro:if>
   <!-- Switch between Gazebo-Simulation and Real Robot -->
-    <xacro:if value="$(arg sim_mode)">
-      <xacro:include filename="$(find pm_robot_description)/urdf/ros2_control_gazebo.xacro" />
-    </xacro:if>
-    <xacro:unless value="$(arg sim_mode)">
-      <xacro:include filename="$(find pm_robot_description)/urdf/ros2_control.xacro" />
-    </xacro:unless>
+    <!-- <xacro:if value="$(arg sim_mode)"> -->
+      <!-- <xacro:include filename="$(find pm_robot_description)/urdf/ros2_control_gazebo.xacro" /> -->
+    <!-- </xacro:if> -->
+    <!-- <xacro:unless value="$(arg sim_mode)"> -->
+      <!-- <xacro:include filename="$(find pm_robot_description)/urdf/ros2_control.xacro" /> -->
+    <!-- </xacro:unless> -->
   <xacro:include filename="$(find pm_robot_description)/urdf/sensors.urdf" />
 </robot>

File: pm_robot_moveit_config/config/pm_robot.ros2_control.xacro (robot description, xacro)
@@ -13,4 +13,5 @@
                   <param name="initial_value">${initial_positions['Gonio_Right_Stage_1_Top_Joint']}</param>
                 </state_interface>
+                <state_interface name="position"/>
                 <state_interface name="velocity"/>
             </joint>
@@ -20,4 +21,5 @@
                   <param name="initial_value">${initial_positions['Gonio_Right_Stage_2_Bottom_Joint']}</param>
                 </state_interface>
+                <state_interface name="position"/>
                 <state_interface name="velocity"/>
             </joint>
@@ -27,4 +29,5 @@
                   <param name="initial_value">${initial_positions['Gonio_Left_Stage_1_Top_Joint']}</param>
                 </state_interface>
+                <state_interface name="position"/>
                 <state_interface name="velocity"/>
             </joint>
@@ -34,4 +37,5 @@
                   <param name="initial_value">${initial_positions['Gonio_Left_Stage_2_Bottom_Joint']}</param>
                 </state_interface>
+                <state_interface name="position"/>
                 <state_interface name="velocity"/>
             </joint>
@@ -41,4 +45,5 @@
                   <param name="initial_value">${initial_positions['X_Axis_Joint']}</param>
                 </state_interface>
+                <state_interface name="position"/>
                 <state_interface name="velocity"/>
             </joint>
@@ -48,4 +53,5 @@
                   <param name="initial_value">${initial_positions['Y_Axis_Joint']}</param>
                 </state_interface>
+                <state_interface name="position"/>
                 <state_interface name="velocity"/>
             </joint>
@@ -55,4 +61,5 @@
                   <param name="initial_value">${initial_positions['Z_Axis_Joint']}</param>
                 </state_interface>
+                <state_interface name="position"/>
                 <state_interface name="velocity"/>
             </joint>
@@ -62,4 +69,5 @@
                   <param name="initial_value">${initial_positions['1K_Dispenser_Flap_Joint']}</param>
                 </state_interface>
+                <state_interface name="position"/>
                 <state_interface name="velocity"/>
             </joint>
@@ -69,4 +77,5 @@
                   <param name="initial_value">${initial_positions['T_Axis_Joint']}</param>
                 </state_interface>
+                <state_interface name="position"/>
                 <state_interface name="velocity"/>
             </joint>

File: pm_robot_moveit_config/config/pm_robot.urdf.xacro (robot description, xacro)
@@ -3,5 +3,5 @@
     <xacro:arg name="initial_positions_file" default="initial_positions.yaml" />
     <!-- Import pm_robot urdf file -->
-    <xacro:include filename="$(find pm_robot_description)/urdf/pm_robot_main.xacro" />
+    <xacro:include filename="$(find pm_robot_description)/urdf/pm_robot_main_copy.xacro" />
     <!-- Import control_xacro -->
     <xacro:include filename="pm_robot.ros2_control.xacro" />

Commit message: Moveit Integration

File: pm_robot_description/urdf/pm_robot.xacro (robot description, xacro)
@@ -326,5 +326,5 @@
         <mesh filename="file://$(find pm_robot_description)/meshes/Test_Station.STL" />
       </geometry>
-      <material name="grey"/>
+      <material name="white"/>
     </visual>
     <collision>

File: pm_robot_description/urdf/pm_robot_main.xacro (robot description, xacro)
@@ -4,5 +4,9 @@
   <!-- Configurations -->
   <xacro:include filename="$(find pm_robot_description)/urdf/materials.xacro" />
-  <xacro:arg name="sim_mode"                 default="true" />
+  <!-- <xacro:arg name="launch_mode"                default="fake_HW" /> -->
+  <!-- <xacro:arg name="launch_mode"                default="real_HW" /> -->
+  <xacro:arg name="launch_mode"                     default="sim_HW" />
+  <!-- <xacro:arg name="launch_mode"                default="real_sim_HW" /> -->
+  <xacro:arg name="initial_positions_file"          default="pm_robot_initial_positions.yaml" />
   <xacro:arg name="with_Gonio_Left"                 default="true" />
   <xacro:arg name="with_Gonio_Right"                default="true" />
@@ -30,11 +34,22 @@
       <xacro:include filename="$(find pm_robot_description)/urdf/pm_robot_gonio_left.xacro" />
     </xacro:if>
+    <xacro:include filename="$(find pm_robot_description)/urdf/sensors.urdf" />
   <!-- Switch between Gazebo-Simulation and Real Robot -->
-    <xacro:if value="$(arg sim_mode)">
-      <xacro:include filename="$(find pm_robot_description)/urdf/ros2_control_gazebo.xacro" />
+    <!-- Import control_xacro -->
+    <xacro:include filename="$(find pm_robot_description)/urdf/ros2_control_fake.xacro" />
+    <xacro:include filename="$(find pm_robot_description)/urdf/ros2_control_gazebo.xacro" />
+    <!-- <xacro:include filename="$(find pm_robot_description)/urdf/ros2_control_real.xacro" /> -->
+    <xacro:property name="launch_mode" value="$(arg launch_mode)"/>
+    <xacro:if value="${launch_mode == 'fake_HW'}">
+      <xacro:pm_robot_ros2_control_hw_fake name="Fake_HW" initial_positions_file="$(arg initial_positions_file)"/>
     </xacro:if>
-    <xacro:unless value="$(arg sim_mode)">
-      <xacro:include filename="$(find pm_robot_description)/urdf/ros2_control.xacro" />
-    </xacro:unless>
-  <xacro:include filename="$(find pm_robot_description)/urdf/sensors.urdf" />
+    <xacro:if value="${launch_mode == 'real_HW'}">
+      <xacro:pm_robot_ros2_control_hw_real name="Real_HW"/>
+    </xacro:if>
+    <xacro:if value="${launch_mode == 'sim_HW'}">
+      <xacro:pm_robot_ros2_control_hw_sim name="Sim_HW" initial_positions_file="$(arg initial_positions_file)"/>
+    </xacro:if>
+    <xacro:if value="${launch_mode == 'real_sim_HW'}">
+      <!-- <xacro:pm_robot_ros2_control_hw_fake name="Real_Sim_HW" initial_positions_file="$(arg initial_positions_file)"/> -->
+    </xacro:if>
 </robot>

File: pm_robot_description/urdf/ros2_control_fake.xacro (robot description, xacro)
@@ -1,9 +1,10 @@
 <?xml version="1.0"?>
 <robot xmlns:xacro="http://www.ros.org/wiki/xacro">
-    <xacro:macro name="pm_robot_ros2_control_hw_sim" params="name initial_positions_file">
+    <xacro:macro name="pm_robot_ros2_control_hw_fake" params="name initial_positions_file">
         <xacro:property name="initial_positions" value="${load_yaml(initial_positions_file)['initial_positions']}"/>
-        <ros2_control name="GazeboSystem" type="system">
+        <ros2_control name="${name}" type="system">
             <hardware>
-                <plugin>gazebo_ros2_control/GazeboSystem</plugin>
+                <!-- By default, set up controllers for simulation. This won't work on real hardware -->
+                <plugin>mock_components/GenericSystem</plugin>
             </hardware>
             <joint name="X_Axis_Joint">
@@ -91,32 +92,5 @@
                 <state_interface name="position"/>
             </joint>
-            <xacro:if value="$(arg with_Tool_MPG_10)">
-                <joint name="Tool_Gripper_MPG_10_Jaw_1_Joint">
-                        <command_interface name="position">
-                        </command_interface>
-                        <state_interface name="position"/>
-                    </joint>
-                    <joint name="Tool_Gripper_MPG_10_Jaw_2_Joint">
-                        <param name="mimic">Tool_Gripper_MPG_10_Jaw_1_Joint</param>
-                        <param name="mulltiplier">1</param>
-                        <command_interface name="position">
-                        </command_interface>
-                        <state_interface name="position"/>
-                    </joint>
-            </xacro:if>
         </ros2_control>
-            <gazebo>
-                <plugin name="gazebo_ros2_control" filename="libgazebo_ros2_control.so">
-                    <parameters>$(find pm_robot_description)/config/pm_robot_control.yaml</parameters>
-                    <parameters>$(find pm_robot_description)/config/pm_robot_control_gonio_right.yaml</parameters>
-                    <parameters>$(find pm_robot_description)/config/pm_robot_control_gonio_left.yaml</parameters>
-                    <xacro:if value="$(arg with_Tool_MPG_10)">
-                        <parameters>$(find pm_robot_description)/config/pm_robot_control_gripper.yaml</parameters>
-                    </xacro:if>
-                    <!--robot_param>robot_description</robot_param-->            <!--The location of the robot_description (URDF) on the parameter server, defaults to robot_description-->
-                    <!--robot_param_node>robot_state_publisher</robot_param_node-->            <!-- Name of the node where the robot_param is located, defauls to robot_state_publisher-->
-                    <!--robotNamespace>${arm_id}</robotNamespace-->
-                </plugin>
-            </gazebo>
     </xacro:macro>
 </robot>

File: pm_robot_description/urdf/ros2_control_real.xacro (robot description, xacro)
@@ -1,9 +1,9 @@
 <?xml version="1.0"?>
 <robot xmlns:xacro="http://www.ros.org/wiki/xacro">
-    <xacro:macro name="pm_robot_ros2_control_hw_sim" params="name initial_positions_file">
-        <xacro:property name="initial_positions" value="${load_yaml(initial_positions_file)['initial_positions']}"/>
-        <ros2_control name="GazeboSystem" type="system">
+    <xacro:macro name="pm_robot_ros2_control_hw_real">
+        <ros2_control name="PMSystem" type="system">
             <hardware>
-                <plugin>gazebo_ros2_control/GazeboSystem</plugin>
+                <!-- <plugin>gazebo_ros2_control/GazeboSystem</plugin> -->
+                <plugin>pm_hardware_interface/PMSystem</plugin>
             </hardware>
             <joint name="X_Axis_Joint">
@@ -91,18 +91,16 @@
                 <state_interface name="position"/>
             </joint>
-            <xacro:if value="$(arg with_Tool_MPG_10)">
-                <joint name="Tool_Gripper_MPG_10_Jaw_1_Joint">
-                        <command_interface name="position">
-                        </command_interface>
-                        <state_interface name="position"/>
-                    </joint>
-                    <joint name="Tool_Gripper_MPG_10_Jaw_2_Joint">
-                        <param name="mimic">Tool_Gripper_MPG_10_Jaw_1_Joint</param>
-                        <param name="mulltiplier">1</param>
-                        <command_interface name="position">
-                        </command_interface>
-                        <state_interface name="position"/>
-                    </joint>
-            </xacro:if>
+            <joint name="Tool_Gripper_MPG_10_Jaw_1_Joint">
+                <command_interface name="position">
+                </command_interface>
+                <state_interface name="position"/>
+            </joint>
+            <joint name="Tool_Gripper_MPG_10_Jaw_2_Joint">
+                <param name="mimic">Tool_Gripper_MPG_10_Jaw_1_Joint</param>
+                <param name="mulltiplier">1</param>
+                <command_interface name="position">
+                </command_interface>
+                <state_interface name="position"/>
+            </joint>
         </ros2_control>
             <gazebo>
@@ -111,7 +109,5 @@
                     <parameters>$(find pm_robot_description)/config/pm_robot_control_gonio_right.yaml</parameters>
                     <parameters>$(find pm_robot_description)/config/pm_robot_control_gonio_left.yaml</parameters>
-                    <xacro:if value="$(arg with_Tool_MPG_10)">
-                        <parameters>$(find pm_robot_description)/config/pm_robot_control_gripper.yaml</parameters>
-                    </xacro:if>
+                    <parameters>$(find pm_robot_description)/config/pm_robot_control_gripper.yaml</parameters>
                     <!--robot_param>robot_description</robot_param-->            <!--The location of the robot_description (URDF) on the parameter server, defaults to robot_description-->
                     <!--robot_param_node>robot_state_publisher</robot_param_node-->            <!-- Name of the node where the robot_param is located, defauls to robot_state_publisher-->
