Commit message: calibration.yaml

File: pm_robot_description/urdf/pm_robot.xacro (robot description, xacro)
@@ -3,666 +3,94 @@
      Commit Version: 1.6.0-1-g15f4949  Build Version: 1.6.7594.29634
      For more information, please see http://wiki.ros.org/sw_urdf_exporter -->
-<robot name="pm_robot">
-  <link name="world">
-  </link>
-  <joint name="world_joint" type="fixed">
-    <parent link="world"/>
-    <child link="base_link_empthy"/>
-    <origin xyz="0 0 0" rpy="0 0 0" />
-  </joint>
-<!--%%%%%%%%%%%%% Base Link Definitions %%%%%%%%%%%%%-->
-  <link
-    name="base_link_empthy">
-  </link>
-<!--%%%%%%%%%%%%% PM_Robot Base Link Definitions %%%%%%%%%%%%%-->
- <link
-    name="pm_robot_base_link">
-    <inertial>
-      <origin
-        xyz="0.600186355261373 0.60024822812755 -0.0500803495201262"
-        rpy="0 0 0" />
-      <mass
-        value="143.433412382625" />
-      <inertia
-        ixx="17.331308476166"
-        ixy="-0.000173857700061693"
-        ixz="-0.00010330360577037"
-        iyy="17.3263788236508"
-        iyz="-0.00227792943650154"
-        izz="34.4189883960519" />
-    </inertial>
-    <visual>
-      <origin
-        xyz="0 0 0"
-        rpy="0 0 0" />
-      <geometry>
-        <mesh filename="file://$(find pm_robot_description)/meshes/pm_robot_base_link.STL" />
-      </geometry>
-      <material
-        name="">
-        <color
-          rgba="1 1 1 1" />
-      </material>
-    </visual>
-    <collision>
-      <origin
-        xyz="0 0 0"
-        rpy="0 0 0" />
-      <geometry>
-        <mesh filename="file://$(find pm_robot_description)/meshes/pm_robot_base_link.STL" />
-      </geometry>
-    </collision>
-  </link>
-   <joint
-    name="pm_robot_base_link_joint"
-    type="fixed">
-    <origin
-      xyz="0 0 0.971"
-      rpy="0 0 0" />
-    <parent
-      link="base_link_empthy" />
-    <child
-      link="pm_robot_base_link" />
-    <axis
-      xyz="0 0 0" />
-  </joint>
-  <!--%%%%%%%%%%%%% Axis-Base Definitions %%%%%%%%%%%%%-->
-  <link
-    name="axis_base">
-    <inertial>
-      <origin
-        xyz="0.396220059353836 0.105196690337481 0.307909602405796"
-        rpy="0 0 0" />
-      <mass
-        value="43.6102590245999" />
-      <inertia
-        ixx="0.364950648797973"
-        ixy="-0.000379121082023338"
-        ixz="0.00337088160159615"
-        iyy="2.29090638523672"
-        iyz="0.000705385684699142"
-        izz="2.23411883185999" />
-    </inertial>
-    <visual>
-      <origin
-        xyz="0 0 0"
-        rpy="0 0 0" />
-      <geometry>
-        <mesh filename="file://$(find pm_robot_description)/meshes/axis_base.STL" />
-      </geometry>
-      <material
-        name="">
-        <color
-          rgba="0.752941176470588 0.752941176470588 0.752941176470588 1" />
-      </material>
-    </visual>
-    <collision>
-      <origin
-        xyz="0 0 0"
-        rpy="0 0 0" />
-      <geometry>
-        <mesh filename="file://$(find pm_robot_description)/meshes/axis_base.STL" />
-      </geometry>
-    </collision>
-  </link>
-  <joint
-    name="axis_base_joint"
-    type="fixed">
-    <origin
-      xyz="0.08001 0.632 1.000000000001E-05"
-      rpy="0 0 0" />
-    <parent
-      link="pm_robot_base_link" />
-    <child
-      link="axis_base" />
-    <axis
-      xyz="0 0 0" />
-  </joint>
-  <!--%%%%%%%%%%%%% X Axis Definitions %%%%%%%%%%%%%-->
-  <link
-    name="X_Axis">
-    <inertial>
-      <origin
-        xyz="0.13867117656886 0.0294673421865695 0.0322225410424505"
-        rpy="0 0 0" />
-      <mass
-        value="3.46651857022574" />
-      <inertia
-        ixx="0.0263967056575219"
-        ixy="-0.000746452162875097"
-        ixz="-6.60103497268881E-06"
-        iyy="0.0104790265642698"
-        iyz="-0.000507544087069928"
-        izz="0.0342327102580871" />
-    </inertial>
-    <visual>
-      <origin
-        xyz="0 0 0"
-        rpy="0 0 0" />
-      <geometry>
-        <mesh filename="file://$(find pm_robot_description)/meshes/X_Axis.STL" />
-      </geometry>
-      <material name="orange"/>
-    </visual>
-    <collision>
-      <origin
-        xyz="0 0 0"
-        rpy="0 0 0" />
-      <geometry>
-        <mesh filename="file://$(find pm_robot_description)/meshes/X_Axis.STL" />
-      </geometry>
-    </collision>
-  </link>
-  <joint
-    name="X_Axis_Joint"
-    type="prismatic">
-    <origin
-      xyz="0.64699 0.11775 0.47499"
-      rpy="0 0 0" />
-    <parent
-      link="axis_base" />
-    <child
-      link="X_Axis" />
-    <axis
-      xyz="1 0 0" />
-    <limit lower="-0.745" upper="0.055" effort="0.1" velocity="35" />
-  </joint>
- <!--%%%%%%%%%%%%% Y Axis Definitions %%%%%%%%%%%%%-->
-  <link
-    name="Y_Axis">
-    <inertial>
-      <origin
-        xyz="-0.00196813987548172 -0.3177998990051 0.113823941424653"
-        rpy="0 0 0" />
-      <mass
-        value="5.64847104935336" />
-      <inertia
-        ixx="0.0734343917353869"
-        ixy="-5.65230035141878E-06"
-        ixz="-0.000161953758832679"
-        iyy="0.0377139193260435"
-        iyz="0.00720112978111611"
-        izz="0.0598441739891415" />
-    </inertial>
-    <visual>
-      <origin
-        xyz="0 0 0"
-        rpy="0 0 0" />
-      <geometry>
-        <mesh filename="file://$(find pm_robot_description)/meshes/Y_Axis.STL" />
-      </geometry>
-      <material name="brown"/>
-    </visual>
-    <collision>
-      <origin
-        xyz="0 0 0"
-        rpy="0 0 0" />
-      <geometry>
-        <mesh filename="file://$(find pm_robot_description)/meshes/Y_Axis.STL" />
-      </geometry>
-    </collision>
-  </link>
-  <joint
-    name="Y_Axis_Joint"
-    type="prismatic">
-    <origin
-      xyz="0.10865 0.25835 0.06525"
-      rpy="0 0 0" />
-    <parent
-      link="X_Axis" />
-    <child
-      link="Y_Axis" />
-    <axis
-      xyz="0 1 0" />
-    <limit lower="-0.134000" upper="-0.019700" effort="100" velocity="35" />
-  </joint>
- <!--%%%%%%%%%%%%% Z Axis Definitions %%%%%%%%%%%%%-->
-  <link
-    name="Z_Axis">
-    <inertial>
-      <origin
-        xyz="0.000627664293855634 -0.00434675424374531 -0.2726241124114"
-        rpy="0 0 0" />
-      <mass
-        value="2.64388477073549" />
-      <inertia
-        ixx="0.0168607348742555"
-        ixy="-1.50786678765243E-05"
-        ixz="-0.000199875277453675"
-        iyy="0.0218740034837586"
-        iyz="-8.24046242568125E-05"
-        izz="0.00606496678568248" />
-    </inertial>
-    <visual>
-      <origin
-        xyz="0 0 0"
-        rpy="0 0 0" />
-      <geometry>
-        <mesh filename="file://$(find pm_robot_description)/meshes/Z_Axis.STL" />
-      </geometry>
-      <material name="blue"/>
-    </visual>
-    <collision>
-      <origin
-        xyz="0 0 0"
-        rpy="0 0 0" />
-      <geometry>
-        <mesh filename="file://$(find pm_robot_description)/meshes/Z_Axis.STL" />
-      </geometry>
-    </collision>
-  </link>
-  <!---Gravity off-->
-  <gazebo reference="Z_Axis">
-    <turnGravityOff>true</turnGravityOff>
-  </gazebo>
-  <joint
-    name="Z_Axis_Joint"
-    type="prismatic">
-    <origin
-      xyz="-0.00365 -0.499 0.33875"
-      rpy="0 0 0" />
-    <parent
-      link="Y_Axis" />
-    <child
-      link="Z_Axis" />
-    <axis
-      xyz="0 0 -1" />
-    <limit lower="-0.05262" upper="0.055" effort="100" velocity="35" />
-  </joint>
-  <!--%%%%%%%%%%%%% T Axis Definitions %%%%%%%%%%%%%-->
-  <link
-    name="Gripper_Rot_Plate">
-    <inertial>
-      <origin
-        xyz="-1.74281094778017E-07 2.03483659588777E-07 0.00907792340584457"
-        rpy="0 0 0" />
-      <mass
-        value="0.110297257842221" />
-      <inertia
-        ixx="8.79759467929701E-05"
-        ixy="1.90651210379881E-10"
-        ixz="1.25536613370482E-10"
-        iyy="8.79764882626525E-05"
-        iyz="-1.50065581017382E-10"
-        izz="0.00016565987032676" />
-    </inertial>
-    <visual>
-      <origin
-        xyz="0 0 0"
-        rpy="0 0 0" />
-      <geometry>
-        <mesh filename="file://$(find pm_robot_description)/meshes/Gripper_Rot_Plate.STL" />
-      </geometry>
-      <material name="black"/>
-    </visual>
-    <collision>
-      <origin
-        xyz="0 0 0"
-        rpy="0 0 0" />
-      <geometry>
-        <mesh filename="file://$(find pm_robot_description)/meshes/Gripper_Rot_Plate.STL" />
-      </geometry>
-    </collision>
-  </link>
-  <!---Gravity off-->
-  <gazebo reference="Gripper_Rot_Plate">
-    <turnGravityOff>true</turnGravityOff>
-  </gazebo>
-  <joint
-    name="T_Axis_Joint"
-    type="revolute">
-    <origin
-      xyz="0.0600000000000017 -0.0580000000000003 -0.427500000000004"
-      rpy="0 0 0" />
-    <parent
-      link="Z_Axis" />
-    <child
-      link="Gripper_Rot_Plate" />
-    <axis
-      xyz="0 0 1" />
-    <limit lower="0" upper="12" effort="100" velocity="5" />
-  </joint>
-  <link
-    name="t_axis_toolchanger">
-    <inertial>
-      <origin
-        xyz="2.66657822625138E-05 -6.51697797860451E-05 -0.0173989628147272"
-        rpy="0 0 0" />
-      <mass
-        value="0.0770166396645032" />
-      <inertia
-        ixx="1.38724675369177E-05"
-        ixy="-2.81065278601148E-08"
-        ixz="-4.32931581160332E-09"
-        iyy="1.28173377099281E-05"
-        iyz="-3.69738102041932E-10"
-        izz="2.32495071670115E-05" />
-    </inertial>
-    <visual>
-      <origin
-        xyz="0 0 0"
-        rpy="0 0 0" />
-      <geometry>
-        <mesh filename="file://$(find pm_robot_description)/meshes/t_axis_tool.STL" />
-      </geometry>
-      <material
-        name="">
-        <color
-          rgba="0.75294 0.75294 0.75294 1" />
-      </material>
-    </visual>
-    <collision>
-      <origin
-        xyz="0 0 0"
-        rpy="0 0 0" />
-      <geometry>
-        <mesh filename="file://$(find pm_robot_description)/meshes/t_axis_tool.STL" />
-      </geometry>
-    </collision>
-  </link>
-  <!---Gravity off-->
-  <gazebo reference="t_axis_toolchanger">
-    <turnGravityOff>true</turnGravityOff>
-  </gazebo>
-  <joint
-    name="t_axis_toolchanger_joint"
-    type="fixed">
-    <origin
-      xyz="0 0 0"
-      rpy="0 0 0" />
-    <parent
-      link="Gripper_Rot_Plate" />
-    <child
-      link="t_axis_toolchanger" />
-    <axis
-      xyz="0 0 0" />
-  </joint>
-  <link
-    name="PM_Robot_Tool_TCP">
-  </link>
-  <joint
-    name="PM_Robot_Tool_TCP_Joint"
-    type="fixed">
-    <!--Hier spaeter Variable-->
-    <origin
-      xyz="0 0 -0.08142"
-      rpy="0 0 0" />
-    <parent
-      link="Gripper_Rot_Plate" />
-    <child
-      link="PM_Robot_Tool_TCP" />
-    <axis
-      xyz="0 0 0" />
-  </joint>
-  <!--%%%%%%%%%%%%% 1K Dispenser Flap Definitions %%%%%%%%%%%%%-->
-  <link
-    name="1K_Dispenser_Flap">
-    <inertial>
-      <origin
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
File: pm_robot_description/urdf/pm_robot_main.xacro (robot description, xacro)
@@ -14,4 +14,5 @@
     <xacro:arg name="with_SPT_R_A1000_I500"           default="false"/>
   <xacro:include filename="$(find pm_robot_description)/urdf/pm_robot.xacro" />
+  <xacro:pm_robot />
   <xacro:include filename="$(find pm_robot_description)/urdf/pm_robot_housing.xacro" />
   <!-- Tool Defines-->
