Commit message: calibration added

File: pm_robot_description/urdf/pm_robot.xacro (robot description, xacro)
@@ -4,6 +4,15 @@
      For more information, please see http://wiki.ros.org/sw_urdf_exporter -->
 <robot xmlns:xacro="http://ros.org/wiki/xacro">
-  <xacro:macro name="pm_robot">
-    <xacro:property name="pm_robot_joint_calibraion_file" value="$(find pm_robot_description)/calibration_config/pm_robot_joint_calibration.yaml" />
+  <xacro:macro name="pm_robot" params="launch_mode">
+    <xacro:if value="${launch_mode == 'sim_HW'}">
+      <xacro:property name="pm_robot_joint_calibraion_file" value="$(find pm_robot_description)/calibration_config/pm_robot_joint_calibration.yaml" />
+    </xacro:if>
+    <!-- If launch_mode 'real' a local path can be specified for the calibration file -->
+    <xacro:if value="${launch_mode == 'real_HW'}">
+      <xacro:property name="local_calibration_file_path__file" value="$(find pm_robot_description)/calibration_config/pm_robot_calibration_path.yaml" />
+      <xacro:property name="path_dict" value="${xacro.load_yaml(local_calibration_file_path__file)}"/>
+      <xacro:property name="local_calibration_file_path" value="${path_dict['pm_robot_calibration_file_path']}"/>
+      <xacro:property name="pm_robot_joint_calibraion_file" value="${local_calibration_file_path}" />
+    </xacro:if>
     <xacro:property name="calibration_dict" value="${xacro.load_yaml(pm_robot_joint_calibraion_file)}"/>
     <link name="world">
@@ -384,4 +393,10 @@
       name="PM_Robot_Tool_TCP">
     </link>
+    <xacro:property name="PM_Robot_Tool_TCP_Joint_Cal_x" value="${calibration_dict['PM_Robot_Tool_TCP_Joint']['x_offset']}"/>
+    <xacro:property name="PM_Robot_Tool_TCP_Joint_Cal_y" value="${calibration_dict['PM_Robot_Tool_TCP_Joint']['y_offset']}"/>
+    <xacro:property name="PM_Robot_Tool_TCP_Joint_Cal_z" value="${calibration_dict['PM_Robot_Tool_TCP_Joint']['z_offset']}"/>
+    <xacro:property name="PM_Robot_Tool_TCP_Joint_Cal_rx" value="${calibration_dict['PM_Robot_Tool_TCP_Joint']['rx_offset']}"/>
+    <xacro:property name="PM_Robot_Tool_TCP_Joint_Cal_ry" value="${calibration_dict['PM_Robot_Tool_TCP_Joint']['ry_offset']}"/>
+    <xacro:property name="PM_Robot_Tool_TCP_Joint_Cal_rz" value="${calibration_dict['PM_Robot_Tool_TCP_Joint']['rz_offset']}"/>
     <joint
       name="PM_Robot_Tool_TCP_Joint"
@@ -389,6 +404,13 @@
       <!--Hier spaeter Variable-->
       <origin
-        xyz="0 0 -0.08142"
-        rpy="0 0 0" />
+        xyz="
+        ${0 + PM_Robot_Tool_TCP_Joint_Cal_x * 0.000001}
+        ${0 + PM_Robot_Tool_TCP_Joint_Cal_y * 0.000001}
+        ${-0.08142 + PM_Robot_Tool_TCP_Joint_Cal_z * 0.000001}"
+        rpy="
+        ${0 + PM_Robot_Tool_TCP_Joint_Cal_rx * 3.14159265359/180}
+        ${0 + PM_Robot_Tool_TCP_Joint_Cal_ry * 3.14159265359/180}
+        ${0 + PM_Robot_Tool_TCP_Joint_Cal_rz * 3.14159265359/180}"
+      />
       <parent
         link="Gripper_Rot_Plate" />
@@ -507,10 +529,24 @@
       name="1K_Dispenser_TCP">
     </link>
+    <!-- Property names should not start with a number -->
+    <xacro:property name="Dispenser_1K_TCP_Joint_Cal_x" value="${calibration_dict['1K_Dispenser_TCP_Joint']['x_offset']}"/>
+    <xacro:property name="Dispenser_1K_TCP_Joint_Cal_y" value="${calibration_dict['1K_Dispenser_TCP_Joint']['y_offset']}"/>
+    <xacro:property name="Dispenser_1K_TCP_Joint_Cal_z" value="${calibration_dict['1K_Dispenser_TCP_Joint']['z_offset']}"/>
+    <xacro:property name="Dispenser_1K_TCP_Joint_Cal_rx" value="${calibration_dict['1K_Dispenser_TCP_Joint']['rx_offset']}"/>
+    <xacro:property name="Dispenser_1K_TCP_Joint_Cal_ry" value="${calibration_dict['1K_Dispenser_TCP_Joint']['ry_offset']}"/>
+    <xacro:property name="Dispenser_1K_TCP_Joint_Cal_rz" value="${calibration_dict['1K_Dispenser_TCP_Joint']['rz_offset']}"/>
     <joint
       name="1K_Dispenser_TCP_Joint"
       type="fixed">
       <origin
-        xyz="-0.001 -0.0318 -0.1285"
-        rpy="0 0 0" />
+        xyz="
+        ${-0.001 + Dispenser_1K_TCP_Joint_Cal_x * 0.000001}
+        ${-0.0318 + Dispenser_1K_TCP_Joint_Cal_y * 0.000001}
+        ${-0.1285 + Dispenser_1K_TCP_Joint_Cal_z * 0.000001}"
+        rpy="
+        ${0 + Dispenser_1K_TCP_Joint_Cal_rx * 3.14159265359/180}
+        ${0 + Dispenser_1K_TCP_Joint_Cal_ry * 3.14159265359/180}
+        ${0 + Dispenser_1K_TCP_Joint_Cal_rz * 3.14159265359/180}"
+      />
       <parent
         link="1K_Dispenser" />
@@ -576,10 +612,24 @@
       name="2K_Dispenser_TCP">
     </link>
+        <!-- Property names should not start with a number -->
+    <xacro:property name="Dispenser_2K_TCP_Joint_Cal_x" value="${calibration_dict['2K_Dispenser_TCP_Joint']['x_offset']}"/>
+    <xacro:property name="Dispenser_2K_TCP_Joint_Cal_y" value="${calibration_dict['2K_Dispenser_TCP_Joint']['y_offset']}"/>
+    <xacro:property name="Dispenser_2K_TCP_Joint_Cal_z" value="${calibration_dict['2K_Dispenser_TCP_Joint']['z_offset']}"/>
+    <xacro:property name="Dispenser_2K_TCP_Joint_Cal_rx" value="${calibration_dict['2K_Dispenser_TCP_Joint']['rx_offset']}"/>
+    <xacro:property name="Dispenser_2K_TCP_Joint_Cal_ry" value="${calibration_dict['2K_Dispenser_TCP_Joint']['ry_offset']}"/>
+    <xacro:property name="Dispenser_2K_TCP_Joint_Cal_rz" value="${calibration_dict['2K_Dispenser_TCP_Joint']['rz_offset']}"/>
     <joint
       name="2K_Dispenser_TCP_Joint"
       type="fixed">
       <origin
-        xyz="0 -0.045 -0.04614"
-        rpy="0 0 0" />
+        xyz="
+        ${0 + Dispenser_2K_TCP_Joint_Cal_x * 0.000001}
+        ${-0.045 + Dispenser_2K_TCP_Joint_Cal_y * 0.000001}
+        ${-0.04614 + Dispenser_2K_TCP_Joint_Cal_z * 0.000001}"
+        rpy="
+        ${0 + Dispenser_2K_TCP_Joint_Cal_rx * 3.14159265359/180}
+        ${0 + Dispenser_2K_TCP_Joint_Cal_ry * 3.14159265359/180}
+        ${0 + Dispenser_2K_TCP_Joint_Cal_rz * 3.14159265359/180}"
+      />
       <parent
         link="2K_Dispenser_Cartridge" />
@@ -632,10 +682,23 @@
       <turnGravityOff>true</turnGravityOff>
     </gazebo>
+    <xacro:property name="Cam1_Toolhead_TCP_Joint_Cal_x" value="${calibration_dict['Cam1_Toolhead_TCP_Joint']['x_offset']}"/>
+    <xacro:property name="Cam1_Toolhead_TCP_Joint_Cal_y" value="${calibration_dict['Cam1_Toolhead_TCP_Joint']['y_offset']}"/>
+    <xacro:property name="Cam1_Toolhead_TCP_Joint_Cal_z" value="${calibration_dict['Cam1_Toolhead_TCP_Joint']['z_offset']}"/>
+    <xacro:property name="Cam1_Toolhead_TCP_Joint_Cal_rx" value="${calibration_dict['Cam1_Toolhead_TCP_Joint']['rx_offset']}"/>
+    <xacro:property name="Cam1_Toolhead_TCP_Joint_Cal_ry" value="${calibration_dict['Cam1_Toolhead_TCP_Joint']['ry_offset']}"/>
+    <xacro:property name="Cam1_Toolhead_TCP_Joint_Cal_rz" value="${calibration_dict['Cam1_Toolhead_TCP_Joint']['rz_offset']}"/>
     <joint
       name="Cam1_Toolhead_TCP_Joint"
       type="fixed">
       <origin
-        xyz="-0.0320000000000003 -0.0579999999999998 -0.515338706"
-        rpy="0 0 0" />
+        xyz="
+        ${-0.0320000000000003 + Cam1_Toolhead_TCP_Joint_Cal_x * 0.000001}
+        ${-0.0579999999999998 + Cam1_Toolhead_TCP_Joint_Cal_y * 0.000001}
+        ${-0.515338706 + Cam1_Toolhead_TCP_Joint_Cal_z * 0.000001}"
+        rpy="
+        ${0 + Cam1_Toolhead_TCP_Joint_Cal_rx * 3.14159265359/180}
+        ${0 + Cam1_Toolhead_TCP_Joint_Cal_ry * 3.14159265359/180}
+        ${0 + Cam1_Toolhead_TCP_Joint_Cal_rz * 3.14159265359/180}"
+      />
       <parent
         link="Z_Axis" />
@@ -691,4 +754,7 @@
       <xacro:property name="Laser_Toolhead_TCP_Joint_Cal_y" value="${calibration_dict['Laser_Toolhead_TCP_Joint']['y_offset']}"/>
       <xacro:property name="Laser_Toolhead_TCP_Joint_Cal_z" value="${calibration_dict['Laser_Toolhead_TCP_Joint']['z_offset']}"/>
+      <xacro:property name="Laser_Toolhead_TCP_Joint_Cal_rx" value="${calibration_dict['Laser_Toolhead_TCP_Joint']['rx_offset']}"/>
+      <xacro:property name="Laser_Toolhead_TCP_Joint_Cal_ry" value="${calibration_dict['Laser_Toolhead_TCP_Joint']['ry_offset']}"/>
+      <xacro:property name="Laser_Toolhead_TCP_Joint_Cal_rz" value="${calibration_dict['Laser_Toolhead_TCP_Joint']['rz_offset']}"/>
       <joint
         name="Laser_Toolhead_TCP_Joint"
@@ -699,5 +765,9 @@
           ${-0.0899999732334101 + Laser_Toolhead_TCP_Joint_Cal_y*0.000001}
           ${-0.495500000000011+ Laser_Toolhead_TCP_Joint_Cal_z*0.000001}"
-          rpy="0 0 0" />
+          rpy="
+          ${0 + Laser_Toolhead_TCP_Joint_Cal_rx*3.14159265359/180}
+          ${0 + Laser_Toolhead_TCP_Joint_Cal_ry*3.14159265359/180}
+          ${0 + Laser_Toolhead_TCP_Joint_Cal_rz*3.14159265359/180}"
+          />
         <parent
           link="Z_Axis" />
@@ -806,10 +876,23 @@
       name="Camera_Station_TCP">
     </link>
+    <xacro:property name="Camera_Station_TCP_Joint_Cal_x" value="${calibration_dict['Camera_Station_TCP_Joint']['x_offset']}"/>
+    <xacro:property name="Camera_Station_TCP_Joint_Cal_y" value="${calibration_dict['Camera_Station_TCP_Joint']['y_offset']}"/>
+    <xacro:property name="Camera_Station_TCP_Joint_Cal_z" value="${calibration_dict['Camera_Station_TCP_Joint']['z_offset']}"/>
+    <xacro:property name="Camera_Station_TCP_Joint_Cal_rx" value="${calibration_dict['Camera_Station_TCP_Joint']['rx_offset']}"/>
+    <xacro:property name="Camera_Station_TCP_Joint_Cal_ry" value="${calibration_dict['Camera_Station_TCP_Joint']['ry_offset']}"/>
+    <xacro:property name="Camera_Station_TCP_Joint_Cal_rz" value="${calibration_dict['Camera_Station_TCP_Joint']['rz_offset']}"/>
     <joint
       name="Camera_Station_TCP_Joint"
       type="fixed">
       <origin
-        xyz="0.08 0.092783 0.3045"
-        rpy="0 0 0" />
+        xyz="
+        ${0.08 + Camera_Station_TCP_Joint_Cal_x*0.000001}
+        ${0.092783 + Camera_Station_TCP_Joint_Cal_y*0.000001}
+        ${0.3045 + Camera_Station_TCP_Joint_Cal_z*0.000001}"
+        rpy="
+        ${0 + Camera_Station_TCP_Joint_Cal_rx*3.14159265359/180}
+        ${0 + Camera_Station_TCP_Joint_Cal_ry*3.14159265359/180}
+        ${0 + Camera_Station_TCP_Joint_Cal_rz*3.14159265359/180}"
+      />
       <parent
         link="Camera_Station" />
@@ -857,10 +940,23 @@
         </collision>
       </link>
+      <xacro:property name="Station_Laser_Bottom_TCP_Joint_Cal_x" value="${calibration_dict['Station_Laser_Bottom_TCP_Joint']['x_offset']}"/>
+      <xacro:property name="Station_Laser_Bottom_TCP_Joint_Cal_y" value="${calibration_dict['Station_Laser_Bottom_TCP_Joint']['y_offset']}"/>
+      <xacro:property name="Station_Laser_Bottom_TCP_Joint_Cal_z" value="${calibration_dict['Station_Laser_Bottom_TCP_Joint']['z_offset']}"/>
+      <xacro:property name="Station_Laser_Bottom_TCP_Joint_Cal_rx" value="${calibration_dict['Station_Laser_Bottom_TCP_Joint']['rx_offset']}"/>
+      <xacro:property name="Station_Laser_Bottom_TCP_Joint_Cal_ry" value="${calibration_dict['Station_Laser_Bottom_TCP_Joint']['ry_offset']}"/>
+      <xacro:property name="Station_Laser_Bottom_TCP_Joint_Cal_rz" value="${calibration_dict['Station_Laser_Bottom_TCP_Joint']['rz_offset']}"/>
       <joint
         name="Station_Laser_Bottom_TCP_Joint"
         type="fixed">
         <origin
-          xyz="0.1799989100971 0.0939999732334095 0.328499853483917"
-          rpy="0 0 0" />
+        xyz="
+          ${0.1799989100971 + Station_Laser_Bottom_TCP_Joint_Cal_x*0.000001}
+          ${0.0939999732334095 + Station_Laser_Bottom_TCP_Joint_Cal_y*0.000001}
+          ${0.328499853483917 + Station_Laser_Bottom_TCP_Joint_Cal_z*0.000001}"
+          rpy="
+          ${0 + Station_Laser_Bottom_TCP_Joint_Cal_rx*3.14159265359/180}
+          ${0 + Station_Laser_Bottom_TCP_Joint_Cal_ry*3.14159265359/180}
+          ${0 + Station_Laser_Bottom_TCP_Joint_Cal_rz*3.14159265359/180}"
+        />
         <parent
           link="Camera_Station" />
@@ -958,10 +1054,23 @@
       <turnGravityOff>true</turnGravityOff>
     </gazebo>
+    <xacro:property name="Calibration_Qube_Joint_Cal_x" value="${calibration_dict['Calibration_Qube_Joint']['x_offset']}"/>
+    <xacro:property name="Calibration_Qube_Joint_Cal_y" value="${calibration_dict['Calibration_Qube_Joint']['y_offset']}"/>
+    <xacro:property name="Calibration_Qube_Joint_Cal_z" value="${calibration_dict['Calibration_Qube_Joint']['z_offset']}"/>
+    <xacro:property name="Calibration_Qube_Joint_Cal_rx" value="${calibration_dict['Calibration_Qube_Joint']['rx_offset']}"/>
+    <xacro:property name="Calibration_Qube_Joint_Cal_ry" value="${calibration_dict['Calibration_Qube_Joint']['ry_offset']}"/>
+    <xacro:property name="Calibration_Qube_Joint_Cal_rz" value="${calibration_dict['Calibration_Qube_Joint']['rz_offset']}"/>
     <joint
       name="Calibration_Qube_Joint"
       type="prismatic">
       <origin
-        xyz="0.152 0.108 0.326"
-        rpy="0 0 0" />
+        xyz="
+          ${0.152 + Calibration_Qube_Joint_Cal_x*0.000001}
+          ${0.108 + Calibration_Qube_Joint_Cal_y*0.000001}
+          ${0.326 + Calibration_Qube_Joint_Cal_z*0.000001}"
+          rpy="
+          ${0 + Calibration_Qube_Joint_Cal_rx*3.14159265359/180}
+          ${0 + Calibration_Qube_Joint_Cal_ry*3.14159265359/180}
+          ${0 + Calibration_Qube_Joint_Cal_rz*3.14159265359/180}"
+      />
       <parent
         link="Camera_Station" />

File: pm_robot_description/urdf/pm_robot_main.xacro (robot description, xacro)
@@ -14,5 +14,5 @@
     <xacro:arg name="with_SPT_R_A1000_I500"           default="false"/>
   <xacro:include filename="$(find pm_robot_description)/urdf/pm_robot.xacro" />
-  <xacro:pm_robot />
+  <xacro:pm_robot launch_mode="$(arg launch_mode)"/>
   <xacro:include filename="$(find pm_robot_description)/urdf/pm_robot_housing.xacro" />
   <!-- Tool Defines-->

Commit message: bringup fixes

File: pm_robot_description/urdf/pm_robot.xacro (robot description, xacro)
@@ -10,9 +10,9 @@
     <!-- If launch_mode 'real' a local path can be specified for the calibration file -->
     <xacro:if value="${launch_mode == 'real_HW'}">
-      <!-- <xacro:property name="local_calibration_file_path__file" value="$(find pm_robot_description)/calibration_config/pm_robot_calibration_path.yaml" />
+      <xacro:property name="local_calibration_file_path__file" value="$(find pm_robot_description)/calibration_config/pm_robot_calibration_path.yaml" />
       <xacro:property name="path_dict" value="${xacro.load_yaml(local_calibration_file_path__file)}"/>
       <xacro:property name="local_calibration_file_path" value="${path_dict['pm_robot_calibration_file_path']}"/>
-      <xacro:property name="pm_robot_joint_calibraion_file" value="${local_calibration_file_path}" /> -->
-      <xacro:property name="pm_robot_joint_calibraion_file" value="$(find pm_robot_description)/calibration_config/pm_robot_joint_calibration.yaml" />
+      <xacro:property name="pm_robot_joint_calibraion_file" value="${local_calibration_file_path}" />
+      <!-- <xacro:property name="pm_robot_joint_calibraion_file" value="$(find pm_robot_description)/calibration_config/pm_robot_joint_calibration.yaml" /> -->
     </xacro:if>
     <xacro:property name="calibration_dict" value="${xacro.load_yaml(pm_robot_joint_calibraion_file)}"/>

File: pm_robot_description/urdf/ros2_control_real_HW.xacro (robot description, xacro)
@@ -33,5 +33,5 @@
                 <state_interface name="velocity"/>
             </joint>
-            <joint name="1K_Dispenser_Flap_Joint">
+            <!-- <joint name="1K_Dispenser_Flap_Joint">
                 <command_interface name="position">
                 </command_interface>
@@ -113,5 +113,5 @@
                     <state_interface name="velocity"/>
                 </joint>
-            </xacro:if>
+            </xacro:if> -->
         </ros2_control>
     </xacro:macro>

File: pm_robot_description/urdf/ros2_control_sim_HW.xacro (robot description, xacro)
@@ -1,7 +1,6 @@
 <?xml version="1.0"?>
 <robot xmlns:xacro="http://www.ros.org/wiki/xacro">
-    <!-- <xacro:macro name="pm_robot_ros2_control_hw_sim" params="name initial_positions_file"> -->
-    <xacro:macro name="pm_robot_ros2_control_hw_sim">
-        <!-- <xacro:property name="initial_positions" value="${load_yaml(initial_positions_file)['initial_positions']}"/> -->
+    <xacro:macro name="pm_robot_ros2_control_hw_sim" params="name initial_positions_file">
+        <xacro:property name="initial_positions" value="${load_yaml(initial_positions_file)['initial_positions']}"/>
         <ros2_control name="GazeboSystem" type="system">
             <hardware>

Commit message: joint limits fixed

File: pm_robot_description/urdf/pm_robot.xacro (robot description, xacro)
@@ -139,5 +139,5 @@
       <child link="Y_Axis" />
       <axis xyz="0 1 0" />
-      <limit lower="-0.134000" upper="-0.019700" effort="100" velocity="35" />
+      <limit lower="-0.134000" upper="0.032400" effort="100" velocity="35" />
     </joint>
     <!--%%%%%%%%%%%%% Z Axis Definitions %%%%%%%%%%%%%-->
@@ -171,5 +171,5 @@
       <child link="Z_Axis" />
       <axis xyz="0 0 -1" />
-      <limit lower="-0.05262" upper="0.055" effort="100" velocity="35" />
+      <limit lower="-0.0562" upper="0.041" effort="100" velocity="35" />
     </joint>
     <!--%%%%%%%%%%%%% T Axis Definitions %%%%%%%%%%%%%-->

Commit message: Movit2 with real HW

File: pm_robot_description/urdf/pm_robot.xacro (robot description, xacro)
@@ -111,5 +111,5 @@
       <child link="X_Axis" />
       <axis xyz="1 0 0" />
-      <limit lower="-0.745" upper="0.055" effort="0.1" velocity="35" />
+      <limit lower="-0.745" upper="0.05" effort="0.1" velocity="35" />
     </joint>
     <!--%%%%%%%%%%%%% Y Axis Definitions %%%%%%%%%%%%%-->
@@ -167,5 +167,5 @@
     </gazebo>
     <joint name="Z_Axis_Joint" type="prismatic">
-      <origin xyz="-0.00365 -0.499 0.33875" rpy="0 0 0" />
+      <origin xyz="-0.00365 -0.499 0.28025" rpy="0 0 0" />
       <parent link="Y_Axis" />
       <child link="Z_Axis" />
