Commit message: modular gonios & new gripper

File: pm_robot_description/urdf/pm_robot.xacro (robot description, xacro)
@@ -26,4 +26,5 @@
     <xacro:property name="current_pm_robot_bringup_config" value="${xacro.load_yaml(pm_robot_bringup_config_file)}"/>
     <xacro:property name="current_pm_robot_1K_dipsenser_tip" value="${current_pm_robot_bringup_config['pm_robot_1K_dispenser_tip']['use_dispenser_tip']}"/>
+    <xacro:property name="current_vacuum_tool" value="${current_pm_robot_bringup_config['pm_robot_tools']['pm_robot_vacuum_tools']['use_tool']}"/>
     <xacro:property name="calibration_dict" value="${xacro.load_yaml(pm_robot_joint_calibraion_file)}"/>
     <link name="world">
@@ -254,4 +255,5 @@
       <axis xyz="0 0 0" />
     </joint>
+<!--
     <link name="PM_Robot_Tool_TCP">
     </link>
@@ -262,10 +264,11 @@
     <xacro:property name="PM_Robot_Tool_TCP_Joint_Cal_ry" value="${calibration_dict['PM_Robot_Tool_TCP_Joint']['ry_offset']}"/>
     <xacro:property name="PM_Robot_Tool_TCP_Joint_Cal_rz" value="${calibration_dict['PM_Robot_Tool_TCP_Joint']['rz_offset']}"/>
+    <xacro:property name="pm_robot_tool_TCP_z_offset" value="$(arg pm_robot_tool_TCP_z_offset)"/>
     <joint name="PM_Robot_Tool_TCP_Joint" type="fixed">
-      <!--Hier spaeter Variable-->
+      Hier spaeter Variable
       <origin xyz="
         ${0 + PM_Robot_Tool_TCP_Joint_Cal_x * 0.000001}
         ${0 + PM_Robot_Tool_TCP_Joint_Cal_y * 0.000001}
-        ${-0.08142 + PM_Robot_Tool_TCP_Joint_Cal_z * 0.000001}" rpy="
+        ${0 + pm_robot_tool_TCP_z_offset + PM_Robot_Tool_TCP_Joint_Cal_z * 0.000001}" rpy="
         ${0 + PM_Robot_Tool_TCP_Joint_Cal_rx * 3.14159265359/180}
         ${0 + PM_Robot_Tool_TCP_Joint_Cal_ry * 3.14159265359/180}
@@ -274,5 +277,5 @@
       <child link="PM_Robot_Tool_TCP" />
       <axis xyz="0 0 0" />
-    </joint>
+    </joint> -->
     <!--%%%%%%%%%%%%% 1K Dispenser Flap Definitions %%%%%%%%%%%%%-->
     <link name="1K_Dispenser_Flap">

File: pm_robot_description/urdf/pm_robot_gonio_left.xacro (robot description, xacro)
@@ -3,5 +3,30 @@
      Commit Version: 1.6.0-1-g15f4949  Build Version: 1.6.7594.29634
      For more information, please see http://wiki.ros.org/sw_urdf_exporter -->
-<robot name="pm_robot_gonio_left">
+<robot xmlns:xacro="http://ros.org/wiki/xacro">
+    <xacro:macro name="pm_robot_gonio_left" params="launch_mode">
+  <!-- Loading of the Robot Joint calibrations -->
+  <xacro:if value="${launch_mode == 'sim_HW'}">
+    <xacro:property name="pm_robot_joint_calibraion_file" value="$(find pm_robot_description)/calibration_config/pm_robot_joint_calibration.yaml" />
+    <xacro:property name="pm_robot_bringup_config_file" value="$(find pm_robot_bringup)/config/pm_robot_bringup_config.yaml" />
+  </xacro:if>
+  <!-- If launch_mode 'real' a local path can be specified for the calibration file -->
+  <xacro:if value="${launch_mode == 'real_HW'}">
+    <xacro:property name="local_file_paths__file" value="$(find pm_robot_description)/calibration_config/pm_robot_path_real_HW.yaml" />
+    <xacro:property name="path_dict" value="${xacro.load_yaml(local_file_paths__file)}"/>
+    <xacro:property name="local_calibration_file_path" value="${path_dict['pm_robot_calibration_file_path']}"/>
+    <xacro:property name="local_robot_bringup_file_path" value="${path_dict['pm_robot_bringup_config_file_path']}"/>
+    <!-- REAL -->
+    <!-- <xacro:property name="pm_robot_joint_calibraion_file" value="${local_calibration_file_path}" />
+    <xacro:property name="pm_robot_bringup_config_file" value="${local_robot_bringup_file_path}"/> -->
+    <!-- SIM -->
+    <xacro:property name="pm_robot_joint_calibraion_file" value="$(find pm_robot_description)/calibration_config/pm_robot_joint_calibration.yaml" />
+    <xacro:property name="pm_robot_bringup_config_file" value="$(find pm_robot_bringup)/config/pm_robot_bringup_config.yaml" />
+  </xacro:if>
+  <xacro:property name="current_pm_robot_bringup_config" value="${xacro.load_yaml(pm_robot_bringup_config_file)}"/>
+  <xacro:property name="current_gonio_left_chuck" value="${current_pm_robot_bringup_config['pm_robot_gonio_left']['use_chuck']}"/>
+  <xacro:property name="calibration_dict" value="${xacro.load_yaml(pm_robot_joint_calibraion_file)}"/>
+  <!-- Init Definition of gonio chuck dict -->
+  <xacro:property name="gonio_left_configs_file" value="$(find pm_robot_description)/urdf/urdf_configs/gonio_left_chuck_config.yaml" />
+  <xacro:property name="gonio_left_configs_dict" value="${xacro.load_yaml(gonio_left_configs_file)}"/>
  <!--%%%%%%%%%%%%% Gonio Station Left Definitions-->
   <link
@@ -160,8 +185,8 @@
   <!--%%%%%%%%%%%%% Gonio Left Chuck Definitions-->
   <link
-    name="Gonio_Left_Chuck">
-  </link>
-  <joint
-    name="Gonio_Left_Chuck_Joint"
+    name="Gonio_Left_Chuck_Origin">
+  </link>
+  <joint
+    name="Gonio_Left_Chuck_Origin_Joint"
     type="fixed">
     <origin
@@ -171,8 +196,77 @@
       link="Gonio_Left_Stage_2_Bottom" />
     <child
-      link="Gonio_Left_Chuck" />
+      link="Gonio_Left_Chuck_Origin" />
     <axis
       xyz="0 0 0" />
   </joint>
+  <!--%%%%%%%%%%%%% Gonio Left Example Chuck Definitions-->
+  <!--%%%%%%%%%%%%% This is for the Chuck  -->
+  <xacro:property name="gonio_chuck_tcp_offset_x" value="${gonio_left_configs_dict[current_gonio_left_chuck]['tcp_offset_from_gonio_x']}"/>
+  <xacro:property name="gonio_chuck_tcp_offset_y" value="${gonio_left_configs_dict[current_gonio_left_chuck]['tcp_offset_from_gonio_y']}"/>
+  <xacro:property name="gonio_chuck_tcp_offset_z" value="${gonio_left_configs_dict[current_gonio_left_chuck]['tcp_offset_from_gonio_z']}"/>
+  <xacro:property name="gonio_chuck_xyz" value="${gonio_left_configs_dict[current_gonio_left_chuck]['xyz']}"/>
+  <xacro:property name="gonio_chuck_xyz" value="${gonio_left_configs_dict[current_gonio_left_chuck]['xyz']}"/>
+  <xacro:property name="gonio_chuck_xyz" value="${gonio_left_configs_dict[current_gonio_left_chuck]['xyz']}"/>
+  <xacro:property name="gonio_chuck_rpy" value="${gonio_left_configs_dict[current_gonio_left_chuck]['rpy']}"/>
+  <xacro:property name="gonio_chuck_mass" value="${gonio_left_configs_dict[current_gonio_left_chuck]['mass']}"/>
+  <xacro:property name="gonio_chuck_inertia_ixx" value="${gonio_left_configs_dict[current_gonio_left_chuck]['inertia_ixx']}"/>
+  <xacro:property name="gonio_chuck_inertia_ixy" value="${gonio_left_configs_dict[current_gonio_left_chuck]['inertia_ixy']}"/>
+  <xacro:property name="gonio_chuck_inertia_ixz" value="${gonio_left_configs_dict[current_gonio_left_chuck]['inertia_ixz']}"/>
+  <xacro:property name="gonio_chuck_inertia_iyy" value="${gonio_left_configs_dict[current_gonio_left_chuck]['inertia_iyy']}"/>
+  <xacro:property name="gonio_chuck_inertia_iyz" value="${gonio_left_configs_dict[current_gonio_left_chuck]['inertia_iyz']}"/>
+  <xacro:property name="gonio_chuck_inertia_izz" value="${gonio_left_configs_dict[current_gonio_left_chuck]['inertia_izz']}"/>
+  <xacro:property name="gonio_chuck_color" value="${gonio_left_configs_dict[current_gonio_left_chuck]['color']}"/>
+  <xacro:property name="gonio_chuck_visual_filename" value="${gonio_left_configs_dict[current_gonio_left_chuck]['visual_filename']}"/>
+  <xacro:property name="gonio_chuck_collision_filename" value="${gonio_left_configs_dict[current_gonio_left_chuck]['collision_filename']}"/>
+<link
+  name="Gonio_Left_Chuck">
+  <inertial>
+    <origin
+      xyz="${gonio_chuck_xyz}"
+      rpy="${gonio_chuck_rpy}"/>
+    <mass
+      value="${gonio_chuck_mass}"/>
+    <inertia
+      ixx="${gonio_chuck_inertia_ixx}"
+      ixy="${gonio_chuck_inertia_ixy}"
+      ixz="${gonio_chuck_inertia_ixz}"
+      iyy="${gonio_chuck_inertia_iyy}"
+      iyz="${gonio_chuck_inertia_iyz}"
+      izz="${gonio_chuck_inertia_izz}" />
+  </inertial>
+  <visual>
+    <origin
+      xyz="0 0 0"
+      rpy="0 0 0" />
+    <geometry>
+      <mesh filename="file://$(find pm_robot_description)/meshes/Gonio_Left/Gonio_Left_Chucks/${gonio_chuck_visual_filename}" />
+    </geometry>
+    <material
+      name="${gonio_chuck_color}">
+    </material>
+  </visual>
+  <collision>
+    <origin
+      xyz="0 0 0"
+      rpy="0 0 0" />
+    <geometry>
+      <mesh filename="file://$(find pm_robot_description)/meshes/Gonio_Left/Gonio_Left_Chucks/${gonio_chuck_collision_filename}" />
+    </geometry>
+  </collision>
+</link>
+<joint
+  name="Gonio_Left_Chuck_Joint"
+  type="fixed">
+  <origin
+    xyz="0 0 0"
+    rpy="0 0 0" />
+  <parent
+    link="Gonio_Left_Chuck_Origin" />
+  <child
+    link="Gonio_Left_Chuck" />
+  <axis
+    xyz="0 0 0" />
+</joint>
+  <!--%%%%%%%%%%%%% Gonio Left Part Origin -->
   <link
     name="Gonio_Left_Part_Origin">
@@ -182,8 +276,8 @@
     type="fixed">
     <origin
-      xyz="0 0 0"
-      rpy="0 0 0" />
-    <parent
-      link="Gonio_Left_Chuck" />
+      xyz="${gonio_chuck_tcp_offset_x} ${gonio_chuck_tcp_offset_y} ${gonio_chuck_tcp_offset_z}"
+      rpy="0 0 0" />
+    <parent
+      link="Gonio_Left_Chuck_Origin" />
     <child
       link="Gonio_Left_Part_Origin" />
@@ -191,60 +285,8 @@
       xyz="0 0 0" />
   </joint>
-  <!--%%%%%%%%%%%%% Gonio Left Example Chuck Definitions-->
-  <link
-    name="Gonio_Left_Example_Chuck">
-    <inertial>
-      <origin
-        xyz="0.00851660407252697 0.00736263697453748 0.0446054201819609"
-        rpy="0 0 0" />
-      <mass
-        value="0.193859196068301" />
-      <inertia
-        ixx="6.74557361964199E-05"
-        ixy="-1.48218596250914E-05"
-        ixz="-9.56044333605206E-07"
-        iyy="0.000514689088229689"
-        iyz="-1.14966587929801E-06"
-        izz="0.00047114586366426" />
-    </inertial>
-    <visual>
-      <origin
-        xyz="0 0 0"
-        rpy="0 0 0" />
-      <geometry>
-        <mesh filename="file://$(find pm_robot_description)/meshes/Gonio_Left/Gonio_Left_Chuck.STL" />
-      </geometry>
-      <material
-        name="">
-        <color
-          rgba="0.752941176470588 0.752941176470588 0.752941176470588 1" />
-      </material>
-    </visual>
-    <collision>
-      <origin
-        xyz="0 0 0"
-        rpy="0 0 0" />
-      <geometry>
-        <mesh filename="file://$(find pm_robot_description)/meshes/Gonio_Left/Gonio_Left_Chuck.STL" />
-      </geometry>
-    </collision>
-  </link>
   <!---Gravity off-->
-  <gazebo reference="Gonio_Left_Example_Chuck">
+  <gazebo reference="Gonio_Left_Chuck">
     <turnGravityOff>true</turnGravityOff>
   </gazebo>
-  <joint
-    name="Gonio_Left_Example_Chuck_Joint"
-    type="fixed">
-    <origin
-      xyz="0 0 0"
-      rpy="0 0 0" />
-    <parent
-      link="Gonio_Left_Chuck" />
-    <child
-      link="Gonio_Left_Example_Chuck" />
-    <axis
-      xyz="0 0 0" />
-  </joint>
   <!--%%%%%%%%%%%%% UV Slider X Front Definitions-->
   <link
@@ -443,3 +485,4 @@
     <limit lower="0" upper="0.05" effort="100" velocity="0.05" />
   </joint>
+</xacro:macro>
 </robot>

File: pm_robot_description/urdf/pm_robot_gonio_right.xacro (robot description, xacro)
@@ -3,5 +3,30 @@
      Commit Version: 1.6.0-1-g15f4949  Build Version: 1.6.7594.29634
      For more information, please see http://wiki.ros.org/sw_urdf_exporter -->
-<robot name="pm_robot_Gonio_Right">
+     <robot xmlns:xacro="http://ros.org/wiki/xacro">
+      <xacro:macro name="pm_robot_gonio_right" params="launch_mode">
+    <!-- Loading of the Robot Joint calibrations -->
+    <xacro:if value="${launch_mode == 'sim_HW'}">
+      <xacro:property name="pm_robot_joint_calibraion_file" value="$(find pm_robot_description)/calibration_config/pm_robot_joint_calibration.yaml" />
+      <xacro:property name="pm_robot_bringup_config_file" value="$(find pm_robot_bringup)/config/pm_robot_bringup_config.yaml" />
+    </xacro:if>
+    <!-- If launch_mode 'real' a local path can be specified for the calibration file -->
+    <xacro:if value="${launch_mode == 'real_HW'}">
+      <xacro:property name="local_file_paths__file" value="$(find pm_robot_description)/calibration_config/pm_robot_path_real_HW.yaml" />
+      <xacro:property name="path_dict" value="${xacro.load_yaml(local_file_paths__file)}"/>
+      <xacro:property name="local_calibration_file_path" value="${path_dict['pm_robot_calibration_file_path']}"/>
+      <xacro:property name="local_robot_bringup_file_path" value="${path_dict['pm_robot_bringup_config_file_path']}"/>
+      <!-- REAL -->
+      <!-- <xacro:property name="pm_robot_joint_calibraion_file" value="${local_calibration_file_path}" />
+      <xacro:property name="pm_robot_bringup_config_file" value="${local_robot_bringup_file_path}"/> -->
+      <!-- SIM -->
+      <xacro:property name="pm_robot_joint_calibraion_file" value="$(find pm_robot_description)/calibration_config/pm_robot_joint_calibration.yaml" />
+      <xacro:property name="pm_robot_bringup_config_file" value="$(find pm_robot_bringup)/config/pm_robot_bringup_config.yaml" />
+    </xacro:if>
+    <xacro:property name="current_pm_robot_bringup_config" value="${xacro.load_yaml(pm_robot_bringup_config_file)}"/>
+    <xacro:property name="current_gonio_right_chuck" value="${current_pm_robot_bringup_config['pm_robot_gonio_right']['use_chuck']}"/>
+    <xacro:property name="calibration_dict" value="${xacro.load_yaml(pm_robot_joint_calibraion_file)}"/>
+    <!-- Init Definition of gonio chuck dict -->
+    <xacro:property name="gonio_right_configs_file" value="$(find pm_robot_description)/urdf/urdf_configs/gonio_right_chuck_config.yaml" />
+    <xacro:property name="gonio_right_configs_dict" value="${xacro.load_yaml(gonio_right_configs_file)}"/>
 <!--%%%%%%%%%%%%% Gonio_Right Definitions %%%%%%%%-->
   <link
@@ -212,8 +237,8 @@
   <!--%%%%%%%%%%%%% Gonio Right Chuck Definitions-->
   <link
-    name="Gonio_Right_Chuck">
-  </link>
-  <joint
-    name="Gonio_Right_Chuck_Joint"
+    name="Gonio_Right_Chuck_Origin">
+  </link>
+  <joint
+    name="Gonio_Right_Chuck_Origin_Joint"
     type="fixed">
     <origin
@@ -223,8 +248,75 @@
       link="Gonio_Right_Stage_2_Bottom" />
     <child
-      link="Gonio_Right_Chuck" />
+      link="Gonio_Right_Chuck_Origin" />
     <axis
       xyz="0 0 0" />
   </joint>
+  <!--%%%%%%%%%%%%% This is for the Chuck  -->
+  <xacro:property name="gonio_chuck_tcp_offset_x" value="${gonio_right_configs_dict[current_gonio_right_chuck]['tcp_offset_from_gonio_x']}"/>
+  <xacro:property name="gonio_chuck_tcp_offset_y" value="${gonio_right_configs_dict[current_gonio_right_chuck]['tcp_offset_from_gonio_y']}"/>
+  <xacro:property name="gonio_chuck_tcp_offset_z" value="${gonio_right_configs_dict[current_gonio_right_chuck]['tcp_offset_from_gonio_z']}"/>
+  <xacro:property name="gonio_chuck_xyz" value="${gonio_right_configs_dict[current_gonio_right_chuck]['xyz']}"/>
+  <xacro:property name="gonio_chuck_xyz" value="${gonio_right_configs_dict[current_gonio_right_chuck]['xyz']}"/>
+  <xacro:property name="gonio_chuck_xyz" value="${gonio_right_configs_dict[current_gonio_right_chuck]['xyz']}"/>
+  <xacro:property name="gonio_chuck_rpy" value="${gonio_right_configs_dict[current_gonio_right_chuck]['rpy']}"/>
+  <xacro:property name="gonio_chuck_mass" value="${gonio_right_configs_dict[current_gonio_right_chuck]['mass']}"/>
+  <xacro:property name="gonio_chuck_inertia_ixx" value="${gonio_right_configs_dict[current_gonio_right_chuck]['inertia_ixx']}"/>
+  <xacro:property name="gonio_chuck_inertia_ixy" value="${gonio_right_configs_dict[current_gonio_right_chuck]['inertia_ixy']}"/>
+  <xacro:property name="gonio_chuck_inertia_ixz" value="${gonio_right_configs_dict[current_gonio_right_chuck]['inertia_ixz']}"/>
+  <xacro:property name="gonio_chuck_inertia_iyy" value="${gonio_right_configs_dict[current_gonio_right_chuck]['inertia_iyy']}"/>
+  <xacro:property name="gonio_chuck_inertia_iyz" value="${gonio_right_configs_dict[current_gonio_right_chuck]['inertia_iyz']}"/>
+  <xacro:property name="gonio_chuck_inertia_izz" value="${gonio_right_configs_dict[current_gonio_right_chuck]['inertia_izz']}"/>
+  <xacro:property name="gonio_chuck_color" value="${gonio_right_configs_dict[current_gonio_right_chuck]['color']}"/>
+  <xacro:property name="gonio_chuck_visual_filename" value="${gonio_right_configs_dict[current_gonio_right_chuck]['visual_filename']}"/>
+  <xacro:property name="gonio_chuck_collision_filename" value="${gonio_right_configs_dict[current_gonio_right_chuck]['collision_filename']}"/>
+<link
+  name="Gonio_Right_Chuck">
+  <inertial>
+    <origin
+      xyz="${gonio_chuck_xyz}"
+      rpy="${gonio_chuck_rpy}"/>
+    <mass
+      value="${gonio_chuck_mass}"/>
+    <inertia
+      ixx="${gonio_chuck_inertia_ixx}"
+      ixy="${gonio_chuck_inertia_ixy}"
+      ixz="${gonio_chuck_inertia_ixz}"
+      iyy="${gonio_chuck_inertia_iyy}"
+      iyz="${gonio_chuck_inertia_iyz}"
+      izz="${gonio_chuck_inertia_izz}" />
+  </inertial>
+  <visual>
+    <origin
+      xyz="0 0 0"
+      rpy="0 0 0" />
+    <geometry>
+      <mesh filename="file://$(find pm_robot_description)/meshes/Gonio_Right/Gonio_Right_Chucks/${gonio_chuck_visual_filename}" />
+    </geometry>
+    <material
+      name="${gonio_chuck_color}">
+    </material>
+  </visual>
+  <collision>
+    <origin
+      xyz="0 0 0"
+      rpy="0 0 0" />
+    <geometry>
+      <mesh filename="file://$(find pm_robot_description)/meshes/Gonio_Right/Gonio_Right_Chucks/${gonio_chuck_collision_filename}" />
+    </geometry>
+  </collision>
+</link>
+<joint
+  name="Gonio_Right_Chuck_Joint"
+  type="fixed">
+  <origin
+    xyz="0 0 0"
+    rpy="0 0 0" />
+  <parent
+    link="Gonio_Right_Chuck_Origin" />
+  <child
+    link="Gonio_Right_Chuck" />
+  <axis
+    xyz="0 0 0" />
+</joint>
   <!--%%%%%%%%%%%%% Gonio Right Part Origin -->
   <link
@@ -235,8 +327,8 @@
     type="fixed">
     <origin
-      xyz="0 0 0"
-      rpy="0 0 0" />
-    <parent
-      link="Gonio_Right_Chuck" />
+      xyz="${gonio_chuck_tcp_offset_x} ${gonio_chuck_tcp_offset_y} ${gonio_chuck_tcp_offset_z}"
+      rpy="0 0 0" />
+    <parent
+      link="Gonio_Right_Chuck_Origin" />
     <child
       link="Gonio_Right_Part_Origin" />
@@ -244,55 +336,4 @@
       xyz="0 0 0" />
   </joint>
-  <!--%%%%%%%%%%%%% This is a Chuck Example -->
-  <link
-    name="Gonio_Right_Example_Chuck">
-    <inertial>
-      <origin
-        xyz="-4.91275391850676E-05 -7.08920350384057E-06 0.0216564841336891"
-        rpy="0 0 0" />
-      <mass
-        value="0.133934804202608" />
-      <inertia
-        ixx="3.05433990945277E-05"
-        ixy="-2.55507616624267E-10"
-        ixz="-1.7486699307754E-08"
-        iyy="4.80787890381723E-05"
-        iyz="2.24246430305895E-09"
-        izz="7.18729232269431E-05" />
-    </inertial>
-    <visual>
-      <origin
-        xyz="0 0 0"
-        rpy="0 0 0" />
-      <geometry>
-        <mesh filename="file://$(find pm_robot_description)/meshes/Gonio_Right/Gonio_Right_Chuck.STL" />
-      </geometry>
-      <material
-        name="">
-        <color
-          rgba="0.752941176470588 0.752941176470588 0.752941176470588 1" />
-      </material>
-    </visual>
-    <collision>
-      <origin
-        xyz="0 0 0"
-        rpy="0 0 0" />
-      <geometry>
-        <mesh filename="file://$(find pm_robot_description)/meshes/Gonio_Right/Gonio_Right_Chuck.STL" />
-      </geometry>
-    </collision>
-  </link>
-  <joint
-    name="Gonio_Right_Example_Chuck_Joint"
-    type="fixed">
-    <origin
-      xyz="0 0 0"
-      rpy="0 0 0" />
-    <parent
-      link="Gonio_Right_Chuck" />
-    <child
-      link="Gonio_Right_Example_Chuck" />
-    <axis
-      xyz="0 0 0" />
-  </joint>
+</xacro:macro>
 </robot>
