Commit message: modular gonios & new gripper

File: pm_robot_description/urdf/pm_robot_main.xacro (robot description, xacro)
@@ -4,5 +4,11 @@
   <!-- Configurations -->
   <xacro:include filename="$(find pm_robot_description)/urdf/materials.xacro" />
+  <xacro:include filename="$(find pm_robot_description)/urdf/pm_robot.xacro" />
+  <xacro:include filename="$(find pm_robot_description)/urdf/pm_robot_housing.xacro" />
+  <xacro:include filename="$(find pm_robot_description)/urdf/pm_robot_gonio_left.xacro" />
+  <xacro:include filename="$(find pm_robot_description)/urdf/pm_robot_gonio_right.xacro" />
+  <xacro:include filename="$(find pm_robot_description)/urdf/pm_Schunk_Tools/Schunk_Vacuum_Tools.xacro" />
   <xacro:arg name="launch_mode" default="sim_HW" />
+  <xacro:property name="launch_mode" value="$(arg launch_mode)"/>
   <xacro:arg name="initial_positions_file" default="pm_robot_initial_positions.yaml" />
   <xacro:arg name="with_Gonio_Left" default="true" />
@@ -13,12 +19,30 @@
   <xacro:arg name="with_Tool_SPT_Holder" default="false" />
   <xacro:arg name="with_SPT_R_A1000_I500" default="false"/>
-  <xacro:include filename="$(find pm_robot_description)/urdf/pm_robot.xacro" />
   <xacro:pm_robot launch_mode="$(arg launch_mode)"/>
-  <xacro:include filename="$(find pm_robot_description)/urdf/pm_robot_housing.xacro" />
+  <!-- Loading of the Robot Joint calibrations -->
+  <xacro:if value="${launch_mode == 'sim_HW'}">
+    <xacro:property name="pm_robot_bringup_config_file" value="$(find pm_robot_bringup)/config/pm_robot_bringup_config.yaml" />
+  </xacro:if>
+  <!-- If launch_mode 'real' a local path can be specified for the calibration file -->
+  <xacro:if value="${launch_mode == 'real_HW'}">
+      <xacro:property name="local_file_paths__file" value="$(find pm_robot_description)/calibration_config/pm_robot_path_real_HW.yaml" />
+      <xacro:property name="path_dict" value="${xacro.load_yaml(local_file_paths__file)}"/>
+      <xacro:property name="local_robot_bringup_file_path" value="${path_dict['pm_robot_bringup_config_file_path']}"/>
+      <!-- REAL -->
+      <!-- <xacro:property name="pm_robot_joint_calibraion_file" value="${local_calibration_file_path}" />
+      <xacro:property name="pm_robot_bringup_config_file" value="${local_robot_bringup_file_path}"/> -->
+      <!-- SIM -->
+      <xacro:property name="pm_robot_bringup_config_file" value="$(find pm_robot_bringup)/config/pm_robot_bringup_config.yaml" />
+    </xacro:if>
+    <xacro:property name="current_pm_robot_bringup_config" value="${xacro.load_yaml(pm_robot_bringup_config_file)}"/>
   <!-- Tool Defines-->
+  <xacro:if value="${current_pm_robot_bringup_config['pm_robot_tools']['pm_robot_vacuum_tools']['use_vacuum_tool']}">
+    <xacro:Schunk_Vacuum_Tools launch_mode="$(arg launch_mode)" />
+  </xacro:if>
   <xacro:if value="$(arg with_Tool_MPG_10)">
     <xacro:include filename="$(find pm_robot_description)/urdf/pm_Schunk_Tools/MPG_10_plus.xacro" />
     <xacro:mpg_10_plus use_three_mm_lens="$(arg with_Tool_MPG_10_Jaw_3mm_Lens)" />
   </xacro:if>
+  <!-- This may be deletet in the future -->
   <xacro:if value="$(arg with_Tool_SPT_Holder)">
     <xacro:include filename="$(find pm_robot_description)/urdf/pm_Schunk_Tools/SPT_Vacuumtool.xacro" />
@@ -27,9 +51,9 @@
   <!-- Gonio Right Defines-->
   <xacro:if value="$(arg with_Gonio_Right)">
-    <xacro:include filename="$(find pm_robot_description)/urdf/pm_robot_gonio_right.xacro" />
+    <xacro:pm_robot_gonio_right launch_mode="$(arg launch_mode)"/>
   </xacro:if>
   <!-- Gonio Right Defines-->
   <xacro:if value="$(arg with_Gonio_Left)">
-    <xacro:include filename="$(find pm_robot_description)/urdf/pm_robot_gonio_left.xacro" />
+    <xacro:pm_robot_gonio_left launch_mode="$(arg launch_mode)"/>
   </xacro:if>
   <xacro:include filename="$(find pm_robot_description)/urdf/sensors.urdf" />
@@ -39,5 +63,4 @@
   <xacro:include filename="$(find pm_robot_description)/urdf/ros2_control_sim_HW.xacro" />
   <xacro:include filename="$(find pm_robot_description)/urdf/ros2_control_real_HW.xacro" />
-  <xacro:property name="launch_mode" value="$(arg launch_mode)"/>
   <xacro:if value="${launch_mode == 'fake_HW'}">
     <xacro:pm_robot_ros2_control_hw_fake name="Fake_HW" initial_positions_file="$(arg initial_positions_file)"/>

Commit message: urdf changes + moveit gonio

File: pm_robot_description/urdf/pm_robot.xacro (robot description, xacro)
@@ -226,5 +226,5 @@
       <inertial>
         <origin xyz="2.66657822625138E-05 -6.51697797860451E-05 -0.0173989628147272" rpy="0 0 0" />
-        <mass value="0.0770166396645032" />
+        <mass value="0.0741175653990944" />
         <inertia ixx="1.38724675369177E-05" ixy="-2.81065278601148E-08" ixz="-4.32931581160332E-09" iyy="1.28173377099281E-05" iyz="-3.69738102041932E-10" izz="2.32495071670115E-05" />
       </inertial>
@@ -535,5 +535,5 @@
     <link name="Laser_Toolhead_TCP">
       <inertial>
-        <origin xyz="0.00141971945625508 0.0148011051892054 0.0588118094043311" rpy="0 0 0" />
+        <origin xyz="0.00143426339843722 0.014826109459576 0.0588947661972293" rpy="0 0 0" />
         <mass value="0.185632781644417" />
         <inertia ixx="0.00018384097226268" ixy="5.39428478530615E-09" ixz="-6.26322611599089E-07" iyy="0.000136967759808617" iyz="6.13082513214026E-07" izz="7.65210217467237E-05" />
@@ -567,7 +567,7 @@
     <joint name="Laser_Toolhead_TCP_Joint" type="fixed">
       <origin xyz="
-          ${0.147498952947696 + Laser_Toolhead_TCP_Joint_Cal_x*0.000001}
-          ${-0.0899999732334101 + Laser_Toolhead_TCP_Joint_Cal_y*0.000001}
-          ${-0.495500000000011+ Laser_Toolhead_TCP_Joint_Cal_z*0.000001}" rpy="
+          ${0.147498952947694 + Laser_Toolhead_TCP_Joint_Cal_x*0.000001}
+          ${-0.0739999732334102 + Laser_Toolhead_TCP_Joint_Cal_y*0.000001}
+          ${-0.495500146516092+ Laser_Toolhead_TCP_Joint_Cal_z*0.000001}" rpy="
           ${0 + Laser_Toolhead_TCP_Joint_Cal_rx*3.14159265359/180}
           ${0 + Laser_Toolhead_TCP_Joint_Cal_ry*3.14159265359/180}
@@ -651,44 +651,46 @@
       <axis xyz="0 0 0" />
     </joint>
-    <link name="Station_Laser_Bottom_TCP">
-      <inertial>
-        <origin xyz="0.00141971945625008 -0.0148011051892056 -0.0588118094043316" rpy="0 0 0" />
-        <mass value="0.185632781644417" />
-        <inertia ixx="0.000183840972262678" ixy="-5.39428478522435E-09" ixz="6.26322611589981E-07" iyy="0.000136967759808615" iyz="6.13082513215402E-07" izz="7.65210217467232E-05" />
-      </inertial>
-      <visual>
-        <origin xyz="0 0 0" rpy="0 0 0" />
-        <geometry>
-          <mesh filename="file://$(find pm_robot_description)/meshes/Station_Laser_Bottom_TCP.STL" />
-        </geometry>
-        <material name="">
-          <color rgba="0.752941176470588 0.752941176470588 0.752941176470588 1" />
-        </material>
-      </visual>
-      <collision>
-        <origin xyz="0 0 0" rpy="0 0 0" />
-        <geometry>
-          <mesh filename="file://$(find pm_robot_description)/meshes/Station_Laser_Bottom_TCP.STL" />
-        </geometry>
-      </collision>
-    </link>
-    <xacro:property name="Station_Laser_Bottom_TCP_Joint_Cal_x" value="${calibration_dict['Station_Laser_Bottom_TCP_Joint']['x_offset']}"/>
-    <xacro:property name="Station_Laser_Bottom_TCP_Joint_Cal_y" value="${calibration_dict['Station_Laser_Bottom_TCP_Joint']['y_offset']}"/>
-    <xacro:property name="Station_Laser_Bottom_TCP_Joint_Cal_z" value="${calibration_dict['Station_Laser_Bottom_TCP_Joint']['z_offset']}"/>
-    <xacro:property name="Station_Laser_Bottom_TCP_Joint_Cal_rx" value="${calibration_dict['Station_Laser_Bottom_TCP_Joint']['rx_offset']}"/>
-    <xacro:property name="Station_Laser_Bottom_TCP_Joint_Cal_ry" value="${calibration_dict['Station_Laser_Bottom_TCP_Joint']['ry_offset']}"/>
-    <xacro:property name="Station_Laser_Bottom_TCP_Joint_Cal_rz" value="${calibration_dict['Station_Laser_Bottom_TCP_Joint']['rz_offset']}"/>
-    <joint name="Station_Laser_Bottom_TCP_Joint" type="fixed">
-      <origin xyz="
-          ${0.1799989100971 + Station_Laser_Bottom_TCP_Joint_Cal_x*0.000001}
-          ${0.0939999732334095 + Station_Laser_Bottom_TCP_Joint_Cal_y*0.000001}
-          ${0.328499853483917 + Station_Laser_Bottom_TCP_Joint_Cal_z*0.000001}" rpy="
-          ${0 + Station_Laser_Bottom_TCP_Joint_Cal_rx*3.14159265359/180}
-          ${0 + Station_Laser_Bottom_TCP_Joint_Cal_ry*3.14159265359/180}
-          ${0 + Station_Laser_Bottom_TCP_Joint_Cal_rz*3.14159265359/180}" />
-      <parent link="Camera_Station" />
-      <child link="Station_Laser_Bottom_TCP" />
-      <axis xyz="0 0 0" />
-    </joint>
+    <xacro:if value="${current_pm_robot_bringup_config['measuring_systems']['use_keyence_bottom']}">
+      <link name="Station_Laser_Bottom_TCP">
+        <inertial>
+          <origin xyz="0.00143426339843278 -0.0148261094595752 -0.0588947661972306" rpy="0 0 0" />
+          <mass value="0.185632781644417" />
+          <inertia ixx="0.000183840972262678" ixy="-5.39428478522435E-09" ixz="6.26322611589981E-07" iyy="0.000136967759808615" iyz="6.13082513215402E-07" izz="7.65210217467232E-05" />
+        </inertial>
+        <visual>
+          <origin xyz="0 0 0" rpy="0 0 0" />
+          <geometry>
+            <mesh filename="file://$(find pm_robot_description)/meshes/Station_Laser_Bottom_TCP.STL" />
+          </geometry>
+          <material name="">
+            <color rgba="0.752941176470588 0.752941176470588 0.752941176470588 1" />
+          </material>
+        </visual>
+        <collision>
+          <origin xyz="0 0 0" rpy="0 0 0" />
+          <geometry>
+            <mesh filename="file://$(find pm_robot_description)/meshes/Station_Laser_Bottom_TCP.STL" />
+          </geometry>
+        </collision>
+      </link>
+      <xacro:property name="Station_Laser_Bottom_TCP_Joint_Cal_x" value="${calibration_dict['Station_Laser_Bottom_TCP_Joint']['x_offset']}"/>
+      <xacro:property name="Station_Laser_Bottom_TCP_Joint_Cal_y" value="${calibration_dict['Station_Laser_Bottom_TCP_Joint']['y_offset']}"/>
+      <xacro:property name="Station_Laser_Bottom_TCP_Joint_Cal_z" value="${calibration_dict['Station_Laser_Bottom_TCP_Joint']['z_offset']}"/>
+      <xacro:property name="Station_Laser_Bottom_TCP_Joint_Cal_rx" value="${calibration_dict['Station_Laser_Bottom_TCP_Joint']['rx_offset']}"/>
+      <xacro:property name="Station_Laser_Bottom_TCP_Joint_Cal_ry" value="${calibration_dict['Station_Laser_Bottom_TCP_Joint']['ry_offset']}"/>
+      <xacro:property name="Station_Laser_Bottom_TCP_Joint_Cal_rz" value="${calibration_dict['Station_Laser_Bottom_TCP_Joint']['rz_offset']}"/>
+      <joint name="Station_Laser_Bottom_TCP_Joint" type="fixed">
+        <origin xyz="
+            ${0.179998910097098 + Station_Laser_Bottom_TCP_Joint_Cal_x*0.000001}
+            ${0.0939999732334105 + Station_Laser_Bottom_TCP_Joint_Cal_y*0.000001}
+            ${0.328500000000003 + Station_Laser_Bottom_TCP_Joint_Cal_z*0.000001}" rpy="
+            ${0 + Station_Laser_Bottom_TCP_Joint_Cal_rx*3.14159265359/180}
+            ${0 + Station_Laser_Bottom_TCP_Joint_Cal_ry*3.14159265359/180}
+            ${0 + Station_Laser_Bottom_TCP_Joint_Cal_rz*3.14159265359/180}" />
+        <parent link="Camera_Station" />
+        <child link="Station_Laser_Bottom_TCP" />
+        <axis xyz="0 0 0" />
+      </joint>
+  </xacro:if>
     <!--%%%%%%%%%%%%% Camera Calibration Definitions-->
     <link name="Camera_Calibration_Platelet">

File: pm_robot_description/urdf/pm_robot_gonio_left.xacro (robot description, xacro)
@@ -32,7 +32,8 @@
     <link name="Gonio_Left_Base">
       <inertial>
-        <origin xyz="0.178376501584756 0.0965486243516244 0.101012071321914" rpy="0 0 0" />
-        <mass value="4.83318673735945" />
-        <inertia ixx="0.0115124478906001" ixy="4.00480442649554E-05" ixz="-5.80448319957772E-07" iyy="0.0188689063295654" iyz="-2.7716346407679E-05" izz="0.0269850736598033" />
+        <origin xyz="0.177919402818021 0.0965286177417367 0.101012071345888" rpy="0 0 0" />
+        <mass value="4.83318674398637" />
+        <inertia
+        ixx="0.0115127403940929" ixy="-3.33565784736103E-05" ixz="-1.45496624993124E-06" iyy="0.0188686138682557" iyz="-2.7618864699939E-05" izz="0.026985073699425" />
       </inertial>
       <visual>
@@ -54,5 +55,4 @@
       <parent link="pm_robot_base_link" />
       <child link="Gonio_Left_Base" />
-ö
       <axis xyz="0 0 0" />
     </joint>
@@ -60,7 +60,13 @@
     <link name="Gonio_Left_Stage_1_Top">
       <inertial>
-        <origin xyz="0.059454973286124 0.0107762403389283 -0.0446785627316242" rpy="0 0 0" />
+        <origin xyz="0.059782487896749 0.00877925652714845 -0.0446785627316222" rpy="0 0 0" />
         <mass value="0.578798857286943" />
-        <inertia ixx="0.000410450617020548" ixy="-0.000168393668986117" ixz="9.5803621154249E-07" iyy="0.00156907354726657" iyz="-5.23053452301373E-06" izz="0.00188005175520343" />
+        <inertia
+        ixx="0.000400478324367351"
+        ixy="-0.000129239522587819"
+        ixz="7.82346515336273E-07"
+        iyy="0.00157904583991977"
+        iyz="-5.25968237719779E-06"
+        izz="0.00188005175520343" />
       </inertial>
       <visual>
@@ -92,7 +98,13 @@
     <link name="Gonio_Left_Stage_2_Bottom">
       <inertial>
-        <origin xyz="4.69384364709668E-10 1.57268642553277E-11 -0.00620045721380197" rpy="0 0 0" />
-        <mass value="0.0270626701992899" />
-        <inertia ixx="6.08566105952436E-06" ixy="5.75557428925166E-08" ixz="-8.6517331846629E-13" iyy="4.36978117330268E-06" iyz="-2.89879120608969E-14" izz="9.60640029376035E-06" />
+        <origin xyz="4.69633887334453E-10 4.9960036108132E-16 -0.0212004572137997" rpy="0 0 0" />
+        <mass value="0.02706267019929" />
+        <inertia
+        ixx="6.08758948397044E-06"
+        ixy="4.1172957090613E-14"
+        ixz="-8.65658801813879E-13"
+        iyy="4.36785274885666E-06"
+        iyz="-3.36683105860672E-21"
+        izz="9.6064002937604E-06" />
       </inertial>
       <visual>
@@ -118,5 +130,5 @@
       <parent link="Gonio_Left_Stage_1_Top" />
       <child link="Gonio_Left_Stage_2_Bottom" />
-      <axis xyz="0.0334865202089474 -0.999439169216564 0" />
+      <axis xyz="0 -1 0" />
       <limit lower="-0.17453" upper="0.17453" effort="100" velocity="0.1" />
     </joint>
@@ -125,5 +137,5 @@
     </link>
     <joint name="Gonio_Left_Chuck_Origin_Joint" type="fixed">
-      <origin xyz="0 0 -0.015" rpy="0 0 3.174753954" />
+      <origin xyz="0 0 -0.015" rpy="0 0 0" />
       <parent link="Gonio_Left_Stage_2_Bottom" />
       <child link="Gonio_Left_Chuck_Origin" />

Commit message: make moveit and gonios work a little better

File: pm_robot_description/urdf/pm_robot.xacro (robot description, xacro)
@@ -5,6 +5,6 @@
 <robot xmlns:xacro="http://ros.org/wiki/xacro">
   <xacro:macro name="pm_robot" params="launch_mode">
-  <xacro:include filename="$(find pm_robot_description)/urdf/match_logo.urdf.xacro" />
-  <!-- Loading of the Robot Joint calibrations -->
+    <xacro:include filename="$(find pm_robot_description)/urdf/match_logo.urdf.xacro" />
+    <!-- Loading of the Robot Joint calibrations -->
     <xacro:if value="${launch_mode == 'sim_HW'}">
       <xacro:property name="pm_robot_joint_calibraion_file" value="$(find pm_robot_description)/calibration_config/pm_robot_joint_calibration.yaml" />
@@ -221,5 +221,5 @@
       <child link="Gripper_Rot_Plate" />
       <axis xyz="0 0 1" />
-      <limit lower="0" upper="12" effort="100" velocity="5" />
+      <limit lower="-2.0" upper="2.0" effort="100" velocity="5" />
     </joint>
     <link name="t_axis_toolchanger">
@@ -255,5 +255,5 @@
       <axis xyz="0 0 0" />
     </joint>
-<!--
+    <!--
     <link name="PM_Robot_Tool_TCP">
     </link>
@@ -359,6 +359,5 @@
         ${-0.001 + Dispenser_1K_TCP_Joint_Cal_x * 0.000001}
         ${-0.0318 + Dispenser_1K_TCP_Joint_Cal_y * 0.000001}
-        ${-0.135 + Dispenser_1K_TCP_Joint_Cal_z * 0.000001 + Dispenser_1K_tip_z_offset}"
-        rpy="
+        ${-0.135 + Dispenser_1K_TCP_Joint_Cal_z * 0.000001 + Dispenser_1K_tip_z_offset}" rpy="
         ${0 + Dispenser_1K_TCP_Joint_Cal_rx * 3.14159265359/180}
         ${0 + Dispenser_1K_TCP_Joint_Cal_ry * 3.14159265359/180}
@@ -381,57 +380,36 @@
     <xacro:property name="Dispenser_1K_tip_visual_filename" value="${dispenser_1K_configs_dict[current_pm_robot_1K_dipsenser_tip]['visual_filename']}"/>
     <xacro:property name="Dispenser_1K_tip_collision_filename" value="${dispenser_1K_configs_dict[current_pm_robot_1K_dipsenser_tip]['collision_filename']}"/>
-  <!--%%%%%%%%%%%%% The parameters here are interchangeable %%%%%%%%%%%%%-->
-  <!--%%%%%%%%%%%%% Jaw 1 Definitions %%%%%%%%%%%%%-->
-  <link
-    name="1K_Dispenser_Tip">
-    <inertial>
-      <origin
-        xyz="${Dispenser_1K_tip_xyz}"
-        rpy="${Dispenser_1K_tip_rpy}"/>
-      <mass
-        value="${Dispenser_1K_tip_mass}"/>
-      <inertia
-        ixx="${Dispenser_1K_tip_inertia_ixx}"
-        ixy="${Dispenser_1K_tip_inertia_ixy}"
-        ixz="${Dispenser_1K_tip_inertia_ixz}"
-        iyy="${Dispenser_1K_tip_inertia_iyy}"
-        iyz="${Dispenser_1K_tip_inertia_iyz}"
-        izz="${Dispenser_1K_tip_inertia_izz}" />
-    </inertial>
-    <visual>
-      <origin
-        xyz="0 0 0"
-        rpy="0 0 0" />
-      <geometry>
-        <mesh filename="file://$(find pm_robot_description)/meshes/Dispenser_Tips/${Dispenser_1K_tip_visual_filename}" />
-      </geometry>
-      <material
-        name="${Dispenser_1K_tip_color}">
-      </material>
-    </visual>
-    <collision>
-      <origin
-        xyz="0 0 0"
-        rpy="0 0 0" />
-      <geometry>
-        <mesh filename="file://$(find pm_robot_description)/meshes/Dispenser_Tips/${Dispenser_1K_tip_collision_filename}" />
-      </geometry>
-    </collision>
-  </link>
-  <gazebo reference="1K_Dispenser_Tip">
-    <turnGravityOff>true</turnGravityOff>
-  </gazebo>
-  <joint
-    name="1K_Dispenser_Tip_Joint"
-    type="fixed">
-    <!-- This needs to be corrected in Solidworks -->
-    <origin
-      xyz="0.000 0 0 "
-      rpy="0 0 0" />
-    <parent
-      link="1K_Dispenser_TCP" />
-    <child
-      link="1K_Dispenser_Tip" />
-  </joint>
+    <!--%%%%%%%%%%%%% The parameters here are interchangeable %%%%%%%%%%%%%-->
+    <!--%%%%%%%%%%%%% Jaw 1 Definitions %%%%%%%%%%%%%-->
+    <link name="1K_Dispenser_Tip">
+      <inertial>
+        <origin xyz="${Dispenser_1K_tip_xyz}" rpy="${Dispenser_1K_tip_rpy}"/>
+        <mass value="${Dispenser_1K_tip_mass}"/>
+        <inertia ixx="${Dispenser_1K_tip_inertia_ixx}" ixy="${Dispenser_1K_tip_inertia_ixy}" ixz="${Dispenser_1K_tip_inertia_ixz}" iyy="${Dispenser_1K_tip_inertia_iyy}" iyz="${Dispenser_1K_tip_inertia_iyz}" izz="${Dispenser_1K_tip_inertia_izz}" />
+      </inertial>
+      <visual>
+        <origin xyz="0 0 0" rpy="0 0 0" />
+        <geometry>
+          <mesh filename="file://$(find pm_robot_description)/meshes/Dispenser_Tips/${Dispenser_1K_tip_visual_filename}" />
+        </geometry>
+        <material name="${Dispenser_1K_tip_color}">
+        </material>
+      </visual>
+      <collision>
+        <origin xyz="0 0 0" rpy="0 0 0" />
+        <geometry>
+          <mesh filename="file://$(find pm_robot_description)/meshes/Dispenser_Tips/${Dispenser_1K_tip_collision_filename}" />
+        </geometry>
+      </collision>
+    </link>
+    <gazebo reference="1K_Dispenser_Tip">
+      <turnGravityOff>true</turnGravityOff>
+    </gazebo>
+    <joint name="1K_Dispenser_Tip_Joint" type="fixed">
+      <!-- This needs to be corrected in Solidworks -->
+      <origin xyz="0.000 0 0 " rpy="0 0 0" />
+      <parent link="1K_Dispenser_TCP" />
+      <child link="1K_Dispenser_Tip" />
+    </joint>
     <!--%%%%%%%%%%%%% 2K Dispenser Definitions-->
     <link name="2K_Dispenser_Cartridge">
@@ -692,5 +670,5 @@
         <axis xyz="0 0 0" />
       </joint>
-  </xacro:if>
+    </xacro:if>
     <!--%%%%%%%%%%%%% Camera Calibration Definitions-->
     <link name="Camera_Calibration_Platelet">

File: pm_robot_description/urdf/ros2_control_real_HW.xacro (robot description, xacro)
@@ -33,4 +33,26 @@
                 <state_interface name="velocity"/>
             </joint>
+            <joint name="Gonio_Left_Stage_1_Joint">
+                <command_interface name="position">
+                </command_interface>
+                <state_interface name="position"/>
+            </joint>
+            <joint name="Gonio_Left_Stage_2_Joint">
+                <command_interface name="position">
+                </command_interface>
+                <state_interface name="position"/>
+            </joint>
+            <joint name="Gonio_Right_Stage_1_Joint">
+                <command_interface name="position">
+                </command_interface>
+                <state_interface name="position"/>
+                <state_interface name="velocity"/>
+            </joint>
+            <joint name="Gonio_Right_Stage_2_Joint">
+                <command_interface name="position">
+                </command_interface>
+                <state_interface name="position"/>
+                <state_interface name="velocity"/>
+            </joint>
             <!-- <joint name="1K_Dispenser_Flap_Joint">
                 <command_interface name="position">
@@ -48,27 +70,5 @@
                 <state_interface name="position"/>
             </joint> -->
-            <!-- <joint name="Gonio_Right_Stage_1_Joint">
-                <command_interface name="position">
-                </command_interface>
-                <state_interface name="position"/>
-                <state_interface name="velocity"/>
-            </joint>
-            <joint name="Gonio_Right_Stage_2_Joint">
-                <command_interface name="position">
-                </command_interface>
-                <state_interface name="position"/>
-                <state_interface name="velocity"/>
-            </joint> -->
             <!-- <joint name="Camera_Calibration_Platelet_Joint">
-                <command_interface name="position">
-                </command_interface>
-                <state_interface name="position"/>
-            </joint> -->
-            <!-- <joint name="Gonio_Left_Stage_1_Joint">
-                <command_interface name="position">
-                </command_interface>
-                <state_interface name="position"/>
-            </joint>
-            <joint name="Gonio_Left_Stage_2_Joint">
                 <command_interface name="position">
                 </command_interface>
