Commit message: pneumatic axes listener

File: pm_robot_description/urdf/pm_robot.xacro (robot description, xacro)
@@ -309,5 +309,5 @@
       <child link="1K_Dispenser_Flap" />
       <axis xyz="1 0 0" />
-      <limit lower="0" upper="0.02" effort="100" velocity="0.05" />
+      <limit lower="0.02" upper="0.00" effort="100" velocity="0.5" />
     </joint>
     <!--%%%%%%%%%%%%% 1K Dispenser Definitions %%%%%%%%%%%%%-->
@@ -442,6 +442,6 @@
       <parent link="Z_Axis" />
       <child link="2K_Dispenser_Cartridge" />
-      <axis xyz="0 0 -1" />
-      <limit lower="0" upper="0.02" effort="100" velocity="0.05" />
+      <axis xyz="0 0 1" />
+      <limit lower="-0.04" upper="0.00" effort="100" velocity="0.1" />
     </joint>
     <link name="2K_Dispenser_TCP">
@@ -698,5 +698,5 @@
       <child link="Camera_Calibration_Platelet" />
       <axis xyz="0 -1 0" />
-      <limit lower="-0.04" upper="0.0" effort="100" velocity="0.05" />
+      <limit lower="-0.04" upper="0.0" effort="100" velocity="0.5" />
     </joint>
     <!--%%%%%%%%%%%%% Calibration Qube Definitions-->

File: pm_robot_description/urdf/pm_robot_gonio_left.xacro (robot description, xacro)
@@ -255,5 +255,5 @@
       <child link="UV_LED_Front" />
       <axis xyz="0 1 0" />
-      <limit lower="0" upper="0.01" effort="100" velocity="0.05" />
+      <limit lower="0.05" upper="0.0" effort="100" velocity="0.5" />
     </joint>
     <!--%%%%%%%%%%%%% UV Slider X Back Definitions-->
@@ -311,5 +311,5 @@
       <child link="UV_LED_Back" />
       <axis xyz="0 1 0" />
-      <limit lower="0" upper="0.05" effort="100" velocity="0.05" />
+      <limit lower="-0.05" upper="0.0" effort="100" velocity="0.05" />
     </joint>
   </xacro:macro>

File: pm_robot_description/urdf/pm_robot_main.xacro (robot description, xacro)
@@ -78,4 +78,5 @@
   <xacro:if value="${launch_mode == 'real_HW'}">
     <xacro:pm_robot_ros2_control_hw_real name="Real_HW" initial_positions_file="$(arg initial_positions_file)"/>
+    <xacro:pm_robot_pneumatic_mock  />
     <!-- <xacro:pm_robot_ros2_control_hw_sim name="Sim_HW"/> -->
   </xacro:if>

File: pm_robot_description/urdf/ros2_control_real_HW.xacro (robot description, xacro)
@@ -55,20 +55,11 @@
                 <state_interface name="velocity"/>
             </joint>
-            <!-- <joint name="1K_Dispenser_Flap_Joint">
+<!--
+            <joint name="1K_Dispenser_Flap_Joint">
                 <command_interface name="position">
                 </command_interface>
                 <state_interface name="position"/>
             </joint>
-            <joint name="1K_Dispenser_Joint">
-                <command_interface name="position">
-                </command_interface>
-                <state_interface name="position"/>
-            </joint>
-            <joint name="2K_Dispenser_Joint">
-                <command_interface name="position">
-                </command_interface>
-                <state_interface name="position"/>
-            </joint>
-            <joint name="Camera_Calibration_Platelet_Joint">
+            <joint name="Calibration_Qube_Joint">
                 <command_interface name="position">
                 </command_interface>
@@ -80,20 +71,5 @@
                 <state_interface name="position"/>
             </joint>
-            <joint name="UV_LED_Front_Joint">
-                <command_interface name="position">
-                </command_interface>
-                <state_interface name="position"/>
-            </joint>
             <joint name="UV_Slider_X_Back_Joint">
-                <command_interface name="position">
-                </command_interface>
-                <state_interface name="position"/>
-            </joint>
-            <joint name="UV_LED_Back_Joint">
-                <command_interface name="position">
-                </command_interface>
-                <state_interface name="position"/>
-            </joint>
-            <joint name="Calibration_Qube_Joint">
                 <command_interface name="position">
                 </command_interface>
@@ -150,3 +126,53 @@
         </ros2_control>
     </xacro:macro>
+    <xacro:macro name="pm_robot_pneumatic_mock" >
+        <ros2_control name="PMSystemPneumatic" type="system">
+            <hardware>
+                <plugin>mock_components/GenericSystem</plugin>
+                <!-- <param name="mock_sensor_commands">true</param> -->
+            </hardware>
+            <joint name="1K_Dispenser_Joint">
+                <command_interface name="position" >
+                </command_interface>
+                <state_interface name="position">
+                <param name="initial_value">0.0</param>
+                </state_interface>
+            </joint>
+            <joint name="2K_Dispenser_Joint">
+                <command_interface name="position" >
+                </command_interface>
+                <state_interface name="position">
+                <param name="initial_value">0.0</param>
+                </state_interface>
+            </joint>
+            <joint name="Camera_Calibration_Platelet_Joint">
+                <command_interface name="position">
+                </command_interface>
+                <state_interface name="position">
+                    <param name="initial_value">-0.04</param>
+                </state_interface>
+            </joint>
+            <joint name="UV_LED_Front_Joint">
+                <command_interface name="position" >
+                </command_interface>
+                <state_interface name="position">
+                    <param name="initial_value">0.0</param>
+                </state_interface>
+            </joint>
+            <joint name="UV_LED_Back_Joint">
+                <command_interface name="position">
+                </command_interface>
+                <state_interface name="position">
+                    <param name="initial_value">0.0</param>
+                </state_interface>
+            </joint>
+            <joint name="1K_Dispenser_Flap_Joint">
+                <command_interface name="position">
+                </command_interface>
+                <state_interface name="position">
+                    <param name="initial_value">0.0</param>
+                </state_interface>
+            </joint>
+        </ros2_control>
+    </xacro:macro>
 </robot>

Commit message: mock interface for pneumatic

File: pm_robot_description/urdf/pm_robot.xacro (robot description, xacro)
@@ -309,5 +309,5 @@
       <child link="1K_Dispenser_Flap" />
       <axis xyz="1 0 0" />
-      <limit lower="0.02" upper="0.00" effort="100" velocity="0.5" />
+      <limit lower="0.025" upper="0.00" effort="100" velocity="0.5" />
     </joint>
     <!--%%%%%%%%%%%%% 1K Dispenser Definitions %%%%%%%%%%%%%-->

File: pm_robot_description/urdf/pm_robot_gonio_left.xacro (robot description, xacro)
@@ -255,5 +255,5 @@
       <child link="UV_LED_Front" />
       <axis xyz="0 1 0" />
-      <limit lower="0.05" upper="0.0" effort="100" velocity="0.5" />
+      <limit lower="0.0157" upper="0.0" effort="100" velocity="0.5" />
     </joint>
     <!--%%%%%%%%%%%%% UV Slider X Back Definitions-->
@@ -311,5 +311,5 @@
       <child link="UV_LED_Back" />
       <axis xyz="0 1 0" />
-      <limit lower="-0.05" upper="0.0" effort="100" velocity="0.05" />
+      <limit lower="-0.0157" upper="0.0" effort="100" velocity="0.05" />
     </joint>
   </xacro:macro>

Commit message: changes meshes; package merges, etc

File: pm_robot_description/urdf/pm_robot.xacro (robot description, xacro)
@@ -104,4 +104,9 @@
     </joint>
     <!--%%%%%%%%%%%%% X Axis Definitions %%%%%%%%%%%%%-->
+    <!-- Init Definition of 1K Dispenser tip -->
+    <!-- Property names should not start with a number -->
+    <xacro:property name="X_Axis_Offset" value="${calibration_dict['PM_Robot_XYZ_Calibration']['x_offset']}"/>
+    <xacro:property name="Y_Axis_Offset" value="${calibration_dict['PM_Robot_XYZ_Calibration']['y_offset']}"/>
+    <xacro:property name="Z_Axis_Offset" value="${calibration_dict['PM_Robot_XYZ_Calibration']['z_offset']}"/>
     <link name="X_Axis">
       <inertial>
@@ -125,5 +130,5 @@
     </link>
     <joint name="X_Axis_Joint" type="prismatic">
-      <origin xyz="0.64699 0.11775 0.47499" rpy="0 0 0" />
+      <origin xyz="${0.64699 + X_Axis_Offset*0.000001} 0.11775 0.47499" rpy="0 0 0" />
       <parent link="axis_base" />
       <child link="X_Axis" />
@@ -153,5 +158,5 @@
     </link>
     <joint name="Y_Axis_Joint" type="prismatic">
-      <origin xyz="0.10865 0.25835 0.06525" rpy="0 0 0" />
+      <origin xyz="0.10865 ${0.25835 + Y_Axis_Offset*0.000001} 0.06525" rpy="0 0 0" />
       <parent link="X_Axis" />
       <child link="Y_Axis" />
@@ -185,5 +190,5 @@
     </gazebo>
     <joint name="Z_Axis_Joint" type="prismatic">
-      <origin xyz="-0.00365 -0.499 0.28025" rpy="0 0 0" />
+      <origin xyz="-0.00365 -0.499 ${0.28025 + Z_Axis_Offset*0.000001}" rpy="0 0 0" />
       <parent link="Y_Axis" />
       <child link="Z_Axis" />
@@ -308,6 +313,6 @@
       <parent link="Z_Axis" />
       <child link="1K_Dispenser_Flap" />
-      <axis xyz="1 0 0" />
-      <limit lower="0.025" upper="0.00" effort="100" velocity="0.5" />
+      <axis xyz="-1 0 0" />
+      <limit lower="-0.025" upper="0.00" effort="100" velocity="0.5" />
     </joint>
     <!--%%%%%%%%%%%%% 1K Dispenser Definitions %%%%%%%%%%%%%-->
@@ -661,7 +666,8 @@
       <joint name="Station_Laser_Bottom_TCP_Joint" type="fixed">
         <origin xyz="
-            ${0.179998910097098 + Station_Laser_Bottom_TCP_Joint_Cal_x*0.000001}
+            ${0.181998910097099 + Station_Laser_Bottom_TCP_Joint_Cal_x*0.000001}
             ${0.0939999732334105 + Station_Laser_Bottom_TCP_Joint_Cal_y*0.000001}
-            ${0.328500000000003 + Station_Laser_Bottom_TCP_Joint_Cal_z*0.000001}" rpy="
+            ${0.307500000000001 + Station_Laser_Bottom_TCP_Joint_Cal_z*0.000001}"
+            rpy="
             ${0 + Station_Laser_Bottom_TCP_Joint_Cal_rx*3.14159265359/180}
             ${0 + Station_Laser_Bottom_TCP_Joint_Cal_ry*3.14159265359/180}
@@ -733,7 +739,7 @@
     <joint name="Calibration_Qube_Joint" type="prismatic">
       <origin xyz="
-          ${0.152 + Calibration_Qube_Joint_Cal_x*0.000001}
+          ${0.154 + Calibration_Qube_Joint_Cal_x*0.000001}
           ${0.108 + Calibration_Qube_Joint_Cal_y*0.000001}
-          ${0.326 + Calibration_Qube_Joint_Cal_z*0.000001}" rpy="
+          ${0.305 + Calibration_Qube_Joint_Cal_z*0.000001}" rpy="
           ${0 + Calibration_Qube_Joint_Cal_rx*3.14159265359/180}
           ${0 + Calibration_Qube_Joint_Cal_ry*3.14159265359/180}

File: pm_robot_description/urdf/pm_robot_gonio_left.xacro (robot description, xacro)
@@ -255,5 +255,5 @@
       <child link="UV_LED_Front" />
       <axis xyz="0 1 0" />
-      <limit lower="0.0157" upper="0.0" effort="100" velocity="0.5" />
+      <limit lower="-0.0157" upper="0.0" effort="100" velocity="0.5" />
     </joint>
     <!--%%%%%%%%%%%%% UV Slider X Back Definitions-->

File: pm_robot_description/urdf/ros2_control_sim_HW.xacro (robot description, xacro)
@@ -2,9 +2,9 @@
 <robot xmlns:xacro="http://www.ros.org/wiki/xacro">
     <xacro:macro name="pm_robot_ros2_control_hw_sim" params="name initial_positions_file">
-                <!-- Loading of the Robot bringup config -->
-                <xacro:if value="${launch_mode == 'sim_HW'}">
-                    <xacro:property name="pm_robot_bringup_config_file" value="$(find pm_robot_bringup)/config/pm_robot_bringup_config.yaml" />
-                </xacro:if>
-                <xacro:property name="current_pm_robot_bringup_config" value="${xacro.load_yaml(pm_robot_bringup_config_file)}"/>
+            <!-- Loading of the Robot bringup config -->
+            <xacro:if value="${launch_mode == 'sim_HW'}">
+                <xacro:property name="pm_robot_bringup_config_file" value="$(find pm_robot_bringup)/config/pm_robot_bringup_config.yaml" />
+            </xacro:if>
+            <xacro:property name="current_pm_robot_bringup_config" value="${xacro.load_yaml(pm_robot_bringup_config_file)}"/>
         <xacro:property name="initial_positions" value="${load_yaml(initial_positions_file)['initial_positions']}"/>
         <ros2_control name="GazeboSystem" type="system">

Commit message: confocal_sensors

File: pm_robot_description/urdf/pm_robot.xacro (robot description, xacro)
@@ -678,4 +678,130 @@
       </joint>
     </xacro:if>
+    <xacro:if value="${current_pm_robot_bringup_config['measuring_systems']['use_confocal_bottom']}">
+      <link name="TCP_Confocal_Sensor_Bottom">
+      <inertial>
+            <origin
+              xyz="-0.00247029745512151 0.0425771909752702 -0.0497854338510461"
+              rpy="0 0 0" />
+            <mass
+              value="0.344263397388723" />
+            <inertia
+              ixx="0.000599129085110184"
+              ixy="-1.74073417588787E-05"
+              ixz="-4.10917598198572E-08"
+              iyy="0.000151077936284775"
+              iyz="-8.61442405235731E-06"
+              izz="0.000578610557041608" />
+          </inertial>
+        <visual>
+          <origin xyz="0 0 0" rpy="0 0 0" />
+          <geometry>
+            <mesh filename="file://$(find pm_robot_description)/meshes/Confocal_Sensor_Bottom.STL" />
+          </geometry>
+          <material name="">
+            <color rgba="0.752941176470588 0.752941176470588 0.752941176470588 1" />
+          </material>
+        </visual>
+        <collision>
+          <origin xyz="0 0 0" rpy="0 0 0" />
+          <geometry>
+            <mesh filename="file://$(find pm_robot_description)/meshes/Confocal_Sensor_Bottom.STL" />
+          </geometry>
+        </collision>
+      </link>
+      <xacro:property name="Confocal_Sensor_Bottom_TCP_Joint_Cal_x" value="${calibration_dict['Confocal_Sensor_Bottom_TCP_Joint']['x_offset']}"/>
+      <xacro:property name="Confocal_Sensor_Bottom_TCP_Joint_Cal_y" value="${calibration_dict['Confocal_Sensor_Bottom_TCP_Joint']['y_offset']}"/>
+      <xacro:property name="Confocal_Sensor_Bottom_TCP_Joint_Cal_z" value="${calibration_dict['Confocal_Sensor_Bottom_TCP_Joint']['z_offset']}"/>
+      <xacro:property name="Confocal_Sensor_Bottom_TCP_Joint_Cal_rx" value="${calibration_dict['Confocal_Sensor_Bottom_TCP_Joint']['rx_offset']}"/>
+      <xacro:property name="Confocal_Sensor_Bottom_TCP_Joint_Cal_ry" value="${calibration_dict['Confocal_Sensor_Bottom_TCP_Joint']['ry_offset']}"/>
+      <xacro:property name="Confocal_Sensor_Bottom_TCP_Joint_Cal_rz" value="${calibration_dict['Confocal_Sensor_Bottom_TCP_Joint']['rz_offset']}"/>
+      <joint name="TCP_Confocal_Sensor_Bottom_Joint" type="fixed">
+        <origin xyz="
+            ${0.1925 + Confocal_Sensor_Bottom_TCP_Joint_Cal_x*0.000001}
+            ${0.0938799999999999+ Confocal_Sensor_Bottom_TCP_Joint_Cal_y*0.000001}
+            ${0.30825985348391 + Confocal_Sensor_Bottom_TCP_Joint_Cal_z*0.000001}"
+            rpy="
+            ${0 + Confocal_Sensor_Bottom_TCP_Joint_Cal_rx*3.14159265359/180}
+            ${0 + Confocal_Sensor_Bottom_TCP_Joint_Cal_ry*3.14159265359/180}
+            ${0 + Confocal_Sensor_Bottom_TCP_Joint_Cal_rz*3.14159265359/180}" />
+        <parent link="Camera_Station" />
+        <child link="TCP_Confocal_Sensor_Bottom" />
+        <axis xyz="0 0 0" />
+      </joint>
+    </xacro:if>
+    <xacro:if value="${current_pm_robot_bringup_config['measuring_systems']['use_confocal_head']}">
+      <link name="TCP_Confocal_Sensor_Top">
+      <inertial>
+        <origin
+          xyz="-0.0129743586620629 -0.0179072639596305 0.0489187396629332"
+          rpy="0 0 0" />
+        <mass
+          value="0.0631321031924395" />
+        <inertia
+          ixx="5.72140577879517E-05"
+          ixy="-1.00812729158378E-05"
+          ixz="-1.59225714048641E-06"
+          iyy="3.26664833980595E-05"
+          iyz="-4.19709040215342E-06"
+          izz="3.82911436485178E-05" />
+      </inertial>
+        <visual>
+          <origin xyz="0 0 0" rpy="0 0 0" />
+          <geometry>
+            <mesh filename="file://$(find pm_robot_description)/meshes/Confocal_Sensor_Top.STL" />
+          </geometry>
+          <material name="">
+            <color rgba="0.752941176470588 0.752941176470588 0.752941176470588 1" />
+          </material>
+        </visual>
+        <collision>
+          <origin xyz="0 0 0" rpy="0 0 0" />
+          <geometry>
+            <mesh filename="file://$(find pm_robot_description)/meshes/Confocal_Sensor_Top.STL" />
+          </geometry>
+        </collision>
+      </link>
+      <xacro:property name="Confocal_Sensor_Top_TCP_Joint_Cal_x" value="${calibration_dict['Confocal_Sensor_Top_TCP_Joint']['x_offset']}"/>
+      <xacro:property name="Confocal_Sensor_Top_TCP_Joint_Cal_y" value="${calibration_dict['Confocal_Sensor_Top_TCP_Joint']['y_offset']}"/>
+      <xacro:property name="Confocal_Sensor_Top_TCP_Joint_Cal_z" value="${calibration_dict['Confocal_Sensor_Top_TCP_Joint']['z_offset']}"/>
+      <xacro:property name="Confocal_Sensor_Top_TCP_Joint_Cal_rx" value="${calibration_dict['Confocal_Sensor_Top_TCP_Joint']['rx_offset']}"/>
+      <xacro:property name="Confocal_Sensor_Top_TCP_Joint_Cal_ry" value="${calibration_dict['Confocal_Sensor_Top_TCP_Joint']['ry_offset']}"/>
+      <xacro:property name="Confocal_Sensor_Top_TCP_Joint_Cal_rz" value="${calibration_dict['Confocal_Sensor_Top_TCP_Joint']['rz_offset']}"/>
+      <joint name="TCP_Confocal_Sensor_Top_Joint" type="fixed">
+        <origin xyz="
+            ${0.176999957149375 + Confocal_Sensor_Top_TCP_Joint_Cal_x*0.000001}
+            ${-0.0580000000000008+ Confocal_Sensor_Top_TCP_Joint_Cal_y*0.000001}
+            ${-0.495500000000003 + Confocal_Sensor_Top_TCP_Joint_Cal_z*0.000001}"
+            rpy="
+            ${0 + Confocal_Sensor_Top_TCP_Joint_Cal_rx*3.14159265359/180}
+            ${0 + Confocal_Sensor_Top_TCP_Joint_Cal_ry*3.14159265359/180}
+            ${0 + Confocal_Sensor_Top_TCP_Joint_Cal_rz*3.14159265359/180}" />
+        <parent link="Z_Axis" />
+        <child link="TCP_Confocal_Sensor_Top" />
+        <axis xyz="0 0 0" />
+      </joint>
+      <link
+        name="TCP_Confocal_Sensor_Top_2">
+      </link>
+      <xacro:property name="Confocal_Sensor_Top_TCP_2_Joint_Cal_x" value="${calibration_dict['Confocal_Sensor_Top_TCP_2_Joint']['x_offset']}"/>
+      <xacro:property name="Confocal_Sensor_Top_TCP_2_Joint_Cal_y" value="${calibration_dict['Confocal_Sensor_Top_TCP_2_Joint']['y_offset']}"/>
+      <xacro:property name="Confocal_Sensor_Top_TCP_2_Joint_Cal_z" value="${calibration_dict['Confocal_Sensor_Top_TCP_2_Joint']['z_offset']}"/>
+      <xacro:property name="Confocal_Sensor_Top_TCP_2_Joint_Cal_rx" value="${calibration_dict['Confocal_Sensor_Top_TCP_2_Joint']['rx_offset']}"/>
+      <xacro:property name="Confocal_Sensor_Top_TCP_2_Joint_Cal_ry" value="${calibration_dict['Confocal_Sensor_Top_TCP_2_Joint']['ry_offset']}"/>
+      <xacro:property name="Confocal_Sensor_Top_TCP_2_Joint_Cal_rz" value="${calibration_dict['Confocal_Sensor_Top_TCP_2_Joint']['rz_offset']}"/>
+      <joint name="TCP_Confocal_Sensor_Top_2_Joint" type="fixed">
+        <origin xyz="
+            ${0.147499957149375 + Confocal_Sensor_Top_TCP_2_Joint_Cal_x*0.000001}
+            ${-0.1065 + Confocal_Sensor_Top_TCP_2_Joint_Cal_y*0.000001}
+            ${-0.4955 + Confocal_Sensor_Top_TCP_2_Joint_Cal_z*0.000001}"
+            rpy="
+            ${0 + Confocal_Sensor_Top_TCP_2_Joint_Cal_rx*3.14159265359/180}
+            ${0 + Confocal_Sensor_Top_TCP_2_Joint_Cal_ry*3.14159265359/180}
+            ${0 + Confocal_Sensor_Top_TCP_2_Joint_Cal_rz*3.14159265359/180}" />
+        <parent link="Z_Axis" />
+        <child link="TCP_Confocal_Sensor_Top_2" />
+        <axis xyz="0 0 0" />
+      </joint>
+    </xacro:if>
     <!--%%%%%%%%%%%%% Camera Calibration Definitions-->
     <link name="Camera_Calibration_Platelet">

Commit message: bug fixes

File: pm_robot_description/urdf/pm_robot.xacro (robot description, xacro)
@@ -285,5 +285,5 @@
     </joint> -->
     <!--%%%%%%%%%%%%% 1K Dispenser Flap Definitions %%%%%%%%%%%%%-->
-    <link name="1K_Dispenser_Flap">
+    <link name="1K_Dispenser_Protection">
       <inertial>
         <origin xyz="-0.0475534171935499 -0.0152444446246764 -0.0129366605877314" rpy="0 0 0" />
@@ -306,11 +306,11 @@
     </link>
     <!---Gravity off-->
-    <gazebo reference="1K_Dispenser_Flap">
-      <turnGravityOff>true</turnGravityOff>
-    </gazebo>
-    <joint name="1K_Dispenser_Flap_Joint" type="prismatic">
+    <gazebo reference="1K_Dispenser_Protection">
+      <turnGravityOff>true</turnGravityOff>
+    </gazebo>
+    <joint name="1K_Dispenser_Protection_Joint" type="prismatic">
       <origin xyz="-0.0315 -0.02479 -0.424" rpy="0 0 0" />
       <parent link="Z_Axis" />
-      <child link="1K_Dispenser_Flap" />
+      <child link="1K_Dispenser_Protection" />
       <axis xyz="-1 0 0" />
       <limit lower="-0.025" upper="0.00" effort="100" velocity="0.5" />

File: pm_robot_description/urdf/pm_robot_unity.urdf (robot description, URDF)
Before this commit: robot pm_robot, 56 links, 55 joints
Links:
- removed link 1K_Dispenser_Flap
- added link 1K_Dispenser_Protection, mass 0.0179075605864254; collision mesh filename=file:///home/match-mover/Documents/ros2_ws/install/pm_robot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; visual mesh filename=file:///home/match-mover/Documents/ros2_ws/install/pm_robot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
Joints:
- removed joint 1K_Dispenser_Flap_Joint
- added joint 1K_Dispenser_Protection_Joint: type prismatic, parent Z_Axis, child 1K_Dispenser_Protection, origin xyz=-0.0315 -0.02479 -0.424 rpy=0 0 0, axis -1 0 0, limit lower=-0.025 upper=0.00 effort=100 velocity=0.5

File: pm_robot_description/urdf/ros2_control_real_HW.xacro (robot description, xacro)
@@ -63,5 +63,5 @@
             </joint>
 <!--
-            <joint name="1K_Dispenser_Flap_Joint">
+            <joint name="1K_Dispenser_Protection_Joint">
                 <command_interface name="position">
                 </command_interface>
@@ -174,5 +174,5 @@
                 </state_interface>
             </joint>
-            <joint name="1K_Dispenser_Flap_Joint">
+            <joint name="1K_Dispenser_Protection_Joint">
                 <command_interface name="position">
                 </command_interface>

File: pm_robot_description/urdf/ros2_control_sim_HW.xacro (robot description, xacro)
@@ -36,5 +36,5 @@
                 <state_interface name="velocity"/>
             </joint>
-            <joint name="1K_Dispenser_Flap_Joint">
+            <joint name="1K_Dispenser_Protection_Joint">
                 <command_interface name="position">
                 </command_interface>
