Commit message: config class & bug fixes

File: pm_robot_description/urdf/pm_robot.xacro (robot description, xacro)
@@ -221,10 +221,25 @@
       <turnGravityOff>true</turnGravityOff>
     </gazebo>
+<!-- Property names should not start with a number -->
+    <xacro:property name="T_Axis_Joint_Cal_x" value="${calibration_dict['T_Axis_Joint']['x_offset']}"/>
+    <xacro:property name="T_Axis_Joint_Cal_y" value="${calibration_dict['T_Axis_Joint']['y_offset']}"/>
+    <xacro:property name="T_Axis_Joint_Cal_z" value="${calibration_dict['T_Axis_Joint']['z_offset']}"/>
+    <xacro:property name="T_Axis_Joint_Cal_rx" value="${calibration_dict['T_Axis_Joint']['rx_offset']}"/>
+    <xacro:property name="T_Axis_Joint_Cal_ry" value="${calibration_dict['T_Axis_Joint']['ry_offset']}"/>
+    <xacro:property name="T_Axis_Joint_Cal_rz" value="${calibration_dict['T_Axis_Joint']['rz_offset']}"/>
     <joint name="T_Axis_Joint" type="revolute">
-      <origin xyz="0.0600000000000017 -0.0580000000000003 -0.427500000000004" rpy="0 0 0" />
+      <origin
+      xyz="
+        ${0.0600000000000017 + T_Axis_Joint_Cal_x * 0.000001}
+        ${-0.0580000000000003 + T_Axis_Joint_Cal_y * 0.000001}
+        ${-0.427500000000004 + T_Axis_Joint_Cal_z * 0.000001}"
+        rpy="
+        ${0 + T_Axis_Joint_Cal_rx * 3.14159265359/180}
+        ${0 + T_Axis_Joint_Cal_ry * 3.14159265359/180}
+        ${0 + T_Axis_Joint_Cal_rz * 3.14159265359/180}" />
       <parent link="Z_Axis" />
       <child link="Gripper_Rot_Plate" />
       <axis xyz="0 0 1" />
-      <limit lower="-2.0" upper="2.0" effort="100" velocity="5" />
+      <limit lower="-2.0" upper="2.0" effort="100" velocity="15" />
     </joint>
     <link name="t_axis_toolchanger">

Commit message: calibration

File: pm_robot_description/urdf/pm_robot.xacro (robot description, xacro)
@@ -799,10 +799,10 @@
         name="TCP_Confocal_Sensor_Top_2">
       </link>
-      <xacro:property name="Confocal_Sensor_Top_TCP_2_Joint_Cal_x" value="${calibration_dict['Confocal_Sensor_Top_TCP_2_Joint']['x_offset']}"/>
-      <xacro:property name="Confocal_Sensor_Top_TCP_2_Joint_Cal_y" value="${calibration_dict['Confocal_Sensor_Top_TCP_2_Joint']['y_offset']}"/>
-      <xacro:property name="Confocal_Sensor_Top_TCP_2_Joint_Cal_z" value="${calibration_dict['Confocal_Sensor_Top_TCP_2_Joint']['z_offset']}"/>
-      <xacro:property name="Confocal_Sensor_Top_TCP_2_Joint_Cal_rx" value="${calibration_dict['Confocal_Sensor_Top_TCP_2_Joint']['rx_offset']}"/>
-      <xacro:property name="Confocal_Sensor_Top_TCP_2_Joint_Cal_ry" value="${calibration_dict['Confocal_Sensor_Top_TCP_2_Joint']['ry_offset']}"/>
-      <xacro:property name="Confocal_Sensor_Top_TCP_2_Joint_Cal_rz" value="${calibration_dict['Confocal_Sensor_Top_TCP_2_Joint']['rz_offset']}"/>
+      <xacro:property name="Confocal_Sensor_Top_TCP_2_Joint_Cal_x" value="${calibration_dict['Confocal_Sensor_Top_TCP_Joint']['x_offset']}"/>
+      <xacro:property name="Confocal_Sensor_Top_TCP_2_Joint_Cal_y" value="${calibration_dict['Confocal_Sensor_Top_TCP_Joint']['y_offset']}"/>
+      <xacro:property name="Confocal_Sensor_Top_TCP_2_Joint_Cal_z" value="${calibration_dict['Confocal_Sensor_Top_TCP_Joint']['z_offset']}"/>
+      <xacro:property name="Confocal_Sensor_Top_TCP_2_Joint_Cal_rx" value="${calibration_dict['Confocal_Sensor_Top_TCP_Joint']['rx_offset']}"/>
+      <xacro:property name="Confocal_Sensor_Top_TCP_2_Joint_Cal_ry" value="${calibration_dict['Confocal_Sensor_Top_TCP_Joint']['ry_offset']}"/>
+      <xacro:property name="Confocal_Sensor_Top_TCP_2_Joint_Cal_rz" value="${calibration_dict['Confocal_Sensor_Top_TCP_Joint']['rz_offset']}"/>
       <joint name="TCP_Confocal_Sensor_Top_2_Joint" type="fixed">
         <origin xyz="

Commit message: urdf update confocal sensor

File: pm_robot_description/urdf/pm_robot.xacro (robot description, xacro)
@@ -696,17 +696,17 @@
       <link name="TCP_Confocal_Sensor_Bottom">
       <inertial>
-            <origin
-              xyz="-0.00247029745512151 0.0425771909752702 -0.0497854338510461"
-              rpy="0 0 0" />
-            <mass
-              value="0.344263397388723" />
-            <inertia
-              ixx="0.000599129085110184"
-              ixy="-1.74073417588787E-05"
-              ixz="-4.10917598198572E-08"
-              iyy="0.000151077936284775"
-              iyz="-8.61442405235731E-06"
-              izz="0.000578610557041608" />
-          </inertial>
+      <origin
+          xyz="0.00873210562859661 -0.0528919985243314 -0.048485473461278"
+          rpy="0 0 0" />
+          <mass
+            value="0.282095702939505" />
+          <inertia
+            ixx="0.000459498255002395"
+            ixy="-2.6478647169319E-05"
+            ixz="1.30820197742833E-05"
+            iyy="0.000113874627024508"
+            iyz="8.93478168646323E-06"
+            izz="0.000453112849086854" />
+        </inertial>
         <visual>
           <origin xyz="0 0 0" rpy="0 0 0" />
@@ -733,7 +733,7 @@
       <joint name="TCP_Confocal_Sensor_Bottom_Joint" type="fixed">
         <origin xyz="
-            ${0.1925 + Confocal_Sensor_Bottom_TCP_Joint_Cal_x*0.000001}
-            ${0.0938799999999999+ Confocal_Sensor_Bottom_TCP_Joint_Cal_y*0.000001}
-            ${0.30825985348391 + Confocal_Sensor_Bottom_TCP_Joint_Cal_z*0.000001}"
+            ${0.138 + Confocal_Sensor_Bottom_TCP_Joint_Cal_x*0.000001}
+            ${0.07484+ Confocal_Sensor_Bottom_TCP_Joint_Cal_y*0.000001}
+            ${0.30851 + Confocal_Sensor_Bottom_TCP_Joint_Cal_z*0.000001}"
             rpy="
             ${0 + Confocal_Sensor_Bottom_TCP_Joint_Cal_rx*3.14159265359/180}
@@ -748,16 +748,16 @@
       <link name="TCP_Confocal_Sensor_Top">
       <inertial>
-        <origin
-          xyz="-0.0129743586620629 -0.0179072639596305 0.0489187396629332"
-          rpy="0 0 0" />
-        <mass
-          value="0.0631321031924395" />
-        <inertia
-          ixx="5.72140577879517E-05"
-          ixy="-1.00812729158378E-05"
-          ixz="-1.59225714048641E-06"
-          iyy="3.26664833980595E-05"
-          iyz="-4.19709040215342E-06"
-          izz="3.82911436485178E-05" />
+      <origin
+        xyz="-0.0129992374574083 -0.0182302838306646 0.0532500614504829"
+        rpy="0 0 0" />
+      <mass
+        value="0.0655666647000771" />
+      <inertia
+        ixx="6.2078599619276E-05"
+        ixy="-1.1064871149157E-05"
+        ixz="-1.62845145975249E-06"
+        iyy="3.63712240262645E-05"
+        iyz="-4.78563533641753E-06"
+        izz="4.07979832865319E-05" />
       </inertial>
         <visual>
@@ -787,5 +787,5 @@
             ${0.176999957149375 + Confocal_Sensor_Top_TCP_Joint_Cal_x*0.000001}
             ${-0.0580000000000008+ Confocal_Sensor_Top_TCP_Joint_Cal_y*0.000001}
-            ${-0.495500000000003 + Confocal_Sensor_Top_TCP_Joint_Cal_z*0.000001}"
+            ${-0.502500000000003 + Confocal_Sensor_Top_TCP_Joint_Cal_z*0.000001}"
             rpy="
             ${0 + Confocal_Sensor_Top_TCP_Joint_Cal_rx*3.14159265359/180}
@@ -807,7 +807,7 @@
       <joint name="TCP_Confocal_Sensor_Top_2_Joint" type="fixed">
         <origin xyz="
-            ${0.147499957149375 + Confocal_Sensor_Top_TCP_2_Joint_Cal_x*0.000001}
+            ${0.147499957149374 + Confocal_Sensor_Top_TCP_2_Joint_Cal_x*0.000001}
             ${-0.1065 + Confocal_Sensor_Top_TCP_2_Joint_Cal_y*0.000001}
-            ${-0.4955 + Confocal_Sensor_Top_TCP_2_Joint_Cal_z*0.000001}"
+            ${-0.5025 + Confocal_Sensor_Top_TCP_2_Joint_Cal_z*0.000001}"
             rpy="
             ${0 + Confocal_Sensor_Top_TCP_2_Joint_Cal_rx*3.14159265359/180}
@@ -822,8 +822,17 @@
     <link name="Camera_Calibration_Platelet">
       <inertial>
-        <origin xyz="-0.000344499007125409 0.0696122748122424 0.000295151280628292" rpy="0 0 0" />
-        <mass value="0.0334016358510876" />
-        <inertia ixx="2.05104945364406E-05" ixy="-1.61006130053269E-08" ixz="-7.42638002033627E-6" iyy="2.64967112268826E-06" iyz="4.64472618194223E-07" izz="2.23824646029018E-05" />
-      </inertial>
+      <origin
+        xyz="0.0128792780733884 0.0686361134200075 0.00483645717370385"
+        rpy="0 0 0" />
+      <mass
+        value="0.0528869806353836" />
+      <inertia
+        ixx="2.80210657912113E-05"
+        ixy="-5.13560878472572E-06"
+        ixz="-4.10913124496945E-07"
+        iyy="9.69742442471709E-06"
+        iyz="-2.11158283931519E-07"
+        izz="3.52667510166924E-05" />
+    </inertial>
       <visual>
         <origin xyz="0 0 0" rpy="0 0 0" />
@@ -847,4 +856,22 @@
       <limit lower="-0.04" upper="0.0" effort="100" velocity="0.5" />
     </joint>
+      <link
+        name="Laser_Height_Calibration_Frame">
+      </link>
+      <joint name="Laser_Height_Calibration_Frame_Joint" type="fixed">
+        <origin xyz="0.057308970 0.115944000 0.017870000" rpy="0 0 0" />
+        <parent link="Camera_Calibration_Platelet" />
+        <child link="Laser_Height_Calibration_Frame" />
+        <axis xyz="0 0 0" />
+      </joint>
+      <link
+        name="Calibration_Platelet_Calibration_Frame">
+      </link>
+      <joint name="Calibration_Platelet_Calibration_Frame_Joint" type="fixed">
+        <origin xyz="0.0 0.10405 0.012" rpy="0 0 0" />
+        <parent link="Camera_Calibration_Platelet" />
+        <child link="Calibration_Platelet_Calibration_Frame" />
+        <axis xyz="0 0 0" />
+      </joint>
     <!--%%%%%%%%%%%%% Calibration Qube Definitions-->
     <link name="Calibration_Qube">
@@ -880,5 +907,5 @@
     <joint name="Calibration_Qube_Joint" type="prismatic">
       <origin xyz="
-          ${0.154 + Calibration_Qube_Joint_Cal_x*0.000001}
+          ${0.172 + Calibration_Qube_Joint_Cal_x*0.000001}
           ${0.108 + Calibration_Qube_Joint_Cal_y*0.000001}
           ${0.305 + Calibration_Qube_Joint_Cal_z*0.000001}" rpy="

File: pm_robot_description/urdf/pm_smarpod_station.xacro (robot description, xacro)
@@ -88,5 +88,5 @@
     type="fixed">
     <origin
-      xyz="0.2 0.15 0.2253999999992"
+      xyz="0.1465 0.15 0.2253999999992"
       rpy="0 0 0" />
     <parent

Commit message: urdf changes

File: pm_robot_description/urdf/pm_robot.xacro (robot description, xacro)
@@ -463,5 +463,5 @@
       <child link="2K_Dispenser_Cartridge" />
       <axis xyz="0 0 1" />
-      <limit lower="-0.04" upper="0.00" effort="100" velocity="0.1" />
+      <limit lower="-0.05" upper="0.00" effort="100" velocity="0.1" />
     </joint>
     <link name="2K_Dispenser_TCP">
@@ -734,6 +734,6 @@
         <origin xyz="
             ${0.138 + Confocal_Sensor_Bottom_TCP_Joint_Cal_x*0.000001}
-            ${0.07484+ Confocal_Sensor_Bottom_TCP_Joint_Cal_y*0.000001}
-            ${0.30851 + Confocal_Sensor_Bottom_TCP_Joint_Cal_z*0.000001}"
+            ${0.07964+ Confocal_Sensor_Bottom_TCP_Joint_Cal_y*0.000001}
+            ${0.307 + Confocal_Sensor_Bottom_TCP_Joint_Cal_z*0.000001}"
             rpy="
             ${0 + Confocal_Sensor_Bottom_TCP_Joint_Cal_rx*3.14159265359/180}
@@ -787,5 +787,5 @@
             ${0.176999957149375 + Confocal_Sensor_Top_TCP_Joint_Cal_x*0.000001}
             ${-0.0580000000000008+ Confocal_Sensor_Top_TCP_Joint_Cal_y*0.000001}
-            ${-0.502500000000003 + Confocal_Sensor_Top_TCP_Joint_Cal_z*0.000001}"
+            ${-0.500500000000003 + Confocal_Sensor_Top_TCP_Joint_Cal_z*0.000001}"
             rpy="
             ${0 + Confocal_Sensor_Top_TCP_Joint_Cal_rx*3.14159265359/180}
@@ -850,9 +850,9 @@
     </link>
     <joint name="Camera_Calibration_Platelet_Joint" type="prismatic">
-      <origin xyz="0.08 -0.0805 0.293" rpy="0 0 0" />
+      <origin xyz="0.08 -0.0805 0.2922" rpy="0 0 0" />
       <parent link="Camera_Station" />
       <child link="Camera_Calibration_Platelet" />
       <axis xyz="0 -1 0" />
-      <limit lower="-0.04" upper="0.0" effort="100" velocity="0.5" />
+      <limit lower="-0.048" upper="0.0" effort="100" velocity="0.5" />
     </joint>
       <link
@@ -860,5 +860,5 @@
       </link>
       <joint name="Laser_Height_Calibration_Frame_Joint" type="fixed">
-        <origin xyz="0.057308970 0.115944000 0.017870000" rpy="0 0 0" />
+        <origin xyz="0.058 0.115944000 0.020870000" rpy="0 0 0" />
         <parent link="Camera_Calibration_Platelet" />
         <child link="Laser_Height_Calibration_Frame" />
@@ -869,5 +869,5 @@
       </link>
       <joint name="Calibration_Platelet_Calibration_Frame_Joint" type="fixed">
-        <origin xyz="0.0 0.10405 0.012" rpy="0 0 0" />
+        <origin xyz="0.0 0.1195 0.0135 " rpy="0 0 0" />
         <parent link="Camera_Calibration_Platelet" />
         <child link="Calibration_Platelet_Calibration_Frame" />

Commit message: robot calibration

File: pm_robot_description/urdf/pm_robot.xacro (robot description, xacro)
@@ -361,5 +361,5 @@
       <child link="1K_Dispenser" />
       <axis xyz="0 0 -1" />
-      <limit lower="0" upper="0.04" effort="100" velocity="0.05" />
+      <limit lower="0" upper="0.035" effort="100" velocity="0.05" />
     </joint>
     <link name="1K_Dispenser_TCP">
@@ -786,5 +786,5 @@
         <origin xyz="
             ${0.176999957149375 + Confocal_Sensor_Top_TCP_Joint_Cal_x*0.000001}
-            ${-0.0580000000000008+ Confocal_Sensor_Top_TCP_Joint_Cal_y*0.000001}
+            ${-0.0580000000000008 + Confocal_Sensor_Top_TCP_Joint_Cal_y*0.000001}
             ${-0.500500000000003 + Confocal_Sensor_Top_TCP_Joint_Cal_z*0.000001}"
             rpy="
@@ -918,4 +918,14 @@
       <limit lower="-0.008" upper="0" effort="0" velocity="0.005" />
     </joint>
+    <xacro:property name="Calibration_Cube_Bottom_Joint_Cal_z" value="${calibration_dict['Calibration_Cube_Bottom_Joint']['z_offset']}"/>
+    <link
+      name="Calibration_Cube_Bottom">
+    </link>
+    <joint name="Calibration_Cube_Bottom_Joint" type="fixed">
+      <origin xyz="0.0 0.0 ${-0.004 + Calibration_Cube_Bottom_Joint_Cal_z*0.000001}" rpy="0 0 0" />
+      <parent link="Calibration_Qube" />
+      <child link="Calibration_Cube_Bottom" />
+      <axis xyz="0 0 0" />
+    </joint>
   </xacro:macro>
 </robot>

File: pm_robot_description/urdf/pm_robot_gonio_left.xacro (robot description, xacro)
@@ -147,12 +147,4 @@
     </joint>
     <!--%%%%%%%%%%%%% Gonio Left Chuck Definitions-->
-    <link name="Gonio_Left_Chuck_Origin">
-    </link>
-    <joint name="Gonio_Left_Chuck_Origin_Joint" type="fixed">
-      <origin xyz="0 0 -0.015" rpy="0 0 0" />
-      <parent link="Gonio_Left_Stage_2_Bottom" />
-      <child link="Gonio_Left_Chuck_Origin" />
-      <axis xyz="0 0 0" />
-    </joint>
     <!--%%%%%%%%%%%%% Gonio Left Example Chuck Definitions-->
     <!--%%%%%%%%%%%%% This is for the Chuck  -->
@@ -180,34 +172,42 @@
     <xacro:property name="Gonio_Left_Chuck_Cal_ry" value="${calibration_dict['Gonio_Left_Chuck_Joint']['ry_offset']}"/>
     <xacro:property name="Gonio_Left_Chuck_Cal_rz" value="${calibration_dict['Gonio_Left_Chuck_Joint']['rz_offset']}"/>
-    <link name="Gonio_Left_Chuck">
-      <inertial>
-        <origin xyz="${gonio_chuck_xyz}" rpy="${gonio_chuck_rpy}"/>
-        <mass value="${gonio_chuck_mass}"/>
-        <inertia ixx="${gonio_chuck_inertia_ixx}" ixy="${gonio_chuck_inertia_ixy}" ixz="${gonio_chuck_inertia_ixz}" iyy="${gonio_chuck_inertia_iyy}" iyz="${gonio_chuck_inertia_iyz}" izz="${gonio_chuck_inertia_izz}" />
-      </inertial>
-      <visual>
-        <origin xyz="0 0 0" rpy="0 0 0" />
-        <geometry>
-          <mesh filename="file://$(find pm_robot_description)/meshes/Gonio_Left/Gonio_Left_Chucks/${gonio_chuck_visual_filename}" />
-        </geometry>
-        <material name="${gonio_chuck_color}">
-        </material>
-      </visual>
-      <collision>
-        <origin xyz="0 0 0" rpy="0 0 0" />
-        <geometry>
-          <mesh filename="file://$(find pm_robot_description)/meshes/Gonio_Left/Gonio_Left_Chucks/${gonio_chuck_collision_filename}" />
-        </geometry>
-      </collision>
-    </link>
-    <joint name="Gonio_Left_Chuck_Joint" type="fixed">
-        <origin xyz="
+    <link name="Gonio_Left_Chuck_Origin">
+    </link>
+    <joint name="Gonio_Left_Chuck_Origin_Joint" type="fixed">
+      <origin xyz="
         ${0.0 + Gonio_Left_Chuck_Cal_x * 0.000001}
         ${0.0 + Gonio_Left_Chuck_Cal_y * 0.000001}
-        ${0.0 + Gonio_Left_Chuck_Cal_z * 0.000001}"
+        ${-0.015 + Gonio_Left_Chuck_Cal_z * 0.000001}"
         rpy="
         ${0 + Gonio_Left_Chuck_Cal_rx * 3.14159265359/180}
         ${0 + Gonio_Left_Chuck_Cal_ry * 3.14159265359/180}
         ${0 + Gonio_Left_Chuck_Cal_rz * 3.14159265359/180}" />
+      <parent link="Gonio_Left_Stage_2_Bottom" />
+      <child link="Gonio_Left_Chuck_Origin" />
+      <axis xyz="0 0 0" />
+    </joint>
+    <link name="Gonio_Left_Chuck">
+      <inertial>
+        <origin xyz="${gonio_chuck_xyz}" rpy="${gonio_chuck_rpy}"/>
+        <mass value="${gonio_chuck_mass}"/>
+        <inertia ixx="${gonio_chuck_inertia_ixx}" ixy="${gonio_chuck_inertia_ixy}" ixz="${gonio_chuck_inertia_ixz}" iyy="${gonio_chuck_inertia_iyy}" iyz="${gonio_chuck_inertia_iyz}" izz="${gonio_chuck_inertia_izz}" />
+      </inertial>
+      <visual>
+        <origin xyz="0 0 0" rpy="0 0 0" />
+        <geometry>
+          <mesh filename="file://$(find pm_robot_description)/meshes/Gonio_Left/Gonio_Left_Chucks/${gonio_chuck_visual_filename}" />
+        </geometry>
+        <material name="${gonio_chuck_color}">
+        </material>
+      </visual>
+      <collision>
+        <origin xyz="0 0 0" rpy="0 0 0" />
+        <geometry>
+          <mesh filename="file://$(find pm_robot_description)/meshes/Gonio_Left/Gonio_Left_Chucks/${gonio_chuck_collision_filename}" />
+        </geometry>
+      </collision>
+    </link>
+    <joint name="Gonio_Left_Chuck_Joint" type="fixed">
+      <origin xyz="0 0 0.00" rpy="0 0 0" />
       <parent link="Gonio_Left_Chuck_Origin" />
       <child link="Gonio_Left_Chuck" />

File: pm_robot_description/urdf/pm_robot_gonio_right.xacro (robot description, xacro)
@@ -253,20 +253,4 @@
   </joint>
   <!--%%%%%%%%%%%%% Gonio Right Chuck Definitions-->
-  <link
-    name="Gonio_Right_Chuck_Origin">
-  </link>
-  <joint
-    name="Gonio_Right_Chuck_Origin_Joint"
-    type="fixed">
-    <origin
-      xyz="0 0 -0.05"
-      rpy="0 0 0" />
-    <parent
-      link="Gonio_Right_Stage_2_Bottom" />
-    <child
-      link="Gonio_Right_Chuck_Origin" />
-    <axis
-      xyz="0 0 0" />
-  </joint>
   <!--%%%%%%%%%%%%% This is for the Chuck  -->
   <xacro:property name="gonio_chuck_tcp_offset_x_1" value="${gonio_right_configs_dict[current_gonio_right_chuck]['spawn_1_offset_from_gonio_x']}"/>
@@ -297,4 +281,25 @@
   <xacro:property name="Gonio_Right_Chuck_Cal_rz" value="${calibration_dict['Gonio_Right_Chuck_Joint']['rz_offset']}"/>
   <link
+    name="Gonio_Right_Chuck_Origin">
+  </link>
+  <joint
+    name="Gonio_Right_Chuck_Origin_Joint"
+    type="fixed">
+      <origin xyz="
+      ${0.0 + Gonio_Right_Chuck_Cal_x * 0.000001}
+      ${0.0 + Gonio_Right_Chuck_Cal_y * 0.000001}
+      ${-0.05 + Gonio_Right_Chuck_Cal_z * 0.000001}"
+      rpy="
+      ${0 + Gonio_Right_Chuck_Cal_rx * 3.14159265359/180}
+      ${0 + Gonio_Right_Chuck_Cal_ry * 3.14159265359/180}
+      ${0 + Gonio_Right_Chuck_Cal_rz * 3.14159265359/180}" />
+    <parent
+      link="Gonio_Right_Stage_2_Bottom" />
+    <child
+      link="Gonio_Right_Chuck_Origin" />
+    <axis
+      xyz="0 0 0" />
+  </joint>
+  <link
     name="Gonio_Right_Chuck">
     <inertial>
@@ -336,11 +341,11 @@
     type="fixed">
     <origin xyz="
-      ${0.0 + Gonio_Right_Chuck_Cal_x * 0.000001}
-      ${0.0 + Gonio_Right_Chuck_Cal_y * 0.000001}
-      ${0.0 + Gonio_Right_Chuck_Cal_z * 0.000001}"
+      ${0.0 }
+      ${0.0 }
+      ${0.0 }"
       rpy="
-      ${0 + Gonio_Right_Chuck_Cal_rx * 3.14159265359/180}
-      ${0 + Gonio_Right_Chuck_Cal_ry * 3.14159265359/180}
-      ${0 + Gonio_Right_Chuck_Cal_rz * 3.14159265359/180}" />
+      ${0}
+      ${0}
+      ${0}" />
     <parent
       link="Gonio_Right_Chuck_Origin" />
