Commit message: collision models and planing

File: pm_robot_description/urdf/pm_robot.xacro (robot description, xacro)
@@ -93,5 +93,5 @@
         <origin xyz="0 0 0" rpy="0 0 0" />
         <geometry>
-          <mesh filename="file://$(find pm_robot_description)/meshes/axis_base.STL" />
+          <mesh filename="file://$(find pm_robot_description)/meshes/axis_base_coll.STL" />
         </geometry>
       </collision>
@@ -125,5 +125,5 @@
         <origin xyz="0 0 0" rpy="0 0 0" />
         <geometry>
-          <mesh filename="file://$(find pm_robot_description)/meshes/X_Axis.STL" />
+          <mesh filename="file://$(find pm_robot_description)/meshes/X_Axis_coll.STL" />
         </geometry>
       </collision>
@@ -153,5 +153,5 @@
         <origin xyz="0 0 0" rpy="0 0 0" />
         <geometry>
-          <mesh filename="file://$(find pm_robot_description)/meshes/Y_Axis.STL" />
+          <mesh filename="file://$(find pm_robot_description)/meshes/Y_Axis_coll.STL" />
         </geometry>
       </collision>
@@ -181,5 +181,5 @@
         <origin xyz="0 0 0" rpy="0 0 0" />
         <geometry>
-          <mesh filename="file://$(find pm_robot_description)/meshes/Z_Axis.STL" />
+          <mesh filename="file://$(find pm_robot_description)/meshes/Z_Axis_coll.STL" />
         </geometry>
       </collision>
@@ -213,5 +213,5 @@
         <origin xyz="0 0 0" rpy="0 0 0" />
         <geometry>
-          <mesh filename="file://$(find pm_robot_description)/meshes/Gripper_Rot_Plate.STL" />
+          <mesh filename="file://$(find pm_robot_description)/meshes/Gripper_Rot_Plate_coll.STL" />
         </geometry>
       </collision>
@@ -261,5 +261,5 @@
         <origin xyz="0 0 0" rpy="0 0 0" />
         <geometry>
-          <mesh filename="file://$(find pm_robot_description)/meshes/t_axis_tool.STL" />
+          <mesh filename="file://$(find pm_robot_description)/meshes/t_axis_tool_coll.STL" />
         </geometry>
       </collision>
@@ -316,5 +316,5 @@
         <origin xyz="0 0 0" rpy="0 0 0" />
         <geometry>
-          <mesh filename="file://$(find pm_robot_description)/meshes/Glue_Cartridge_Flap.STL" />
+          <mesh filename="file://$(find pm_robot_description)/meshes/Glue_Cartridge_Flap_Coll.STL" />
         </geometry>
       </collision>
@@ -348,5 +348,5 @@
         <origin xyz="0 0 0" rpy="0 0 0" />
         <geometry>
-          <mesh filename="file://$(find pm_robot_description)/meshes/1K_Dispenser.STL" />
+          <mesh filename="file://$(find pm_robot_description)/meshes/1K_Dispenser_coll.STL" />
         </geometry>
       </collision>
@@ -450,5 +450,5 @@
         <origin xyz="0 0 0" rpy="0 0 0" />
         <geometry>
-          <mesh filename="file://$(find pm_robot_description)/meshes/2K_Glue_Cartridge.STL" />
+          <mesh filename="file://$(find pm_robot_description)/meshes/2K_Glue_Cartridge_Coll.STL" />
         </geometry>
       </collision>
@@ -505,5 +505,5 @@
         <origin xyz="0 0 0" rpy="0 0 0" />
         <geometry>
-          <mesh filename="file://$(find pm_robot_description)/meshes/Cam1_Toolhead_TCP.STL" />
+          <mesh filename="file://$(find pm_robot_description)/meshes/Cam1_Toolhead_TCP_coll.STL" />
         </geometry>
       </collision>
@@ -620,5 +620,5 @@
         <origin xyz="0 0 0" rpy="0 0 0" />
         <geometry>
-          <mesh filename="file://$(find pm_robot_description)/meshes/Camera_Station.STL" />
+          <mesh filename="file://$(find pm_robot_description)/meshes/Camera_Station_coll.STL" />
         </geometry>
       </collision>
@@ -773,5 +773,5 @@
           <origin xyz="0 0 0" rpy="0 0 0" />
           <geometry>
-            <mesh filename="file://$(find pm_robot_description)/meshes/Confocal_Sensor_Top.STL" />
+            <mesh filename="file://$(find pm_robot_description)/meshes/Confocal_Sensor_Top_coll.STL" />
           </geometry>
         </collision>
@@ -845,5 +845,5 @@
         <origin xyz="0 0 0" rpy="0 0 0" />
         <geometry>
-          <mesh filename="file://$(find pm_robot_description)/meshes/Camera_Calibration_Platelet.STL" />
+          <mesh filename="file://$(find pm_robot_description)/meshes/Camera_Calibration_Platelet_coll.STL" />
         </geometry>
       </collision>

File: pm_robot_description/urdf/pm_robot_gonio_left.xacro (robot description, xacro)
@@ -47,5 +47,5 @@
         <origin xyz="0 0 0" rpy="0 0 0" />
         <geometry>
-          <mesh filename="file://$(find pm_robot_description)/meshes/Gonio_Left/Gonio_Left_Base.STL" />
+          <mesh filename="file://$(find pm_robot_description)/meshes/Gonio_Left/Gonio_Left_Base_coll.STL" />
         </geometry>
       </collision>
@@ -244,5 +244,5 @@
         <origin xyz="0 0 0" rpy="0 0 0" />
         <geometry>
-          <mesh filename="file://$(find pm_robot_description)/meshes/Gonio_Left/UV_Cart_X_Front.STL" />
+          <mesh filename="file://$(find pm_robot_description)/meshes/Gonio_Left/UV_Cart_X_Front_Coll.STL" />
         </geometry>
       </collision>
@@ -301,5 +301,5 @@
         <origin xyz="0 0 0" rpy="0 0 0" />
         <geometry>
-          <mesh filename="file://$(find pm_robot_description)/meshes/Gonio_Left/UV_Cart_X_Back.STL" />
+          <mesh filename="file://$(find pm_robot_description)/meshes/Gonio_Left/UV_Cart_X_Back_Coll.STL" />
         </geometry>
       </collision>
@@ -330,5 +330,5 @@
         <origin xyz="0 0 0" rpy="0 0 0" />
         <geometry>
-          <mesh filename="file://$(find pm_robot_description)/meshes/Gonio_Left/UV_Cart_Back.STL" />
+          <mesh filename="file://$(find pm_robot_description)/meshes/Gonio_Left/UV_Cart_Back_Coll.STL" />
         </geometry>
       </collision>

File: pm_robot_description/urdf/pm_robot_gonio_right.xacro (robot description, xacro)
@@ -66,5 +66,5 @@
         rpy="0 0 0" />
       <geometry>
-        <mesh filename="file://$(find pm_robot_description)/meshes/Gonio_Right/Gonio_Base_Right.STL" />
+        <mesh filename="file://$(find pm_robot_description)/meshes/Gonio_Right/Gonio_Base_Right_Coll.STL" />
       </geometry>
     </collision>

Commit message: limit t_axis

File: pm_robot_description/urdf/pm_robot.xacro (robot description, xacro)
@@ -242,5 +242,5 @@
       <child link="Gripper_Rot_Plate" />
       <axis xyz="0 0 1" />
-      <limit lower="-2.0" upper="2.0" effort="100" velocity="15" />
+      <limit lower="${-150 * 3.14159265359/180}" upper="${200 * 3.14159265359/180}" effort="100" velocity="15" />
     </joint>
     <link name="t_axis_toolchanger">
