Commit message: 2k dispenser tip

File: pm_robot_description/urdf/pm_robot.xacro (robot description, xacro)
@@ -27,4 +27,5 @@
     <xacro:property name="current_pm_robot_bringup_config" value="${xacro.load_yaml(pm_robot_bringup_config_file)}"/>
     <xacro:property name="current_pm_robot_1K_dipsenser_tip" value="${current_pm_robot_bringup_config['pm_robot_1K_dispenser_tip']['use_dispenser_tip']}"/>
+    <xacro:property name="current_pm_robot_2K_dipsenser_tip" value="${current_pm_robot_bringup_config['pm_robot_2K_dispenser_tip']['use_dispenser_tip']}"/>
     <xacro:property name="current_vacuum_tool" value="${current_pm_robot_bringup_config['pm_robot_tools']['pm_robot_vacuum_tools']['use_tool']}"/>
     <xacro:property name="calibration_dict" value="${xacro.load_yaml(pm_robot_joint_calibraion_file)}"/>
@@ -381,5 +382,5 @@
         ${-0.001 + Dispenser_1K_TCP_Joint_Cal_x * 0.000001}
         ${-0.0318 + Dispenser_1K_TCP_Joint_Cal_y * 0.000001}
-        ${-0.135 + Dispenser_1K_TCP_Joint_Cal_z * 0.000001 + Dispenser_1K_tip_z_offset}" rpy="
+        ${-0.11 + Dispenser_1K_TCP_Joint_Cal_z * 0.000001 - Dispenser_1K_tip_z_offset}" rpy="
         ${0 + Dispenser_1K_TCP_Joint_Cal_rx * 3.14159265359/180}
         ${0 + Dispenser_1K_TCP_Joint_Cal_ry * 3.14159265359/180}
@@ -403,35 +404,36 @@
     <xacro:property name="Dispenser_1K_tip_collision_filename" value="${dispenser_1K_configs_dict[current_pm_robot_1K_dipsenser_tip]['collision_filename']}"/>
     <!--%%%%%%%%%%%%% The parameters here are interchangeable %%%%%%%%%%%%%-->
-    <!--%%%%%%%%%%%%% Jaw 1 Definitions %%%%%%%%%%%%%-->
-    <link name="1K_Dispenser_Tip">
-      <inertial>
-        <origin xyz="${Dispenser_1K_tip_xyz}" rpy="${Dispenser_1K_tip_rpy}"/>
-        <mass value="${Dispenser_1K_tip_mass}"/>
-        <inertia ixx="${Dispenser_1K_tip_inertia_ixx}" ixy="${Dispenser_1K_tip_inertia_ixy}" ixz="${Dispenser_1K_tip_inertia_ixz}" iyy="${Dispenser_1K_tip_inertia_iyy}" iyz="${Dispenser_1K_tip_inertia_iyz}" izz="${Dispenser_1K_tip_inertia_izz}" />
-      </inertial>
-      <visual>
-        <origin xyz="0 0 0" rpy="0 0 0" />
-        <geometry>
-          <mesh filename="file://$(find pm_robot_description)/meshes/Dispenser_Tips/${Dispenser_1K_tip_visual_filename}" />
-        </geometry>
-        <material name="${Dispenser_1K_tip_color}">
-        </material>
-      </visual>
-      <collision>
-        <origin xyz="0 0 0" rpy="0 0 0" />
-        <geometry>
-          <mesh filename="file://$(find pm_robot_description)/meshes/Dispenser_Tips/${Dispenser_1K_tip_collision_filename}" />
-        </geometry>
-      </collision>
-    </link>
-    <gazebo reference="1K_Dispenser_Tip">
-      <turnGravityOff>true</turnGravityOff>
-    </gazebo>
-    <joint name="1K_Dispenser_Tip_Joint" type="fixed">
-      <!-- This needs to be corrected in Solidworks -->
-      <origin xyz="0.000 0 0 " rpy="0 0 0" />
-      <parent link="1K_Dispenser_TCP" />
-      <child link="1K_Dispenser_Tip" />
-    </joint>
+    <xacro:if value="${current_pm_robot_1K_dipsenser_tip != 'empty'}">
+      <link name="1K_Dispenser_Tip">
+        <inertial>
+          <origin xyz="${Dispenser_1K_tip_xyz}" rpy="${Dispenser_1K_tip_rpy}"/>
+          <mass value="${Dispenser_1K_tip_mass}"/>
+          <inertia ixx="${Dispenser_1K_tip_inertia_ixx}" ixy="${Dispenser_1K_tip_inertia_ixy}" ixz="${Dispenser_1K_tip_inertia_ixz}" iyy="${Dispenser_1K_tip_inertia_iyy}" iyz="${Dispenser_1K_tip_inertia_iyz}" izz="${Dispenser_1K_tip_inertia_izz}" />
+        </inertial>
+        <visual>
+          <origin xyz="0 0 0" rpy="0 0 0" />
+          <geometry>
+            <mesh filename="file://$(find pm_robot_description)/meshes/Dispenser_Tips/${Dispenser_1K_tip_visual_filename}" />
+          </geometry>
+          <material name="${Dispenser_1K_tip_color}">
+          </material>
+        </visual>
+        <collision>
+          <origin xyz="0 0 0" rpy="0 0 0" />
+          <geometry>
+            <mesh filename="file://$(find pm_robot_description)/meshes/Dispenser_Tips/${Dispenser_1K_tip_collision_filename}" />
+          </geometry>
+        </collision>
+      </link>
+      <gazebo reference="1K_Dispenser_Tip">
+        <turnGravityOff>true</turnGravityOff>
+      </gazebo>
+      <joint name="1K_Dispenser_Tip_Joint" type="fixed">
+        <!-- This needs to be corrected in Solidworks -->
+        <origin xyz="0.000 0 0 " rpy="0 0 0" />
+        <parent link="1K_Dispenser_TCP" />
+        <child link="1K_Dispenser_Tip" />
+      </joint>
+    </xacro:if>
     <!--%%%%%%%%%%%%% 2K Dispenser Definitions-->
     <link name="2K_Dispenser_Cartridge">
@@ -468,4 +470,8 @@
     <link name="2K_Dispenser_TCP">
     </link>
+    <!-- Init Definition of 2K Dispenser tip -->
+    <xacro:property name="dispenser_2K_configs_file" value="$(find pm_robot_description)/urdf/urdf_configs/2K_Dispenser_config.yaml" />
+    <xacro:property name="dispenser_2K_configs_dict" value="${xacro.load_yaml(dispenser_2K_configs_file)}"/>
+    <xacro:property name="Dispenser_2K_tip_z_offset" value="${dispenser_2K_configs_dict[current_pm_robot_2K_dipsenser_tip]['2K_dispencer_tcp_offset']}"/>
     <!-- Property names should not start with a number -->
     <xacro:property name="Dispenser_2K_TCP_Joint_Cal_x" value="${calibration_dict['2K_Dispenser_TCP_Joint']['x_offset']}"/>
@@ -479,5 +485,5 @@
         ${0 + Dispenser_2K_TCP_Joint_Cal_x * 0.000001}
         ${-0.045 + Dispenser_2K_TCP_Joint_Cal_y * 0.000001}
-        ${-0.04614 + Dispenser_2K_TCP_Joint_Cal_z * 0.000001}" rpy="
+        ${-0.04 + Dispenser_2K_TCP_Joint_Cal_z * 0.000001 - Dispenser_2K_tip_z_offset}" rpy="
         ${0 + Dispenser_2K_TCP_Joint_Cal_rx * 3.14159265359/180}
         ${0 + Dispenser_2K_TCP_Joint_Cal_ry * 3.14159265359/180}
@@ -487,4 +493,49 @@
       <axis xyz="0 0 0" />
     </joint>
+    <xacro:property name="Dispenser_2K_tip_xyz" value="${dispenser_2K_configs_dict[current_pm_robot_2K_dipsenser_tip]['xyz']}"/>
+    <xacro:property name="Dispenser_2K_tip_rpy" value="${dispenser_2K_configs_dict[current_pm_robot_2K_dipsenser_tip]['rpy']}"/>
+    <xacro:property name="Dispenser_2K_tip_mass" value="${dispenser_2K_configs_dict[current_pm_robot_2K_dipsenser_tip]['mass']}"/>
+    <xacro:property name="Dispenser_2K_tip_inertia_ixx" value="${dispenser_2K_configs_dict[current_pm_robot_2K_dipsenser_tip]['inertia_ixx']}"/>
+    <xacro:property name="Dispenser_2K_tip_inertia_ixy" value="${dispenser_2K_configs_dict[current_pm_robot_2K_dipsenser_tip]['inertia_ixy']}"/>
+    <xacro:property name="Dispenser_2K_tip_inertia_ixz" value="${dispenser_2K_configs_dict[current_pm_robot_2K_dipsenser_tip]['inertia_ixz']}"/>
+    <xacro:property name="Dispenser_2K_tip_inertia_iyy" value="${dispenser_2K_configs_dict[current_pm_robot_2K_dipsenser_tip]['inertia_iyy']}"/>
+    <xacro:property name="Dispenser_2K_tip_inertia_iyz" value="${dispenser_2K_configs_dict[current_pm_robot_2K_dipsenser_tip]['inertia_iyz']}"/>
+    <xacro:property name="Dispenser_2K_tip_inertia_izz" value="${dispenser_2K_configs_dict[current_pm_robot_2K_dipsenser_tip]['inertia_izz']}"/>
+    <xacro:property name="Dispenser_2K_tip_color" value="${dispenser_2K_configs_dict[current_pm_robot_2K_dipsenser_tip]['color']}"/>
+    <xacro:property name="Dispenser_2K_tip_visual_filename" value="${dispenser_2K_configs_dict[current_pm_robot_2K_dipsenser_tip]['visual_filename']}"/>
+    <xacro:property name="Dispenser_2K_tip_collision_filename" value="${dispenser_2K_configs_dict[current_pm_robot_2K_dipsenser_tip]['collision_filename']}"/>
+    <!--%%%%%%%%%%%%% The parameters here are interchangeable %%%%%%%%%%%%%-->
+    <xacro:if value="${current_pm_robot_2K_dipsenser_tip != 'empty'}">
+      <link name="2K_Dispenser_Tip">
+        <inertial>
+          <origin xyz="${Dispenser_2K_tip_xyz}" rpy="${Dispenser_2K_tip_rpy}"/>
+          <mass value="${Dispenser_2K_tip_mass}"/>
+          <inertia ixx="${Dispenser_2K_tip_inertia_ixx}" ixy="${Dispenser_2K_tip_inertia_ixy}" ixz="${Dispenser_2K_tip_inertia_ixz}" iyy="${Dispenser_2K_tip_inertia_iyy}" iyz="${Dispenser_2K_tip_inertia_iyz}" izz="${Dispenser_2K_tip_inertia_izz}" />
+        </inertial>
+        <visual>
+          <origin xyz="0 0 0" rpy="0 0 0" />
+          <geometry>
+            <mesh filename="file://$(find pm_robot_description)/meshes/Dispenser_Tips/${Dispenser_2K_tip_visual_filename}" />
+          </geometry>
+          <material name="${Dispenser_2K_tip_color}">
+          </material>
+        </visual>
+        <collision>
+          <origin xyz="0 0 0" rpy="0 0 0" />
+          <geometry>
+            <mesh filename="file://$(find pm_robot_description)/meshes/Dispenser_Tips/${Dispenser_2K_tip_collision_filename}" />
+          </geometry>
+        </collision>
+      </link>
+      <gazebo reference="2K_Dispenser_Tip">
+        <turnGravityOff>true</turnGravityOff>
+      </gazebo>
+      <joint name="2K_Dispenser_Tip_Joint" type="fixed">
+        <!-- This needs to be corrected in Solidworks -->
+        <origin xyz="0.0 0 0 " rpy="0 0 0" />
+        <parent link="2K_Dispenser_TCP" />
+        <child link="2K_Dispenser_Tip" />
+      </joint>
+    </xacro:if>
     <!--%%%%%%%%%%%%% Top Camera Definitions-->
     <link name="Cam1_Toolhead_TCP">

Commit message: distance sensor config + config checker

File: pm_robot_description/urdf/pm_robot.xacro (robot description, xacro)
@@ -29,4 +29,9 @@
     <xacro:property name="current_pm_robot_2K_dipsenser_tip" value="${current_pm_robot_bringup_config['pm_robot_2K_dispenser_tip']['use_dispenser_tip']}"/>
     <xacro:property name="current_vacuum_tool" value="${current_pm_robot_bringup_config['pm_robot_tools']['pm_robot_vacuum_tools']['use_tool']}"/>
+    <!-- The selected confocal head supplies both its geometry and its TCP offset. -->
+    <xacro:property name="distance_sensor_configs_file" value="$(find pm_robot_description)/urdf/urdf_configs/distance_sensors.yaml" />
+    <xacro:property name="distance_sensor_configs" value="${xacro.load_yaml(distance_sensor_configs_file)}"/>
+    <xacro:property name="current_confocal_sensor_head" value="${current_pm_robot_bringup_config['confocal_sensor_head']['use_config']}"/>
+    <xacro:property name="current_confocal_sensor_head_config" value="${distance_sensor_configs[current_confocal_sensor_head]}"/>
     <xacro:property name="calibration_dict" value="${xacro.load_yaml(pm_robot_joint_calibraion_file)}"/>
     <link name="world">
@@ -816,5 +821,5 @@
           <origin xyz="0 0 0" rpy="0 0 0" />
           <geometry>
-            <mesh filename="file://$(find pm_robot_description)/meshes/Confocal_Sensor_Top.STL" />
+            <mesh filename="file://$(find pm_robot_description)/meshes/distance_sensors/${current_confocal_sensor_head_config['visual_filename']}" />
           </geometry>
           <material name="">
@@ -825,5 +830,5 @@
           <origin xyz="0 0 0" rpy="0 0 0" />
           <geometry>
-            <mesh filename="file://$(find pm_robot_description)/meshes/Confocal_Sensor_Top_coll.STL" />
+            <mesh filename="file://$(find pm_robot_description)/meshes/distance_sensors/${current_confocal_sensor_head_config['collision_filename']}" />
           </geometry>
         </collision>
@@ -835,9 +840,12 @@
       <xacro:property name="Confocal_Sensor_Top_TCP_Joint_Cal_ry" value="${calibration_dict['Confocal_Sensor_Top_TCP_Joint']['ry_offset']}"/>
       <xacro:property name="Confocal_Sensor_Top_TCP_Joint_Cal_rz" value="${calibration_dict['Confocal_Sensor_Top_TCP_Joint']['rz_offset']}"/>
+      <xacro:property name="Confocal_Sensor_Head_Offset_x" value="${float(current_confocal_sensor_head_config['x'])}"/>
+      <xacro:property name="Confocal_Sensor_Head_Offset_y" value="${float(current_confocal_sensor_head_config['y'])}"/>
+      <xacro:property name="Confocal_Sensor_Head_Offset_z" value="${float(current_confocal_sensor_head_config['z'])}"/>
       <joint name="TCP_Confocal_Sensor_Top_Joint" type="fixed">
         <origin xyz="
-            ${0.176999957149375 + Confocal_Sensor_Top_TCP_Joint_Cal_x*0.000001}
-            ${-0.0580000000000008 + Confocal_Sensor_Top_TCP_Joint_Cal_y*0.000001}
-            ${-0.500500000000003 + Confocal_Sensor_Top_TCP_Joint_Cal_z*0.000001}"
+            ${0.148 + Confocal_Sensor_Head_Offset_x + Confocal_Sensor_Top_TCP_Joint_Cal_x*0.000001}
+            ${-0.074 + Confocal_Sensor_Head_Offset_y + Confocal_Sensor_Top_TCP_Joint_Cal_y*0.000001}
+            ${-0.4955 - Confocal_Sensor_Head_Offset_z + Confocal_Sensor_Top_TCP_Joint_Cal_z*0.000001}"
             rpy="
             ${0 + Confocal_Sensor_Top_TCP_Joint_Cal_rx*3.14159265359/180}
@@ -846,26 +854,4 @@
         <parent link="Z_Axis" />
         <child link="TCP_Confocal_Sensor_Top" />
-        <axis xyz="0 0 0" />
-      </joint>
-      <link
-        name="TCP_Confocal_Sensor_Top_2">
-      </link>
-      <xacro:property name="Confocal_Sensor_Top_TCP_2_Joint_Cal_x" value="${calibration_dict['Confocal_Sensor_Top_TCP_Joint']['x_offset']}"/>
-      <xacro:property name="Confocal_Sensor_Top_TCP_2_Joint_Cal_y" value="${calibration_dict['Confocal_Sensor_Top_TCP_Joint']['y_offset']}"/>
-      <xacro:property name="Confocal_Sensor_Top_TCP_2_Joint_Cal_z" value="${calibration_dict['Confocal_Sensor_Top_TCP_Joint']['z_offset']}"/>
-      <xacro:property name="Confocal_Sensor_Top_TCP_2_Joint_Cal_rx" value="${calibration_dict['Confocal_Sensor_Top_TCP_Joint']['rx_offset']}"/>
-      <xacro:property name="Confocal_Sensor_Top_TCP_2_Joint_Cal_ry" value="${calibration_dict['Confocal_Sensor_Top_TCP_Joint']['ry_offset']}"/>
-      <xacro:property name="Confocal_Sensor_Top_TCP_2_Joint_Cal_rz" value="${calibration_dict['Confocal_Sensor_Top_TCP_Joint']['rz_offset']}"/>
-      <joint name="TCP_Confocal_Sensor_Top_2_Joint" type="fixed">
-        <origin xyz="
-            ${0.147499957149374 + Confocal_Sensor_Top_TCP_2_Joint_Cal_x*0.000001}
-            ${-0.1065 + Confocal_Sensor_Top_TCP_2_Joint_Cal_y*0.000001}
-            ${-0.5025 + Confocal_Sensor_Top_TCP_2_Joint_Cal_z*0.000001}"
-            rpy="
-            ${0 + Confocal_Sensor_Top_TCP_2_Joint_Cal_rx*3.14159265359/180}
-            ${0 + Confocal_Sensor_Top_TCP_2_Joint_Cal_ry*3.14159265359/180}
-            ${0 + Confocal_Sensor_Top_TCP_2_Joint_Cal_rz*3.14159265359/180}" />
-        <parent link="Z_Axis" />
-        <child link="TCP_Confocal_Sensor_Top_2" />
         <axis xyz="0 0 0" />
       </joint>
