Commit message: smarpod fixes

File: pm_robot_description/urdf/pm_robot_gonio_right.xacro (robot description, xacro)
@@ -30,4 +30,10 @@
     <xacro:property name="gonio_right_configs_dict" value="${xacro.load_yaml(gonio_right_configs_file)}"/>
 <!--%%%%%%%%%%%%% Gonio_Right Definitions %%%%%%%%-->
+  <xacro:property name="gonio_offset_smarpod_x" value="0.0"/>
+  <xacro:property name="gonio_offset_smarpod_y" value="0.0"/>
+  <xacro:if value="${current_pm_robot_bringup_config['pm_smparpod_station']['with_smarpod_station']}">
+    <xacro:property name="gonio_offset_smarpod_x" value="0.0"/>
+    <xacro:property name="gonio_offset_smarpod_y" value="0.6"/>
+  </xacro:if>
   <link
     name="Gonio_Base_Right">
@@ -68,5 +74,5 @@
     type="fixed">
     <origin
-      xyz="0.750000000000003 0.31 0"
+      xyz="${0.750000000000003+gonio_offset_smarpod_x} ${0.31+gonio_offset_smarpod_y} 0"
       rpy="0 0 0" />
     <parent

File: pm_robot_description/urdf/pm_smarpod_station.xacro (robot description, xacro)
@@ -72,5 +72,5 @@
     type="fixed">
     <origin
-      xyz="0.750000000000003 0.31 0"
+      xyz="0.750000000000003 0.315 0"
       rpy="0 0 0" />
     <parent

Commit message: sensing jaws

File: pm_robot_description/urdf/pm_robot_gonio_right.xacro (robot description, xacro)
@@ -373,20 +373,22 @@
     </joint>
     <!--%%%%%%%%%%%%% Gonio Right Part 2 Origin -->
-    <link
-      name="Gonio_Right_Part_2_Origin">
-    </link>
-    <joint
-      name="Gonio_Right_Part_2_Origin_Joint"
-      type="fixed">
-      <origin
-        xyz="${gonio_chuck_tcp_offset_x_2} ${gonio_chuck_tcp_offset_y_2} ${gonio_chuck_tcp_offset_z_2}"
-        rpy="0 0 0" />
-      <parent
-        link="Gonio_Right_Chuck_Origin" />
-      <child
-        link="Gonio_Right_Part_2_Origin" />
-      <axis
-        xyz="0 0 0" />
-    </joint>
+    <xacro:if value="${gonio_chuck_tcp_offset_x_2 != 0.0 or gonio_chuck_tcp_offset_y_2 != 0.0 or gonio_chuck_tcp_offset_z_2 != 0.0}">
+      <link
+        name="Gonio_Right_Part_2_Origin">
+      </link>
+      <joint
+        name="Gonio_Right_Part_2_Origin_Joint"
+        type="fixed">
+        <origin
+          xyz="${gonio_chuck_tcp_offset_x_2} ${gonio_chuck_tcp_offset_y_2} ${gonio_chuck_tcp_offset_z_2}"
+          rpy="0 0 0" />
+        <parent
+          link="Gonio_Right_Chuck_Origin" />
+        <child
+          link="Gonio_Right_Part_2_Origin" />
+        <axis
+          xyz="0 0 0" />
+      </joint>
+    </xacro:if>
   </xacro:macro>
 </robot>
