Commit message: Tool_SPT_added

File: pm_robot_description/urdf/pm_robot_main.xacro (robot description, xacro)
@@ -3,20 +3,20 @@
   xmlns:xacro="https://ros.org/wiki/xacro">
   <!-- Configurations -->
-  <xacro:arg name="with_Tool_MPG_10"                default="false" />
-  <xacro:arg name="with_Tool_MPG_10_Jaw_3mm_Lens"   default="false"/>
   <xacro:arg name="with_Gonio_Left"                 default="false" />
   <xacro:arg name="with_Gonio_Right"                default="true" />
+    <!-- Tools -->
+    <xacro:arg name="with_Tool_MPG_10"                default="false" />
+    <xacro:arg name="with_Tool_MPG_10_Jaw_3mm_Lens"   default="false"/>
+    <xacro:arg name="with_Tool_SPT_Holder"            default="false" />
+    <xacro:arg name="with_SPT_R_A1000_I500"           default="false"/>
   <xacro:include filename="$(find pm_robot_description)/urdf/pm_robot.xacro" />
   <!-- Tool Defines-->
-    <!-- <xacro:if value="$(arg with_Tool_MPG_10)">
-      	<xacro:macro name="Gripper" params="gazebo:=false">
-          <xacro:arg name="with_Tool_MPG_10_Jaw_3mm_Lens" default="true" />
-          <xacro:include filename="$(find pm_robot_description)/urdf/pm_Schunk_Tools/MPG_10_plus.xacro" />
-      </xacro:macro>
-	    <xacro:Gripper gazebo="true" />
-    </xacro:if> -->
     <xacro:if value="$(arg with_Tool_MPG_10)">
       <xacro:include filename="$(find pm_robot_description)/urdf/pm_Schunk_Tools/MPG_10_plus.xacro" />
       <xacro:mpg_10_plus use_three_mm_lens="$(arg with_Tool_MPG_10_Jaw_3mm_Lens)" />
+    </xacro:if>
+    <xacro:if value="$(arg with_Tool_SPT_Holder)">
+      <xacro:include filename="$(find pm_robot_description)/urdf/pm_Schunk_Tools/SPT_Vacuumtool.xacro" />
+      <xacro:SPT_Vacuumtool use_R_A1000_I500="$(arg with_SPT_R_A1000_I500)" />
     </xacro:if>
     <!-- Gonio Right Defines-->

Commit message: Moveit + Gazebo working

File: pm_robot_description/urdf/pm_robot_main.xacro (robot description, xacro)
@@ -4,8 +4,5 @@
   <!-- Configurations -->
   <xacro:include filename="$(find pm_robot_description)/urdf/materials.xacro" />
-  <!-- <xacro:arg name="launch_mode"                default="fake_HW" /> -->
-  <!-- <xacro:arg name="launch_mode"                default="real_HW" /> -->
   <xacro:arg name="launch_mode"                     default="sim_HW" />
-  <!-- <xacro:arg name="launch_mode"                default="real_sim_HW" /> -->
   <xacro:arg name="initial_positions_file"          default="pm_robot_initial_positions.yaml" />
   <xacro:arg name="with_Gonio_Left"                 default="true" />

File: pm_robot_description/urdf/ros2_control_fake.xacro (robot description, xacro)
@@ -92,4 +92,18 @@
                 <state_interface name="position"/>
             </joint>
+            <xacro:if value="$(arg with_Tool_MPG_10)">
+                <joint name="Tool_Gripper_MPG_10_Jaw_1_Joint">
+                        <command_interface name="position">
+                        </command_interface>
+                        <state_interface name="position"/>
+                    </joint>
+                    <joint name="Tool_Gripper_MPG_10_Jaw_2_Joint">
+                        <param name="mimic">Tool_Gripper_MPG_10_Jaw_1_Joint</param>
+                        <param name="mulltiplier">1</param>
+                        <command_interface name="position">
+                        </command_interface>
+                        <state_interface name="position"/>
+                    </joint>
+            </xacro:if>
         </ros2_control>
     </xacro:macro>

File: pm_robot_moveit_config/config/pm_robot.urdf.xacro (robot description, xacro)
@@ -3,5 +3,5 @@
     <xacro:arg name="initial_positions_file" default="initial_positions.yaml" />
     <!-- Import pm_robot urdf file -->
-    <xacro:include filename="$(find pm_robot_description)/urdf/pm_robot_main_copy.xacro" />
+    <xacro:include filename="$(find pm_robot_description)/urdf/pm_robot_main.xacro" />
     <!-- Import control_xacro -->
     <xacro:include filename="pm_robot.ros2_control.xacro" />

Commit message: fix bugs in pm hardware interface
pm hardware interface can now successfully connect and interact
with the opcua server specified in ros2_control.xacro

File: pm_robot_description/urdf/pm_robot_main.xacro (robot description, xacro)
@@ -4,37 +4,37 @@
   <!-- Configurations -->
   <xacro:include filename="$(find pm_robot_description)/urdf/materials.xacro" />
-  <xacro:arg name="sim_mode"                 default="true" />
-  <xacro:arg name="with_Gonio_Left"                 default="true" />
-  <xacro:arg name="with_Gonio_Right"                default="true" />
-    <!-- Tools -->
-    <xacro:arg name="with_Tool_MPG_10"                default="false" />
-    <xacro:arg name="with_Tool_MPG_10_Jaw_3mm_Lens"   default="false"/>
-    <xacro:arg name="with_Tool_SPT_Holder"            default="false" />
-    <xacro:arg name="with_SPT_R_A1000_I500"           default="false"/>
+  <xacro:arg name="sim_mode" default="true" />
+  <xacro:arg name="with_Gonio_Left" default="true" />
+  <xacro:arg name="with_Gonio_Right" default="true" />
+  <!-- Tools -->
+  <xacro:arg name="with_Tool_MPG_10" default="false" />
+  <xacro:arg name="with_Tool_MPG_10_Jaw_3mm_Lens" default="false"/>
+  <xacro:arg name="with_Tool_SPT_Holder" default="false" />
+  <xacro:arg name="with_SPT_R_A1000_I500" default="false"/>
   <xacro:include filename="$(find pm_robot_description)/urdf/pm_robot.xacro" />
   <!-- Tool Defines-->
-    <xacro:if value="$(arg with_Tool_MPG_10)">
-      <xacro:include filename="$(find pm_robot_description)/urdf/pm_Schunk_Tools/MPG_10_plus.xacro" />
-      <xacro:mpg_10_plus use_three_mm_lens="$(arg with_Tool_MPG_10_Jaw_3mm_Lens)" />
-    </xacro:if>
-    <xacro:if value="$(arg with_Tool_SPT_Holder)">
-      <xacro:include filename="$(find pm_robot_description)/urdf/pm_Schunk_Tools/SPT_Vacuumtool.xacro" />
-      <xacro:SPT_Vacuumtool use_R_A1000_I500="$(arg with_SPT_R_A1000_I500)" />
-    </xacro:if>
-    <!-- Gonio Right Defines-->
-    <xacro:if value="$(arg with_Gonio_Right)">
-      <xacro:include filename="$(find pm_robot_description)/urdf/pm_robot_gonio_right.xacro" />
-    </xacro:if>
-    <!-- Gonio Right Defines-->
-    <xacro:if value="$(arg with_Gonio_Left)">
-      <xacro:include filename="$(find pm_robot_description)/urdf/pm_robot_gonio_left.xacro" />
-    </xacro:if>
+  <xacro:if value="$(arg with_Tool_MPG_10)">
+    <xacro:include filename="$(find pm_robot_description)/urdf/pm_Schunk_Tools/MPG_10_plus.xacro" />
+    <xacro:mpg_10_plus use_three_mm_lens="$(arg with_Tool_MPG_10_Jaw_3mm_Lens)" />
+  </xacro:if>
+  <xacro:if value="$(arg with_Tool_SPT_Holder)">
+    <xacro:include filename="$(find pm_robot_description)/urdf/pm_Schunk_Tools/SPT_Vacuumtool.xacro" />
+    <xacro:SPT_Vacuumtool use_R_A1000_I500="$(arg with_SPT_R_A1000_I500)" />
+  </xacro:if>
+  <!-- Gonio Right Defines-->
+  <xacro:if value="$(arg with_Gonio_Right)">
+    <xacro:include filename="$(find pm_robot_description)/urdf/pm_robot_gonio_right.xacro" />
+  </xacro:if>
+  <!-- Gonio Right Defines-->
+  <xacro:if value="$(arg with_Gonio_Left)">
+    <xacro:include filename="$(find pm_robot_description)/urdf/pm_robot_gonio_left.xacro" />
+  </xacro:if>
   <!-- Switch between Gazebo-Simulation and Real Robot -->
-    <xacro:if value="$(arg sim_mode)">
-      <xacro:include filename="$(find pm_robot_description)/urdf/ros2_control_gazebo.xacro" />
-    </xacro:if>
-    <xacro:unless value="$(arg sim_mode)">
-      <xacro:include filename="$(find pm_robot_description)/urdf/ros2_control.xacro" />
-    </xacro:unless>
+  <xacro:if value="$(arg sim_mode)">
+    <xacro:include filename="$(find pm_robot_description)/urdf/ros2_control_gazebo.xacro" />
+  </xacro:if>
+  <xacro:unless value="$(arg sim_mode)">
+    <xacro:include filename="$(find pm_robot_description)/urdf/ros2_control.xacro" />
+  </xacro:unless>
   <xacro:include filename="$(find pm_robot_description)/urdf/sensors.urdf" />
 </robot>

File: pm_robot_description/urdf/ros2_control.xacro (robot description, xacro)
@@ -6,4 +6,6 @@
             <!-- <plugin>gazebo_ros2_control/GazeboSystem</plugin> -->
             <plugin>pm_hardware_interface/PMSystem</plugin>
+            <param name="opcua_endpoint">opc.tcp://PC1M0484-1:4840</param>
+            <!-- <param name="opcua_endpoint">opc.tcp://localhost:4840</param> -->
         </hardware>
         <joint name="X_Axis_Joint">
@@ -31,5 +33,5 @@
             <state_interface name="velocity"/>
         </joint>
-        <joint name="1K_Dispenser_Flap_Joint">
+        <!-- <joint name="1K_Dispenser_Flap_Joint">
             <command_interface name="position">
             </command_interface>
@@ -102,12 +104,12 @@
             </command_interface>
             <state_interface name="position"/>
-        </joint>
+        </joint> -->
     </ros2_control>
     <gazebo>
         <plugin name="gazebo_ros2_control" filename="libgazebo_ros2_control.so">
             <parameters>$(find pm_robot_description)/config/pm_robot_control.yaml</parameters>
-            <parameters>$(find pm_robot_description)/config/pm_robot_control_gonio_right.yaml</parameters>
-            <parameters>$(find pm_robot_description)/config/pm_robot_control_gonio_left.yaml</parameters>
-            <parameters>$(find pm_robot_description)/config/pm_robot_control_gripper.yaml</parameters>
+            <!-- <parameters>$(find pm_robot_description)/config/pm_robot_control_gonio_right.yaml</parameters> -->
+            <!-- <parameters>$(find pm_robot_description)/config/pm_robot_control_gonio_left.yaml</parameters> -->
+            <!-- <parameters>$(find pm_robot_description)/config/pm_robot_control_gripper.yaml</parameters> -->
             <!--robot_param>robot_description</robot_param-->            <!--The location of the robot_description (URDF) on the parameter server, defaults to robot_description-->
             <!--robot_param_node>robot_state_publisher</robot_param_node-->            <!-- Name of the node where the robot_param is located, defauls to robot_state_publisher-->

Commit message: robot_bringup

File: pm_robot_description/urdf/pm_robot_main.xacro (robot description, xacro)
@@ -36,7 +36,7 @@
   <!-- Switch between Gazebo-Simulation and Real Robot -->
   <!-- Import control_xacro -->
-  <xacro:include filename="$(find pm_robot_description)/urdf/ros2_control_fake.xacro" />
-  <xacro:include filename="$(find pm_robot_description)/urdf/ros2_control_gazebo.xacro" />
-  <!-- <xacro:include filename="$(find pm_robot_description)/urdf/ros2_control_real.xacro" /> -->
+  <xacro:include filename="$(find pm_robot_description)/urdf/ros2_control_fake_HW.xacro" />
+  <xacro:include filename="$(find pm_robot_description)/urdf/ros2_control_sim_HW.xacro" />
+  <xacro:include filename="$(find pm_robot_description)/urdf/ros2_control_real_HW.xacro" />
   <xacro:property name="launch_mode" value="$(arg launch_mode)"/>
   <xacro:if value="${launch_mode == 'fake_HW'}">
@@ -44,5 +44,6 @@
   </xacro:if>
   <xacro:if value="${launch_mode == 'real_HW'}">
-    <xacro:pm_robot_ros2_control_hw_real name="Real_HW"/>
+    <xacro:pm_robot_ros2_control_hw_real name="Real_HW" initial_positions_file="$(arg initial_positions_file)"/>
+    <!-- <xacro:pm_robot_ros2_control_hw_sim name="Sim_HW"/> -->
   </xacro:if>
   <xacro:if value="${launch_mode == 'sim_HW'}">

File: pm_robot_description/urdf/ros2_control_real_HW.xacro (robot description, xacro)
@@ -1,9 +1,11 @@
 <?xml version="1.0"?>
 <robot xmlns:xacro="http://www.ros.org/wiki/xacro">
-    <xacro:macro name="pm_robot_ros2_control_hw_sim" params="name initial_positions_file">
+    <xacro:macro name="pm_robot_ros2_control_hw_real" params="name initial_positions_file">
         <xacro:property name="initial_positions" value="${load_yaml(initial_positions_file)['initial_positions']}"/>
-        <ros2_control name="GazeboSystem" type="system">
+        <ros2_control name="PMSystem" type="system">
             <hardware>
-                <plugin>gazebo_ros2_control/GazeboSystem</plugin>
+                <plugin>pm_hardware_interface/PMSystem</plugin>
+                <param name="opcua_endpoint">opc.tcp://PC1M0484-1:4840</param>
+                <!-- <param name="opcua_endpoint">opc.tcp://localhost:4840</param> -->
             </hardware>
             <joint name="X_Axis_Joint">
@@ -113,18 +115,4 @@
             </xacro:if>
         </ros2_control>
-            <gazebo>
-                <plugin name="gazebo_ros2_control" filename="libgazebo_ros2_control.so">
-                    <parameters>$(find pm_robot_description)/config/pm_robot_control_fakeHW.yaml</parameters>
-                    <parameters>$(find pm_robot_description)/config/pm_robot_control_gonio_right.yaml</parameters>
-                    <parameters>$(find pm_robot_description)/config/pm_robot_control_gonio_left.yaml</parameters>
-                    <xacro:if value="$(arg with_Tool_MPG_10)">
-                        <parameters>$(find pm_robot_description)/config/pm_robot_control_gripper.yaml</parameters>
-                    </xacro:if>
-                    <parameters>$(find pm_robot_description)/config/pm_robot_control_gazebo_param.yaml</parameters>
-                    <!--robot_param>robot_description</robot_param-->            <!--The location of the robot_description (URDF) on the parameter server, defaults to robot_description-->
-                    <!--robot_param_node>robot_state_publisher</robot_param_node-->            <!-- Name of the node where the robot_param is located, defauls to robot_state_publisher-->
-                    <!--robotNamespace>${arm_id}</robotNamespace-->
-                </plugin>
-            </gazebo>
     </xacro:macro>
 </robot>

File: pm_robot_description/urdf/ros2_control_sim_HW.xacro (robot description, xacro)
@@ -1,11 +1,10 @@
 <?xml version="1.0"?>
 <robot xmlns:xacro="http://www.ros.org/wiki/xacro">
-    <xacro:macro name="pm_robot_ros2_control_hw_real">
-        <ros2_control name="PMSystem" type="system">
+    <!-- <xacro:macro name="pm_robot_ros2_control_hw_sim" params="name initial_positions_file"> -->
+    <xacro:macro name="pm_robot_ros2_control_hw_sim">
+        <!-- <xacro:property name="initial_positions" value="${load_yaml(initial_positions_file)['initial_positions']}"/> -->
+        <ros2_control name="GazeboSystem" type="system">
             <hardware>
-                <!-- <plugin>gazebo_ros2_control/GazeboSystem</plugin> -->
-                <plugin>pm_hardware_interface/PMSystem</plugin>
-                <param name="opcua_endpoint">opc.tcp://PC1M0484-1:4840</param>
-                <!-- <param name="opcua_endpoint">opc.tcp://localhost:4840</param> -->
+                <plugin>gazebo_ros2_control/GazeboSystem</plugin>
             </hardware>
             <joint name="X_Axis_Joint">
@@ -105,5 +104,5 @@
                     <state_interface name="velocity"/>
                 </joint>
-                <joint name="pm_robot_Tool_Parallel_Joint_2">
+                <joint name="pm_robot_Tool_Parallel_Joint_mimic">
                     <param name="mimic">pm_robot_Tool_Parallel_Joint</param>
                     <param name="mulltiplier">1</param>
@@ -117,8 +116,10 @@
         <gazebo>
             <plugin name="gazebo_ros2_control" filename="libgazebo_ros2_control.so">
-                <parameters>$(find pm_robot_description)/config/pm_robot_control_realHW.yaml</parameters>
-                <parameters>$(find pm_robot_description)/config/pm_robot_control_gonio_right.yaml</parameters>
-                <parameters>$(find pm_robot_description)/config/pm_robot_control_gonio_left.yaml</parameters>
-                <parameters>$(find pm_robot_description)/config/pm_robot_control_gripper.yaml</parameters>
+                <parameters>$(find pm_robot_description)/config/pm_robot_control_sim_HW.yaml</parameters>
+                <parameters>$(find pm_robot_description)/config/pm_robot_control_gonio_right_sim_HW.yaml</parameters>
+                <parameters>$(find pm_robot_description)/config/pm_robot_control_gonio_left_sim_HW.yaml</parameters>
+                <xacro:if value="$(arg with_Tool_MPG_10)">
+                    <parameters>$(find pm_robot_description)/config/pm_robot_control_gripper_sim_HW.yaml</parameters>
+                </xacro:if>
                 <!--robot_param>robot_description</robot_param-->                <!--The location of the robot_description (URDF) on the parameter server, defaults to robot_description-->
                 <!--robot_param_node>robot_state_publisher</robot_param_node-->                <!-- Name of the node where the robot_param is located, defauls to robot_state_publisher-->

Commit message: Cameras activated

File: pm_robot_description/urdf/pm_robot_main.xacro (robot description, xacro)
@@ -33,5 +33,5 @@
     <xacro:include filename="$(find pm_robot_description)/urdf/pm_robot_gonio_left.xacro" />
   </xacro:if>
-  <!--xacro:include filename="$(find pm_robot_description)/urdf/sensors.urdf" /-->
+  <xacro:include filename="$(find pm_robot_description)/urdf/sensors.urdf" />
   <!-- Switch between Gazebo-Simulation and Real Robot -->
   <!-- Import control_xacro -->

File: pm_robot_description/urdf/sensors.urdf (robot description, URDF)
Before this commit: robot pm_robot, 5 links, 5 joints
Joints:
- joint Camera_Bottom_View_Joint: origin xyz=0.0645 0.287 -0.754 rpy=0 -1.570796 0  -> xyz=0.0 0 -0.754 rpy=0 -1.570796 0 ; parent Camera_System -> Camera_Station_TCP
- joint Camera_Top_View_Link_Joint: parent Camera_Top_View -> Cam1_Toolhead_TCP

Commit message: generation of unity_urdf

File: pm_robot_description/urdf/pm_robot_main.xacro (robot description, xacro)
@@ -91,7 +91,5 @@
   <xacro:include filename="$(find pm_robot_description)/urdf/ros2_control_real_HW.xacro" />
   <xacro:if value="${launch_mode == 'real_HW'}">
-    <xacro:pm_robot_ros2_control_hw_real name="Real_HW" initial_positions_file="$(arg initial_positions_file)"/>
-    <!-- <xacro:pm_robot_pneumatic_mock  />  -->
-    <!-- <xacro:pm_robot_ros2_control_hw_sim name="Sim_HW"/> -->
+    <xacro:pm_robot_ros2_control_hw_real name="Real_HW" initial_positions_file="$(arg initial_positions_file)" launch_mode="$(arg launch_mode)"/>
   </xacro:if>
   <xacro:if value="${launch_mode == 'sim_HW'}">

File: pm_robot_description/urdf/ros2_control_real_HW.xacro (robot description, xacro)
@@ -1,11 +1,18 @@
 <?xml version="1.0"?>
 <robot xmlns:xacro="http://www.ros.org/wiki/xacro">
-    <xacro:macro name="pm_robot_ros2_control_hw_real" params="name initial_positions_file">
+    <xacro:macro name="pm_robot_ros2_control_hw_real" params="name initial_positions_file launch_mode">
         <xacro:property name="initial_positions" value="${load_yaml(initial_positions_file)['initial_positions']}"/>
         <ros2_control name="PMSystem" type="system">
             <hardware>
                 <plugin>pm_hardware_interface/PMSystem</plugin>
-                <param name="opcua_endpoint">opc.tcp://PC1M0484-1:4840</param>
+                <!-- <param name="opcua_endpoint">opc.tcp://PC1M0484-1:4840</param> -->
                 <!-- <param name="opcua_endpoint">opc.tcp://localhost:4840</param> -->
+                <!-- Conditionally set the opcua_endpoint based on launch_mode -->
+                <xacro:if value="${launch_mode == 'sim_HW'}">
+                    <param name="opcua_endpoint">opc.tcp://PC1M0484-1:4840</param>
+                </xacro:if>
+                <xacro:if value="${launch_mode == 'real_HW'}">
+                    <param name="opcua_endpoint">opc.tcp://localhost:4840</param>
+                </xacro:if>
             </hardware>
             <joint name="X_Axis_Joint">

Commit message: launch with unity hw

File: pm_robot_description/urdf/pm_robot_main.xacro (robot description, xacro)
@@ -11,5 +11,7 @@
   <xacro:include filename="$(find pm_robot_description)/urdf/pm_Schunk_Tools/Schunk_Vacuum_Tools.xacro" />
   <xacro:arg name="launch_mode" default="sim_HW" />
+  <xacro:arg name="hardware" default="unity" />
   <xacro:property name="launch_mode" value="$(arg launch_mode)"/>
+  <xacro:property name="simulation" value="$(arg simulation)"/>
   <xacro:arg name="initial_positions_file" default="pm_robot_initial_positions.yaml" />
   <!-- <xacro:arg name="with_Gonio_Left" default="true" />
@@ -91,5 +93,5 @@
   <xacro:include filename="$(find pm_robot_description)/urdf/ros2_control_real_HW.xacro" />
   <xacro:if value="${launch_mode == 'real_HW'}">
-    <xacro:pm_robot_ros2_control_hw_real name="Real_HW" initial_positions_file="$(arg initial_positions_file)" launch_mode="$(arg launch_mode)"/>
+    <xacro:pm_robot_ros2_control_hw_real name="Real_HW" initial_positions_file="$(arg initial_positions_file)" launch_mode="$(arg launch_mode)" hardware="$(arg hardware)"/>
   </xacro:if>
   <xacro:if value="${launch_mode == 'sim_HW'}">

File: pm_robot_description/urdf/ros2_control_real_HW.xacro (robot description, xacro)
@@ -1,5 +1,5 @@
 <?xml version="1.0"?>
 <robot xmlns:xacro="http://www.ros.org/wiki/xacro">
-    <xacro:macro name="pm_robot_ros2_control_hw_real" params="name initial_positions_file launch_mode">
+    <xacro:macro name="pm_robot_ros2_control_hw_real" params="name initial_positions_file launch_mode hardware">
         <xacro:property name="initial_positions" value="${load_yaml(initial_positions_file)['initial_positions']}"/>
         <ros2_control name="PMSystem" type="system">
@@ -9,8 +9,8 @@
                 <!-- <param name="opcua_endpoint">opc.tcp://localhost:4840</param> -->
                 <!-- Conditionally set the opcua_endpoint based on launch_mode -->
-                <xacro:if value="${launch_mode == 'sim_HW'}">
+                <xacro:if value="${hardware == 'robot'}">
                     <param name="opcua_endpoint">opc.tcp://PC1M0484-1:4840</param>
                 </xacro:if>
-                <xacro:if value="${launch_mode == 'real_HW'}">
+                <xacro:if value="${hardware == 'unity'}">
                     <param name="opcua_endpoint">opc.tcp://localhost:4840</param>
                 </xacro:if>
