Commit message: bug fixes

File: pm_robot_description/urdf/pm_robot_main.xacro (robot description, xacro)
@@ -94,4 +94,5 @@
   <xacro:if value="${launch_mode == 'real_HW'}">
     <xacro:pm_robot_ros2_control_hw_real name="Real_HW" initial_positions_file="$(arg initial_positions_file)" launch_mode="$(arg launch_mode)" hardware="$(arg hardware)"/>
+    <xacro:pm_robot_pneumatic_mock_2 />
   </xacro:if>
   <xacro:if value="${launch_mode == 'sim_HW'}">

File: pm_robot_description/urdf/ros2_control_real_HW.xacro (robot description, xacro)
@@ -72,14 +72,4 @@
                 <state_interface name="velocity"/>
             </joint>
-            <joint name="UV_Slider_X_Front_Joint">
-                <command_interface name="position">
-                </command_interface>
-                <state_interface name="position"/>
-            </joint>
-            <joint name="UV_Slider_X_Back_Joint">
-                <command_interface name="position">
-                </command_interface>
-                <state_interface name="position"/>
-            </joint>
 <!--
             <joint name="1K_Dispenser_Protection_Joint">
@@ -150,9 +140,9 @@
         </ros2_control>
     </xacro:macro>
+<!--
     <xacro:macro name="pm_robot_pneumatic_mock" >
         <ros2_control name="PMSystemPneumatic" type="system">
             <hardware>
                 <plugin>mock_components/GenericSystem</plugin>
-                <!-- <param name="mock_sensor_commands">true</param> -->
             </hardware>
             <joint name="1K_Dispenser_Joint">
@@ -199,4 +189,26 @@
             </joint>
         </ros2_control>
+    </xacro:macro> -->
+    <xacro:macro name="pm_robot_pneumatic_mock_2" >
+        <ros2_control name="PMSystemPneumatic_2" type="system">
+            <hardware>
+                <plugin>mock_components/GenericSystem</plugin>
+                <!-- <param name="mock_sensor_commands">true</param> -->
+            </hardware>
+            <joint name="UV_Slider_X_Front_Joint">
+                <command_interface name="position">
+                </command_interface>
+                <state_interface name="position">
+                    <param name="initial_value">0.0</param>
+                </state_interface>
+            </joint>
+            <joint name="UV_Slider_X_Back_Joint">
+                <command_interface name="position">
+                </command_interface>
+                <state_interface name="position">
+                    <param name="initial_value">0.0</param>
+                </state_interface>
+            </joint>
+        </ros2_control>
     </xacro:macro>
 </robot>

Commit message: consistent bringup config

File: pm_robot_description/urdf/pm_robot_main.xacro (robot description, xacro)
@@ -13,4 +13,5 @@
   <xacro:arg name="hardware" default="unity" />
   <xacro:property name="launch_mode" value="$(arg launch_mode)"/>
+  <xacro:property name="hardware" value="$(arg hardware)"/>
   <xacro:property name="simulation" value="$(arg simulation)"/>
   <xacro:arg name="initial_positions_file" default="pm_robot_initial_positions.yaml" />
@@ -21,17 +22,14 @@
   <!-- START - Loading Config Files-->
     <!-- Loading of the Robot bringup config -->
-    <xacro:if value="${launch_mode == 'sim_HW'}">
+    <!-- hardware=='unity' uses local package config; hardware=='robot' (real hardware) uses the server path.-->
+    <xacro:if value="${launch_mode == 'sim_HW' or hardware == 'unity'}">
       <xacro:property name="pm_robot_bringup_config_file" value="$(find pm_robot_bringup)/config/pm_robot_bringup_config.yaml" />
     </xacro:if>
-    <!-- If launch_mode 'real' a local path can be specified for the calibration file -->
-    <xacro:if value="${launch_mode == 'real_HW'}">
+    <xacro:if value="${(launch_mode == 'real_HW' and hardware != 'unity') or hardware == 'robot'}">
         <xacro:property name="local_file_paths__file" value="$(find pm_robot_description)/calibration_config/pm_robot_path_real_HW.yaml" />
         <xacro:property name="path_dict" value="${xacro.load_yaml(local_file_paths__file)}"/>
         <xacro:property name="local_robot_bringup_file_path" value="${path_dict['pm_robot_bringup_config_file_path']}"/>
         <!-- REAL -->
-        <!-- <xacro:property name="pm_robot_joint_calibraion_file" value="${local_calibration_file_path}" />
-        <xacro:property name="pm_robot_bringup_config_file" value="${local_robot_bringup_file_path}"/> -->
-        <!-- SIM -->
-        <xacro:property name="pm_robot_bringup_config_file" value="$(find pm_robot_bringup)/config/pm_robot_bringup_config.yaml" />
+        <xacro:property name="pm_robot_bringup_config_file" value="${local_robot_bringup_file_path}"/>
       </xacro:if>
   <xacro:property name="current_pm_robot_bringup_config" value="${xacro.load_yaml(pm_robot_bringup_config_file)}"/>

File: pm_robot_description/urdf/pm_smarpod_station.xacro (robot description, xacro)
@@ -7,10 +7,10 @@
     <xacro:include filename="$(find smaract_hexapod_description)/urdf/smaract_hexapod_macro.xacro" />
     <!-- Loading of the Robot Joint calibrations -->
-    <xacro:if value="${launch_mode == 'sim_HW'}">
+    <!-- hardware=='unity' uses the local package config; hardware=='robot' (real hardware) uses the server paths. -->
+    <xacro:if value="${launch_mode == 'sim_HW' or hardware == 'unity'}">
       <xacro:property name="pm_robot_joint_calibraion_file" value="$(find pm_robot_description)/calibration_config/pm_robot_joint_calibration.yaml" />
       <xacro:property name="pm_robot_bringup_config_file" value="$(find pm_robot_bringup)/config/pm_robot_bringup_config.yaml" />
     </xacro:if>
-    <!-- If launch_mode 'real' a local path can be specified for the calibration file -->
-    <xacro:if value="${launch_mode == 'real_HW'}">
+    <xacro:if value="${(launch_mode == 'real_HW' and hardware != 'unity') or hardware == 'robot'}">
       <xacro:property name="local_file_paths__file" value="$(find pm_robot_description)/calibration_config/pm_robot_path_real_HW.yaml" />
       <xacro:property name="path_dict" value="${xacro.load_yaml(local_file_paths__file)}"/>
@@ -20,7 +20,4 @@
       <xacro:property name="pm_robot_joint_calibraion_file" value="${local_calibration_file_path}" />
       <xacro:property name="pm_robot_bringup_config_file" value="${local_robot_bringup_file_path}"/>
-      <!-- SIM -->
-      <!-- <xacro:property name="pm_robot_joint_calibraion_file" value="$(find pm_robot_description)/calibration_config/pm_robot_joint_calibration.yaml" />
-      <xacro:property name="pm_robot_bringup_config_file" value="$(find pm_robot_bringup)/config/pm_robot_bringup_config.yaml" /> -->
     </xacro:if>
     <xacro:property name="current_pm_robot_bringup_config" value="${xacro.load_yaml(pm_robot_bringup_config_file)}"/>

File: pm_robot_description/urdf/ros2_control_real_HW.xacro (robot description, xacro)
@@ -3,5 +3,10 @@
     <xacro:macro name="pm_robot_ros2_control_hw_real" params="name initial_positions_file launch_mode hardware">
         <xacro:property name="initial_positions" value="${load_yaml(initial_positions_file)['initial_positions']}"/>
-        <xacro:if value="${launch_mode == 'real_HW'}">
+        <!-- hardware=='unity' uses the local package config; hardware=='robot' (real hardware) uses the server paths. -->
+        <xacro:if value="${launch_mode == 'sim_HW' or hardware == 'unity'}">
+            <xacro:property name="pm_robot_joint_calibraion_file" value="$(find pm_robot_description)/calibration_config/pm_robot_joint_calibration.yaml" />
+            <xacro:property name="pm_robot_bringup_config_file" value="$(find pm_robot_bringup)/config/pm_robot_bringup_config.yaml" />
+        </xacro:if>
+        <xacro:if value="${(launch_mode == 'real_HW' and hardware != 'unity') or hardware == 'robot'}">
             <xacro:property name="local_file_paths__file" value="$(find pm_robot_description)/calibration_config/pm_robot_path_real_HW.yaml" />
             <xacro:property name="path_dict" value="${xacro.load_yaml(local_file_paths__file)}"/>
