Commit message: majer client rework

File: pm_robot_description/urdf/pm_robot_main.xacro (robot description, xacro)
@@ -93,5 +93,4 @@
     <xacro:pm_robot_ros2_control_hw_real name="Real_HW" initial_positions_file="$(arg initial_positions_file)" launch_mode="$(arg launch_mode)" hardware="$(arg hardware)"/>
     <xacro:pm_robot_pneumatic_mock_2 />
-    <xacro:pm_robot_gripper_mock />
   </xacro:if>
   <xacro:if value="${launch_mode == 'sim_HW'}">

File: pm_robot_description/urdf/pm_smarpod_station.xacro (robot description, xacro)
@@ -22,4 +22,10 @@
     </xacro:if>
     <xacro:property name="current_pm_robot_bringup_config" value="${xacro.load_yaml(pm_robot_bringup_config_file)}"/>
+    <!-- Real SmarPod is a separate hardware component from PMSystem. -->
+    <xacro:if value="${launch_mode == 'real_HW'}">
+      <xacro:include filename="$(find smaract_hexapod_description)/urdf/ros2_control.xacro" />
+      <xacro:smaract_hexapod_ros2_control_sim_hw launch_mode="${launch_mode}"
+        startup_pivot="${current_pm_robot_bringup_config['pm_smparpod_station'].get('startup_pivot', '0 0 0')}" />
+    </xacro:if>
     <xacro:property name="calibration_dict" value="${xacro.load_yaml(pm_robot_joint_calibraion_file)}"/>
     <xacro:property name="smarpod_chuck_calibration" value="${calibration_dict.get('Smarpod_Chuck', dict())}"/>

File: pm_robot_description/urdf/ros2_control_real_HW.xacro (robot description, xacro)
@@ -3,10 +3,5 @@
     <xacro:macro name="pm_robot_ros2_control_hw_real" params="name initial_positions_file launch_mode hardware">
         <xacro:property name="initial_positions" value="${load_yaml(initial_positions_file)['initial_positions']}"/>
-        <!-- hardware=='unity' uses the local package config; hardware=='robot' (real hardware) uses the server paths. -->
-        <xacro:if value="${launch_mode == 'sim_HW' or hardware == 'unity'}">
-            <xacro:property name="pm_robot_joint_calibraion_file" value="$(find pm_robot_description)/calibration_config/pm_robot_joint_calibration.yaml" />
-            <xacro:property name="pm_robot_bringup_config_file" value="$(find pm_robot_bringup)/config/pm_robot_bringup_config.yaml" />
-        </xacro:if>
-        <xacro:if value="${(launch_mode == 'real_HW' and hardware != 'unity') or hardware == 'robot'}">
+        <xacro:if value="${launch_mode == 'real_HW'}">
             <xacro:property name="local_file_paths__file" value="$(find pm_robot_description)/calibration_config/pm_robot_path_real_HW.yaml" />
             <xacro:property name="path_dict" value="${xacro.load_yaml(local_file_paths__file)}"/>
@@ -30,4 +25,9 @@
                     <param name="opcua_endpoint">opc.tcp://localhost:4840</param>
                 </xacro:if>
+                <!-- Keep slow auxiliary traffic off the 10 Hz motion path. -->
+                <param name="opcua_timeout_ms">1000</param>
+                <param name="auxiliary_io_poll_rate_hz">10</param>
+                <param name="auxiliary_sensor_poll_rate_hz">10</param>
+                <param name="auxiliary_lighting_poll_rate_hz">2</param>
             </hardware>
             <joint name="X_Axis_Joint">
@@ -114,120 +114,36 @@
                 </joint>
             </xacro:if>  -->
+            <!-- Only if gripper with two jaws is selected -->
+            <xacro:if value="${current_pm_robot_bringup_config['pm_robot_tools']['pm_robot_tool_parallel_gripper_2_jaws']['use_paralell_gripper']}">
+                <joint name="Tool_Parallel_Gripper_Jaw_1_Joint">
+                    <command_interface name="position">
+                    </command_interface>
+                    <state_interface name="position"/>
+                </joint>
+                <joint name="Tool_Parallel_Gripper_Jaw_2_Joint">
+                    <command_interface name="position">
+                    </command_interface>
+                    <state_interface name="position"/>
+                </joint>
+                <!-- <joint name="Tool_Parallel_Gripper_Jaw_2_Joint">
+                    <param name="mimic">Tool_Parallel_Gripper_Jaw_1_Joint</param>
+                    <param name="mulltiplier">1</param>
+                    <command_interface name="position">
+                    </command_interface>
+                    <state_interface name="position"/>
+                    <state_interface name="velocity"/>
+                </joint> -->
+            </xacro:if>
+            <!-- If parallel gripper with one jaw is selected -->
+            <xacro:if value="${current_pm_robot_bringup_config['pm_robot_tools']['pm_robot_tool_parallel_gripper_1_jaw']['use_paralell_gripper']}">
+                <joint name="Tool_Parallel_Gripper_Jaw_Joint">
+                    <command_interface name="position">
+                    </command_interface>
+                    <state_interface name="position"/>
+                </joint>
+            </xacro:if>
         </ros2_control>
-        <!-- SmarPod Hardware Interface -->
-        <xacro:if value="${current_pm_robot_bringup_config['pm_smparpod_station']['with_smarpod_station']}">
-            <ros2_control name="SmarPodSystem" type="system">
-                <hardware>
-                    <plugin>smaract_hexapod_hw_interface/SmarPodSystem</plugin>
-                    <param name="model_number">10006</param>
-                    <!-- The value of the starup pivot has been manually calibrated. it is the difference from the hexapod internal model to the kinematic model we created. we measured the top surface with the laser to make sure the pivot is at a certain point below the top surface. -->
-                    <!-- <param name="startup_pivot">0.0 0.0 -0.003812</param> -->
-                    <param name="startup_pivot">0.0 0.0 -0.003372</param>
-                    <!-- <param name="startup_pivot">0.0 0.0 -0.005282</param> -->
-                    <!-- Set the sensor mode. options: disabled, enabled, power_save -->
-                    <param name="sensor_mode">power_save</param>
-                    <!-- Set the maximum frequency of the sensor, this value should never exceed 12000 -->
-                    <param name="maximum_frequency">7000</param>
-                </hardware>
-                <!-- SmarPod Joint Definitions -->
-                <joint name="SP_X_Joint">
-                    <command_interface name="position"/>
-                    <state_interface name="position"/>
-                    <state_interface name="velocity"/>
-                </joint>
-                <joint name="SP_Y_Joint">
-                    <command_interface name="position"/>
-                    <state_interface name="position"/>
-                    <state_interface name="velocity"/>
-                </joint>
-                <joint name="SP_Z_Joint">
-                    <command_interface name="position"/>
-                    <state_interface name="position"/>
-                    <state_interface name="velocity"/>
-                </joint>
-                <joint name="SP_A_Joint">
-                    <command_interface name="position"/>
-                    <state_interface name="position"/>
-                    <state_interface name="velocity"/>
-                </joint>
-                <joint name="SP_B_Joint">
-                    <command_interface name="position"/>
-                    <state_interface name="position"/>
-                    <state_interface name="velocity"/>
-                </joint>
-                <joint name="SP_C_Joint">
-                    <command_interface name="position"/>
-                    <state_interface name="position"/>
-                    <state_interface name="velocity"/>
-                </joint>
-                <!-- SmarPod Stage Joints (State only) -->
-                <joint name="Smarpod_A_Stage_1_Joint">
-                    <state_interface name="position"/>
-                </joint>
-                <joint name="Smarpod_A_Stage_2_Joint">
-                    <state_interface name="position"/>
-                </joint>
-                <joint name="Smarpod_A_Stage_3_Joint">
-                    <state_interface name="position"/>
-                </joint>
-                <joint name="Smarpod_B_Stage_1_Joint">
-                    <state_interface name="position"/>
-                </joint>
-                <joint name="Smarpod_B_Stage_2_Joint">
-                    <state_interface name="position"/>
-                </joint>
-                <joint name="Smarpod_B_Stage_3_Joint">
-                    <state_interface name="position"/>
-                </joint>
-                <joint name="Smarpod_C_Stage_1_Joint">
-                    <state_interface name="position"/>
-                </joint>
-                <joint name="Smarpod_C_Stage_2_Joint">
-                    <state_interface name="position"/>
-                </joint>
-                <joint name="Smarpod_C_Stage_3_Joint">
-                    <state_interface name="position"/>
-                </joint>
-            </ros2_control>
-        </xacro:if>
     </xacro:macro>
-    <!-- Mock hardware for parallel gripper (separate from PMSystem) -->
-    <xacro:macro name="pm_robot_gripper_mock">
-        <xacro:if value="${current_pm_robot_bringup_config['pm_robot_tools']['pm_robot_tool_parallel_gripper_1_jaw']['use_paralell_gripper']}">
-            <ros2_control name="PMSystemGripper" type="system">
-                <hardware>
-                    <plugin>mock_components/GenericSystem</plugin>
-                </hardware>
-                <joint name="Tool_Parallel_Gripper_Jaw_Joint">
-                    <command_interface name="position">
-                    </command_interface>
-                    <state_interface name="position">
-                        <param name="initial_value">0.0</param>
-                    </state_interface>
-                </joint>
-            </ros2_control>
-        </xacro:if>
-        <xacro:if value="${current_pm_robot_bringup_config['pm_robot_tools']['pm_robot_tool_parallel_gripper_2_jaws']['use_paralell_gripper']}">
-            <ros2_control name="PMSystemGripper" type="system">
-                <hardware>
-                    <plugin>mock_components/GenericSystem</plugin>
-                </hardware>
-                <joint name="Tool_Parallel_Gripper_Jaw_1_Joint">
-                    <command_interface name="position">
-                    </command_interface>
-                    <state_interface name="position">
-                        <param name="initial_value">0.0</param>
-                    </state_interface>
-                </joint>
-                <joint name="Tool_Parallel_Gripper_Jaw_2_Joint">
-                    <command_interface name="position">
-                    </command_interface>
-                    <state_interface name="position">
-                        <param name="initial_value">0.0</param>
-                    </state_interface>
-                </joint>
-            </ros2_control>
-        </xacro:if>
-    </xacro:macro>
+<!--
     <xacro:macro name="pm_robot_pneumatic_mock" >
         <ros2_control name="PMSystemPneumatic" type="system">
@@ -278,5 +194,5 @@
             </joint>
         </ros2_control>
-    </xacro:macro>
+    </xacro:macro> -->
     <xacro:macro name="pm_robot_pneumatic_mock_2" >
         <ros2_control name="PMSystemPneumatic_2" type="system">
