Commit message: smarpod real hw added

File: pm_robot_description/urdf/pm_smarpod_station.xacro (robot description, xacro)
@@ -6,25 +6,22 @@
   <xacro:macro name="pm_smarpod_station" params="launch_mode">
     <xacro:include filename="$(find smaract_hexapod_description)/urdf/smaract_hexapod_macro.xacro" />
-    <!-- Loading of the Robot Joint calibrations -->
+      <!-- Loading of the Robot bringup config -->
     <xacro:if value="${launch_mode == 'sim_HW'}">
-      <xacro:property name="pm_robot_joint_calibraion_file" value="$(find pm_robot_description)/calibration_config/pm_robot_joint_calibration.yaml" />
       <xacro:property name="pm_robot_bringup_config_file" value="$(find pm_robot_bringup)/config/pm_robot_bringup_config.yaml" />
     </xacro:if>
     <!-- If launch_mode 'real' a local path can be specified for the calibration file -->
     <xacro:if value="${launch_mode == 'real_HW'}">
-      <xacro:property name="local_file_paths__file" value="$(find pm_robot_description)/calibration_config/pm_robot_path_real_HW.yaml" />
-      <xacro:property name="path_dict" value="${xacro.load_yaml(local_file_paths__file)}"/>
-      <xacro:property name="local_calibration_file_path" value="${path_dict['pm_robot_calibration_file_path']}"/>
-      <xacro:property name="local_robot_bringup_file_path" value="${path_dict['pm_robot_bringup_config_file_path']}"/>
-      <!-- REAL -->
-      <xacro:property name="pm_robot_joint_calibraion_file" value="${local_calibration_file_path}" />
-      <xacro:property name="pm_robot_bringup_config_file" value="${local_robot_bringup_file_path}"/>
-      <!-- SIM -->
-      <!-- <xacro:property name="pm_robot_joint_calibraion_file" value="$(find pm_robot_description)/calibration_config/pm_robot_joint_calibration.yaml" />
-      <xacro:property name="pm_robot_bringup_config_file" value="$(find pm_robot_bringup)/config/pm_robot_bringup_config.yaml" /> -->
-    </xacro:if>
+        <xacro:property name="local_file_paths__file" value="$(find pm_robot_description)/calibration_config/pm_robot_path_real_HW.yaml" />
+        <xacro:property name="path_dict" value="${xacro.load_yaml(local_file_paths__file)}"/>
+        <xacro:property name="local_robot_bringup_file_path" value="${path_dict['pm_robot_bringup_config_file_path']}"/>
+        <!-- REAL -->
+        <!-- <xacro:property name="pm_robot_joint_calibraion_file" value="${local_calibration_file_path}" />
+        <xacro:property name="pm_robot_bringup_config_file" value="${local_robot_bringup_file_path}"/> -->
+        <!-- SIM -->
+        <xacro:property name="pm_robot_bringup_config_file" value="$(find pm_robot_bringup)/config/pm_robot_bringup_config.yaml" />
+      </xacro:if>
     <xacro:property name="current_pm_robot_bringup_config" value="${xacro.load_yaml(pm_robot_bringup_config_file)}"/>
     <xacro:property name="calibration_dict" value="${xacro.load_yaml(pm_robot_joint_calibraion_file)}"/>
-    <xacro:smaract_hexapod launch_mode="$(arg launch_mode)" base_link="Smarpod_Station_Base" chuck="${current_pm_robot_bringup_config['pm_smparpod_station']['use_chuck']}"/>
+    <xacro:smaract_hexapod launch_mode="${launch_mode}" base_link="Smarpod_Station_Base" chuck="${current_pm_robot_bringup_config['pm_smparpod_station']['use_chuck']}"/>
     <!-- Smarpod Station -->
     <link

File: pm_robot_description/urdf/ros2_control_real_HW.xacro (robot description, xacro)
@@ -131,5 +131,5 @@
             </xacro:if>
             <!-- If parallel gripper with one jaw is selected -->
-            <!-- <xacro:if value="${current_pm_robot_bringup_config['pm_robot_tools']['pm_robot_tool_parallel_gripper_1_jaw']['use_paralell_gripper']}">
+            <xacro:if value="${current_pm_robot_bringup_config['pm_robot_tools']['pm_robot_tool_parallel_gripper_1_jaw']['use_paralell_gripper']}">
                 <joint name="Tool_Parallel_Gripper_Jaw_Joint">
                     <command_interface name="position">
@@ -137,6 +137,78 @@
                     <state_interface name="position"/>
                 </joint>
-            </xacro:if> -->
+            </xacro:if>
         </ros2_control>
+        <!-- SmarPod Hardware Interface -->
+        <xacro:if value="${current_pm_robot_bringup_config['pm_smparpod_station']['with_smarpod_station']}">
+            <ros2_control name="SmarPodSystem" type="system">
+                <hardware>
+                    <plugin>smaract_hexapod_hw_interface/SmarPodSystem</plugin>
+                    <param name="model_number">1011</param>
+                    <!-- Set the sensor mode. options: disabled, enabled, power_save -->
+                    <param name="sensor_mode">power_save</param>
+                    <!-- Set the maximum frequency of the sensor, this value should never exceed XXX -->
+                    <param name="maximum_frequency">17000</param>
+                </hardware>
+                <!-- SmarPod Joint Definitions -->
+                <joint name="SP_X_Joint">
+                    <command_interface name="position"/>
+                    <state_interface name="position"/>
+                    <state_interface name="velocity"/>
+                </joint>
+                <joint name="SP_Y_Joint">
+                    <command_interface name="position"/>
+                    <state_interface name="position"/>
+                    <state_interface name="velocity"/>
+                </joint>
+                <joint name="SP_Z_Joint">
+                    <command_interface name="position"/>
+                    <state_interface name="position"/>
+                    <state_interface name="velocity"/>
+                </joint>
+                <joint name="SP_A_Joint">
+                    <command_interface name="position"/>
+                    <state_interface name="position"/>
+                    <state_interface name="velocity"/>
+                </joint>
+                <joint name="SP_B_Joint">
+                    <command_interface name="position"/>
+                    <state_interface name="position"/>
+                    <state_interface name="velocity"/>
+                </joint>
+                <joint name="SP_C_Joint">
+                    <command_interface name="position"/>
+                    <state_interface name="position"/>
+                    <state_interface name="velocity"/>
+                </joint>
+                <!-- SmarPod Stage Joints (State only) -->
+                <joint name="Smarpod_A_Stage_1_Joint">
+                    <state_interface name="position"/>
+                </joint>
+                <joint name="Smarpod_A_Stage_2_Joint">
+                    <state_interface name="position"/>
+                </joint>
+                <joint name="Smarpod_A_Stage_3_Joint">
+                    <state_interface name="position"/>
+                </joint>
+                <joint name="Smarpod_B_Stage_1_Joint">
+                    <state_interface name="position"/>
+                </joint>
+                <joint name="Smarpod_B_Stage_2_Joint">
+                    <state_interface name="position"/>
+                </joint>
+                <joint name="Smarpod_B_Stage_3_Joint">
+                    <state_interface name="position"/>
+                </joint>
+                <joint name="Smarpod_C_Stage_1_Joint">
+                    <state_interface name="position"/>
+                </joint>
+                <joint name="Smarpod_C_Stage_2_Joint">
+                    <state_interface name="position"/>
+                </joint>
+                <joint name="Smarpod_C_Stage_3_Joint">
+                    <state_interface name="position"/>
+                </joint>
+            </ros2_control>
+        </xacro:if>
     </xacro:macro>
 <!--

Commit message: smarpod_calibration init

File: pm_robot_description/urdf/pm_smarpod_station.xacro (robot description, xacro)
@@ -81,10 +81,22 @@
     name="Smarpod_Station_Base">
   </link>
+  <xacro:property name="Smarpod_Station_Joint_Cal_x" value="${calibration_dict['Smarpod_Station']['x_offset']}"/>
+  <xacro:property name="Smarpod_Station_Joint_Cal_y" value="${calibration_dict['Smarpod_Station']['y_offset']}"/>
+  <xacro:property name="Smarpod_Station_Joint_Cal_z" value="${calibration_dict['Smarpod_Station']['z_offset']}"/>
+  <xacro:property name="Smarpod_Station_Joint_Cal_rx" value="${calibration_dict['Smarpod_Station']['rx_offset']}"/>
+  <xacro:property name="Smarpod_Station_Joint_Cal_ry" value="${calibration_dict['Smarpod_Station']['ry_offset']}"/>
+  <xacro:property name="Smarpod_Station_Joint_Cal_rz" value="${calibration_dict['Smarpod_Station']['rz_offset']}"/>
   <joint
     name="Smarpod_Station_Base_Joint"
     type="fixed">
     <origin
-      xyz="0.1465 0.1 0.2253999999992"
-      rpy="0 0 0" />
+      xyz="
+        ${0.1465 + Smarpod_Station_Joint_Cal_x * 0.000001}
+        ${0.1 + Smarpod_Station_Joint_Cal_y * 0.000001}
+        ${0.2254 + Smarpod_Station_Joint_Cal_z * 0.000001}"
+        rpy="
+        ${0 + Smarpod_Station_Joint_Cal_rx * 3.14159265359/180}
+        ${0 + Smarpod_Station_Joint_Cal_ry * 3.14159265359/180}
+        ${0 + Smarpod_Station_Joint_Cal_rz * 3.14159265359/180}" />
     <parent
       link="Smarpod_Station" />
