Commit message: smarpod calibration joint added

File: pm_robot_description/urdf/pm_smarpod_station.xacro (robot description, xacro)
@@ -79,4 +79,26 @@
   </joint>
   <link
+    name="Smarpod_Station_Base_Calibration">
+  </link>
+  <joint
+    name="Smarpod_Station_Base_Calibration_Joint"
+    type="fixed">
+    <origin
+      xyz="
+        0.1465
+        0.1
+        0.2254"
+        rpy="
+        0
+        0
+        0" />
+    <parent
+      link="Smarpod_Station" />
+    <child
+      link="Smarpod_Station_Base_Calibration" />
+    <axis
+      xyz="0 0 0" />
+  </joint>
+  <link
     name="Smarpod_Station_Base">
   </link>
@@ -92,7 +114,7 @@
     <origin
       xyz="
-        ${0.1465 + Smarpod_Station_Joint_Cal_x * 0.000001}
-        ${0.1 + Smarpod_Station_Joint_Cal_y * 0.000001}
-        ${0.2254 + Smarpod_Station_Joint_Cal_z * 0.000001}"
+        ${0.0 + Smarpod_Station_Joint_Cal_x * 0.000001}
+        ${0.0 + Smarpod_Station_Joint_Cal_y * 0.000001}
+        ${0.0 + Smarpod_Station_Joint_Cal_z * 0.000001}"
         rpy="
         ${0 + Smarpod_Station_Joint_Cal_rx * 3.14159265359/180}
@@ -100,5 +122,5 @@
         ${0 + Smarpod_Station_Joint_Cal_rz * 3.14159265359/180}" />
     <parent
-      link="Smarpod_Station" />
+      link="Smarpod_Station_Base_Calibration" />
     <child
       link="Smarpod_Station_Base" />

File: pm_robot_description/urdf/ros2_control_real_HW.xacro (robot description, xacro)
@@ -120,9 +120,9 @@
                 <hardware>
                     <plugin>smaract_hexapod_hw_interface/SmarPodSystem</plugin>
-                    <param name="model_number">1011</param>
+                    <param name="model_number">10006</param>
                     <!-- Set the sensor mode. options: disabled, enabled, power_save -->
                     <param name="sensor_mode">power_save</param>
-                    <!-- Set the maximum frequency of the sensor, this value should never exceed XXX -->
-                    <param name="maximum_frequency">17000</param>
+                    <!-- Set the maximum frequency of the sensor, this value should never exceed 12000 -->
+                    <param name="maximum_frequency">7000</param>
                 </hardware>
                 <!-- SmarPod Joint Definitions -->

Commit message: moveit server fix

File: pm_robot_description/urdf/pm_smarpod_station.xacro (robot description, xacro)
@@ -23,5 +23,23 @@
     <xacro:property name="current_pm_robot_bringup_config" value="${xacro.load_yaml(pm_robot_bringup_config_file)}"/>
     <xacro:property name="calibration_dict" value="${xacro.load_yaml(pm_robot_joint_calibraion_file)}"/>
-    <xacro:smaract_hexapod launch_mode="${launch_mode}" base_link="Smarpod_Station_Base" chuck="${current_pm_robot_bringup_config['pm_smparpod_station']['use_chuck']}" chuck_center="${current_pm_robot_bringup_config['pm_smparpod_station']['use_chuck_center']}"/>
+    <xacro:property name="smarpod_chuck_calibration" value="${calibration_dict.get('Smarpod_Chuck', dict())}"/>
+    <xacro:property name="smarpod_chuck_center_calibration" value="${calibration_dict.get('Smarpod_Chuck_Center', dict())}"/>
+    <xacro:smaract_hexapod
+      launch_mode="${launch_mode}"
+      base_link="Smarpod_Station_Base"
+      chuck="${current_pm_robot_bringup_config['pm_smparpod_station']['use_chuck']}"
+      chuck_center="${current_pm_robot_bringup_config['pm_smparpod_station']['use_chuck_center']}"
+      chuck_x_offset="${smarpod_chuck_calibration.get('x_offset', 0.0)}"
+      chuck_y_offset="${smarpod_chuck_calibration.get('y_offset', 0.0)}"
+      chuck_z_offset="${smarpod_chuck_calibration.get('z_offset', 0.0)}"
+      chuck_rx_offset="${smarpod_chuck_calibration.get('rx_offset', 0.0)}"
+      chuck_ry_offset="${smarpod_chuck_calibration.get('ry_offset', 0.0)}"
+      chuck_rz_offset="${smarpod_chuck_calibration.get('rz_offset', 0.0)}"
+      chuck_center_x_offset="${smarpod_chuck_center_calibration.get('x_offset', 0.0)}"
+      chuck_center_y_offset="${smarpod_chuck_center_calibration.get('y_offset', 0.0)}"
+      chuck_center_z_offset="${smarpod_chuck_center_calibration.get('z_offset', 0.0)}"
+      chuck_center_rx_offset="${smarpod_chuck_center_calibration.get('rx_offset', 0.0)}"
+      chuck_center_ry_offset="${smarpod_chuck_center_calibration.get('ry_offset', 0.0)}"
+      chuck_center_rz_offset="${smarpod_chuck_center_calibration.get('rz_offset', 0.0)}"/>
     <!-- Smarpod Station -->
     <link

File: pm_robot_description/urdf/ros2_control_real_HW.xacro (robot description, xacro)
@@ -122,5 +122,7 @@
                     <param name="model_number">10006</param>
                     <!-- The value of the starup pivot has been manually calibrated. it is the difference from the hexapod internal model to the kinematic model we created. we measured the top surface with the laser to make sure the pivot is at a certain point below the top surface. -->
-                    <param name="startup_pivot">0.0 0.0 -0.003812</param>
+                    <!-- <param name="startup_pivot">0.0 0.0 -0.003812</param> -->
+                    <param name="startup_pivot">0.0 0.0 -0.003372</param>
+                    <!-- <param name="startup_pivot">0.0 0.0 -0.005282</param> -->
                     <!-- Set the sensor mode. options: disabled, enabled, power_save -->
                     <param name="sensor_mode">power_save</param>
