Commit message: generate unity urdf

File: pm_robot_description/urdf/pm_robot_unity.urdf (robot description, URDF)
Before this commit: robot pm_robot, 159 links, 127 joints
Links:
- removed link 1K_Dispenser_Protection
- removed link 1K_Dispenser_Tip
- removed link 2K_Dispenser_Cartridge
- removed link Gonio_Left_Chuck
- removed link Gonio_Left_Stage_1_Top
- removed link Gonio_Left_Stage_2_Bottom
- removed link Gonio_Right_Chuck
- removed link Gonio_Right_Stage_1_Bottom
- removed link Gonio_Right_Stage_1_Top
- removed link Gonio_Right_Stage_2_Bottom
- removed link Laser_Toolhead_TCP
- removed link TCP_Confocal_Sensor_Bottom
- removed link TCP_Confocal_Sensor_Top
- removed link UV_LED_Back
- removed link UV_LED_Front
- removed link UV_Slider_X_Back
- removed link UV_Slider_X_Front
- removed link chuck_gonio_right_double_lens_holder_12_7
- removed link left_match_logo_font
- removed link t_axis_toolchanger
- added link Gonio_Left_Part_Origin__unity_source__Chuck_ASG_Dummy
- added link Gonio_Left_Part_Origin__unity_source__Chuck_Carrier_Demo
- added link Gonio_Left_Part_Origin__unity_source__Chuck_Siemens_Carrier_P39
- added link Gonio_Left_Part_Origin__unity_source__Chuck_Siemens_Carrier_P39_V2
- added link Gonio_Left_Part_Origin__unity_source__chuck_gonio_left_IPEG_Demonstrator
- added link Gonio_Left_Part_Origin__unity_source__chuck_gonio_left_Siemens_Carrier
- added link Gonio_Left_Part_Origin__unity_source__chuck_gonio_left_Siemens_Carrier_SIN
- added link Gonio_Left_Part_Origin__unity_source__chuck_gonio_left_Siemens_Sensor
- added link Gonio_Right_Chuck_ASG_Bruecke, mass 0.0856656121839983; collision mesh filename=meshes/Gonio_Right/Gonio_Right_Chucks/Gonio_Right_Chuck_ASG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; visual mesh filename=meshes/Gonio_Right/Gonio_Right_Chucks/Gonio_Right_Chuck_ASG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
- added link Gonio_Right_Part_1_Origin__unity_source__chuck_gonio_right_ASG_bridge
- added link Gonio_Right_Part_1_Origin__unity_source__chuck_gonio_right_Siemens_UFC
- added link Gonio_Right_Part_1_Origin__unity_source__chuck_gonio_right_double_lens_holder_12_7
- added link Gonio_Right_Part_1_Origin__unity_source__chuck_gonio_right_ipeg_active_alignment_station
- added link Gonio_Right_Part_1_Origin__unity_source__chuck_gonio_right_siemens_SIN
- added link Gonio_Right_Part_2_Origin__unity_source__chuck_gonio_right_double_lens_holder_12_7
Joints:
- removed joint Gonio_Right_Part_2_Origin_Joint_chuck_gonio_right_double_lens_holder_12_7
- added joint Gonio_Left_Part_Origin_Joint_unity_source_Chuck_ASG_Dummy: type fixed, parent Gonio_Left_Chuck_Origin, child Gonio_Left_Part_Origin__unity_source__Chuck_ASG_Dummy, origin xyz=0.0164 0.00859 0.1 rpy=0 0 0, axis 0 0 0
- added joint Gonio_Left_Part_Origin_Joint_unity_source_Chuck_Carrier_Demo: type fixed, parent Gonio_Left_Chuck_Origin, child Gonio_Left_Part_Origin__unity_source__Chuck_Carrier_Demo, origin xyz=0.1022 0.0107 0.0695 rpy=0 0 0, axis 0 0 0
- added joint Gonio_Left_Part_Origin_Joint_unity_source_Chuck_Siemens_Carrier_P39: type fixed, parent Gonio_Left_Chuck_Origin, child Gonio_Left_Part_Origin__unity_source__Chuck_Siemens_Carrier_P39, origin xyz=0.0301 0.0 0.0695 rpy=0 0 0, axis 0 0 0
- added joint Gonio_Left_Part_Origin_Joint_unity_source_Chuck_Siemens_Carrier_P39_V2: type fixed, parent Gonio_Left_Chuck_Origin, child Gonio_Left_Part_Origin__unity_source__Chuck_Siemens_Carrier_P39_V2, origin xyz=0.0301 0.0 0.069 rpy=0 0 0, axis 0 0 0
- added joint Gonio_Left_Part_Origin_Joint_unity_source_chuck_gonio_left_IPEG_Demonstrator: type fixed, parent Gonio_Left_Chuck_Origin, child Gonio_Left_Part_Origin__unity_source__chuck_gonio_left_IPEG_Demonstrator, origin xyz=0.01 0.015 0.10105 rpy=0 0 0, axis 0 0 0
- added joint Gonio_Left_Part_Origin_Joint_unity_source_chuck_gonio_left_Siemens_Carrier: type fixed, parent Gonio_Left_Chuck_Origin, child Gonio_Left_Part_Origin__unity_source__chuck_gonio_left_Siemens_Carrier, origin xyz=0.1022 0.0107 0.0695 rpy=0 0 0, axis 0 0 0
- added joint Gonio_Left_Part_Origin_Joint_unity_source_chuck_gonio_left_Siemens_Carrier_SIN: type fixed, parent Gonio_Left_Chuck_Origin, child Gonio_Left_Part_Origin__unity_source__chuck_gonio_left_Siemens_Carrier_SIN, origin xyz=0.1022 -0.0107 0.1055 rpy=0 0 0, axis 0 0 0
- added joint Gonio_Left_Part_Origin_Joint_unity_source_chuck_gonio_left_Siemens_Sensor: type fixed, parent Gonio_Left_Chuck_Origin, child Gonio_Left_Part_Origin__unity_source__chuck_gonio_left_Siemens_Sensor, origin xyz=0.0175 0.023 0.09655 rpy=0 0 0, axis 0 0 0
- added joint Gonio_Right_Part_1_Origin_Joint_unity_source_chuck_gonio_right_ASG_bridge: type fixed, parent Gonio_Right_Chuck_Origin, child Gonio_Right_Part_1_Origin__unity_source__chuck_gonio_right_ASG_bridge, origin xyz=0.04009 0.01093 0.038 rpy=0 0 0, axis 0 0 0
- added joint Gonio_Right_Part_1_Origin_Joint_unity_source_chuck_gonio_right_Siemens_UFC: type fixed, parent Gonio_Right_Chuck_Origin, child Gonio_Right_Part_1_Origin__unity_source__chuck_gonio_right_Siemens_UFC, origin xyz=0.0175 0.01025 0.0525 rpy=0 0 0, axis 0 0 0
- added joint Gonio_Right_Part_1_Origin_Joint_unity_source_chuck_gonio_right_double_lens_holder_12_7: type fixed, parent Gonio_Right_Chuck_Origin, child Gonio_Right_Part_1_Origin__unity_source__chuck_gonio_right_double_lens_holder_12_7, origin xyz=0.009782273 0.0 0.056053231 rpy=0 0 0, axis 0 0 0
- added joint Gonio_Right_Part_1_Origin_Joint_unity_source_chuck_gonio_right_ipeg_active_alignment_station: type fixed, parent Gonio_Right_Chuck_Origin, child Gonio_Right_Part_1_Origin__unity_source__chuck_gonio_right_ipeg_active_alignment_station, origin xyz=0.0035 0.1 0.0476 rpy=0 0 0, axis 0 0 0
- added joint Gonio_Right_Part_1_Origin_Joint_unity_source_chuck_gonio_right_siemens_SIN: type fixed, parent Gonio_Right_Chuck_Origin, child Gonio_Right_Part_1_Origin__unity_source__chuck_gonio_right_siemens_SIN, origin xyz=0.01774801 0.01093 0.054 rpy=0 0 0, axis 0 0 0
- added joint Gonio_Right_Part_2_Origin_Joint_unity_source_chuck_gonio_right_double_lens_holder_12_7: type fixed, parent Gonio_Right_Chuck_Origin, child Gonio_Right_Part_2_Origin__unity_source__chuck_gonio_right_double_lens_holder_12_7, origin xyz=-0.009782273 0.0 0.056053231 rpy=0 0 0, axis 0 0 0
- joint 1K_Dispenser_Protection_Joint: child 1K_Dispenser_Protection -> Glue_Cartridge_Flap
- joint 1K_Dispenser_Tip_Joint: child 1K_Dispenser_Tip -> Dis_Tip_Red_I_250_A520_L12700
- joint 2K_Dispenser_Joint: child 2K_Dispenser_Cartridge -> 2K_Glue_Cartridge
- joint 2K_Dispenser_TCP_Joint: parent 2K_Dispenser_Cartridge -> 2K_Glue_Cartridge
- joint Gonio_Left_Chuck_Joint: child Gonio_Left_Chuck -> Chuck_Carrier_Demo
- joint Gonio_Left_Chuck_Origin_Joint: parent Gonio_Left_Stage_2_Bottom -> Gonio_Left_Stage_2
- joint Gonio_Left_Part_Origin_Joint: origin xyz=0.0301 0.0 0.069 rpy=0 0 0 -> xyz=0.0164 0.00859 0.1 rpy=0 0 0
- joint Gonio_Left_Stage_1_Joint: child Gonio_Left_Stage_1_Top -> Gonio_Left_Stage_1
- joint Gonio_Left_Stage_2_Joint: child Gonio_Left_Stage_2_Bottom -> Gonio_Left_Stage_2; parent Gonio_Left_Stage_1_Top -> Gonio_Left_Stage_1
- joint Gonio_Right_Chuck_Joint: child Gonio_Right_Chuck -> Gonio_Right_Chuck_ASG_Bruecke
- joint Gonio_Right_Chuck_Origin_Joint: parent Gonio_Right_Stage_2_Bottom -> Gonio_Right_Stage_2_Upper
- joint Gonio_Right_Part_1_Origin_Joint: origin xyz=0.0035 0.1 0.0476 rpy=0 0 0 -> xyz=0.04009 0.01093 0.038 rpy=0 0 0
- joint Gonio_Right_Stage_1_Bottom_Joint: child Gonio_Right_Stage_1_Bottom -> Gonio_Right_Stage_1
- joint Gonio_Right_Stage_1_Joint: child Gonio_Right_Stage_1_Top -> Gonio_Right_Stage_1_Upper; parent Gonio_Right_Stage_1_Bottom -> Gonio_Right_Stage_1
- joint Gonio_Right_Stage_2_Joint: child Gonio_Right_Stage_2_Bottom -> Gonio_Right_Stage_2_Upper; parent Gonio_Right_Stage_1_Top -> Gonio_Right_Stage_1_Upper
- joint Laser_Toolhead_TCP_Joint: child Laser_Toolhead_TCP -> Laser_Kopf_TCP
- joint PM_Robot_Tool_TCP_Joint_Schunk_MPG_20_plus_Jaw_ASG_Gripper: origin xyz=       0.0        0.0        -0.04542 rpy=       0.0        0.0        0.0 -> xyz=       0.0        0.0        -0.08843000000000001 rpy=       0.0        0.0        0.0
- joint TCP_Confocal_Sensor_Bottom_Joint: child TCP_Confocal_Sensor_Bottom -> Confocal_Sensor_Bottom
- joint TCP_Confocal_Sensor_Top_Joint: child TCP_Confocal_Sensor_Top -> Confocal_Sensor_Top
- joint Tool_Parallel_Gripper_Body_Joint_Schunk_MPG_10_plus_Jaw_3mm_Lens: parent t_axis_toolchanger -> Gripper_Rot_Plate
- joint Tool_Parallel_Gripper_Body_Joint_Schunk_MPG_20_plus_Jaw_ASG_Gripper: parent t_axis_toolchanger -> Gripper_Rot_Plate
- joint Tool_Parallel_Gripper_Body_Joint_SmarAct_Piezo_Gripper_Default_Jaw: parent t_axis_toolchanger -> Gripper_Rot_Plate
- joint Tool_Parallel_Gripper_Body_Joint_SmarAct_Piezo_Gripper_flat_Default_Jaw: parent t_axis_toolchanger -> Gripper_Rot_Plate
- joint Tool_Parallel_Gripper_Body_Joint_SmarAct_Piezo_Gripper_flat_Flat_Jaw: parent t_axis_toolchanger -> Gripper_Rot_Plate
- joint Tool_Parallel_Gripper_Body_Joint_SmarAct_Piezo_Gripper_flat_Sensing_Jaw: parent t_axis_toolchanger -> Gripper_Rot_Plate
- joint UV_LED_Back_Joint: child UV_LED_Back -> UV_Cart_Back; parent UV_Slider_X_Back -> UV_Cart_X_Back
- joint UV_LED_Front_Joint: child UV_LED_Front -> UV_Cart_Front; parent UV_Slider_X_Front -> UV_Cart_X_Front
- joint UV_Slider_X_Back_Joint: child UV_Slider_X_Back -> UV_Cart_X_Back
- joint UV_Slider_X_Front_Joint: child UV_Slider_X_Front -> UV_Cart_X_Front
- joint left_match_logo_font_joint: child left_match_logo_font -> match_font
- joint t_axis_toolchanger_joint: child t_axis_toolchanger -> t_axis_tool

Commit message: generate urdf fix

File: pm_robot_description/urdf/pm_robot_unity.urdf (robot description, URDF)
Before this commit: robot pm_robot, 154 links, 140 joints
Links:
- added link Dis_Tip_Lavender_I_150_A310_L12700_2K, mass 0.00266749600701752; collision mesh filename=meshes/Dispenser_Tips/Dis_Tip_Lavender_I_150_A310_L12700.STL; visual mesh filename=meshes/Dispenser_Tips/Dis_Tip_Lavender_I_150_A310_L12700.STL
- added link Dis_Tip_Red_I_250_A520_L12700_2K, mass 0.00266749600701752; collision mesh filename=meshes/Dispenser_Tips/Dis_Tip_Red_I_250_A520_L12700.STL; visual mesh filename=meshes/Dispenser_Tips/Dis_Tip_Red_I_250_A520_L12700.STL
- added link Dis_Tip_Yellow_I_100_A240_L12700_2K, mass 0.00266749600701752; collision mesh filename=meshes/Dispenser_Tips/Dis_Tip_Yellow_I_100_A240_L12700.STL; visual mesh filename=meshes/Dispenser_Tips/Dis_Tip_Yellow_I_100_A240_L12700.STL
Joints:
- added joint 2K_Dispenser_Tip_Joint: type fixed, parent 2K_Dispenser_TCP, child Dis_Tip_Red_I_250_A520_L12700_2K, origin xyz=0.0 0 0  rpy=0 0 0
- joint 1K_Dispenser_TCP_Joint: origin xyz=         -0.001          -0.0318          -0.11800000000000001 rpy=         0.0          0.0          0.0 -> xyz=         -0.001         -0.0318         -0.127 rpy=         0.0         0.0         0.0
- joint 2K_Dispenser_TCP_Joint: origin xyz=         0.0          -0.045          -0.04614 rpy=         0.0          0.0          0.0 -> xyz=         0.0         -0.045         -0.057 rpy=         0.0         0.0         0.0
- joint Cam1_Toolhead_TCP_Joint: origin xyz=         -0.0320000000000003          -0.0579999999999998          -0.517313246516092 rpy=         0.0          0.0          0.0 -> xyz=         -0.0320000000000003          -0.0579999999999998          -0.517313247 rpy=         0.0          0.0          0.0
- joint Gonio_Left_Chuck_Origin_Joint: origin xyz=         0.0          0.0          -0.015 rpy=         0.0          0.0          0.0 -> xyz=         0.0          0.0          -0.004999999999999999 rpy=         0.0          0.0          0.0
- joint PM_Robot_Tool_TCP_Joint_Schunk_MPG_20_plus_Jaw_ASG_Gripper: origin xyz=       0.0        0.0        -0.08843000000000001 rpy=       0.0        0.0        0.0 -> xyz=       0.0        0.0        -0.07843 rpy=       0.0        0.0        1.5707963267950003
