Commit message: materials

File: pm_robot_description/urdf/pm_Schunk_Tools/SPT_Vacuumtool.xacro (robot description, xacro)
@@ -17,7 +17,5 @@
                     <mesh filename="file://$(find pm_robot_description)/meshes/Tools/SPT_Vacuumtools/Tool_Schunk_base_link.STL" />
                 </geometry>
-                <material name="">
-                    <color rgba="0.75294 0.75294 0.75294 1" />
-                </material>
+                <material name="orange"/>
             </visual>
             <collision>
@@ -62,7 +60,5 @@
                         <mesh filename="file://$(find pm_robot_description)/meshes/Tools/SPT_Vacuumtools/Tools/Tool_TCP_SPT_R_A1000_I500.STL" />
                     </geometry>
-                    <material name="">
-                        <color rgba="0.79216 0.81961 0.93333 1" />
-                    </material>
+                    <material name="grey"/>
                 </visual>
                 <collision>

File: pm_robot_description/urdf/pm_robot.xacro (robot description, xacro)
@@ -29,7 +29,5 @@
         <mesh filename="file://$(find pm_robot_description)/meshes/base_link.STL" />
       </geometry>
-      <material name="">
-        <color rgba="0.792156862745098 0.819607843137255 0.933333333333333 1" />
-      </material>
+      <material name="grey"/>
     </visual>
     <collision>
@@ -52,4 +50,5 @@
         <mesh filename="file://$(find pm_robot_description)/meshes/X_Axis.STL" />
       </geometry>
+      <material name="orange"/>
     </visual>
     <collision>
@@ -79,4 +78,5 @@
         <mesh filename="file://$(find pm_robot_description)/meshes/Y_Axis.STL" />
       </geometry>
+      <material name="brown"/>
     </visual>
     <collision>
@@ -106,4 +106,5 @@
         <mesh filename="file://$(find pm_robot_description)/meshes/Z_Axis.STL" />
       </geometry>
+      <material name="blue"/>
     </visual>
     <collision>
@@ -137,4 +138,5 @@
         <mesh filename="file://$(find pm_robot_description)/meshes/Gripper_Rot_Plate.STL" />
       </geometry>
+      <material name="black"/>
     </visual>
     <collision>
@@ -197,4 +199,5 @@
         <mesh filename="file://$(find pm_robot_description)/meshes/1K_Dispenser_Flap.STL" />
       </geometry>
+      <material name="white"/>
     </visual>
     <collision>
@@ -228,4 +231,5 @@
         <mesh filename="file://$(find pm_robot_description)/meshes/1K_Dispenser.STL" />
       </geometry>
+      <material name="red"/>
     </visual>
     <collision>
@@ -259,4 +263,5 @@
         <mesh filename="file://$(find pm_robot_description)/meshes/2K_Dispenser.STL" />
       </geometry>
+      <material name="orange"/>
     </visual>
     <collision>
@@ -290,4 +295,5 @@
         <mesh filename="file://$(find pm_robot_description)/meshes/Camera_Top_View.STL" />
       </geometry>
+      <material name="white"/>
     </visual>
     <collision>
@@ -320,4 +326,5 @@
         <mesh filename="file://$(find pm_robot_description)/meshes/Test_Station.STL" />
       </geometry>
+      <material name="grey"/>
     </visual>
     <collision>
@@ -374,4 +381,5 @@
         <mesh filename="file://$(find pm_robot_description)/meshes/Camera_System.STL" />
       </geometry>
+      <material name="white"/>
     </visual>
     <collision>
@@ -400,4 +408,5 @@
         <mesh filename="file://$(find pm_robot_description)/meshes/Camera_Calibration.STL" />
       </geometry>
+      <material name="green"/>
     </visual>
     <collision>

File: pm_robot_description/urdf/pm_robot_main.xacro (robot description, xacro)
@@ -3,4 +3,5 @@
   xmlns:xacro="https://ros.org/wiki/xacro">
   <!-- Configurations -->
+  <xacro:include filename="$(find pm_robot_description)/urdf/materials.xacro" />
   <xacro:arg name="with_Gonio_Left"                 default="true" />
   <xacro:arg name="with_Gonio_Right"                default="true" />

Commit message: small changes

File: pm_robot_description/urdf/pm_Schunk_Tools/SPT_Vacuumtool.xacro (robot description, xacro)
@@ -32,5 +32,6 @@
         </gazebo>
         <joint name="Tool_Schunk_SPT_Toolholder_joint" type="fixed">
-            <origin xyz="0 0 -0.06" rpy="0 0 0" />
+            <!-- <origin xyz="0 0 -0.06" rpy="0 0 0" /> -->
+            <origin xyz="0 0 -0.03" rpy="0 0 0" />
             <parent link="Gripper_Rot_Plate" />
             <child link="Tool_Schunk_SPT_Toolholder" />

File: pm_robot_description/urdf/pm_robot.xacro (robot description, xacro)
@@ -64,5 +64,5 @@
     <child link="X_Axis" />
     <axis xyz="-1 0 0" />
-    <limit lower="-0.745" upper="0.055" effort="0.1" velocity="100" />
+    <limit lower="-0.745" upper="0.055" effort="0.1" velocity="35" />
   </joint>
  <!--%%%%%%%%%%%%% Y Axis Definitions %%%%%%%%%%%%%-->
@@ -92,5 +92,5 @@
     <child link="Y_Axis" />
     <axis xyz="0 -1 0" />
-    <limit lower="-0.134000" upper="-0.019700" effort="100" velocity="100" />
+    <limit lower="-0.134000" upper="-0.019700" effort="100" velocity="35" />
   </joint>
  <!--%%%%%%%%%%%%% Z Axis Definitions %%%%%%%%%%%%%-->
@@ -124,5 +124,5 @@
     <child link="Z_Axis" />
     <axis xyz="0 0 -1" />
-    <limit lower="-0.05262" upper="0.055" effort="100" velocity="0.05" />
+    <limit lower="-0.05262" upper="0.055" effort="100" velocity="35" />
   </joint>
    <!--%%%%%%%%%%%%% T Axis Definitions %%%%%%%%%%%%%-->
@@ -156,6 +156,15 @@
     <child link="Gripper_Rot_Plate" />
     <axis xyz="0 0 1" />
-    <limit lower="0" upper="12" effort="100" velocity="2" />
-  </joint>
+    <limit lower="0" upper="12" effort="100" velocity="5" />
+  </joint>
+  <link
+      name="PM_Robot_TCP">
+    </link>
+    <joint name="PM_Robot_TCP_Joint" type="fixed">
+        <origin xyz="0 0 -0.1" rpy="0 0 0" />
+        <parent link="Gripper_Rot_Plate" />
+        <child link="PM_Robot_TCP" />
+        <axis xyz="0 0 0" />
+    </joint>
   <!--
   Gripper Definitions
