Commit message: changeable Jaws & Moveit Gripper fix

File: pm_robot_description/urdf/pm_Schunk_Tools/MPG_10_plus.xacro (robot description, xacro)
@@ -113,5 +113,5 @@
       lower="0"
       upper="0.001"
-      effort="100"
+      effort="20"
       velocity="0.05" />
   </joint>
@@ -177,5 +177,5 @@
     </gazebo>
   <joint
-    name="pm_robot_Tool_Parallel_Joint_mimic"
+    name="pm_robot_Tool_Parallel_Joint_2"
     type="prismatic">
     <origin
@@ -191,135 +191,184 @@
         lower="0"
         upper="0.001"
-        effort="100"
+        effort="20"
         velocity="0.05" />
-  </joint>
+    <mimic joint="pm_robot_Tool_Parallel_Joint" />
+  </joint>
+  <link
+    name="Tool_Gripper_MPG_10_Jaw_2_Point">
+  </link>
+  <joint
+    name="Tool_Gripper_MPG_10_Jaw_2_Point_Joint"
+    type="fixed">
+    <origin
+      xyz="0 0.0014 -0.0075"
+      rpy="0 0 0" />
+    <parent
+      link="Tool_Gripper_MPG_10_Jaw_2" />
+    <child
+      link="Tool_Gripper_MPG_10_Jaw_2_Point" />
+    <axis
+      xyz="0 0 0" />
+  </joint>
+  <!--%%%%%%%%%%%%% Jaw Definitions %%%%%%%%%%%%%-->
+    <xacro:property name="mpg_10_plus_jaw_define_file" value="$(find pm_robot_description)/urdf/pm_Schunk_Tools/MPG_10_plus_jaws.yaml" />
+    <xacro:property name="jaw_dict" value="${xacro.load_yaml(mpg_10_plus_jaw_define_file)}"/>
+    <!--%%%%%%%%%%%%% Default Jaw Definitions %%%%%%%%%%%%%-->
+    <xacro:property name="Gripper_jaw_1_xyz" value="${jaw_dict['lens_jaw_3_mm_1']['xyz']}"/>
+    <xacro:property name="Gripper_jaw_1_rpy" value="${jaw_dict['lens_jaw_3_mm_1']['rpy']}"/>
+    <xacro:property name="Gripper_jaw_1_mass" value="${jaw_dict['lens_jaw_3_mm_1']['mass']}"/>
+    <xacro:property name="Gripper_jaw_1_inertia_ixx" value="${jaw_dict['lens_jaw_3_mm_1']['inertia_ixx']}"/>
+    <xacro:property name="Gripper_jaw_1_inertia_ixy" value="${jaw_dict['lens_jaw_3_mm_1']['inertia_ixy']}"/>
+    <xacro:property name="Gripper_jaw_1_inertia_ixz" value="${jaw_dict['lens_jaw_3_mm_1']['inertia_ixz']}"/>
+    <xacro:property name="Gripper_jaw_1_inertia_iyy" value="${jaw_dict['lens_jaw_3_mm_1']['inertia_iyy']}"/>
+    <xacro:property name="Gripper_jaw_1_inertia_iyz" value="${jaw_dict['lens_jaw_3_mm_1']['inertia_iyz']}"/>
+    <xacro:property name="Gripper_jaw_1_inertia_izz" value="${jaw_dict['lens_jaw_3_mm_1']['inertia_izz']}"/>
+    <xacro:property name="Gripper_jaw_1_visual_filename" value="${jaw_dict['lens_jaw_3_mm_1']['visual_filename']}"/>
+    <xacro:property name="Gripper_jaw_1_collision_filename" value="${jaw_dict['lens_jaw_3_mm_1']['collision_filename']}"/>
+    <xacro:property name="Gripper_jaw_2_xyz" value="${jaw_dict['lens_jaw_3_mm_2']['xyz']}"/>
+    <xacro:property name="Gripper_jaw_2_rpy" value="${jaw_dict['lens_jaw_3_mm_2']['rpy']}"/>
+    <xacro:property name="Gripper_jaw_2_mass" value="${jaw_dict['lens_jaw_3_mm_2']['mass']}"/>
+    <xacro:property name="Gripper_jaw_2_inertia_ixx" value="${jaw_dict['lens_jaw_3_mm_2']['inertia_ixx']}"/>
+    <xacro:property name="Gripper_jaw_2_inertia_ixy" value="${jaw_dict['lens_jaw_3_mm_2']['inertia_ixy']}"/>
+    <xacro:property name="Gripper_jaw_2_inertia_ixz" value="${jaw_dict['lens_jaw_3_mm_2']['inertia_ixz']}"/>
+    <xacro:property name="Gripper_jaw_2_inertia_iyy" value="${jaw_dict['lens_jaw_3_mm_2']['inertia_iyy']}"/>
+    <xacro:property name="Gripper_jaw_2_inertia_iyz" value="${jaw_dict['lens_jaw_3_mm_2']['inertia_iyz']}"/>
+    <xacro:property name="Gripper_jaw_2_inertia_izz" value="${jaw_dict['lens_jaw_3_mm_2']['inertia_izz']}"/>
+    <xacro:property name="Gripper_jaw_2_visual_filename" value="${jaw_dict['lens_jaw_3_mm_2']['visual_filename']}"/>
+    <xacro:property name="Gripper_jaw_2_collision_filename" value="${jaw_dict['lens_jaw_3_mm_2']['collision_filename']}"/>
+    <!--%%%%%%%%%%%%% 3MM Lens Jaw 1 Definitions %%%%%%%%%%%%%-->
+    <xacro:if value="${use_three_mm_lens}">
+      <xacro:property name="Gripper_jaw_1_xyz" value="${jaw_dict['lens_jaw_3_mm_1']['xyz']}"/>
+      <xacro:property name="Gripper_jaw_1_rpy" value="${jaw_dict['lens_jaw_3_mm_1']['rpy']}"/>
+      <xacro:property name="Gripper_jaw_1_mass" value="${jaw_dict['lens_jaw_3_mm_1']['mass']}"/>
+      <xacro:property name="Gripper_jaw_1_inertia_ixx" value="${jaw_dict['lens_jaw_3_mm_1']['inertia_ixx']}"/>
+      <xacro:property name="Gripper_jaw_1_inertia_ixy" value="${jaw_dict['lens_jaw_3_mm_1']['inertia_ixy']}"/>
+      <xacro:property name="Gripper_jaw_1_inertia_ixz" value="${jaw_dict['lens_jaw_3_mm_1']['inertia_ixz']}"/>
+      <xacro:property name="Gripper_jaw_1_inertia_iyy" value="${jaw_dict['lens_jaw_3_mm_1']['inertia_iyy']}"/>
+      <xacro:property name="Gripper_jaw_1_inertia_iyz" value="${jaw_dict['lens_jaw_3_mm_1']['inertia_iyz']}"/>
+      <xacro:property name="Gripper_jaw_1_inertia_izz" value="${jaw_dict['lens_jaw_3_mm_1']['inertia_izz']}"/>
+      <xacro:property name="Gripper_jaw_1_visual_filename" value="${jaw_dict['lens_jaw_3_mm_1']['visual_filename']}"/>
+      <xacro:property name="Gripper_jaw_1_collision_filename" value="${jaw_dict['lens_jaw_3_mm_1']['collision_filename']}"/>
+      <xacro:property name="Gripper_jaw_2_xyz" value="${jaw_dict['lens_jaw_3_mm_2']['xyz']}"/>
+      <xacro:property name="Gripper_jaw_2_rpy" value="${jaw_dict['lens_jaw_3_mm_2']['rpy']}"/>
+      <xacro:property name="Gripper_jaw_2_mass" value="${jaw_dict['lens_jaw_3_mm_2']['mass']}"/>
+      <xacro:property name="Gripper_jaw_2_inertia_ixx" value="${jaw_dict['lens_jaw_3_mm_2']['inertia_ixx']}"/>
+      <xacro:property name="Gripper_jaw_2_inertia_ixy" value="${jaw_dict['lens_jaw_3_mm_2']['inertia_ixy']}"/>
+      <xacro:property name="Gripper_jaw_2_inertia_ixz" value="${jaw_dict['lens_jaw_3_mm_2']['inertia_ixz']}"/>
+      <xacro:property name="Gripper_jaw_2_inertia_iyy" value="${jaw_dict['lens_jaw_3_mm_2']['inertia_iyy']}"/>
+      <xacro:property name="Gripper_jaw_2_inertia_iyz" value="${jaw_dict['lens_jaw_3_mm_2']['inertia_iyz']}"/>
+      <xacro:property name="Gripper_jaw_2_inertia_izz" value="${jaw_dict['lens_jaw_3_mm_2']['inertia_izz']}"/>
+      <xacro:property name="Gripper_jaw_2_visual_filename" value="${jaw_dict['lens_jaw_3_mm_2']['visual_filename']}"/>
+      <xacro:property name="Gripper_jaw_2_collision_filename" value="${jaw_dict['lens_jaw_3_mm_2']['collision_filename']}"/>
+    </xacro:if>
+    <!--%%%%%%%%%%%%% The parameters here are interchangeable %%%%%%%%%%%%%-->
+    <!--%%%%%%%%%%%%% Jaw 1 Definitions %%%%%%%%%%%%%-->
     <link
-      name="Tool_Gripper_MPG_10_Jaw_2_Point">
+      name="Tool_Gripper_MPG_10_Jaw_1_changeable">
+      <inertial>
+        <origin
+          xyz="${Gripper_jaw_1_xyz}"
+          rpy="${Gripper_jaw_1_rpy}"/>
+        <mass
+          value="${Gripper_jaw_1_mass}"/>
+        <inertia
+          ixx="${Gripper_jaw_1_inertia_ixx}"
+          ixy="${Gripper_jaw_1_inertia_ixy}"
+          ixz="${Gripper_jaw_1_inertia_ixz}"
+          iyy="${Gripper_jaw_1_inertia_iyy}"
+          iyz="${Gripper_jaw_1_inertia_iyz}"
+          izz="${Gripper_jaw_1_inertia_izz}" />
+      </inertial>
+      <visual>
+        <origin
+          xyz="0 0 0"
+          rpy="0 0 0" />
+        <geometry>
+          <mesh filename="file://$(find pm_robot_description)/meshes/Tools/MPG_10_plus/Jaws/${Gripper_jaw_1_visual_filename}" />
+        </geometry>
+        <material
+          name="">
+          <color
+            rgba="0.780392156862745 0.76078431372549 0.741176470588235 1" />
+        </material>
+      </visual>
+      <collision>
+        <origin
+          xyz="0 0 0"
+          rpy="0 0 0" />
+        <geometry>
+          <mesh filename="file://$(find pm_robot_description)/meshes/Tools/MPG_10_plus/Jaws/${Gripper_jaw_1_visual_filename}" />
+        </geometry>
+      </collision>
     </link>
+    <gazebo reference="Tool_Gripper_Jaw_1">
+      <turnGravityOff>true</turnGravityOff>
+    </gazebo>
     <joint
-      name="Tool_Gripper_MPG_10_Jaw_2_Point_Joint"
+      name="Tool_Gripper_MPG_10_Jaw_1_changeable_Joint"
       type="fixed">
-      <origin
-        xyz="0 0.0014 -0.0075"
+      <!-- This needs to be corrected in Solidworks -->
+      <origin
+        xyz="0.002 0 0 "
         rpy="0 0 0" />
       <parent
-        link="Tool_Gripper_MPG_10_Jaw_2" />
+        link="Tool_Gripper_MPG_10_Jaw_1_Point" />
       <child
+        link="Tool_Gripper_MPG_10_Jaw_1_changeable" />
+    </joint>
+    <!--%%%%%%%%%%%%% Jaw 2 Definitions %%%%%%%%%%%%%-->
+    <link
+      name="Tool_Gripper_MPG_10_Jaw_2_changeable">
+      <inertial>
+        <origin
+          xyz="${Gripper_jaw_2_xyz}"
+          rpy="${Gripper_jaw_2_rpy}"/>
+        <mass
+          value="${Gripper_jaw_2_mass}"/>
+        <inertia
+          ixx="${Gripper_jaw_2_inertia_ixx}"
+          ixy="${Gripper_jaw_2_inertia_ixy}"
+          ixz="${Gripper_jaw_2_inertia_ixz}"
+          iyy="${Gripper_jaw_2_inertia_iyy}"
+          iyz="${Gripper_jaw_2_inertia_iyz}"
+          izz="${Gripper_jaw_2_inertia_izz}" />
+      </inertial>
+      <visual>
+        <origin
+          xyz="0 0 0"
+          rpy="0 0 0" />
+        <geometry>
+          <mesh filename="file://$(find pm_robot_description)/meshes/Tools/MPG_10_plus/Jaws/${Gripper_jaw_2_visual_filename}" />
+        </geometry>
+        <material
+          name="">
+          <color
+            rgba="0.780392156862745 0.76078431372549 0.741176470588235 1" />
+        </material>
+      </visual>
+      <collision>
+        <origin
+          xyz="0 0 0"
+          rpy="0 0 0" />
+        <geometry>
+          <mesh filename="file://$(find pm_robot_description)/meshes/Tools/MPG_10_plus/Jaws/${Gripper_jaw_2_visual_filename}" />
+        </geometry>
+      </collision>
+    </link>
+    <gazebo reference="Tool_Gripper_MPG_10_Jaw_2_changeable">
+      <turnGravityOff>true</turnGravityOff>
+    </gazebo>
+    <joint
+      name="Tool_Gripper_MPG_10_Jaw_2_changeable_Joint"
+      type="fixed">
+      <!-- This needs to be corrected in Solidworks -->
+      <origin
+        xyz="0.002 0  0 "
+        rpy="1.5708 0 0" />
+      <parent
         link="Tool_Gripper_MPG_10_Jaw_2_Point" />
-      <axis
-        xyz="0 0 0" />
+      <child
+        link="Tool_Gripper_MPG_10_Jaw_2_changeable" />
     </joint>
-    <!-- <xacro:property name="with_Tool_MPG_10_Jaw_3mm_Lens" value="true" /> -->
-  <!--%%%%%%%%%%%%% Jaw Definitions %%%%%%%%%%%%%-->
-    <xacro:if value="${use_three_mm_lens}">
-      <!--%%%%%%%%%%%%% 3MM Lens Jaw 1 Definitions %%%%%%%%%%%%%-->
-        <link
-          name="Tool_Gripper_Jaw_1_3MM_Lens">
-          <inertial>
-            <origin
-              xyz="-0.00222703440519818 -1.24600850470724E-13 -0.0015303266892263"
-              rpy="0 0 0" />
-            <mass
-              value="0.000118476289547731" />
-            <inertia
-              ixx="5.50616566102928E-10"
-              ixy="1.15823081964001E-21"
-              ixz="1.51586534634799E-10"
-              iyy="6.62228324828861E-10"
-              iyz="2.68654227697881E-20"
-              izz="4.05699592387869E-10" />
-          </inertial>
-          <visual>
-            <origin
-              xyz="0 0 0"
-              rpy="0 0 0" />
-            <geometry>
-              <mesh
-              filename="file://$(find pm_robot_description)/meshes/Tools/MPG_10_plus/Jaws/Gripper_Jaw_1_3MM_Lens_for_MPG_10.STL" />
-            </geometry>
-            <material
-              name="">
-              <color
-                rgba="0.780392156862745 0.76078431372549 0.741176470588235 1" />
-            </material>
-          </visual>
-          <collision>
-            <origin
-              xyz="0 0 0"
-              rpy="0 0 0" />
-            <geometry>
-              <mesh
-              filename="file://$(find pm_robot_description)/meshes/Tools/MPG_10_plus/Jaws/Gripper_Jaw_1_3MM_Lens_for_MPG_10.STL" />           </geometry>
-          </collision>
-        </link>
-        <gazebo reference="Tool_Gripper_Jaw_1_3MM_Lens">
-          <turnGravityOff>true</turnGravityOff>
-        </gazebo>
-        <joint
-          name="Tool_Gripper_Jaw_1_3MM_Lens_Joint"
-          type="fixed">
-          <origin
-            xyz="0 0 0"
-            rpy="0 0 0" />
-          <parent
-            link="Tool_Gripper_MPG_10_Jaw_1_Point" />
-          <child
-            link="Tool_Gripper_Jaw_1_3MM_Lens" />
-        </joint>
-      <!--%%%%%%%%%%%%% 3MM Lens Jaw 2 Definitions %%%%%%%%%%%%%-->
-        <link
-          name="Tool_Gripper_Jaw_2_3MM_Lens">
-          <inertial>
-            <origin
-              xyz="-0.00224080580616211 -0.00152543365786503 1.2528765306995E-13"
-              rpy="0 0 0" />
-            <mass
-              value="0.000117826998616915" />
-            <inertia
-              ixx="5.504084274466E-10"
-              ixy="1.50894936754082E-10"
-              ixz="-1.43349001887448E-21"
-              iyy="4.00144751949544E-10"
-              iyz="-2.68169098626193E-20"
-              izz="6.58370363267184E-10" />
-          </inertial>
-          <visual>
-            <origin
-              xyz="0 0 0"
-              rpy="0 0 0" />
-            <geometry>
-              <mesh
-              filename="file://$(find pm_robot_description)/meshes/Tools/MPG_10_plus/Jaws/Gripper_Jaw_2_3MM_Lens_for_MPG_10.STL" />
-            </geometry>
-            <material
-              name="">
-              <color
-                rgba="0.780392156862745 0.76078431372549 0.741176470588235 1" />
-            </material>
-          </visual>
-          <collision>
-            <origin
-              xyz="0 0 0"
-              rpy="0 0 0" />
-            <geometry>
-              <mesh
-              filename="file://$(find pm_robot_description)/meshes/Tools/MPG_10_plus/Jaws/Gripper_Jaw_2_3MM_Lens_for_MPG_10.STL" />           </geometry>
-          </collision>
-        </link>
-        <gazebo reference="Tool_Gripper_Jaw_2_3MM_Lens">
-          <turnGravityOff>true</turnGravityOff>
-        </gazebo>
-        <joint
-          name="Tool_Gripper_Jaw_2_3MM_Lens_Joint"
-          type="fixed">
-          <origin
-            xyz="0 0 0"
-            rpy="1.5708 0 0" />
-          <parent
-            link="Tool_Gripper_MPG_10_Jaw_2_Point" />
-          <child
-            link="Tool_Gripper_Jaw_2_3MM_Lens" />
-        </joint>
-    </xacro:if>
-  </xacro:macro>
+</xacro:macro>
 </robot>

File: pm_robot_description/urdf/pm_Schunk_Tools/SPT_Vacuumtool.xacro (robot description, xacro)
@@ -65,5 +65,5 @@
         <xacro:if value="${use_R_A1000_I500}">
             <!--%%%%%%%%%%%% Tool_TCP_SPT_R_A1000_I500 %%%%%%%%%%%%%-->
-            <link name="Tool_SPT_TCP_link">
+            <link name="Tool_SPT_changeable">
                 <inertial>
                     <origin
@@ -97,12 +97,12 @@
             </link>
             <!--Gravity off-->
-            <gazebo reference="Tool_SPT_TCP_link">
+            <gazebo reference="Tool_SPT_changeable">
                 <turnGravityOff>true</turnGravityOff>
                 <color>1.0 0 0.5 1.0</color>
             </gazebo>
-            <joint name="Tool_SPT_TCP_link_joint" type="fixed">
+            <joint name="Tool_SPT_changeable_joint" type="fixed">
                 <origin xyz="0 0 0" rpy="0 0 0" />
                 <parent link="PM_Robot_Tool_TCP" />
-                <child link="Tool_SPT_TCP_link" />
+                <child link="Tool_SPT_changeable" />
                 <axis xyz="0 0 0" />
             </joint>

File: pm_robot_description/urdf/ros2_control_gazebo.xacro (robot description, xacro)
@@ -101,4 +101,5 @@
                     </command_interface>
                     <state_interface name="position"/>
+                    <state_interface name="velocity"/>
                 </joint>
                 <joint name="pm_robot_Tool_Parallel_Joint_mimic">
@@ -108,4 +109,5 @@
                     </command_interface>
                     <state_interface name="position"/>
+                    <state_interface name="velocity"/>
                 </joint>
             </xacro:if>

File: pm_robot_description/urdf/ros2_control_real.xacro (robot description, xacro)
@@ -103,15 +103,17 @@
             <xacro:if value="$(arg with_Tool_MPG_10)">
                 <joint name="pm_robot_Tool_Parallel_Joint">
-                        <command_interface name="position">
-                        </command_interface>
-                        <state_interface name="position"/>
-                    </joint>
-                    <joint name="pm_robot_Tool_Parallel_Joint_mimic">
-                        <param name="mimic">pm_robot_Tool_Parallel_Joint</param>
-                        <param name="mulltiplier">1</param>
-                        <command_interface name="position">
-                        </command_interface>
-                        <state_interface name="position"/>
-                    </joint>
+                    <command_interface name="position">
+                    </command_interface>
+                    <state_interface name="position"/>
+                    <state_interface name="velocity"/>
+                </joint>
+                <joint name="pm_robot_Tool_Parallel_Joint_2">
+                    <param name="mimic">pm_robot_Tool_Parallel_Joint</param>
+                    <param name="mulltiplier">1</param>
+                    <command_interface name="position">
+                    </command_interface>
+                    <state_interface name="position"/>
+                    <state_interface name="velocity"/>
+                </joint>
             </xacro:if>
         </ros2_control>
