Commit message: robot calibration

File: pm_robot_description/urdf/pm_Schunk_Tools/Schunk_Vacuum_Tools.xacro (robot description, xacro)
@@ -62,4 +62,24 @@
     <xacro:property name="pm_robot_tool_TCP_y_offset" value="${vacuum_tool_holder_configs_dict['tool_TCP_y_offset']}"/>
     <xacro:property name="pm_robot_tool_TCP_x_offset" value="${vacuum_tool_holder_configs_dict['tool_TCP_x_offset']}"/>
+  <link name="PM_Robot_Tool_TCP">
+  </link>
+  <xacro:property name="PM_Robot_Tool_TCP_Joint_Cal_x" value="${calibration_dict['PM_Robot_Tool_TCP_Joint']['x_offset']}"/>
+  <xacro:property name="PM_Robot_Tool_TCP_Joint_Cal_y" value="${calibration_dict['PM_Robot_Tool_TCP_Joint']['y_offset']}"/>
+  <xacro:property name="PM_Robot_Tool_TCP_Joint_Cal_z" value="${calibration_dict['PM_Robot_Tool_TCP_Joint']['z_offset']}"/>
+  <xacro:property name="PM_Robot_Tool_TCP_Joint_Cal_rx" value="${calibration_dict['PM_Robot_Tool_TCP_Joint']['rx_offset']}"/>
+  <xacro:property name="PM_Robot_Tool_TCP_Joint_Cal_ry" value="${calibration_dict['PM_Robot_Tool_TCP_Joint']['ry_offset']}"/>
+  <xacro:property name="PM_Robot_Tool_TCP_Joint_Cal_rz" value="${calibration_dict['PM_Robot_Tool_TCP_Joint']['rz_offset']}"/>
+  <joint name="PM_Robot_Tool_TCP_Joint" type="fixed">
+    <origin xyz="
+      ${0 + pm_robot_tool_TCP_x_offset + PM_Robot_Tool_TCP_Joint_Cal_x * 0.000001}
+      ${0 + pm_robot_tool_TCP_y_offset + PM_Robot_Tool_TCP_Joint_Cal_y * 0.000001}
+      ${0 - 0.04542 - pm_robot_tool_TCP_z_offset + PM_Robot_Tool_TCP_Joint_Cal_z * 0.000001}" rpy="
+      ${0 + PM_Robot_Tool_TCP_Joint_Cal_rx * 3.14159265359/180}
+      ${0 + PM_Robot_Tool_TCP_Joint_Cal_ry * 3.14159265359/180}
+      ${0 + PM_Robot_Tool_TCP_Joint_Cal_rz * 3.14159265359/180}" />
+    <parent link="Gripper_Rot_Plate" />
+    <child link="PM_Robot_Tool_TCP" />
+    <axis xyz="0 0 0" />
+  </joint>
   <link
     name="PM_Robot_Vacuum_Tool">
@@ -170,24 +190,4 @@
       xyz="0 0 0" />
   </joint>
-  <link name="PM_Robot_Tool_TCP">
-  </link>
-  <xacro:property name="PM_Robot_Tool_TCP_Joint_Cal_x" value="${calibration_dict['PM_Robot_Tool_TCP_Joint']['x_offset']}"/>
-  <xacro:property name="PM_Robot_Tool_TCP_Joint_Cal_y" value="${calibration_dict['PM_Robot_Tool_TCP_Joint']['y_offset']}"/>
-  <xacro:property name="PM_Robot_Tool_TCP_Joint_Cal_z" value="${calibration_dict['PM_Robot_Tool_TCP_Joint']['z_offset']}"/>
-  <xacro:property name="PM_Robot_Tool_TCP_Joint_Cal_rx" value="${calibration_dict['PM_Robot_Tool_TCP_Joint']['rx_offset']}"/>
-  <xacro:property name="PM_Robot_Tool_TCP_Joint_Cal_ry" value="${calibration_dict['PM_Robot_Tool_TCP_Joint']['ry_offset']}"/>
-  <xacro:property name="PM_Robot_Tool_TCP_Joint_Cal_rz" value="${calibration_dict['PM_Robot_Tool_TCP_Joint']['rz_offset']}"/>
-  <joint name="PM_Robot_Tool_TCP_Joint" type="fixed">
-    <origin xyz="
-      ${0 + pm_robot_tool_TCP_x_offset + PM_Robot_Tool_TCP_Joint_Cal_x * 0.000001}
-      ${0 + pm_robot_tool_TCP_y_offset + PM_Robot_Tool_TCP_Joint_Cal_y * 0.000001}
-      ${0 - 0.04542 - pm_robot_tool_TCP_z_offset + PM_Robot_Tool_TCP_Joint_Cal_z * 0.000001}" rpy="
-      ${0 + PM_Robot_Tool_TCP_Joint_Cal_rx * 3.14159265359/180}
-      ${0 + PM_Robot_Tool_TCP_Joint_Cal_ry * 3.14159265359/180}
-      ${0 + PM_Robot_Tool_TCP_Joint_Cal_rz * 3.14159265359/180}" />
-    <parent link="Gripper_Rot_Plate" />
-    <child link="PM_Robot_Tool_TCP" />
-    <axis xyz="0 0 0" />
-  </joint>
 </xacro:macro>
 </robot>

File: pm_robot_description/urdf/pm_robot.xacro (robot description, xacro)
@@ -850,9 +850,9 @@
     </link>
     <joint name="Camera_Calibration_Platelet_Joint" type="prismatic">
-      <origin xyz="0.08 -0.0805 0.2922" rpy="0 0 0" />
+      <origin xyz="0.08 -0.0815 0.293" rpy="0 0 0" />
       <parent link="Camera_Station" />
       <child link="Camera_Calibration_Platelet" />
       <axis xyz="0 -1 0" />
-      <limit lower="-0.048" upper="0.0" effort="100" velocity="0.5" />
+      <limit lower="-0.050" upper="0.00" effort="100" velocity="0.5" />
     </joint>
       <link
@@ -869,5 +869,5 @@
       </link>
       <joint name="Calibration_Platelet_Calibration_Frame_Joint" type="fixed">
-        <origin xyz="0.0 0.1195 0.0135 " rpy="0 0 0" />
+        <origin xyz="0.0 0.1245 0.0135 " rpy="0 0 0" />
         <parent link="Camera_Calibration_Platelet" />
         <child link="Calibration_Platelet_Calibration_Frame" />
