Commit message: gripper 1 jaw

File: pm_robot_description/urdf/pm_Schunk_Tools/Parallel_Gripper_1_Jaw/SmarAct_Piezo_Gripper.xacro (robot description, xacro)
@@ -26,6 +26,11 @@
     <!-- <xacro:property name="current_vacuum_tool" value="${current_pm_robot_bringup_config['pm_robot_tools']['pm_robot_vacuum_tools']['use_tool']}"/>
     <xacro:property name="current_vacuum_tool_tip" value="${current_pm_robot_bringup_config['pm_robot_tools']['pm_robot_vacuum_tools']['use_tip']}"/> -->
+    <xacro:property name="current_tool" value="${current_pm_robot_bringup_config['pm_robot_tools']['pm_robot_tool_parallel_gripper_1_jaw']['use_tool']}"/>
+    <xacro:property name="current_jaw_attachement" value="${current_pm_robot_bringup_config['pm_robot_tools']['pm_robot_tool_parallel_gripper_1_jaw']['use_jaw_type']}"/>
+    <xacro:property name="parallel_gripper_1_jaw_file" value="$(find pm_robot_description)/urdf/urdf_configs/parallel_gripper_1_jaw.yaml" />
+    <xacro:property name="parallel_gripper_configs" value="${xacro.load_yaml(parallel_gripper_1_jaw_file)}"/>
+    <xacro:property name="Gripper_jaw_1_dict" value="${parallel_gripper_configs[current_tool][current_jaw_attachement]}"/>
     <xacro:property name="calibration_dict" value="${xacro.load_yaml(pm_robot_joint_calibraion_file)}"/>
-    <!--%%%%%%%%%%%%% Base Parallel Gripper Definitions %%%%%%%%%%%%%-->
+    <xacro:property name="joint_offset_value" value="${Gripper_jaw_1_dict['joint_offset_value']}"/>
     <link
     name="Tool_Parallel_Gripper_Body">
@@ -97,5 +102,5 @@
           <mesh filename="file://$(find pm_robot_description)/meshes/Tools/Parallel_Gripper_1_Jaw/SmarAct_Piezo_Gripper/SmarAct_Gripper_Jaw.STL" />
         </geometry>
-        <material name="grey"/>
+        <material name="white"/>
       </visual>
       <collision>
@@ -116,5 +121,5 @@
       type="prismatic">
       <origin
-        xyz="0.00134999999999982 -0.00399999999999992 -0.0248"
+        xyz="${-0.0025+joint_offset_value*0.001} 0.00100000018813534 -0.0520000000000005"
         rpy="0 0 0" />
       <parent
@@ -123,5 +128,5 @@
         link="Tool_Parallel_Gripper_Jaw" />
       <axis
-        xyz="0 1 0" />
+        xyz="1 0 0" />
       <limit
         lower="0"
@@ -137,5 +142,5 @@
       type="fixed">
       <origin
-        xyz="0 0.0014 -0.0075"
+        xyz="0.00250 0.001 -0.052"
         rpy="0 0 0" />
       <parent
@@ -153,5 +158,5 @@
       type="fixed">
       <origin
-      xyz="-0.0014 0 -0.0075"
+      xyz="0.0 0 0.0"
       rpy="0 0 0" />
       <parent
@@ -163,180 +168,155 @@
     </joint>
   <!--%%%%%%%%%%%%% Jaw Definitions %%%%%%%%%%%%%-->
-    <!-- <xacro:property name="mpg_10_plus_jaw_define_file" value="$(find pm_robot_description)/urdf/pm_Schunk_Tools/MPG_10_plus_jaws.yaml" />
-    <xacro:property name="jaw_dict" value="${xacro.load_yaml(mpg_10_plus_jaw_define_file)}"/> -->
-    <!--%%%%%%%%%%%%% Default Jaw Definitions %%%%%%%%%%%%%-->
-    <!-- <xacro:property name="Gripper_jaw_1_xyz" value="${jaw_dict['lens_jaw_3_mm_1']['xyz']}"/>
-    <xacro:property name="Gripper_jaw_1_rpy" value="${jaw_dict['lens_jaw_3_mm_1']['rpy']}"/>
-    <xacro:property name="Gripper_jaw_1_mass" value="${jaw_dict['lens_jaw_3_mm_1']['mass']}"/>
-    <xacro:property name="Gripper_jaw_1_inertia_ixx" value="${jaw_dict['lens_jaw_3_mm_1']['inertia_ixx']}"/>
-    <xacro:property name="Gripper_jaw_1_inertia_ixy" value="${jaw_dict['lens_jaw_3_mm_1']['inertia_ixy']}"/>
-    <xacro:property name="Gripper_jaw_1_inertia_ixz" value="${jaw_dict['lens_jaw_3_mm_1']['inertia_ixz']}"/>
-    <xacro:property name="Gripper_jaw_1_inertia_iyy" value="${jaw_dict['lens_jaw_3_mm_1']['inertia_iyy']}"/>
-    <xacro:property name="Gripper_jaw_1_inertia_iyz" value="${jaw_dict['lens_jaw_3_mm_1']['inertia_iyz']}"/>
-    <xacro:property name="Gripper_jaw_1_inertia_izz" value="${jaw_dict['lens_jaw_3_mm_1']['inertia_izz']}"/>
-    <xacro:property name="Gripper_jaw_1_visual_filename" value="${jaw_dict['lens_jaw_3_mm_1']['visual_filename']}"/>
-    <xacro:property name="Gripper_jaw_1_collision_filename" value="${jaw_dict['lens_jaw_3_mm_1']['collision_filename']}"/>
-    <xacro:property name="Gripper_jaw_2_xyz" value="${jaw_dict['lens_jaw_3_mm_2']['xyz']}"/>
-    <xacro:property name="Gripper_jaw_2_rpy" value="${jaw_dict['lens_jaw_3_mm_2']['rpy']}"/>
-    <xacro:property name="Gripper_jaw_2_mass" value="${jaw_dict['lens_jaw_3_mm_2']['mass']}"/>
-    <xacro:property name="Gripper_jaw_2_inertia_ixx" value="${jaw_dict['lens_jaw_3_mm_2']['inertia_ixx']}"/>
-    <xacro:property name="Gripper_jaw_2_inertia_ixy" value="${jaw_dict['lens_jaw_3_mm_2']['inertia_ixy']}"/>
-    <xacro:property name="Gripper_jaw_2_inertia_ixz" value="${jaw_dict['lens_jaw_3_mm_2']['inertia_ixz']}"/>
-    <xacro:property name="Gripper_jaw_2_inertia_iyy" value="${jaw_dict['lens_jaw_3_mm_2']['inertia_iyy']}"/>
-    <xacro:property name="Gripper_jaw_2_inertia_iyz" value="${jaw_dict['lens_jaw_3_mm_2']['inertia_iyz']}"/>
-    <xacro:property name="Gripper_jaw_2_inertia_izz" value="${jaw_dict['lens_jaw_3_mm_2']['inertia_izz']}"/>
-    <xacro:property name="Gripper_jaw_2_visual_filename" value="${jaw_dict['lens_jaw_3_mm_2']['visual_filename']}"/>
-    <xacro:property name="Gripper_jaw_2_collision_filename" value="${jaw_dict['lens_jaw_3_mm_2']['collision_filename']}"/> -->
-    <!--%%%%%%%%%%%%% 3MM Lens Jaw 1 Definitions %%%%%%%%%%%%%-->
-    <!-- <xacro:if value="${use_three_mm_lens}">
-      <xacro:property name="Gripper_jaw_1_xyz" value="${jaw_dict['lens_jaw_3_mm_1']['xyz']}"/>
-      <xacro:property name="Gripper_jaw_1_rpy" value="${jaw_dict['lens_jaw_3_mm_1']['rpy']}"/>
-      <xacro:property name="Gripper_jaw_1_mass" value="${jaw_dict['lens_jaw_3_mm_1']['mass']}"/>
-      <xacro:property name="Gripper_jaw_1_inertia_ixx" value="${jaw_dict['lens_jaw_3_mm_1']['inertia_ixx']}"/>
-      <xacro:property name="Gripper_jaw_1_inertia_ixy" value="${jaw_dict['lens_jaw_3_mm_1']['inertia_ixy']}"/>
-      <xacro:property name="Gripper_jaw_1_inertia_ixz" value="${jaw_dict['lens_jaw_3_mm_1']['inertia_ixz']}"/>
-      <xacro:property name="Gripper_jaw_1_inertia_iyy" value="${jaw_dict['lens_jaw_3_mm_1']['inertia_iyy']}"/>
-      <xacro:property name="Gripper_jaw_1_inertia_iyz" value="${jaw_dict['lens_jaw_3_mm_1']['inertia_iyz']}"/>
-      <xacro:property name="Gripper_jaw_1_inertia_izz" value="${jaw_dict['lens_jaw_3_mm_1']['inertia_izz']}"/>
-      <xacro:property name="Gripper_jaw_1_visual_filename" value="${jaw_dict['lens_jaw_3_mm_1']['visual_filename']}"/>
-      <xacro:property name="Gripper_jaw_1_collision_filename" value="${jaw_dict['lens_jaw_3_mm_1']['collision_filename']}"/>
-      <xacro:property name="Gripper_jaw_2_xyz" value="${jaw_dict['lens_jaw_3_mm_2']['xyz']}"/>
-      <xacro:property name="Gripper_jaw_2_rpy" value="${jaw_dict['lens_jaw_3_mm_2']['rpy']}"/>
-      <xacro:property name="Gripper_jaw_2_mass" value="${jaw_dict['lens_jaw_3_mm_2']['mass']}"/>
-      <xacro:property name="Gripper_jaw_2_inertia_ixx" value="${jaw_dict['lens_jaw_3_mm_2']['inertia_ixx']}"/>
-      <xacro:property name="Gripper_jaw_2_inertia_ixy" value="${jaw_dict['lens_jaw_3_mm_2']['inertia_ixy']}"/>
-      <xacro:property name="Gripper_jaw_2_inertia_ixz" value="${jaw_dict['lens_jaw_3_mm_2']['inertia_ixz']}"/>
-      <xacro:property name="Gripper_jaw_2_inertia_iyy" value="${jaw_dict['lens_jaw_3_mm_2']['inertia_iyy']}"/>
-      <xacro:property name="Gripper_jaw_2_inertia_iyz" value="${jaw_dict['lens_jaw_3_mm_2']['inertia_iyz']}"/>
-      <xacro:property name="Gripper_jaw_2_inertia_izz" value="${jaw_dict['lens_jaw_3_mm_2']['inertia_izz']}"/>
-      <xacro:property name="Gripper_jaw_2_visual_filename" value="${jaw_dict['lens_jaw_3_mm_2']['visual_filename']}"/>
-      <xacro:property name="Gripper_jaw_2_collision_filename" value="${jaw_dict['lens_jaw_3_mm_2']['collision_filename']}"/>
-    </xacro:if> -->
-    <!--%%%%%%%%%%%%% The parameters here are interchangeable %%%%%%%%%%%%%-->
-    <!--%%%%%%%%%%%%% Jaw 1 Definitions %%%%%%%%%%%%%-->
-    <!-- <link
-      name="Tool_Gripper_MPG_10_Jaw_1_changeable">
-      <inertial>
-        <origin
-          xyz="${Gripper_jaw_1_xyz}"
-          rpy="${Gripper_jaw_1_rpy}"/>
-        <mass
-          value="${Gripper_jaw_1_mass}"/>
-        <inertia
-          ixx="${Gripper_jaw_1_inertia_ixx}"
-          ixy="${Gripper_jaw_1_inertia_ixy}"
-          ixz="${Gripper_jaw_1_inertia_ixz}"
-          iyy="${Gripper_jaw_1_inertia_iyy}"
-          iyz="${Gripper_jaw_1_inertia_iyz}"
-          izz="${Gripper_jaw_1_inertia_izz}" />
-      </inertial>
-      <visual>
-        <origin
-          xyz="0 0 0"
-          rpy="0 0 0" />
-        <geometry>
-          <mesh filename="file://$(find pm_robot_description)/meshes/Tools/MPG_10_plus/Jaws/${Gripper_jaw_1_visual_filename}" />
-        </geometry>
-        <material
-          name="">
-          <color
-            rgba="0.780392156862745 0.76078431372549 0.741176470588235 1" />
-        </material>
-      </visual>
-      <collision>
-        <origin
-          xyz="0 0 0"
-          rpy="0 0 0" />
-        <geometry>
-          <mesh filename="file://$(find pm_robot_description)/meshes/Tools/MPG_10_plus/Jaws/${Gripper_jaw_1_visual_filename}" />
-        </geometry>
-      </collision>
-    </link>
-    <gazebo reference="Tool_Gripper_Jaw_1">
-      <turnGravityOff>true</turnGravityOff>
-    </gazebo>
-    <joint
-      name="Tool_Gripper_MPG_10_Jaw_1_changeable_Joint"
-      type="fixed">
-      <origin
-        xyz="0.002 0 0 "
-        rpy="0 0 0" />
-      <parent
-        link="Tool_Gripper_MPG_10_Jaw_1_Point" />
-      <child
-        link="Tool_Gripper_MPG_10_Jaw_1_changeable" />
-    </joint>
-    <link
-      name="Tool_Gripper_MPG_10_Jaw_2_changeable">
-      <inertial>
-        <origin
-          xyz="${Gripper_jaw_2_xyz}"
-          rpy="${Gripper_jaw_2_rpy}"/>
-        <mass
-          value="${Gripper_jaw_2_mass}"/>
-        <inertia
-          ixx="${Gripper_jaw_2_inertia_ixx}"
-          ixy="${Gripper_jaw_2_inertia_ixy}"
-          ixz="${Gripper_jaw_2_inertia_ixz}"
-          iyy="${Gripper_jaw_2_inertia_iyy}"
-          iyz="${Gripper_jaw_2_inertia_iyz}"
-          izz="${Gripper_jaw_2_inertia_izz}" />
-      </inertial>
-      <visual>
-        <origin
-          xyz="0 0 0"
-          rpy="0 0 0" />
-        <geometry>
-          <mesh filename="file://$(find pm_robot_description)/meshes/Tools/MPG_10_plus/Jaws/${Gripper_jaw_2_visual_filename}" />
-        </geometry>
-        <material
-          name="">
-          <color
-            rgba="0.780392156862745 0.76078431372549 0.741176470588235 1" />
-        </material>
-      </visual>
-      <collision>
-        <origin
-          xyz="0 0 0"
-          rpy="0 0 0" />
-        <geometry>
-          <mesh filename="file://$(find pm_robot_description)/meshes/Tools/MPG_10_plus/Jaws/${Gripper_jaw_2_visual_filename}" />
-        </geometry>
-      </collision>
-    </link>
-    <gazebo reference="Tool_Gripper_MPG_10_Jaw_2_changeable">
-      <turnGravityOff>true</turnGravityOff>
-    </gazebo>
-    <joint
-      name="Tool_Gripper_MPG_10_Jaw_2_changeable_Joint"
-      type="fixed">
-      <origin
-        xyz="0.002 0  0 "
-        rpy="1.5708 0 0" />
-      <parent
-        link="Tool_Gripper_MPG_10_Jaw_2_Point" />
-      <child
-        link="Tool_Gripper_MPG_10_Jaw_2_changeable" />
-    </joint> -->
-  <link name="PM_Robot_Tool_TCP">
+  <xacro:property name="Gripper_jaw_1_xyz" value="${Gripper_jaw_1_dict['Jaw_1']['inertia_xyz']}"/>
+  <xacro:property name="Gripper_jaw_1_rpy" value="${Gripper_jaw_1_dict['Jaw_1']['inertia_rpy']}"/>
+  <xacro:property name="Gripper_jaw_1_mass" value="${Gripper_jaw_1_dict['Jaw_1']['mass']}"/>
+  <xacro:property name="Gripper_jaw_1_inertia_ixx" value="${Gripper_jaw_1_dict['Jaw_1']['inertia_ixx']}"/>
+  <xacro:property name="Gripper_jaw_1_inertia_ixy" value="${Gripper_jaw_1_dict['Jaw_1']['inertia_ixy']}"/>
+  <xacro:property name="Gripper_jaw_1_inertia_ixz" value="${Gripper_jaw_1_dict['Jaw_1']['inertia_ixz']}"/>
+  <xacro:property name="Gripper_jaw_1_inertia_iyy" value="${Gripper_jaw_1_dict['Jaw_1']['inertia_iyy']}"/>
+  <xacro:property name="Gripper_jaw_1_inertia_iyz" value="${Gripper_jaw_1_dict['Jaw_1']['inertia_iyz']}"/>
+  <xacro:property name="Gripper_jaw_1_inertia_izz" value="${Gripper_jaw_1_dict['Jaw_1']['inertia_izz']}"/>
+  <xacro:property name="Gripper_jaw_1_visual_filename" value="${Gripper_jaw_1_dict['Jaw_1']['visual_filename']}"/>
+  <xacro:property name="Gripper_jaw_1_collision_filename" value="${Gripper_jaw_1_dict['Jaw_1']['collision_filename']}"/>
+  <xacro:property name="Gripper_jaw_2_xyz" value="${Gripper_jaw_1_dict['Jaw_2']['inertia_xyz']}"/>
+  <xacro:property name="Gripper_jaw_2_rpy" value="${Gripper_jaw_1_dict['Jaw_2']['inertia_rpy']}"/>
+  <xacro:property name="Gripper_jaw_2_mass" value="${Gripper_jaw_1_dict['Jaw_2']['mass']}"/>
+  <xacro:property name="Gripper_jaw_2_inertia_ixx" value="${Gripper_jaw_1_dict['Jaw_2']['inertia_ixx']}"/>
+  <xacro:property name="Gripper_jaw_2_inertia_ixy" value="${Gripper_jaw_1_dict['Jaw_2']['inertia_ixy']}"/>
+  <xacro:property name="Gripper_jaw_2_inertia_ixz" value="${Gripper_jaw_1_dict['Jaw_2']['inertia_ixz']}"/>
+  <xacro:property name="Gripper_jaw_2_inertia_iyy" value="${Gripper_jaw_1_dict['Jaw_2']['inertia_iyy']}"/>
+  <xacro:property name="Gripper_jaw_2_inertia_iyz" value="${Gripper_jaw_1_dict['Jaw_2']['inertia_iyz']}"/>
+  <xacro:property name="Gripper_jaw_2_inertia_izz" value="${Gripper_jaw_1_dict['Jaw_2']['inertia_izz']}"/>
+  <xacro:property name="Gripper_jaw_2_visual_filename" value="${Gripper_jaw_1_dict['Jaw_2']['visual_filename']}"/>
+  <xacro:property name="Gripper_jaw_2_collision_filename" value="${Gripper_jaw_1_dict['Jaw_2']['collision_filename']}"/>
+  <xacro:property name="tool_tcp_offset_x" value="${Gripper_jaw_1_dict['tool_TCP_x_offset']}"/>
+  <xacro:property name="tool_tcp_offset_y" value="${Gripper_jaw_1_dict['tool_TCP_y_offset']}"/>
+  <xacro:property name="tool_tcp_offset_z" value="${Gripper_jaw_1_dict['tool_TCP_z_offset']}"/>
+  <!--%%%%%%%%%%%%% The parameters here are interchangeable %%%%%%%%%%%%%-->
+  <!--%%%%%%%%%%%%% Jaw 1 Definitions %%%%%%%%%%%%%-->
+  <link
+    name="Tool_Parallel_Gripper_Jaw_1_attachment">
+    <inertial>
+      <origin
+        xyz="${Gripper_jaw_1_xyz}"
+        rpy="${Gripper_jaw_1_rpy}"/>
+      <mass
+        value="${Gripper_jaw_1_mass}"/>
+      <inertia
+        ixx="${Gripper_jaw_1_inertia_ixx}"
+        ixy="${Gripper_jaw_1_inertia_ixy}"
+        ixz="${Gripper_jaw_1_inertia_ixz}"
+        iyy="${Gripper_jaw_1_inertia_iyy}"
+        iyz="${Gripper_jaw_1_inertia_iyz}"
+        izz="${Gripper_jaw_1_inertia_izz}" />
+    </inertial>
+    <visual>
+      <origin
+        xyz="0 0 0"
+        rpy="0 0 0" />
+      <geometry>
+        <mesh filename="file://$(find pm_robot_description)/meshes/Tools/Parallel_Gripper_1_Jaw/SmarAct_Piezo_Gripper/${Gripper_jaw_1_visual_filename}" />
+      </geometry>
+      <material
+        name="">
+        <color
+          rgba="0.780392156862745 0.76078431372549 0.741176470588235 1" />
+      </material>
+    </visual>
+    <collision>
+      <origin
+        xyz="0 0 0"
+        rpy="0 0 0" />
+      <geometry>
+        <mesh filename="file://$(find pm_robot_description)/meshes/Tools/Parallel_Gripper_1_Jaw/SmarAct_Piezo_Gripper/${Gripper_jaw_1_visual_filename}" />
+      </geometry>
+    </collision>
   </link>
-  <xacro:property name="PM_Robot_Tool_TCP_Joint_Cal_x" value="${calibration_dict['PM_Robot_Tool_TCP_Joint']['x_offset']}"/>
-  <xacro:property name="PM_Robot_Tool_TCP_Joint_Cal_y" value="${calibration_dict['PM_Robot_Tool_TCP_Joint']['y_offset']}"/>
-  <xacro:property name="PM_Robot_Tool_TCP_Joint_Cal_z" value="${calibration_dict['PM_Robot_Tool_TCP_Joint']['z_offset']}"/>
-  <xacro:property name="PM_Robot_Tool_TCP_Joint_Cal_rx" value="${calibration_dict['PM_Robot_Tool_TCP_Joint']['rx_offset']}"/>
-  <xacro:property name="PM_Robot_Tool_TCP_Joint_Cal_ry" value="${calibration_dict['PM_Robot_Tool_TCP_Joint']['ry_offset']}"/>
-  <xacro:property name="PM_Robot_Tool_TCP_Joint_Cal_rz" value="${calibration_dict['PM_Robot_Tool_TCP_Joint']['rz_offset']}"/>
-  <joint name="PM_Robot_Tool_TCP_Joint" type="fixed">
-    <origin xyz="
-      ${0  + PM_Robot_Tool_TCP_Joint_Cal_x * 0.000001}
-      ${0  + PM_Robot_Tool_TCP_Joint_Cal_y * 0.000001}
-      ${0 - 0.04542 + PM_Robot_Tool_TCP_Joint_Cal_z * 0.000001}" rpy="
-      ${0 + PM_Robot_Tool_TCP_Joint_Cal_rx * 3.14159265359/180}
-      ${0 + PM_Robot_Tool_TCP_Joint_Cal_ry * 3.14159265359/180}
-      ${0 + PM_Robot_Tool_TCP_Joint_Cal_rz * 3.14159265359/180}" />
-    <parent link="Gripper_Rot_Plate" />
-    <child link="PM_Robot_Tool_TCP" />
-    <axis xyz="0 0 0" />
+  <gazebo reference="Tool_Parallel_Gripper_Jaw_1_attachment">
+    <turnGravityOff>true</turnGravityOff>
+  </gazebo>
+  <joint
+    name="Tool_Parallel_Gripper_Jaw_1_attachment_Joint"
+    type="fixed">
+    <origin
+      xyz="0.0 0.0 0 "
+      rpy="1.570796327 0 3.141592654" />
+    <parent
+      link="Tool_Parallel_Gripper_Jaw_1_Point" />
+    <child
+      link="Tool_Parallel_Gripper_Jaw_1_attachment" />
   </joint>
+  <link
+    name="Tool_Parallel_Gripper_Jaw_2_attachment">
+    <inertial>
+      <origin
+        xyz="${Gripper_jaw_2_xyz}"
+        rpy="${Gripper_jaw_2_rpy}"/>
+      <mass
+        value="${Gripper_jaw_2_mass}"/>
+      <inertia
+        ixx="${Gripper_jaw_2_inertia_ixx}"
+        ixy="${Gripper_jaw_2_inertia_ixy}"
+        ixz="${Gripper_jaw_2_inertia_ixz}"
+        iyy="${Gripper_jaw_2_inertia_iyy}"
+        iyz="${Gripper_jaw_2_inertia_iyz}"
+        izz="${Gripper_jaw_2_inertia_izz}" />
+    </inertial>
+    <visual>
+      <origin
+        xyz="0 0 0"
+        rpy="1.570796327 0 0" />
+      <geometry>
+        <mesh filename="file://$(find pm_robot_description)/meshes/Tools/Parallel_Gripper_1_Jaw/SmarAct_Piezo_Gripper/${Gripper_jaw_2_visual_filename}" />
+      </geometry>
+      <material
+        name="">
+        <color
+          rgba="0.780392156862745 0.76078431372549 0.741176470588235 1" />
+      </material>
+    </visual>
+    <collision>
+      <origin
+        xyz="0 0 0"
+        rpy="0 0 0" />
+      <geometry>
+        <mesh filename="file://$(find pm_robot_description)/meshes/Tools/Parallel_Gripper_1_Jaw/SmarAct_Piezo_Gripper/${Gripper_jaw_2_visual_filename}" />
+      </geometry>
+    </collision>
+  </link>
+  <gazebo reference="Tool_Parallel_Gripper_Jaw_2_attachment">
+    <turnGravityOff>true</turnGravityOff>
+  </gazebo>
+  <joint
+    name="Tool_Parallel_Gripper_Jaw_2_attachment_Joint"
+    type="fixed">
+    <origin
+      xyz="0.0 0 0 "
+      rpy="0 0 3.141592654" />
+    <parent
+      link="Tool_Parallel_Gripper_Jaw_2_Point" />
+    <child
+      link="Tool_Parallel_Gripper_Jaw_2_attachment" />
+  </joint>
+<link name="PM_Robot_Tool_TCP">
+</link>
+<xacro:property name="PM_Robot_Tool_TCP_Joint_Cal_x" value="${calibration_dict['PM_Robot_Tool_TCP_Joint']['x_offset']}"/>
+<xacro:property name="PM_Robot_Tool_TCP_Joint_Cal_y" value="${calibration_dict['PM_Robot_Tool_TCP_Joint']['y_offset']}"/>
+<xacro:property name="PM_Robot_Tool_TCP_Joint_Cal_z" value="${calibration_dict['PM_Robot_Tool_TCP_Joint']['z_offset']}"/>
+<xacro:property name="PM_Robot_Tool_TCP_Joint_Cal_rx" value="${calibration_dict['PM_Robot_Tool_TCP_Joint']['rx_offset']}"/>
+<xacro:property name="PM_Robot_Tool_TCP_Joint_Cal_ry" value="${calibration_dict['PM_Robot_Tool_TCP_Joint']['ry_offset']}"/>
+<xacro:property name="PM_Robot_Tool_TCP_Joint_Cal_rz" value="${calibration_dict['PM_Robot_Tool_TCP_Joint']['rz_offset']}"/>
+<joint name="PM_Robot_Tool_TCP_Joint" type="fixed">
+  <origin xyz="
+    ${0 + tool_tcp_offset_x  + PM_Robot_Tool_TCP_Joint_Cal_x * 0.000001}
+    ${0 + tool_tcp_offset_y  + PM_Robot_Tool_TCP_Joint_Cal_y * 0.000001}
+    ${0 + tool_tcp_offset_z - 0.04542 + PM_Robot_Tool_TCP_Joint_Cal_z * 0.000001}" rpy="
+    ${0 + PM_Robot_Tool_TCP_Joint_Cal_rx * 3.14159265359/180}
+    ${0 + PM_Robot_Tool_TCP_Joint_Cal_ry * 3.14159265359/180}
+    ${0 + PM_Robot_Tool_TCP_Joint_Cal_rz * 3.14159265359/180}" />
+  <parent link="Gripper_Rot_Plate" />
+  <child link="PM_Robot_Tool_TCP" />
+  <axis xyz="0 0 0" />
+</joint>
 </xacro:macro>
 </robot>

File: pm_robot_description/urdf/pm_Schunk_Tools/Parallel_Gripper_1_Jaw/SmarAct_Piezo_Gripper_flat.xacro (robot description, xacro)
@@ -28,5 +28,9 @@
     <xacro:property name="current_tool" value="${current_pm_robot_bringup_config['pm_robot_tools']['pm_robot_tool_parallel_gripper_1_jaw']['use_tool']}"/>
     <xacro:property name="current_jaw_attachement" value="${current_pm_robot_bringup_config['pm_robot_tools']['pm_robot_tool_parallel_gripper_1_jaw']['use_jaw_type']}"/>
+    <xacro:property name="parallel_gripper_1_jaw_file" value="$(find pm_robot_description)/urdf/urdf_configs/parallel_gripper_1_jaw.yaml" />
+    <xacro:property name="parallel_gripper_configs" value="${xacro.load_yaml(parallel_gripper_1_jaw_file)}"/>
+    <xacro:property name="Gripper_jaw_1_dict" value="${parallel_gripper_configs[current_tool][current_jaw_attachement]}"/>
     <xacro:property name="calibration_dict" value="${xacro.load_yaml(pm_robot_joint_calibraion_file)}"/>
+    <xacro:property name="joint_offset_value" value="${Gripper_jaw_1_dict['joint_offset_value']}"/>
     <!--%%%%%%%%%%%%% Base Parallel Gripper Definitions %%%%%%%%%%%%%-->
     <link
@@ -99,5 +103,5 @@
           <mesh filename="file://$(find pm_robot_description)/meshes/Tools/Parallel_Gripper_1_Jaw/SmarAct_Piezo_Gripper/SmarAct_Gripper_Jaw_flat.STL" />
         </geometry>
-        <material name="grey"/>
+        <material name="white"/>
       </visual>
       <collision>
@@ -118,5 +122,5 @@
       type="prismatic">
       <origin
-        xyz="-0.00549999981186566 0.00150000018813442 -0.0318"
+        xyz="${0.00551408822663166+joint_offset_value*0.001} 0.00150000018813439 -0.0318"
         rpy="0 0 0" />
       <parent
@@ -125,5 +129,5 @@
         link="Tool_Parallel_Gripper_Jaw" />
       <axis
-        xyz="0 1 0" />
+        xyz="1 0 0" />
       <limit
         lower="0"
@@ -155,5 +159,5 @@
       type="fixed">
       <origin
-      xyz="0.011060767270484 0 0"
+      xyz="0.0 0 0"
       rpy="0 0 0" />
       <parent
@@ -165,8 +169,4 @@
     </joint>
   <!--%%%%%%%%%%%%% Jaw Definitions %%%%%%%%%%%%%-->
-    <xacro:property name="parallel_gripper_1_jaw_file" value="$(find pm_robot_description)/urdf/urdf_configs/parallel_gripper_1_jaw.yaml" />
-    <xacro:property name="parallel_gripper_configs" value="${xacro.load_yaml(parallel_gripper_1_jaw_file)}"/>
-    <!--%%%%%%%%%%%%% Default Jaw Definitions %%%%%%%%%%%%%-->
-    <xacro:property name="Gripper_jaw_1_dict" value="${parallel_gripper_configs[current_tool][current_jaw_attachement]}"/>
     <xacro:property name="Gripper_jaw_1_xyz" value="${Gripper_jaw_1_dict['Jaw_1']['inertia_xyz']}"/>
     <xacro:property name="Gripper_jaw_1_rpy" value="${Gripper_jaw_1_dict['Jaw_1']['inertia_rpy']}"/>
@@ -241,5 +241,5 @@
       type="fixed">
       <origin
-        xyz="0.0 0 0 "
+        xyz="0.0 0.0 0 "
         rpy="0 0 0" />
       <parent
