Commit message: gripper 1 jaw

File: pm_robot_description/urdf/pm_smarpod_station.xacro (robot description, xacro)
@@ -72,5 +72,5 @@
     type="fixed">
     <origin
-      xyz="0.750000000000003 0.315 0"
+      xyz="0.6 0.31 0"
       rpy="0 0 0" />
     <parent
@@ -83,41 +83,4 @@
   <link
     name="Smarpod_Station_Base">
-    <!-- <inertial>
-      <origin
-        xyz="0.00218806954398554 0.016740010574494 -0.0260350780485463"
-        rpy="0 0 0" />
-      <mass
-        value="0.782282249809798" />
-      <inertia
-        ixx="0.00477442216909529"
-        ixy="-5.89281059976034E-08"
-        ixz="2.37578030999863E-10"
-        iyy="0.00354235482448058"
-        iyz="2.44320538923888E-08"
-        izz="0.00631238764877303" />
-    </inertial>
-    <visual>
-      <origin
-        xyz="0 0 0"
-        rpy="0 0 0" />
-      <geometry>
-        <mesh
-          filename="package://BAUGRUPPE_PM_ROBOT_Export_22052024_2/meshes/Smarpod_Station_Base.STL" />
-      </geometry>
-      <material
-        name="">
-        <color
-          rgba="0.752941176470588 0.752941176470588 0.752941176470588 1" />
-      </material>
-    </visual>
-    <collision>
-      <origin
-        xyz="0 0 0"
-        rpy="0 0 0" />
-      <geometry>
-        <mesh
-          filename="package://BAUGRUPPE_PM_ROBOT_Export_22052024_2/meshes/Smarpod_Station_Base.STL" />
-      </geometry>
-    </collision> -->
   </link>
   <joint
@@ -125,5 +88,5 @@
     type="fixed">
     <origin
-      xyz="0.09 0.0899999999999999 0.2136999999992"
+      xyz="0.2 0.15 0.2253999999992"
       rpy="0 0 0" />
     <parent

File: pm_robot_description/urdf/ros2_control_real_HW.xacro (robot description, xacro)
@@ -105,5 +105,4 @@
                     </command_interface>
                     <state_interface name="position"/>
-                    <state_interface name="velocity"/>
                 </joint>
                 <joint name="Tool_Parallel_Gripper_Jaw_2_Joint">
@@ -111,5 +110,4 @@
                     </command_interface>
                     <state_interface name="position"/>
-                    <state_interface name="velocity"/>
                 </joint>
                 <!-- <joint name="Tool_Parallel_Gripper_Jaw_2_Joint">
@@ -128,5 +126,4 @@
                     </command_interface>
                     <state_interface name="position"/>
-                    <state_interface name="velocity"/>
                 </joint>
             </xacro:if>

File: pm_robot_description/urdf/ros2_control_sim_HW.xacro (robot description, xacro)
@@ -111,5 +111,4 @@
                     </command_interface>
                     <state_interface name="position"/>
-                    <state_interface name="velocity"/>
                 </joint>
                <joint name="Tool_Parallel_Gripper_Jaw_2_Joint">
@@ -117,5 +116,4 @@
                     </command_interface>
                     <state_interface name="position"/>
-                    <state_interface name="velocity"/>
                 </joint>
                 <!-- <joint name="Tool_Parallel_Gripper_Jaw_2_Joint">
@@ -134,5 +132,4 @@
                     </command_interface>
                     <state_interface name="position"/>
-                    <state_interface name="velocity"/>
                 </joint>
             </xacro:if>

Commit message: local pm_robot_config

File: pm_robot_description/urdf/pm_Schunk_Tools/Parallel_Gripper_1_Jaw/SmarAct_Piezo_Gripper.xacro (robot description, xacro)
@@ -5,22 +5,23 @@
 <robot xmlns:xacro="http://ros.org/wiki/xacro">
   <xacro:macro name="Tool_Parallel_Gripper_1_Jaw" params="launch_mode">
-          <xacro:if value="${launch_mode == 'sim_HW'}">
-              <xacro:property name="pm_robot_joint_calibraion_file" value="$(find pm_robot_description)/calibration_config/pm_robot_joint_calibration.yaml" />
-              <xacro:property name="pm_robot_bringup_config_file" value="$(find pm_robot_bringup)/config/pm_robot_bringup_config.yaml" />
-          </xacro:if>
+    <xacro:if value="${launch_mode == 'sim_HW'}">
+        <xacro:property name="pm_robot_joint_calibraion_file" value="$(find pm_robot_description)/calibration_config/pm_robot_joint_calibration.yaml" />
+        <xacro:property name="pm_robot_bringup_config_file" value="$(find pm_robot_bringup)/config/pm_robot_bringup_config.yaml" />
+    </xacro:if>
     <!-- Loading of the Robot Joint calibrations and bringup config -->
     <!-- If launch_mode 'real' a local path can be specified for the calibration file -->
-          <xacro:if value="${launch_mode == 'real_HW'}">
-              <xacro:property name="local_file_paths__file" value="$(find pm_robot_description)/calibration_config/pm_robot_path_real_HW.yaml" />
-              <xacro:property name="path_dict" value="${xacro.load_yaml(local_file_paths__file)}"/>
-              <xacro:property name="local_calibration_file_path" value="${path_dict['pm_robot_calibration_file_path']}"/>
-              <xacro:property name="local_robot_bringup_file_path" value="${path_dict['pm_robot_bringup_config_file_path']}"/>
-              <!-- REAL -->
-              <!-- <xacro:property name="pm_robot_joint_calibraion_file" value="${local_calibration_file_path}" />
-              <xacro:property name="pm_robot_bringup_config_file" value="${local_robot_bringup_file_path}"/> -->
-              <!-- SIM -->
-              <xacro:property name="pm_robot_joint_calibraion_file" value="$(find pm_robot_description)/calibration_config/pm_robot_joint_calibration.yaml" />
-              <xacro:property name="pm_robot_bringup_config_file" value="$(find pm_robot_bringup)/config/pm_robot_bringup_config.yaml" />
-          </xacro:if>
+    <!-- If launch_mode 'real' a local path can be specified for the calibration file -->
+    <xacro:if value="${launch_mode == 'real_HW'}">
+      <xacro:property name="local_file_paths__file" value="$(find pm_robot_description)/calibration_config/pm_robot_path_real_HW.yaml" />
+      <xacro:property name="path_dict" value="${xacro.load_yaml(local_file_paths__file)}"/>
+      <xacro:property name="local_calibration_file_path" value="${path_dict['pm_robot_calibration_file_path']}"/>
+      <xacro:property name="local_robot_bringup_file_path" value="${path_dict['pm_robot_bringup_config_file_path']}"/>
+      <!-- REAL -->
+      <xacro:property name="pm_robot_joint_calibraion_file" value="${local_calibration_file_path}" />
+      <xacro:property name="pm_robot_bringup_config_file" value="${local_robot_bringup_file_path}"/>
+      <!-- SIM -->
+      <!-- <xacro:property name="pm_robot_joint_calibraion_file" value="$(find pm_robot_description)/calibration_config/pm_robot_joint_calibration.yaml" />
+      <xacro:property name="pm_robot_bringup_config_file" value="$(find pm_robot_bringup)/config/pm_robot_bringup_config.yaml" /> -->
+    </xacro:if>
     <xacro:property name="current_pm_robot_bringup_config" value="${xacro.load_yaml(pm_robot_bringup_config_file)}"/>
     <!-- <xacro:property name="current_vacuum_tool" value="${current_pm_robot_bringup_config['pm_robot_tools']['pm_robot_vacuum_tools']['use_tool']}"/>

File: pm_robot_description/urdf/pm_Schunk_Tools/Parallel_Gripper_1_Jaw/SmarAct_Piezo_Gripper_flat.xacro (robot description, xacro)
@@ -11,16 +11,16 @@
     <!-- Loading of the Robot Joint calibrations and bringup config -->
     <!-- If launch_mode 'real' a local path can be specified for the calibration file -->
-          <xacro:if value="${launch_mode == 'real_HW'}">
-              <xacro:property name="local_file_paths__file" value="$(find pm_robot_description)/calibration_config/pm_robot_path_real_HW.yaml" />
-              <xacro:property name="path_dict" value="${xacro.load_yaml(local_file_paths__file)}"/>
-              <xacro:property name="local_calibration_file_path" value="${path_dict['pm_robot_calibration_file_path']}"/>
-              <xacro:property name="local_robot_bringup_file_path" value="${path_dict['pm_robot_bringup_config_file_path']}"/>
-              <!-- REAL -->
-              <!-- <xacro:property name="pm_robot_joint_calibraion_file" value="${local_calibration_file_path}" />
-              <xacro:property name="pm_robot_bringup_config_file" value="${local_robot_bringup_file_path}"/> -->
-              <!-- SIM -->
-              <xacro:property name="pm_robot_joint_calibraion_file" value="$(find pm_robot_description)/calibration_config/pm_robot_joint_calibration.yaml" />
-              <xacro:property name="pm_robot_bringup_config_file" value="$(find pm_robot_bringup)/config/pm_robot_bringup_config.yaml" />
-          </xacro:if>
+    <xacro:if value="${launch_mode == 'real_HW'}">
+      <xacro:property name="local_file_paths__file" value="$(find pm_robot_description)/calibration_config/pm_robot_path_real_HW.yaml" />
+      <xacro:property name="path_dict" value="${xacro.load_yaml(local_file_paths__file)}"/>
+      <xacro:property name="local_calibration_file_path" value="${path_dict['pm_robot_calibration_file_path']}"/>
+      <xacro:property name="local_robot_bringup_file_path" value="${path_dict['pm_robot_bringup_config_file_path']}"/>
+      <!-- REAL -->
+      <xacro:property name="pm_robot_joint_calibraion_file" value="${local_calibration_file_path}" />
+      <xacro:property name="pm_robot_bringup_config_file" value="${local_robot_bringup_file_path}"/>
+      <!-- SIM -->
+      <!-- <xacro:property name="pm_robot_joint_calibraion_file" value="$(find pm_robot_description)/calibration_config/pm_robot_joint_calibration.yaml" />
+      <xacro:property name="pm_robot_bringup_config_file" value="$(find pm_robot_bringup)/config/pm_robot_bringup_config.yaml" /> -->
+    </xacro:if>
     <xacro:property name="current_pm_robot_bringup_config" value="${xacro.load_yaml(pm_robot_bringup_config_file)}"/>
     <!-- <xacro:property name="current_vacuum_tool" value="${current_pm_robot_bringup_config['pm_robot_tools']['pm_robot_vacuum_tools']['use_tool']}"/>

File: pm_robot_description/urdf/pm_Schunk_Tools/Parallel_Gripper_2_Jaws/MPG_10_plus.xacro (robot description, xacro)
@@ -11,16 +11,17 @@
     <!-- Loading of the Robot Joint calibrations and bringup config -->
     <!-- If launch_mode 'real' a local path can be specified for the calibration file -->
-          <xacro:if value="${launch_mode == 'real_HW'}">
-              <xacro:property name="local_file_paths__file" value="$(find pm_robot_description)/calibration_config/pm_robot_path_real_HW.yaml" />
-              <xacro:property name="path_dict" value="${xacro.load_yaml(local_file_paths__file)}"/>
-              <xacro:property name="local_calibration_file_path" value="${path_dict['pm_robot_calibration_file_path']}"/>
-              <xacro:property name="local_robot_bringup_file_path" value="${path_dict['pm_robot_bringup_config_file_path']}"/>
-              <!-- REAL -->
-              <!-- <xacro:property name="pm_robot_joint_calibraion_file" value="${local_calibration_file_path}" />
-              <xacro:property name="pm_robot_bringup_config_file" value="${local_robot_bringup_file_path}"/> -->
-              <!-- SIM -->
-              <xacro:property name="pm_robot_joint_calibraion_file" value="$(find pm_robot_description)/calibration_config/pm_robot_joint_calibration.yaml" />
-              <xacro:property name="pm_robot_bringup_config_file" value="$(find pm_robot_bringup)/config/pm_robot_bringup_config.yaml" />
-          </xacro:if>
+    <!-- If launch_mode 'real' a local path can be specified for the calibration file -->
+    <xacro:if value="${launch_mode == 'real_HW'}">
+      <xacro:property name="local_file_paths__file" value="$(find pm_robot_description)/calibration_config/pm_robot_path_real_HW.yaml" />
+      <xacro:property name="path_dict" value="${xacro.load_yaml(local_file_paths__file)}"/>
+      <xacro:property name="local_calibration_file_path" value="${path_dict['pm_robot_calibration_file_path']}"/>
+      <xacro:property name="local_robot_bringup_file_path" value="${path_dict['pm_robot_bringup_config_file_path']}"/>
+      <!-- REAL -->
+      <xacro:property name="pm_robot_joint_calibraion_file" value="${local_calibration_file_path}" />
+      <xacro:property name="pm_robot_bringup_config_file" value="${local_robot_bringup_file_path}"/>
+      <!-- SIM -->
+      <!-- <xacro:property name="pm_robot_joint_calibraion_file" value="$(find pm_robot_description)/calibration_config/pm_robot_joint_calibration.yaml" />
+      <xacro:property name="pm_robot_bringup_config_file" value="$(find pm_robot_bringup)/config/pm_robot_bringup_config.yaml" /> -->
+    </xacro:if>
     <xacro:property name="current_pm_robot_bringup_config" value="${xacro.load_yaml(pm_robot_bringup_config_file)}"/>
     <!-- <xacro:property name="current_vacuum_tool" value="${current_pm_robot_bringup_config['pm_robot_tools']['pm_robot_vacuum_tools']['use_tool']}"/>

File: pm_robot_description/urdf/pm_Schunk_Tools/Schunk_Vacuum_Tools.xacro (robot description, xacro)
@@ -12,16 +12,16 @@
     <!-- Loading of the Robot Joint calibrations and bringup config -->
     <!-- If launch_mode 'real' a local path can be specified for the calibration file -->
-          <xacro:if value="${launch_mode == 'real_HW'}">
-              <xacro:property name="local_file_paths__file" value="$(find pm_robot_description)/calibration_config/pm_robot_path_real_HW.yaml" />
-              <xacro:property name="path_dict" value="${xacro.load_yaml(local_file_paths__file)}"/>
-              <xacro:property name="local_calibration_file_path" value="${path_dict['pm_robot_calibration_file_path']}"/>
-              <xacro:property name="local_robot_bringup_file_path" value="${path_dict['pm_robot_bringup_config_file_path']}"/>
-              <!-- REAL -->
-              <!-- <xacro:property name="pm_robot_joint_calibraion_file" value="${local_calibration_file_path}" />
-              <xacro:property name="pm_robot_bringup_config_file" value="${local_robot_bringup_file_path}"/> -->
-              <!-- SIM -->
-              <xacro:property name="pm_robot_joint_calibraion_file" value="$(find pm_robot_description)/calibration_config/pm_robot_joint_calibration.yaml" />
-              <xacro:property name="pm_robot_bringup_config_file" value="$(find pm_robot_bringup)/config/pm_robot_bringup_config.yaml" />
-          </xacro:if>
+    <xacro:if value="${launch_mode == 'real_HW'}">
+      <xacro:property name="local_file_paths__file" value="$(find pm_robot_description)/calibration_config/pm_robot_path_real_HW.yaml" />
+      <xacro:property name="path_dict" value="${xacro.load_yaml(local_file_paths__file)}"/>
+      <xacro:property name="local_calibration_file_path" value="${path_dict['pm_robot_calibration_file_path']}"/>
+      <xacro:property name="local_robot_bringup_file_path" value="${path_dict['pm_robot_bringup_config_file_path']}"/>
+      <!-- REAL -->
+      <xacro:property name="pm_robot_joint_calibraion_file" value="${local_calibration_file_path}" />
+      <xacro:property name="pm_robot_bringup_config_file" value="${local_robot_bringup_file_path}"/>
+      <!-- SIM -->
+      <!-- <xacro:property name="pm_robot_joint_calibraion_file" value="$(find pm_robot_description)/calibration_config/pm_robot_joint_calibration.yaml" />
+      <xacro:property name="pm_robot_bringup_config_file" value="$(find pm_robot_bringup)/config/pm_robot_bringup_config.yaml" /> -->
+    </xacro:if>
     <xacro:property name="current_pm_robot_bringup_config" value="${xacro.load_yaml(pm_robot_bringup_config_file)}"/>
     <xacro:property name="current_vacuum_tool" value="${current_pm_robot_bringup_config['pm_robot_tools']['pm_robot_vacuum_tools']['use_tool']}"/>

File: pm_robot_description/urdf/pm_robot.xacro (robot description, xacro)
@@ -18,9 +18,9 @@
       <xacro:property name="local_robot_bringup_file_path" value="${path_dict['pm_robot_bringup_config_file_path']}"/>
       <!-- REAL -->
-      <!-- <xacro:property name="pm_robot_joint_calibraion_file" value="${local_calibration_file_path}" />
-      <xacro:property name="pm_robot_bringup_config_file" value="${local_robot_bringup_file_path}"/> -->
+      <xacro:property name="pm_robot_joint_calibraion_file" value="${local_calibration_file_path}" />
+      <xacro:property name="pm_robot_bringup_config_file" value="${local_robot_bringup_file_path}"/>
       <!-- SIM -->
-      <xacro:property name="pm_robot_joint_calibraion_file" value="$(find pm_robot_description)/calibration_config/pm_robot_joint_calibration.yaml" />
-      <xacro:property name="pm_robot_bringup_config_file" value="$(find pm_robot_bringup)/config/pm_robot_bringup_config.yaml" />
+      <!-- <xacro:property name="pm_robot_joint_calibraion_file" value="$(find pm_robot_description)/calibration_config/pm_robot_joint_calibration.yaml" />
+      <xacro:property name="pm_robot_bringup_config_file" value="$(find pm_robot_bringup)/config/pm_robot_bringup_config.yaml" /> -->
     </xacro:if>
     <xacro:property name="current_pm_robot_bringup_config" value="${xacro.load_yaml(pm_robot_bringup_config_file)}"/>

File: pm_robot_description/urdf/pm_robot_gonio_left.xacro (robot description, xacro)
@@ -17,9 +17,9 @@
       <xacro:property name="local_robot_bringup_file_path" value="${path_dict['pm_robot_bringup_config_file_path']}"/>
       <!-- REAL -->
-      <!-- <xacro:property name="pm_robot_joint_calibraion_file" value="${local_calibration_file_path}" />
-    <xacro:property name="pm_robot_bringup_config_file" value="${local_robot_bringup_file_path}"/> -->
+      <xacro:property name="pm_robot_joint_calibraion_file" value="${local_calibration_file_path}" />
+      <xacro:property name="pm_robot_bringup_config_file" value="${local_robot_bringup_file_path}"/>
       <!-- SIM -->
-      <xacro:property name="pm_robot_joint_calibraion_file" value="$(find pm_robot_description)/calibration_config/pm_robot_joint_calibration.yaml" />
-      <xacro:property name="pm_robot_bringup_config_file" value="$(find pm_robot_bringup)/config/pm_robot_bringup_config.yaml" />
+      <!-- <xacro:property name="pm_robot_joint_calibraion_file" value="$(find pm_robot_description)/calibration_config/pm_robot_joint_calibration.yaml" />
+      <xacro:property name="pm_robot_bringup_config_file" value="$(find pm_robot_bringup)/config/pm_robot_bringup_config.yaml" /> -->
     </xacro:if>
     <xacro:property name="current_pm_robot_bringup_config" value="${xacro.load_yaml(pm_robot_bringup_config_file)}"/>

File: pm_robot_description/urdf/pm_robot_gonio_right.xacro (robot description, xacro)
@@ -17,9 +17,9 @@
       <xacro:property name="local_robot_bringup_file_path" value="${path_dict['pm_robot_bringup_config_file_path']}"/>
       <!-- REAL -->
-      <!-- <xacro:property name="pm_robot_joint_calibraion_file" value="${local_calibration_file_path}" />
-      <xacro:property name="pm_robot_bringup_config_file" value="${local_robot_bringup_file_path}"/> -->
+      <xacro:property name="pm_robot_joint_calibraion_file" value="${local_calibration_file_path}" />
+      <xacro:property name="pm_robot_bringup_config_file" value="${local_robot_bringup_file_path}"/>
       <!-- SIM -->
-      <xacro:property name="pm_robot_joint_calibraion_file" value="$(find pm_robot_description)/calibration_config/pm_robot_joint_calibration.yaml" />
-      <xacro:property name="pm_robot_bringup_config_file" value="$(find pm_robot_bringup)/config/pm_robot_bringup_config.yaml" />
+      <!-- <xacro:property name="pm_robot_joint_calibraion_file" value="$(find pm_robot_description)/calibration_config/pm_robot_joint_calibration.yaml" />
+      <xacro:property name="pm_robot_bringup_config_file" value="$(find pm_robot_bringup)/config/pm_robot_bringup_config.yaml" /> -->
     </xacro:if>
     <xacro:property name="current_pm_robot_bringup_config" value="${xacro.load_yaml(pm_robot_bringup_config_file)}"/>

File: pm_robot_description/urdf/pm_smarpod_station.xacro (robot description, xacro)
@@ -18,9 +18,9 @@
       <xacro:property name="local_robot_bringup_file_path" value="${path_dict['pm_robot_bringup_config_file_path']}"/>
       <!-- REAL -->
-      <!-- <xacro:property name="pm_robot_joint_calibraion_file" value="${local_calibration_file_path}" />
-    <xacro:property name="pm_robot_bringup_config_file" value="${local_robot_bringup_file_path}"/> -->
+      <xacro:property name="pm_robot_joint_calibraion_file" value="${local_calibration_file_path}" />
+      <xacro:property name="pm_robot_bringup_config_file" value="${local_robot_bringup_file_path}"/>
       <!-- SIM -->
-      <xacro:property name="pm_robot_joint_calibraion_file" value="$(find pm_robot_description)/calibration_config/pm_robot_joint_calibration.yaml" />
-      <xacro:property name="pm_robot_bringup_config_file" value="$(find pm_robot_bringup)/config/pm_robot_bringup_config.yaml" />
+      <!-- <xacro:property name="pm_robot_joint_calibraion_file" value="$(find pm_robot_description)/calibration_config/pm_robot_joint_calibration.yaml" />
+      <xacro:property name="pm_robot_bringup_config_file" value="$(find pm_robot_bringup)/config/pm_robot_bringup_config.yaml" /> -->
     </xacro:if>
     <xacro:property name="current_pm_robot_bringup_config" value="${xacro.load_yaml(pm_robot_bringup_config_file)}"/>

File: pm_robot_description/urdf/ros2_control_real_HW.xacro (robot description, xacro)
@@ -3,4 +3,14 @@
     <xacro:macro name="pm_robot_ros2_control_hw_real" params="name initial_positions_file launch_mode hardware">
         <xacro:property name="initial_positions" value="${load_yaml(initial_positions_file)['initial_positions']}"/>
+        <xacro:if value="${launch_mode == 'real_HW'}">
+            <xacro:property name="local_file_paths__file" value="$(find pm_robot_description)/calibration_config/pm_robot_path_real_HW.yaml" />
+            <xacro:property name="path_dict" value="${xacro.load_yaml(local_file_paths__file)}"/>
+            <xacro:property name="local_calibration_file_path" value="${path_dict['pm_robot_calibration_file_path']}"/>
+            <xacro:property name="local_robot_bringup_file_path" value="${path_dict['pm_robot_bringup_config_file_path']}"/>
+            <!-- REAL -->
+            <xacro:property name="pm_robot_joint_calibraion_file" value="${local_calibration_file_path}" />
+            <xacro:property name="pm_robot_bringup_config_file" value="${local_robot_bringup_file_path}"/>
+        </xacro:if>
+        <xacro:property name="current_pm_robot_bringup_config" value="${xacro.load_yaml(pm_robot_bringup_config_file)}"/>
         <ros2_control name="PMSystem" type="system">
             <hardware>
