Commit message: vacuum tool angled

File: pm_robot_description/urdf/pm_Schunk_Tools/Parallel_Gripper_1_Jaw/SmarAct_Piezo_Gripper.xacro (robot description, xacro)
@@ -194,4 +194,7 @@
   <xacro:property name="tool_tcp_offset_y" value="${Gripper_jaw_1_dict['tool_TCP_y_offset']}"/>
   <xacro:property name="tool_tcp_offset_z" value="${Gripper_jaw_1_dict['tool_TCP_z_offset']}"/>
+  <xacro:property name="tool_tcp_offset_rx" value="${Gripper_jaw_1_dict['tool_TCP_rx_offset']}"/>
+  <xacro:property name="tool_tcp_offset_ry" value="${Gripper_jaw_1_dict['tool_TCP_ry_offset']}"/>
+  <xacro:property name="tool_tcp_offset_rz" value="${Gripper_jaw_1_dict['tool_TCP_rz_offset']}"/>
   <!--%%%%%%%%%%%%% The parameters here are interchangeable %%%%%%%%%%%%%-->
   <!--%%%%%%%%%%%%% Jaw 1 Definitions %%%%%%%%%%%%%-->
@@ -313,7 +316,7 @@
     ${0 + tool_tcp_offset_y  + PM_Robot_Tool_TCP_Joint_Cal_y * 0.000001}
     ${0 + tool_tcp_offset_z - 0.04542 + PM_Robot_Tool_TCP_Joint_Cal_z * 0.000001}" rpy="
-    ${0 + PM_Robot_Tool_TCP_Joint_Cal_rx * 3.14159265359/180}
-    ${0 + PM_Robot_Tool_TCP_Joint_Cal_ry * 3.14159265359/180}
-    ${0 + PM_Robot_Tool_TCP_Joint_Cal_rz * 3.14159265359/180}" />
+    ${tool_tcp_offset_rx * 3.14159265359/180 + PM_Robot_Tool_TCP_Joint_Cal_rx * 3.14159265359/180}
+    ${tool_tcp_offset_ry * 3.14159265359/180 + PM_Robot_Tool_TCP_Joint_Cal_ry * 3.14159265359/180}
+    ${tool_tcp_offset_rz * 3.14159265359/180 + PM_Robot_Tool_TCP_Joint_Cal_rz * 3.14159265359/180}" />
   <parent link="Gripper_Rot_Plate" />
   <child link="PM_Robot_Tool_TCP" />

File: pm_robot_description/urdf/pm_Schunk_Tools/Parallel_Gripper_1_Jaw/SmarAct_Piezo_Gripper_flat.xacro (robot description, xacro)
@@ -194,4 +194,7 @@
     <xacro:property name="tool_tcp_offset_y" value="${Gripper_jaw_1_dict['tool_TCP_y_offset']}"/>
     <xacro:property name="tool_tcp_offset_z" value="${Gripper_jaw_1_dict['tool_TCP_z_offset']}"/>
+    <xacro:property name="tool_tcp_offset_rx" value="${Gripper_jaw_1_dict['tool_TCP_rx_offset']}"/>
+    <xacro:property name="tool_tcp_offset_ry" value="${Gripper_jaw_1_dict['tool_TCP_ry_offset']}"/>
+    <xacro:property name="tool_tcp_offset_rz" value="${Gripper_jaw_1_dict['tool_TCP_rz_offset']}"/>
     <!--%%%%%%%%%%%%% The parameters here are interchangeable %%%%%%%%%%%%%-->
     <!--%%%%%%%%%%%%% Jaw 1 Definitions %%%%%%%%%%%%%-->
@@ -313,7 +316,7 @@
       ${0 + tool_tcp_offset_y  + PM_Robot_Tool_TCP_Joint_Cal_y * 0.000001}
       ${0 + tool_tcp_offset_z - 0.04542 + PM_Robot_Tool_TCP_Joint_Cal_z * 0.000001}" rpy="
-      ${0 + PM_Robot_Tool_TCP_Joint_Cal_rx * 3.14159265359/180}
-      ${0 + PM_Robot_Tool_TCP_Joint_Cal_ry * 3.14159265359/180}
-      ${0 + PM_Robot_Tool_TCP_Joint_Cal_rz * 3.14159265359/180}" />
+      ${tool_tcp_offset_rx * 3.14159265359/180 + PM_Robot_Tool_TCP_Joint_Cal_rx * 3.14159265359/180}
+      ${tool_tcp_offset_ry * 3.14159265359/180 + PM_Robot_Tool_TCP_Joint_Cal_ry * 3.14159265359/180}
+      ${tool_tcp_offset_rz * 3.14159265359/180 + PM_Robot_Tool_TCP_Joint_Cal_rz * 3.14159265359/180}" />
     <parent link="Gripper_Rot_Plate" />
     <child link="PM_Robot_Tool_TCP" />

File: pm_robot_description/urdf/pm_Schunk_Tools/Schunk_Vacuum_Tools.xacro (robot description, xacro)
@@ -62,4 +62,7 @@
     <xacro:property name="pm_robot_tool_TCP_y_offset" value="${vacuum_tool_holder_configs_dict['tool_TCP_y_offset']}"/>
     <xacro:property name="pm_robot_tool_TCP_x_offset" value="${vacuum_tool_holder_configs_dict['tool_TCP_x_offset']}"/>
+    <xacro:property name="pm_robot_tool_TCP_rx_offset" value="${vacuum_tool_holder_configs_dict['tool_TCP_rx_offset']}"/>
+    <xacro:property name="pm_robot_tool_TCP_ry_offset" value="${vacuum_tool_holder_configs_dict['tool_TCP_ry_offset']}"/>
+    <xacro:property name="pm_robot_tool_TCP_rz_offset" value="${vacuum_tool_holder_configs_dict['tool_TCP_rz_offset']}"/>
   <link name="PM_Robot_Tool_TCP">
   </link>
@@ -75,7 +78,7 @@
       ${0 + pm_robot_tool_TCP_y_offset + PM_Robot_Tool_TCP_Joint_Cal_y * 0.000001}
       ${0 - 0.04542 - pm_robot_tool_TCP_z_offset + PM_Robot_Tool_TCP_Joint_Cal_z * 0.000001}" rpy="
-      ${0 + PM_Robot_Tool_TCP_Joint_Cal_rx * 3.14159265359/180}
-      ${0 + PM_Robot_Tool_TCP_Joint_Cal_ry * 3.14159265359/180}
-      ${0 + PM_Robot_Tool_TCP_Joint_Cal_rz * 3.14159265359/180}" />
+      ${pm_robot_tool_TCP_rx_offset * 3.14159265359/180 + PM_Robot_Tool_TCP_Joint_Cal_rx * 3.14159265359/180}
+      ${pm_robot_tool_TCP_ry_offset * 3.14159265359/180 + PM_Robot_Tool_TCP_Joint_Cal_ry * 3.14159265359/180}
+      ${pm_robot_tool_TCP_rz_offset * 3.14159265359/180 + PM_Robot_Tool_TCP_Joint_Cal_rz * 3.14159265359/180}" />
     <parent link="Gripper_Rot_Plate" />
     <child link="PM_Robot_Tool_TCP" />

Commit message: unity calibration_file & confocal_bottom

File: pm_robot_description/urdf/pm_Schunk_Tools/Parallel_Gripper_1_Jaw/SmarAct_Piezo_Gripper.xacro (robot description, xacro)
@@ -4,6 +4,6 @@
      For more information, please see http://wiki.ros.org/sw_urdf_exporter -->
 <robot xmlns:xacro="http://ros.org/wiki/xacro">
-  <xacro:macro name="Tool_Parallel_Gripper_1_Jaw" params="launch_mode">
-    <xacro:if value="${launch_mode == 'sim_HW'}">
+  <xacro:macro name="Tool_Parallel_Gripper_1_Jaw" params="launch_mode hardware:=''">
+    <xacro:if value="${launch_mode == 'sim_HW' or hardware == 'unity'}">
         <xacro:property name="pm_robot_joint_calibraion_file" value="$(find pm_robot_description)/calibration_config/pm_robot_joint_calibration.yaml" />
         <xacro:property name="pm_robot_bringup_config_file" value="$(find pm_robot_bringup)/config/pm_robot_bringup_config.yaml" />
@@ -12,5 +12,5 @@
     <!-- If launch_mode 'real' a local path can be specified for the calibration file -->
     <!-- If launch_mode 'real' a local path can be specified for the calibration file -->
-    <xacro:if value="${launch_mode == 'real_HW'}">
+    <xacro:if value="${(launch_mode == 'real_HW' and hardware != 'unity') or hardware == 'robot'}">
       <xacro:property name="local_file_paths__file" value="$(find pm_robot_description)/calibration_config/pm_robot_path_real_HW.yaml" />
       <xacro:property name="path_dict" value="${xacro.load_yaml(local_file_paths__file)}"/>

File: pm_robot_description/urdf/pm_Schunk_Tools/Parallel_Gripper_1_Jaw/SmarAct_Piezo_Gripper_flat.xacro (robot description, xacro)
@@ -4,6 +4,6 @@
      For more information, please see http://wiki.ros.org/sw_urdf_exporter -->
 <robot xmlns:xacro="http://ros.org/wiki/xacro">
-  <xacro:macro name="Tool_Parallel_Gripper_1_Jaw" params="launch_mode">
-          <xacro:if value="${launch_mode == 'sim_HW'}">
+  <xacro:macro name="Tool_Parallel_Gripper_1_Jaw" params="launch_mode hardware:=''">
+          <xacro:if value="${launch_mode == 'sim_HW' or hardware == 'unity'}">
               <xacro:property name="pm_robot_joint_calibraion_file" value="$(find pm_robot_description)/calibration_config/pm_robot_joint_calibration.yaml" />
               <xacro:property name="pm_robot_bringup_config_file" value="$(find pm_robot_bringup)/config/pm_robot_bringup_config.yaml" />
@@ -11,5 +11,5 @@
     <!-- Loading of the Robot Joint calibrations and bringup config -->
     <!-- If launch_mode 'real' a local path can be specified for the calibration file -->
-    <xacro:if value="${launch_mode == 'real_HW'}">
+    <xacro:if value="${(launch_mode == 'real_HW' and hardware != 'unity') or hardware == 'robot'}">
       <xacro:property name="local_file_paths__file" value="$(find pm_robot_description)/calibration_config/pm_robot_path_real_HW.yaml" />
       <xacro:property name="path_dict" value="${xacro.load_yaml(local_file_paths__file)}"/>

File: pm_robot_description/urdf/pm_Schunk_Tools/Parallel_Gripper_2_Jaws/MPG_10_plus.xacro (robot description, xacro)
@@ -4,6 +4,6 @@
      For more information, please see http://wiki.ros.org/sw_urdf_exporter -->
 <robot xmlns:xacro="http://ros.org/wiki/xacro">
-  <xacro:macro name="Tool_Parallel_Gripper_2_Jaws" params="launch_mode">
-          <xacro:if value="${launch_mode == 'sim_HW'}">
+  <xacro:macro name="Tool_Parallel_Gripper_2_Jaws" params="launch_mode hardware:=''">
+          <xacro:if value="${launch_mode == 'sim_HW' or hardware == 'unity'}">
               <xacro:property name="pm_robot_joint_calibraion_file" value="$(find pm_robot_description)/calibration_config/pm_robot_joint_calibration.yaml" />
               <xacro:property name="pm_robot_bringup_config_file" value="$(find pm_robot_bringup)/config/pm_robot_bringup_config.yaml" />
@@ -12,5 +12,5 @@
     <!-- If launch_mode 'real' a local path can be specified for the calibration file -->
     <!-- If launch_mode 'real' a local path can be specified for the calibration file -->
-    <xacro:if value="${launch_mode == 'real_HW'}">
+    <xacro:if value="${(launch_mode == 'real_HW' and hardware != 'unity') or hardware == 'robot'}">
       <xacro:property name="local_file_paths__file" value="$(find pm_robot_description)/calibration_config/pm_robot_path_real_HW.yaml" />
       <xacro:property name="path_dict" value="${xacro.load_yaml(local_file_paths__file)}"/>

File: pm_robot_description/urdf/pm_Schunk_Tools/Schunk_Vacuum_Tools.xacro (robot description, xacro)
@@ -4,7 +4,7 @@
      For more information, please see http://wiki.ros.org/sw_urdf_exporter -->
 <robot xmlns:xacro="http://ros.org/wiki/xacro">
-    <xacro:macro name="Schunk_Vacuum_Tools" params="launch_mode">
+    <xacro:macro name="Schunk_Vacuum_Tools" params="launch_mode hardware:=''">
     <!-- Loading of the Robot Joint calibrations and bringup config -->
-          <xacro:if value="${launch_mode == 'sim_HW'}">
+          <xacro:if value="${launch_mode == 'sim_HW' or hardware == 'unity'}">
               <xacro:property name="pm_robot_joint_calibraion_file" value="$(find pm_robot_description)/calibration_config/pm_robot_joint_calibration.yaml" />
               <xacro:property name="pm_robot_bringup_config_file" value="$(find pm_robot_bringup)/config/pm_robot_bringup_config.yaml" />
@@ -12,5 +12,5 @@
     <!-- Loading of the Robot Joint calibrations and bringup config -->
     <!-- If launch_mode 'real' a local path can be specified for the calibration file -->
-    <xacro:if value="${launch_mode == 'real_HW'}">
+    <xacro:if value="${(launch_mode == 'real_HW' and hardware != 'unity') or hardware == 'robot'}">
       <xacro:property name="local_file_paths__file" value="$(find pm_robot_description)/calibration_config/pm_robot_path_real_HW.yaml" />
       <xacro:property name="path_dict" value="${xacro.load_yaml(local_file_paths__file)}"/>

File: pm_robot_description/urdf/pm_robot.xacro (robot description, xacro)
@@ -4,13 +4,14 @@
      For more information, please see http://wiki.ros.org/sw_urdf_exporter -->
 <robot xmlns:xacro="http://ros.org/wiki/xacro">
-  <xacro:macro name="pm_robot" params="launch_mode">
+  <xacro:macro name="pm_robot" params="launch_mode hardware:=''">
     <xacro:include filename="$(find pm_robot_description)/urdf/match_logo.urdf.xacro" />
     <!-- Loading of the Robot Joint calibrations -->
-    <xacro:if value="${launch_mode == 'sim_HW'}">
+    <!-- hardware=='unity' forces sim_HW calibration paths; hardware=='robot' forces real_HW paths -->
+    <xacro:if value="${launch_mode == 'sim_HW' or hardware == 'unity'}">
       <xacro:property name="pm_robot_joint_calibraion_file" value="$(find pm_robot_description)/calibration_config/pm_robot_joint_calibration.yaml" />
       <xacro:property name="pm_robot_bringup_config_file" value="$(find pm_robot_bringup)/config/pm_robot_bringup_config.yaml" />
     </xacro:if>
     <!-- If launch_mode 'real' a local path can be specified for the calibration file -->
-    <xacro:if value="${launch_mode == 'real_HW'}">
+    <xacro:if value="${(launch_mode == 'real_HW' and hardware != 'unity') or hardware == 'robot'}">
       <xacro:property name="local_file_paths__file" value="$(find pm_robot_description)/calibration_config/pm_robot_path_real_HW.yaml" />
       <xacro:property name="path_dict" value="${xacro.load_yaml(local_file_paths__file)}"/>

File: pm_robot_description/urdf/pm_robot_gonio_left.xacro (robot description, xacro)
@@ -4,12 +4,12 @@
      For more information, please see http://wiki.ros.org/sw_urdf_exporter -->
 <robot xmlns:xacro="http://ros.org/wiki/xacro">
-  <xacro:macro name="pm_robot_gonio_left" params="launch_mode">
+  <xacro:macro name="pm_robot_gonio_left" params="launch_mode hardware:=''">
     <!-- Loading of the Robot Joint calibrations -->
-    <xacro:if value="${launch_mode == 'sim_HW'}">
+    <xacro:if value="${launch_mode == 'sim_HW' or hardware == 'unity'}">
       <xacro:property name="pm_robot_joint_calibraion_file" value="$(find pm_robot_description)/calibration_config/pm_robot_joint_calibration.yaml" />
       <xacro:property name="pm_robot_bringup_config_file" value="$(find pm_robot_bringup)/config/pm_robot_bringup_config.yaml" />
     </xacro:if>
     <!-- If launch_mode 'real' a local path can be specified for the calibration file -->
-    <xacro:if value="${launch_mode == 'real_HW'}">
+    <xacro:if value="${(launch_mode == 'real_HW' and hardware != 'unity') or hardware == 'robot'}">
       <xacro:property name="local_file_paths__file" value="$(find pm_robot_description)/calibration_config/pm_robot_path_real_HW.yaml" />
       <xacro:property name="path_dict" value="${xacro.load_yaml(local_file_paths__file)}"/>

File: pm_robot_description/urdf/pm_robot_gonio_right.xacro (robot description, xacro)
@@ -4,12 +4,12 @@
      For more information, please see http://wiki.ros.org/sw_urdf_exporter -->
      <robot xmlns:xacro="http://ros.org/wiki/xacro">
-      <xacro:macro name="pm_robot_gonio_right" params="launch_mode">
+      <xacro:macro name="pm_robot_gonio_right" params="launch_mode hardware:=''">
     <!-- Loading of the Robot Joint calibrations -->
-    <xacro:if value="${launch_mode == 'sim_HW'}">
+    <xacro:if value="${launch_mode == 'sim_HW' or hardware == 'unity'}">
       <xacro:property name="pm_robot_joint_calibraion_file" value="$(find pm_robot_description)/calibration_config/pm_robot_joint_calibration.yaml" />
       <xacro:property name="pm_robot_bringup_config_file" value="$(find pm_robot_bringup)/config/pm_robot_bringup_config.yaml" />
     </xacro:if>
     <!-- If launch_mode 'real' a local path can be specified for the calibration file -->
-    <xacro:if value="${launch_mode == 'real_HW'}">
+    <xacro:if value="${(launch_mode == 'real_HW' and hardware != 'unity') or hardware == 'robot'}">
       <xacro:property name="local_file_paths__file" value="$(find pm_robot_description)/calibration_config/pm_robot_path_real_HW.yaml" />
       <xacro:property name="path_dict" value="${xacro.load_yaml(local_file_paths__file)}"/>

File: pm_robot_description/urdf/pm_robot_main.xacro (robot description, xacro)
@@ -18,5 +18,5 @@
   <xacro:arg name="with_Gonio_Right" default="true" />
   <xacro:arg name="with_smarpod_station" default="false" /> -->
-  <xacro:pm_robot launch_mode="$(arg launch_mode)"/>
+  <xacro:pm_robot launch_mode="$(arg launch_mode)" hardware="$(arg hardware)"/>
   <!-- START - Loading Config Files-->
     <!-- Loading of the Robot bringup config -->
@@ -40,5 +40,5 @@
   <!-- If Vacuum Tool is selected-->
     <xacro:if value="${current_pm_robot_bringup_config['pm_robot_tools']['pm_robot_vacuum_tools']['use_vacuum_tool']}">
-      <xacro:Schunk_Vacuum_Tools launch_mode="$(arg launch_mode)"/>
+      <xacro:Schunk_Vacuum_Tools launch_mode="$(arg launch_mode)" hardware="$(arg hardware)"/>
     </xacro:if>
   <!-- If 2 Jaws Parallel Gripper is selected-->
@@ -51,5 +51,5 @@
       <xacro:include filename="$(find pm_robot_description)/urdf/pm_Schunk_Tools/Parallel_Gripper_2_Jaws/${current_parallel_gripper_xacro}" />
       <!-- Create the included xacro -->
-      <xacro:Tool_Parallel_Gripper_2_Jaws launch_mode="$(arg launch_mode)"/>
+      <xacro:Tool_Parallel_Gripper_2_Jaws launch_mode="$(arg launch_mode)" hardware="$(arg hardware)"/>
     </xacro:if>
     <!-- If 1 Jaws Parallel Gripper is selected-->
@@ -62,5 +62,5 @@
       <xacro:include filename="$(find pm_robot_description)/urdf/pm_Schunk_Tools/Parallel_Gripper_1_Jaw/${current_parallel_gripper_xacro}" />
       <!-- Create the included xacro -->
-      <xacro:Tool_Parallel_Gripper_1_Jaw launch_mode="$(arg launch_mode)"/>
+      <xacro:Tool_Parallel_Gripper_1_Jaw launch_mode="$(arg launch_mode)" hardware="$(arg hardware)"/>
     </xacro:if>
   <!-- END - Tool Defines-->
@@ -68,5 +68,5 @@
   <!-- Gonio Right Defines-->
   <xacro:if value="${current_pm_robot_bringup_config['pm_robot_gonio_right']['with_Gonio_Right']}">
-    <xacro:pm_robot_gonio_right launch_mode="$(arg launch_mode)"/>
+    <xacro:pm_robot_gonio_right launch_mode="$(arg launch_mode)" hardware="$(arg hardware)"/>
   </xacro:if>
   <!-- Gonio Right old version-->
@@ -76,5 +76,5 @@
   <!-- Gonio Right Defines-->
   <xacro:if value="${current_pm_robot_bringup_config['pm_robot_gonio_left']['with_Gonio_Left']}">
-    <xacro:pm_robot_gonio_left launch_mode="$(arg launch_mode)"/>
+    <xacro:pm_robot_gonio_left launch_mode="$(arg launch_mode)" hardware="$(arg hardware)"/>
   </xacro:if>
   <!-- Gonio Left old version-->
