Commit message: path user adaption

File: pm_robot_description/urdf/pm_Schunk_Tools/Parallel_Gripper_1_Jaw/SmarAct_Piezo_Gripper.xacro (robot description, xacro)
@@ -15,6 +15,6 @@
       <xacro:property name="local_file_paths__file" value="$(find pm_robot_description)/calibration_config/pm_robot_path_real_HW.yaml" />
       <xacro:property name="path_dict" value="${xacro.load_yaml(local_file_paths__file)}"/>
-      <xacro:property name="local_calibration_file_path" value="${path_dict['pm_robot_calibration_file_path']}"/>
-      <xacro:property name="local_robot_bringup_file_path" value="${path_dict['pm_robot_bringup_config_file_path']}"/>
+      <xacro:property name="local_calibration_file_path" value="${path_dict['pm_robot_calibration_file_path'].replace('$HOME', '$(env HOME)')}"/>
+      <xacro:property name="local_robot_bringup_file_path" value="${path_dict['pm_robot_bringup_config_file_path'].replace('$HOME', '$(env HOME)')}"/>
       <!-- REAL -->
       <xacro:property name="pm_robot_joint_calibraion_file" value="${local_calibration_file_path}" />

File: pm_robot_description/urdf/pm_Schunk_Tools/Parallel_Gripper_1_Jaw/SmarAct_Piezo_Gripper_flat.xacro (robot description, xacro)
@@ -14,6 +14,6 @@
       <xacro:property name="local_file_paths__file" value="$(find pm_robot_description)/calibration_config/pm_robot_path_real_HW.yaml" />
       <xacro:property name="path_dict" value="${xacro.load_yaml(local_file_paths__file)}"/>
-      <xacro:property name="local_calibration_file_path" value="${path_dict['pm_robot_calibration_file_path']}"/>
-      <xacro:property name="local_robot_bringup_file_path" value="${path_dict['pm_robot_bringup_config_file_path']}"/>
+      <xacro:property name="local_calibration_file_path" value="${path_dict['pm_robot_calibration_file_path'].replace('$HOME', '$(env HOME)')}"/>
+      <xacro:property name="local_robot_bringup_file_path" value="${path_dict['pm_robot_bringup_config_file_path'].replace('$HOME', '$(env HOME)')}"/>
       <!-- REAL -->
       <xacro:property name="pm_robot_joint_calibraion_file" value="${local_calibration_file_path}" />

File: pm_robot_description/urdf/pm_Schunk_Tools/Parallel_Gripper_2_Jaws/MPG_10_plus.xacro (robot description, xacro)
@@ -15,6 +15,6 @@
       <xacro:property name="local_file_paths__file" value="$(find pm_robot_description)/calibration_config/pm_robot_path_real_HW.yaml" />
       <xacro:property name="path_dict" value="${xacro.load_yaml(local_file_paths__file)}"/>
-      <xacro:property name="local_calibration_file_path" value="${path_dict['pm_robot_calibration_file_path']}"/>
-      <xacro:property name="local_robot_bringup_file_path" value="${path_dict['pm_robot_bringup_config_file_path']}"/>
+      <xacro:property name="local_calibration_file_path" value="${path_dict['pm_robot_calibration_file_path'].replace('$HOME', '$(env HOME)')}"/>
+      <xacro:property name="local_robot_bringup_file_path" value="${path_dict['pm_robot_bringup_config_file_path'].replace('$HOME', '$(env HOME)')}"/>
       <!-- REAL -->
       <xacro:property name="pm_robot_joint_calibraion_file" value="${local_calibration_file_path}" />

File: pm_robot_description/urdf/pm_Schunk_Tools/Parallel_Gripper_2_Jaws/MPG_20_plus.xacro (robot description, xacro)
@@ -15,6 +15,6 @@
       <xacro:property name="local_file_paths__file" value="$(find pm_robot_description)/calibration_config/pm_robot_path_real_HW.yaml" />
       <xacro:property name="path_dict" value="${xacro.load_yaml(local_file_paths__file)}"/>
-      <xacro:property name="local_calibration_file_path" value="${path_dict['pm_robot_calibration_file_path']}"/>
-      <xacro:property name="local_robot_bringup_file_path" value="${path_dict['pm_robot_bringup_config_file_path']}"/>
+      <xacro:property name="local_calibration_file_path" value="${path_dict['pm_robot_calibration_file_path'].replace('$HOME', '$(env HOME)')}"/>
+      <xacro:property name="local_robot_bringup_file_path" value="${path_dict['pm_robot_bringup_config_file_path'].replace('$HOME', '$(env HOME)')}"/>
       <!-- REAL -->
       <xacro:property name="pm_robot_joint_calibraion_file" value="${local_calibration_file_path}" />

File: pm_robot_description/urdf/pm_Schunk_Tools/Schunk_Vacuum_Tools.xacro (robot description, xacro)
@@ -15,6 +15,6 @@
       <xacro:property name="local_file_paths__file" value="$(find pm_robot_description)/calibration_config/pm_robot_path_real_HW.yaml" />
       <xacro:property name="path_dict" value="${xacro.load_yaml(local_file_paths__file)}"/>
-      <xacro:property name="local_calibration_file_path" value="${path_dict['pm_robot_calibration_file_path']}"/>
-      <xacro:property name="local_robot_bringup_file_path" value="${path_dict['pm_robot_bringup_config_file_path']}"/>
+      <xacro:property name="local_calibration_file_path" value="${path_dict['pm_robot_calibration_file_path'].replace('$HOME', '$(env HOME)')}"/>
+      <xacro:property name="local_robot_bringup_file_path" value="${path_dict['pm_robot_bringup_config_file_path'].replace('$HOME', '$(env HOME)')}"/>
       <!-- REAL -->
       <xacro:property name="pm_robot_joint_calibraion_file" value="${local_calibration_file_path}" />

File: pm_robot_description/urdf/pm_robot.xacro (robot description, xacro)
@@ -16,6 +16,6 @@
       <xacro:property name="local_file_paths__file" value="$(find pm_robot_description)/calibration_config/pm_robot_path_real_HW.yaml" />
       <xacro:property name="path_dict" value="${xacro.load_yaml(local_file_paths__file)}"/>
-      <xacro:property name="local_calibration_file_path" value="${path_dict['pm_robot_calibration_file_path']}"/>
-      <xacro:property name="local_robot_bringup_file_path" value="${path_dict['pm_robot_bringup_config_file_path']}"/>
+      <xacro:property name="local_calibration_file_path" value="${path_dict['pm_robot_calibration_file_path'].replace('$HOME', '$(env HOME)')}"/>
+      <xacro:property name="local_robot_bringup_file_path" value="${path_dict['pm_robot_bringup_config_file_path'].replace('$HOME', '$(env HOME)')}"/>
       <!-- REAL -->
       <xacro:property name="pm_robot_joint_calibraion_file" value="${local_calibration_file_path}" />

File: pm_robot_description/urdf/pm_robot_gonio_left.xacro (robot description, xacro)
@@ -14,6 +14,6 @@
       <xacro:property name="local_file_paths__file" value="$(find pm_robot_description)/calibration_config/pm_robot_path_real_HW.yaml" />
       <xacro:property name="path_dict" value="${xacro.load_yaml(local_file_paths__file)}"/>
-      <xacro:property name="local_calibration_file_path" value="${path_dict['pm_robot_calibration_file_path']}"/>
-      <xacro:property name="local_robot_bringup_file_path" value="${path_dict['pm_robot_bringup_config_file_path']}"/>
+      <xacro:property name="local_calibration_file_path" value="${path_dict['pm_robot_calibration_file_path'].replace('$HOME', '$(env HOME)')}"/>
+      <xacro:property name="local_robot_bringup_file_path" value="${path_dict['pm_robot_bringup_config_file_path'].replace('$HOME', '$(env HOME)')}"/>
       <!-- REAL -->
       <xacro:property name="pm_robot_joint_calibraion_file" value="${local_calibration_file_path}" />

File: pm_robot_description/urdf/pm_robot_gonio_right.xacro (robot description, xacro)
@@ -14,6 +14,6 @@
       <xacro:property name="local_file_paths__file" value="$(find pm_robot_description)/calibration_config/pm_robot_path_real_HW.yaml" />
       <xacro:property name="path_dict" value="${xacro.load_yaml(local_file_paths__file)}"/>
-      <xacro:property name="local_calibration_file_path" value="${path_dict['pm_robot_calibration_file_path']}"/>
-      <xacro:property name="local_robot_bringup_file_path" value="${path_dict['pm_robot_bringup_config_file_path']}"/>
+      <xacro:property name="local_calibration_file_path" value="${path_dict['pm_robot_calibration_file_path'].replace('$HOME', '$(env HOME)')}"/>
+      <xacro:property name="local_robot_bringup_file_path" value="${path_dict['pm_robot_bringup_config_file_path'].replace('$HOME', '$(env HOME)')}"/>
       <!-- REAL -->
       <xacro:property name="pm_robot_joint_calibraion_file" value="${local_calibration_file_path}" />

File: pm_robot_description/urdf/pm_robot_main.xacro (robot description, xacro)
@@ -29,5 +29,5 @@
         <xacro:property name="local_file_paths__file" value="$(find pm_robot_description)/calibration_config/pm_robot_path_real_HW.yaml" />
         <xacro:property name="path_dict" value="${xacro.load_yaml(local_file_paths__file)}"/>
-        <xacro:property name="local_robot_bringup_file_path" value="${path_dict['pm_robot_bringup_config_file_path']}"/>
+        <xacro:property name="local_robot_bringup_file_path" value="${path_dict['pm_robot_bringup_config_file_path'].replace('$HOME', '$(env HOME)')}"/>
         <!-- REAL -->
         <xacro:property name="pm_robot_bringup_config_file" value="${local_robot_bringup_file_path}"/>

File: pm_robot_description/urdf/pm_smarpod_station.xacro (robot description, xacro)
@@ -15,6 +15,6 @@
       <xacro:property name="local_file_paths__file" value="$(find pm_robot_description)/calibration_config/pm_robot_path_real_HW.yaml" />
       <xacro:property name="path_dict" value="${xacro.load_yaml(local_file_paths__file)}"/>
-      <xacro:property name="local_calibration_file_path" value="${path_dict['pm_robot_calibration_file_path']}"/>
-      <xacro:property name="local_robot_bringup_file_path" value="${path_dict['pm_robot_bringup_config_file_path']}"/>
+      <xacro:property name="local_calibration_file_path" value="${path_dict['pm_robot_calibration_file_path'].replace('$HOME', '$(env HOME)')}"/>
+      <xacro:property name="local_robot_bringup_file_path" value="${path_dict['pm_robot_bringup_config_file_path'].replace('$HOME', '$(env HOME)')}"/>
       <!-- REAL -->
       <xacro:property name="pm_robot_joint_calibraion_file" value="${local_calibration_file_path}" />

File: pm_robot_description/urdf/ros2_control_real_HW.xacro (robot description, xacro)
@@ -6,6 +6,6 @@
             <xacro:property name="local_file_paths__file" value="$(find pm_robot_description)/calibration_config/pm_robot_path_real_HW.yaml" />
             <xacro:property name="path_dict" value="${xacro.load_yaml(local_file_paths__file)}"/>
-            <xacro:property name="local_calibration_file_path" value="${path_dict['pm_robot_calibration_file_path']}"/>
-            <xacro:property name="local_robot_bringup_file_path" value="${path_dict['pm_robot_bringup_config_file_path']}"/>
+            <xacro:property name="local_calibration_file_path" value="${path_dict['pm_robot_calibration_file_path'].replace('$HOME', '$(env HOME)')}"/>
+            <xacro:property name="local_robot_bringup_file_path" value="${path_dict['pm_robot_bringup_config_file_path'].replace('$HOME', '$(env HOME)')}"/>
             <!-- REAL -->
             <xacro:property name="pm_robot_joint_calibraion_file" value="${local_calibration_file_path}" />
