Commit message: smaract gripper + other meshes

File: pm_robot_description/urdf/pm_Schunk_Tools/Parallel_Gripper_1_Jaw/SmarAct_Piezo_Gripper_flat.xacro (robot description, xacro)
@@ -26,4 +26,6 @@
     <!-- <xacro:property name="current_vacuum_tool" value="${current_pm_robot_bringup_config['pm_robot_tools']['pm_robot_vacuum_tools']['use_tool']}"/>
     <xacro:property name="current_vacuum_tool_tip" value="${current_pm_robot_bringup_config['pm_robot_tools']['pm_robot_vacuum_tools']['use_tip']}"/> -->
+    <xacro:property name="current_tool" value="${current_pm_robot_bringup_config['pm_robot_tools']['pm_robot_tool_parallel_gripper_1_jaw']['use_tool']}"/>
+    <xacro:property name="current_jaw_attachement" value="${current_pm_robot_bringup_config['pm_robot_tools']['pm_robot_tool_parallel_gripper_1_jaw']['use_jaw_type']}"/>
     <xacro:property name="calibration_dict" value="${xacro.load_yaml(pm_robot_joint_calibraion_file)}"/>
     <!--%%%%%%%%%%%%% Base Parallel Gripper Definitions %%%%%%%%%%%%%-->
@@ -32,5 +34,5 @@
     <inertial>
       <origin
-        xyz="-0.00355668393665556 -0.000432533962047624 -0.011659024185547"
+        xyz="0.000310146269457783 0.0111566792086014 -0.0108754044082004"
         rpy="0 0 0" />
       <mass
@@ -49,5 +51,5 @@
         rpy="0 0 0" />
       <geometry>
-        <mesh filename="file://$(find pm_robot_description)/meshes/Tools/Parallel_Gripper_1_Jaw/SmarAct_Piezo_Gripper/SmarAct_Gripper_Base.STL" />
+        <mesh filename="file://$(find pm_robot_description)/meshes/Tools/Parallel_Gripper_1_Jaw/SmarAct_Piezo_Gripper/Tool_Parallel_Gripper_Base_flat.STL" />
       </geometry>
       <material name="grey"/>
@@ -58,5 +60,5 @@
         rpy="0 0 0" />
       <geometry>
-        <mesh filename="file://$(find pm_robot_description)/meshes/Tools/Parallel_Gripper_1_Jaw/SmarAct_Piezo_Gripper/SmarAct_Gripper_Base.STL" />
+        <mesh filename="file://$(find pm_robot_description)/meshes/Tools/Parallel_Gripper_1_Jaw/SmarAct_Piezo_Gripper/Tool_Parallel_Gripper_Base_flat.STL" />
       </geometry>
     </collision>
@@ -95,5 +97,5 @@
           rpy="0 0 0" />
         <geometry>
-          <mesh filename="file://$(find pm_robot_description)/meshes/Tools/Parallel_Gripper_1_Jaw/SmarAct_Piezo_Gripper/SmarAct_Gripper_Jaw.STL" />
+          <mesh filename="file://$(find pm_robot_description)/meshes/Tools/Parallel_Gripper_1_Jaw/SmarAct_Piezo_Gripper/SmarAct_Gripper_Jaw_flat.STL" />
         </geometry>
         <material name="grey"/>
@@ -104,5 +106,5 @@
           rpy="0 0 0" />
         <geometry>
-          <mesh filename="file://$(find pm_robot_description)/meshes/Tools/Parallel_Gripper_1_Jaw/SmarAct_Piezo_Gripper/SmarAct_Gripper_Jaw.STL" />
+          <mesh filename="file://$(find pm_robot_description)/meshes/Tools/Parallel_Gripper_1_Jaw/SmarAct_Piezo_Gripper/SmarAct_Gripper_Jaw_flat.STL" />
         </geometry>
       </collision>
@@ -116,5 +118,5 @@
       type="prismatic">
       <origin
-        xyz="0.00134999999999982 -0.00399999999999992 -0.0248"
+        xyz="-0.00549999981186566 0.00150000018813442 -0.0318"
         rpy="0 0 0" />
       <parent
@@ -137,5 +139,5 @@
       type="fixed">
       <origin
-        xyz="0 0.0014 -0.0075"
+        xyz="-0.00549999981186566 0.00150000018813442 -0.0318"
         rpy="0 0 0" />
       <parent
@@ -153,5 +155,5 @@
       type="fixed">
       <origin
-      xyz="-0.0014 0 -0.0075"
+      xyz="0.011060767270484 0 0"
       rpy="0 0 0" />
       <parent
@@ -163,58 +165,37 @@
     </joint>
   <!--%%%%%%%%%%%%% Jaw Definitions %%%%%%%%%%%%%-->
-    <!-- <xacro:property name="mpg_10_plus_jaw_define_file" value="$(find pm_robot_description)/urdf/pm_Schunk_Tools/MPG_10_plus_jaws.yaml" />
-    <xacro:property name="jaw_dict" value="${xacro.load_yaml(mpg_10_plus_jaw_define_file)}"/> -->
+    <xacro:property name="parallel_gripper_1_jaw_file" value="$(find pm_robot_description)/urdf/urdf_configs/parallel_gripper_1_jaw.yaml" />
+    <xacro:property name="parallel_gripper_configs" value="${xacro.load_yaml(parallel_gripper_1_jaw_file)}"/>
     <!--%%%%%%%%%%%%% Default Jaw Definitions %%%%%%%%%%%%%-->
-    <!-- <xacro:property name="Gripper_jaw_1_xyz" value="${jaw_dict['lens_jaw_3_mm_1']['xyz']}"/>
-    <xacro:property name="Gripper_jaw_1_rpy" value="${jaw_dict['lens_jaw_3_mm_1']['rpy']}"/>
-    <xacro:property name="Gripper_jaw_1_mass" value="${jaw_dict['lens_jaw_3_mm_1']['mass']}"/>
-    <xacro:property name="Gripper_jaw_1_inertia_ixx" value="${jaw_dict['lens_jaw_3_mm_1']['inertia_ixx']}"/>
-    <xacro:property name="Gripper_jaw_1_inertia_ixy" value="${jaw_dict['lens_jaw_3_mm_1']['inertia_ixy']}"/>
-    <xacro:property name="Gripper_jaw_1_inertia_ixz" value="${jaw_dict['lens_jaw_3_mm_1']['inertia_ixz']}"/>
-    <xacro:property name="Gripper_jaw_1_inertia_iyy" value="${jaw_dict['lens_jaw_3_mm_1']['inertia_iyy']}"/>
-    <xacro:property name="Gripper_jaw_1_inertia_iyz" value="${jaw_dict['lens_jaw_3_mm_1']['inertia_iyz']}"/>
-    <xacro:property name="Gripper_jaw_1_inertia_izz" value="${jaw_dict['lens_jaw_3_mm_1']['inertia_izz']}"/>
-    <xacro:property name="Gripper_jaw_1_visual_filename" value="${jaw_dict['lens_jaw_3_mm_1']['visual_filename']}"/>
-    <xacro:property name="Gripper_jaw_1_collision_filename" value="${jaw_dict['lens_jaw_3_mm_1']['collision_filename']}"/>
-    <xacro:property name="Gripper_jaw_2_xyz" value="${jaw_dict['lens_jaw_3_mm_2']['xyz']}"/>
-    <xacro:property name="Gripper_jaw_2_rpy" value="${jaw_dict['lens_jaw_3_mm_2']['rpy']}"/>
-    <xacro:property name="Gripper_jaw_2_mass" value="${jaw_dict['lens_jaw_3_mm_2']['mass']}"/>
-    <xacro:property name="Gripper_jaw_2_inertia_ixx" value="${jaw_dict['lens_jaw_3_mm_2']['inertia_ixx']}"/>
-    <xacro:property name="Gripper_jaw_2_inertia_ixy" value="${jaw_dict['lens_jaw_3_mm_2']['inertia_ixy']}"/>
-    <xacro:property name="Gripper_jaw_2_inertia_ixz" value="${jaw_dict['lens_jaw_3_mm_2']['inertia_ixz']}"/>
-    <xacro:property name="Gripper_jaw_2_inertia_iyy" value="${jaw_dict['lens_jaw_3_mm_2']['inertia_iyy']}"/>
-    <xacro:property name="Gripper_jaw_2_inertia_iyz" value="${jaw_dict['lens_jaw_3_mm_2']['inertia_iyz']}"/>
-    <xacro:property name="Gripper_jaw_2_inertia_izz" value="${jaw_dict['lens_jaw_3_mm_2']['inertia_izz']}"/>
-    <xacro:property name="Gripper_jaw_2_visual_filename" value="${jaw_dict['lens_jaw_3_mm_2']['visual_filename']}"/>
-    <xacro:property name="Gripper_jaw_2_collision_filename" value="${jaw_dict['lens_jaw_3_mm_2']['collision_filename']}"/> -->
-    <!--%%%%%%%%%%%%% 3MM Lens Jaw 1 Definitions %%%%%%%%%%%%%-->
-    <!-- <xacro:if value="${use_three_mm_lens}">
-      <xacro:property name="Gripper_jaw_1_xyz" value="${jaw_dict['lens_jaw_3_mm_1']['xyz']}"/>
-      <xacro:property name="Gripper_jaw_1_rpy" value="${jaw_dict['lens_jaw_3_mm_1']['rpy']}"/>
-      <xacro:property name="Gripper_jaw_1_mass" value="${jaw_dict['lens_jaw_3_mm_1']['mass']}"/>
-      <xacro:property name="Gripper_jaw_1_inertia_ixx" value="${jaw_dict['lens_jaw_3_mm_1']['inertia_ixx']}"/>
-      <xacro:property name="Gripper_jaw_1_inertia_ixy" value="${jaw_dict['lens_jaw_3_mm_1']['inertia_ixy']}"/>
-      <xacro:property name="Gripper_jaw_1_inertia_ixz" value="${jaw_dict['lens_jaw_3_mm_1']['inertia_ixz']}"/>
-      <xacro:property name="Gripper_jaw_1_inertia_iyy" value="${jaw_dict['lens_jaw_3_mm_1']['inertia_iyy']}"/>
-      <xacro:property name="Gripper_jaw_1_inertia_iyz" value="${jaw_dict['lens_jaw_3_mm_1']['inertia_iyz']}"/>
-      <xacro:property name="Gripper_jaw_1_inertia_izz" value="${jaw_dict['lens_jaw_3_mm_1']['inertia_izz']}"/>
-      <xacro:property name="Gripper_jaw_1_visual_filename" value="${jaw_dict['lens_jaw_3_mm_1']['visual_filename']}"/>
-      <xacro:property name="Gripper_jaw_1_collision_filename" value="${jaw_dict['lens_jaw_3_mm_1']['collision_filename']}"/>
-      <xacro:property name="Gripper_jaw_2_xyz" value="${jaw_dict['lens_jaw_3_mm_2']['xyz']}"/>
-      <xacro:property name="Gripper_jaw_2_rpy" value="${jaw_dict['lens_jaw_3_mm_2']['rpy']}"/>
-      <xacro:property name="Gripper_jaw_2_mass" value="${jaw_dict['lens_jaw_3_mm_2']['mass']}"/>
-      <xacro:property name="Gripper_jaw_2_inertia_ixx" value="${jaw_dict['lens_jaw_3_mm_2']['inertia_ixx']}"/>
-      <xacro:property name="Gripper_jaw_2_inertia_ixy" value="${jaw_dict['lens_jaw_3_mm_2']['inertia_ixy']}"/>
-      <xacro:property name="Gripper_jaw_2_inertia_ixz" value="${jaw_dict['lens_jaw_3_mm_2']['inertia_ixz']}"/>
-      <xacro:property name="Gripper_jaw_2_inertia_iyy" value="${jaw_dict['lens_jaw_3_mm_2']['inertia_iyy']}"/>
-      <xacro:property name="Gripper_jaw_2_inertia_iyz" value="${jaw_dict['lens_jaw_3_mm_2']['inertia_iyz']}"/>
-      <xacro:property name="Gripper_jaw_2_inertia_izz" value="${jaw_dict['lens_jaw_3_mm_2']['inertia_izz']}"/>
-      <xacro:property name="Gripper_jaw_2_visual_filename" value="${jaw_dict['lens_jaw_3_mm_2']['visual_filename']}"/>
-      <xacro:property name="Gripper_jaw_2_collision_filename" value="${jaw_dict['lens_jaw_3_mm_2']['collision_filename']}"/>
-    </xacro:if> -->
+    <xacro:property name="Gripper_jaw_1_dict" value="${parallel_gripper_configs[current_tool][current_jaw_attachement]}"/>
+    <xacro:property name="Gripper_jaw_1_xyz" value="${Gripper_jaw_1_dict['Jaw_1']['inertia_xyz']}"/>
+    <xacro:property name="Gripper_jaw_1_rpy" value="${Gripper_jaw_1_dict['Jaw_1']['inertia_rpy']}"/>
+    <xacro:property name="Gripper_jaw_1_mass" value="${Gripper_jaw_1_dict['Jaw_1']['mass']}"/>
+    <xacro:property name="Gripper_jaw_1_inertia_ixx" value="${Gripper_jaw_1_dict['Jaw_1']['inertia_ixx']}"/>
+    <xacro:property name="Gripper_jaw_1_inertia_ixy" value="${Gripper_jaw_1_dict['Jaw_1']['inertia_ixy']}"/>
+    <xacro:property name="Gripper_jaw_1_inertia_ixz" value="${Gripper_jaw_1_dict['Jaw_1']['inertia_ixz']}"/>
+    <xacro:property name="Gripper_jaw_1_inertia_iyy" value="${Gripper_jaw_1_dict['Jaw_1']['inertia_iyy']}"/>
+    <xacro:property name="Gripper_jaw_1_inertia_iyz" value="${Gripper_jaw_1_dict['Jaw_1']['inertia_iyz']}"/>
+    <xacro:property name="Gripper_jaw_1_inertia_izz" value="${Gripper_jaw_1_dict['Jaw_1']['inertia_izz']}"/>
+    <xacro:property name="Gripper_jaw_1_visual_filename" value="${Gripper_jaw_1_dict['Jaw_1']['visual_filename']}"/>
+    <xacro:property name="Gripper_jaw_1_collision_filename" value="${Gripper_jaw_1_dict['Jaw_1']['collision_filename']}"/>
+    <xacro:property name="Gripper_jaw_2_xyz" value="${Gripper_jaw_1_dict['Jaw_2']['inertia_xyz']}"/>
+    <xacro:property name="Gripper_jaw_2_rpy" value="${Gripper_jaw_1_dict['Jaw_2']['inertia_rpy']}"/>
+    <xacro:property name="Gripper_jaw_2_mass" value="${Gripper_jaw_1_dict['Jaw_2']['mass']}"/>
+    <xacro:property name="Gripper_jaw_2_inertia_ixx" value="${Gripper_jaw_1_dict['Jaw_2']['inertia_ixx']}"/>
+    <xacro:property name="Gripper_jaw_2_inertia_ixy" value="${Gripper_jaw_1_dict['Jaw_2']['inertia_ixy']}"/>
+    <xacro:property name="Gripper_jaw_2_inertia_ixz" value="${Gripper_jaw_1_dict['Jaw_2']['inertia_ixz']}"/>
+    <xacro:property name="Gripper_jaw_2_inertia_iyy" value="${Gripper_jaw_1_dict['Jaw_2']['inertia_iyy']}"/>
+    <xacro:property name="Gripper_jaw_2_inertia_iyz" value="${Gripper_jaw_1_dict['Jaw_2']['inertia_iyz']}"/>
+    <xacro:property name="Gripper_jaw_2_inertia_izz" value="${Gripper_jaw_1_dict['Jaw_2']['inertia_izz']}"/>
+    <xacro:property name="Gripper_jaw_2_visual_filename" value="${Gripper_jaw_1_dict['Jaw_2']['visual_filename']}"/>
+    <xacro:property name="Gripper_jaw_2_collision_filename" value="${Gripper_jaw_1_dict['Jaw_2']['collision_filename']}"/>
+    <xacro:property name="tool_tcp_offset_x" value="${Gripper_jaw_1_dict['tool_TCP_x_offset']}"/>
+    <xacro:property name="tool_tcp_offset_y" value="${Gripper_jaw_1_dict['tool_TCP_y_offset']}"/>
+    <xacro:property name="tool_tcp_offset_z" value="${Gripper_jaw_1_dict['tool_TCP_z_offset']}"/>
     <!--%%%%%%%%%%%%% The parameters here are interchangeable %%%%%%%%%%%%%-->
     <!--%%%%%%%%%%%%% Jaw 1 Definitions %%%%%%%%%%%%%-->
-    <!-- <link
-      name="Tool_Gripper_MPG_10_Jaw_1_changeable">
+    <link
+      name="Tool_Parallel_Gripper_Jaw_1_attachment">
       <inertial>
         <origin
@@ -236,5 +217,5 @@
           rpy="0 0 0" />
         <geometry>
-          <mesh filename="file://$(find pm_robot_description)/meshes/Tools/MPG_10_plus/Jaws/${Gripper_jaw_1_visual_filename}" />
+          <mesh filename="file://$(find pm_robot_description)/meshes/Tools/Parallel_Gripper_1_Jaw/SmarAct_Piezo_Gripper/${Gripper_jaw_1_visual_filename}" />
         </geometry>
         <material
@@ -249,24 +230,24 @@
           rpy="0 0 0" />
         <geometry>
-          <mesh filename="file://$(find pm_robot_description)/meshes/Tools/MPG_10_plus/Jaws/${Gripper_jaw_1_visual_filename}" />
+          <mesh filename="file://$(find pm_robot_description)/meshes/Tools/Parallel_Gripper_1_Jaw/SmarAct_Piezo_Gripper/${Gripper_jaw_1_visual_filename}" />
         </geometry>
       </collision>
     </link>
-    <gazebo reference="Tool_Gripper_Jaw_1">
+    <gazebo reference="Tool_Parallel_Gripper_Jaw_1_attachment">
       <turnGravityOff>true</turnGravityOff>
     </gazebo>
     <joint
-      name="Tool_Gripper_MPG_10_Jaw_1_changeable_Joint"
+      name="Tool_Parallel_Gripper_Jaw_1_attachment_Joint"
       type="fixed">
       <origin
-        xyz="0.002 0 0 "
-        rpy="0 0 0" />
-      <parent
-        link="Tool_Gripper_MPG_10_Jaw_1_Point" />
-      <child
-        link="Tool_Gripper_MPG_10_Jaw_1_changeable" />
-    </joint>
-    <link
-      name="Tool_Gripper_MPG_10_Jaw_2_changeable">
+        xyz="0.0 0 0 "
+        rpy="0 0 0" />
+      <parent
+        link="Tool_Parallel_Gripper_Jaw_1_Point" />
+      <child
+        link="Tool_Parallel_Gripper_Jaw_1_attachment" />
+    </joint>
+    <link
+      name="Tool_Parallel_Gripper_Jaw_2_attachment">
       <inertial>
         <origin
@@ -288,5 +269,5 @@
           rpy="0 0 0" />
         <geometry>
-          <mesh filename="file://$(find pm_robot_description)/meshes/Tools/MPG_10_plus/Jaws/${Gripper_jaw_2_visual_filename}" />
+          <mesh filename="file://$(find pm_robot_description)/meshes/Tools/Parallel_Gripper_1_Jaw/SmarAct_Piezo_Gripper/${Gripper_jaw_2_visual_filename}" />
         </geometry>
         <material
@@ -301,22 +282,22 @@
           rpy="0 0 0" />
         <geometry>
-          <mesh filename="file://$(find pm_robot_description)/meshes/Tools/MPG_10_plus/Jaws/${Gripper_jaw_2_visual_filename}" />
+          <mesh filename="file://$(find pm_robot_description)/meshes/Tools/Parallel_Gripper_1_Jaw/SmarAct_Piezo_Gripper/${Gripper_jaw_2_visual_filename}" />
         </geometry>
       </collision>
     </link>
-    <gazebo reference="Tool_Gripper_MPG_10_Jaw_2_changeable">
+    <gazebo reference="Tool_Parallel_Gripper_Jaw_2_attachment">
       <turnGravityOff>true</turnGravityOff>
     </gazebo>
     <joint
-      name="Tool_Gripper_MPG_10_Jaw_2_changeable_Joint"
+      name="Tool_Parallel_Gripper_Jaw_2_attachment_Joint"
       type="fixed">
       <origin
-        xyz="0.002 0  0 "
-        rpy="1.5708 0 0" />
-      <parent
-        link="Tool_Gripper_MPG_10_Jaw_2_Point" />
-      <child
-        link="Tool_Gripper_MPG_10_Jaw_2_changeable" />
-    </joint> -->
+        xyz="0.0 0 0 "
+        rpy="0 0 0" />
+      <parent
+        link="Tool_Parallel_Gripper_Jaw_2_Point" />
+      <child
+        link="Tool_Parallel_Gripper_Jaw_2_attachment" />
+    </joint>
   <link name="PM_Robot_Tool_TCP">
   </link>
@@ -329,7 +310,7 @@
   <joint name="PM_Robot_Tool_TCP_Joint" type="fixed">
     <origin xyz="
-      ${0  + PM_Robot_Tool_TCP_Joint_Cal_x * 0.000001}
-      ${0  + PM_Robot_Tool_TCP_Joint_Cal_y * 0.000001}
-      ${0 - 0.04542 + PM_Robot_Tool_TCP_Joint_Cal_z * 0.000001}" rpy="
+      ${0 + tool_tcp_offset_x  + PM_Robot_Tool_TCP_Joint_Cal_x * 0.000001}
+      ${0 + tool_tcp_offset_y  + PM_Robot_Tool_TCP_Joint_Cal_y * 0.000001}
+      ${0 + tool_tcp_offset_z - 0.04542 + PM_Robot_Tool_TCP_Joint_Cal_z * 0.000001}" rpy="
       ${0 + PM_Robot_Tool_TCP_Joint_Cal_rx * 3.14159265359/180}
       ${0 + PM_Robot_Tool_TCP_Joint_Cal_ry * 3.14159265359/180}

Commit message: hwi gripper fix

File: pm_robot_description/urdf/pm_Schunk_Tools/Parallel_Gripper_1_Jaw/SmarAct_Piezo_Gripper_flat.xacro (robot description, xacro)
@@ -251,4 +251,5 @@
         link="Tool_Parallel_Gripper_Jaw_1_attachment" />
     </joint>
+    <!-- Tool_Parallel_Gripper_Jaw_2_attachment DISABLED
     <link
       name="Tool_Parallel_Gripper_Jaw_2_attachment">
@@ -303,4 +304,5 @@
         link="Tool_Parallel_Gripper_Jaw_2_attachment" />
     </joint>
+    -->
   <link name="PM_Robot_Tool_TCP">
   </link>

File: pm_robot_description/urdf/pm_robot_main.xacro (robot description, xacro)
@@ -95,4 +95,5 @@
     <xacro:pm_robot_ros2_control_hw_real name="Real_HW" initial_positions_file="$(arg initial_positions_file)" launch_mode="$(arg launch_mode)" hardware="$(arg hardware)"/>
     <xacro:pm_robot_pneumatic_mock_2 />
+    <xacro:pm_robot_gripper_mock />
   </xacro:if>
   <xacro:if value="${launch_mode == 'sim_HW'}">

File: pm_robot_description/urdf/ros2_control_real_HW.xacro (robot description, xacro)
@@ -109,33 +109,4 @@
                 </joint>
             </xacro:if>  -->
-            <!-- Only if gripper with two jaws is selected -->
-            <xacro:if value="${current_pm_robot_bringup_config['pm_robot_tools']['pm_robot_tool_parallel_gripper_2_jaws']['use_paralell_gripper']}">
-                <joint name="Tool_Parallel_Gripper_Jaw_1_Joint">
-                    <command_interface name="position">
-                    </command_interface>
-                    <state_interface name="position"/>
-                </joint>
-                <joint name="Tool_Parallel_Gripper_Jaw_2_Joint">
-                    <command_interface name="position">
-                    </command_interface>
-                    <state_interface name="position"/>
-                </joint>
-                <!-- <joint name="Tool_Parallel_Gripper_Jaw_2_Joint">
-                    <param name="mimic">Tool_Parallel_Gripper_Jaw_1_Joint</param>
-                    <param name="mulltiplier">1</param>
-                    <command_interface name="position">
-                    </command_interface>
-                    <state_interface name="position"/>
-                    <state_interface name="velocity"/>
-                </joint> -->
-            </xacro:if>
-            <!-- If parallel gripper with one jaw is selected -->
-            <xacro:if value="${current_pm_robot_bringup_config['pm_robot_tools']['pm_robot_tool_parallel_gripper_1_jaw']['use_paralell_gripper']}">
-                <joint name="Tool_Parallel_Gripper_Jaw_Joint">
-                    <command_interface name="position">
-                    </command_interface>
-                    <state_interface name="position"/>
-                </joint>
-            </xacro:if>
         </ros2_control>
         <!-- SmarPod Hardware Interface -->
@@ -212,5 +183,42 @@
         </xacro:if>
     </xacro:macro>
-<!--
+    <!-- Mock hardware for parallel gripper (separate from PMSystem) -->
+    <xacro:macro name="pm_robot_gripper_mock">
+        <xacro:if value="${current_pm_robot_bringup_config['pm_robot_tools']['pm_robot_tool_parallel_gripper_1_jaw']['use_paralell_gripper']}">
+            <ros2_control name="PMSystemGripper" type="system">
+                <hardware>
+                    <plugin>mock_components/GenericSystem</plugin>
+                </hardware>
+                <joint name="Tool_Parallel_Gripper_Jaw_Joint">
+                    <command_interface name="position">
+                    </command_interface>
+                    <state_interface name="position">
+                        <param name="initial_value">0.0</param>
+                    </state_interface>
+                </joint>
+            </ros2_control>
+        </xacro:if>
+        <xacro:if value="${current_pm_robot_bringup_config['pm_robot_tools']['pm_robot_tool_parallel_gripper_2_jaws']['use_paralell_gripper']}">
+            <ros2_control name="PMSystemGripper" type="system">
+                <hardware>
+                    <plugin>mock_components/GenericSystem</plugin>
+                </hardware>
+                <joint name="Tool_Parallel_Gripper_Jaw_1_Joint">
+                    <command_interface name="position">
+                    </command_interface>
+                    <state_interface name="position">
+                        <param name="initial_value">0.0</param>
+                    </state_interface>
+                </joint>
+                <joint name="Tool_Parallel_Gripper_Jaw_2_Joint">
+                    <command_interface name="position">
+                    </command_interface>
+                    <state_interface name="position">
+                        <param name="initial_value">0.0</param>
+                    </state_interface>
+                </joint>
+            </ros2_control>
+        </xacro:if>
+    </xacro:macro>
     <xacro:macro name="pm_robot_pneumatic_mock" >
         <ros2_control name="PMSystemPneumatic" type="system">
@@ -261,5 +269,5 @@
             </joint>
         </ros2_control>
-    </xacro:macro> -->
+    </xacro:macro>
     <xacro:macro name="pm_robot_pneumatic_mock_2" >
         <ros2_control name="PMSystemPneumatic_2" type="system">
