Commit message: major fix brinup config

File: pm_robot_description/urdf/pm_Schunk_Tools/Parallel_Gripper_1_Jaw/SmarAct_Piezo_Gripper_flat.xacro (robot description, xacro)
@@ -24,6 +24,4 @@
     </xacro:if>
     <xacro:property name="current_pm_robot_bringup_config" value="${xacro.load_yaml(pm_robot_bringup_config_file)}"/>
-    <!-- <xacro:property name="current_vacuum_tool" value="${current_pm_robot_bringup_config['pm_robot_tools']['pm_robot_vacuum_tools']['use_tool']}"/>
-    <xacro:property name="current_vacuum_tool_tip" value="${current_pm_robot_bringup_config['pm_robot_tools']['pm_robot_vacuum_tools']['use_tip']}"/> -->
     <xacro:property name="current_tool" value="${current_pm_robot_bringup_config['pm_robot_tools']['pm_robot_tool_parallel_gripper_1_jaw']['use_tool']}"/>
     <xacro:property name="current_jaw_attachement" value="${current_pm_robot_bringup_config['pm_robot_tools']['pm_robot_tool_parallel_gripper_1_jaw']['use_jaw_type']}"/>

File: pm_robot_description/urdf/pm_Schunk_Tools/Parallel_Gripper_2_Jaws/MPG_20_plus.xacro (robot description, xacro)
@@ -25,4 +25,6 @@
     </xacro:if>
     <xacro:property name="current_pm_robot_bringup_config" value="${xacro.load_yaml(pm_robot_bringup_config_file)}"/>
+    <xacro:property name="calibration_dict" value="${xacro.load_yaml(pm_robot_joint_calibraion_file)}"/>
+    <xacro:property name="current_pm_robot_bringup_config" value="${xacro.load_yaml(pm_robot_bringup_config_file)}"/>
     <xacro:property name="current_tool" value="${current_pm_robot_bringup_config['pm_robot_tools']['pm_robot_tool_parallel_gripper_2_jaws']['use_tool']}"/>
     <xacro:property name="current_jaw_attachement" value="${current_pm_robot_bringup_config['pm_robot_tools']['pm_robot_tool_parallel_gripper_2_jaws']['use_jaw_type']}"/>
@@ -30,5 +32,4 @@
     <xacro:property name="parallel_gripper_configs" value="${xacro.load_yaml(parallel_gripper_2_jaw_file)}"/>
     <xacro:property name="Gripper_jaw_2_dict" value="${parallel_gripper_configs[current_tool][current_jaw_attachement]}"/>
-    <xacro:property name="calibration_dict" value="${xacro.load_yaml(pm_robot_joint_calibraion_file)}"/>
     <!--%%%%%%%%%%%%% MPG 10-plus Base Parallel Gripper Definitions %%%%%%%%%%%%%-->
     <link
@@ -36,15 +37,15 @@
     <inertial>
       <origin
-        xyz="5.30403682906828E-05 -4.81468891081322E-05 -0.00753129191051478"
+        xyz="-0.000335975164371893 0.005953622519278 -0.00961798832647953"
         rpy="0 0 0" />
       <mass
-        value="0.0183798400393325" />
+        value="0.0219734801011759" />
       <inertia
-        ixx="2.20562725075551E-05"
-        ixy="3.27141658492019E-05"
-        ixz="1.66797947446843E-05"
-        iyy="1.61047701086979E-05"
-        iyz="7.34159323199958E-05"
-        izz="3.58202149775683E-05" />
+        ixx="2.8061799609194E-06"
+        ixy="3.07435258273047E-08"
+        ixz="-1.63779024253226E-09"
+        iyy="1.86483681914571E-06"
+        iyz="3.87737851095455E-09"
+        izz="4.26150237576402E-06" />
     </inertial>
     <visual>
@@ -53,5 +54,5 @@
         rpy="0 0 0" />
       <geometry>
-        <mesh filename="file://$(find pm_robot_description)/meshes/Tools/Parallel_Gripper_2_Jaws/MPG_10_plus/Tool_MPG_10_Base.STL" />
+        <mesh filename="file://$(find pm_robot_description)/meshes/Tools/Parallel_Gripper_2_Jaws/MPG_20_plus/Tool_MPG_20_Body.STL" />
       </geometry>
       <material name="grey"/>
@@ -62,5 +63,5 @@
         rpy="0 0 0" />
       <geometry>
-        <mesh filename="file://$(find pm_robot_description)/meshes/Tools/Parallel_Gripper_2_Jaws/MPG_10_plus/Tool_MPG_10_Base.STL" />
+        <mesh filename="file://$(find pm_robot_description)/meshes/Tools/Parallel_Gripper_2_Jaws/MPG_20_plus/Tool_MPG_20_Body.STL" />
       </geometry>
     </collision>
@@ -77,5 +78,5 @@
     <axis xyz="0 0 0" />
   </joint>
-  <!--%%%%%%%%%%%%% MPG 10-plus Jaw 2 Parallel Gripper Definitions %%%%%%%%%%%%%-->
+  <!--%%%%%%%%%%%%% MPG 20-plus Jaw 1 Parallel Gripper Definitions %%%%%%%%%%%%%-->
       <link
       name="Tool_Parallel_Gripper_Jaw_2">
@@ -99,5 +100,5 @@
           rpy="0 0 0" />
         <geometry>
-          <mesh filename="file://$(find pm_robot_description)/meshes/Tools/Parallel_Gripper_2_Jaws/MPG_10_plus/MPG_10_Jaw_2.STL" />
+          <mesh filename="file://$(find pm_robot_description)/meshes/Tools/Parallel_Gripper_2_Jaws/MPG_20_plus/MPG_20_Jaw_2.STL" />
         </geometry>
         <material name="grey"/>
@@ -108,5 +109,5 @@
           rpy="0 0 0" />
         <geometry>
-          <mesh filename="file://$(find pm_robot_description)/meshes/Tools/Parallel_Gripper_2_Jaws/MPG_10_plus/MPG_10_Jaw_2.STL" />
+          <mesh filename="file://$(find pm_robot_description)/meshes/Tools/Parallel_Gripper_2_Jaws/MPG_20_plus/MPG_20_Jaw_2.STL" />
         </geometry>
       </collision>
@@ -120,6 +121,6 @@
       type="prismatic">
       <origin
-        xyz="0.00134999999999982 -0.00399999999999992 -0.0248"
-        rpy="0 0 0" />
+      xyz="0.009317 0 -0.02"
+      rpy="0 0 0" />
       <parent
         link="Tool_Parallel_Gripper_Body_2_Jaws" />
@@ -127,8 +128,8 @@
         link="Tool_Parallel_Gripper_Jaw_2" />
       <axis
-        xyz="0 1 0" />
+        xyz="-1 0 0" />
       <limit
         lower="0"
-        upper="0.001"
+        upper="0.002"
         effort="20"
         velocity="0.05" />
@@ -141,5 +142,5 @@
       type="fixed">
       <origin
-      xyz="-0.0014 0 -0.0075"
+      xyz="0.0 0 0.0"
       rpy="0 0 0" />
       <parent
@@ -150,5 +151,5 @@
         xyz="0 0 0" />
     </joint>
-    <!--%%%%%%%%%%%%% MPG 10-plus Jaw 1 Parallel Gripper Definitions %%%%%%%%%%%%%-->
+    <!--%%%%%%%%%%%%% MPG 20-plus Jaw 1 Parallel Gripper Definitions %%%%%%%%%%%%%-->
       <link
       name="Tool_Parallel_Gripper_Jaw_1">
@@ -172,5 +173,5 @@
           rpy="0 0 0" />
         <geometry>
-          <mesh filename="file://$(find pm_robot_description)/meshes/Tools/Parallel_Gripper_2_Jaws/MPG_10_plus/MPG_10_Jaw_1.STL" />
+          <mesh filename="file://$(find pm_robot_description)/meshes/Tools/Parallel_Gripper_2_Jaws/MPG_20_plus/MPG_20_Jaw_1.STL" />
         </geometry>
         <material name="grey"/>
@@ -181,5 +182,5 @@
           rpy="0 0 0" />
         <geometry>
-          <mesh filename="file://$(find pm_robot_description)/meshes/Tools/Parallel_Gripper_2_Jaws/MPG_10_plus/MPG_10_Jaw_1.STL" />
+          <mesh filename="file://$(find pm_robot_description)/meshes/Tools/Parallel_Gripper_2_Jaws/MPG_20_plus/MPG_20_Jaw_1.STL" />
         </geometry>
       </collision>
@@ -193,6 +194,6 @@
       type="prismatic">
       <origin
-        xyz="-0.00135 0.004 -0.0248"
-        rpy="0 0 0" />
+      xyz="-0.009317 0 -0.02"
+      rpy="0 0 0" />
       <parent
         link="Tool_Parallel_Gripper_Body_2_Jaws" />
@@ -200,8 +201,8 @@
         link="Tool_Parallel_Gripper_Jaw_1" />
       <axis
-        xyz="0 -1 0" />
+        xyz="1 0 0" />
       <limit
         lower="0"
-        upper="0.001"
+        upper="0.002"
         effort="20"
         velocity="0.05" />
@@ -214,5 +215,5 @@
       type="fixed">
       <origin
-        xyz="0 0.0014 -0.0075"
+        xyz="0 0.0 0.0"
         rpy="0 0 0" />
       <parent
@@ -275,5 +276,5 @@
           rpy="0 0 0" />
         <geometry>
-          <mesh filename="file://$(find pm_robot_description)/meshes/Tools/Parallel_Gripper_2_Jaws/MPG_10_plus/Jaws/${Gripper_jaw_1_visual_filename}" />
+          <mesh filename="file://$(find pm_robot_description)/meshes/Tools/Parallel_Gripper_2_Jaws/MPG_20_plus/Jaws/${Gripper_jaw_1_visual_filename}" />
         </geometry>
         <material
@@ -288,5 +289,5 @@
           rpy="0 0 0" />
         <geometry>
-          <mesh filename="file://$(find pm_robot_description)/meshes/Tools/Parallel_Gripper_2_Jaws/MPG_10_plus/Jaws/${Gripper_jaw_1_collision_filename}" />
+          <mesh filename="file://$(find pm_robot_description)/meshes/Tools/Parallel_Gripper_2_Jaws/MPG_20_plus/Jaws/${Gripper_jaw_1_collision_filename}" />
         </geometry>
       </collision>
@@ -327,5 +328,5 @@
           rpy="0 0 0" />
         <geometry>
-          <mesh filename="file://$(find pm_robot_description)/meshes/Tools/Parallel_Gripper_2_Jaws/MPG_10_plus/Jaws/${Gripper_jaw_2_visual_filename}" />
+          <mesh filename="file://$(find pm_robot_description)/meshes/Tools/Parallel_Gripper_2_Jaws/MPG_20_plus/Jaws/${Gripper_jaw_2_visual_filename}" />
         </geometry>
         <material
@@ -340,5 +341,5 @@
           rpy="0 0 0" />
         <geometry>
-          <mesh filename="file://$(find pm_robot_description)/meshes/Tools/Parallel_Gripper_2_Jaws/MPG_10_plus/Jaws/${Gripper_jaw_2_collision_filename}" />
+          <mesh filename="file://$(find pm_robot_description)/meshes/Tools/Parallel_Gripper_2_Jaws/MPG_20_plus/Jaws/${Gripper_jaw_2_collision_filename}" />
         </geometry>
       </collision>
